Commit message: create some old robot urdf and xml for better iterations

File: sim/stompy/robot.urdf (robot description, URDF)
Before this commit: robot robot_7dof_arm, 139 links, 138 joints
Joints:
- joint joint_upper_limb_assembly_7_dof_1_full_arm_7_dof_1_lower_arm_3_dof_1_hand_left_1_rmd_x4_24_mock_1_dof_x4: type fixed -> revolute
- joint joint_upper_limb_assembly_7_dof_1_full_arm_7_dof_1_lower_arm_3_dof_1_hand_left_1_slider_1: type fixed -> prismatic
- joint joint_upper_limb_assembly_7_dof_1_full_arm_7_dof_1_lower_arm_3_dof_1_hand_left_1_slider_2: type fixed -> prismatic
- joint joint_upper_limb_assembly_7_dof_1_full_arm_7_dof_2_lower_arm_3_dof_1_hand_left_1_rmd_x4_24_mock_1_dof_x4: type fixed -> revolute
- joint joint_upper_limb_assembly_7_dof_1_full_arm_7_dof_2_lower_arm_3_dof_1_hand_left_1_slider_1: type fixed -> prismatic
- joint joint_upper_limb_assembly_7_dof_1_full_arm_7_dof_2_lower_arm_3_dof_1_hand_left_1_slider_2: type fixed -> prismatic
- joint left ankle pitch: limit lower=0 upper=2 effort=24 velocity=12 -> lower=-1.5707963 upper=2.1816616 effort=24 velocity=5
- joint left ankle roll: limit lower=0.76 upper=2.76 effort=24 velocity=12 -> lower=-2.268928 upper=-1.2217305 effort=24 velocity=5
- joint left elbow pitch: limit lower=2.07 upper=2.071 effort=24 velocity=5 -> lower=1.4486233 upper=5.4454273 effort=24 velocity=5
- joint left hip pitch: limit lower=-0.498 upper=1.502 effort=150 velocity=40 -> lower=-4.712389 upper=4.712389 effort=80 velocity=5
- joint left hip roll: limit lower=-2.57 upper=-0.57 effort=90 velocity=40 -> lower=-3.1415927 upper=3.1415927 effort=90 velocity=5
- joint left hip yaw: limit lower=-3.07 upper=-1.07 effort=90 velocity=40 -> lower=-4.712389 upper=4.712389 effort=90 velocity=5
- joint left knee pitch: limit lower=2.39 upper=4.39 effort=90 velocity=40 -> lower=-4.712389 upper=4.712389 effort=90 velocity=5
- joint left shoulder pitch: limit lower=-0.251 upper=-0.25 effort=90 velocity=5 -> lower=-3.1415927 upper=3.1415927 effort=90 velocity=5
- joint left shoulder roll: limit lower=-1.44 upper=-1.439 effort=24 velocity=5 -> lower=-4.712389 upper=4.712389 effort=24 velocity=5
- joint left shoulder yaw: limit lower=1.82 upper=1.821 effort=90 velocity=5 -> lower=0.97738438 upper=5.3058009 effort=90 velocity=5
- joint left wrist pitch: limit lower=3.33 upper=3.331 effort=24 velocity=5 -> lower=-4.712389 upper=4.712389 effort=24 velocity=5
- joint left wrist roll: limit lower=-2.51 upper=-2.509 effort=24 velocity=5 -> lower=-4.712389 upper=4.712389 effort=24 velocity=5
- joint left wrist yaw: limit lower=0.0628 upper=0.0638 effort=24 velocity=5 -> lower=-4.712389 upper=4.712389 effort=24 velocity=5
- joint right ankle pitch: limit lower=-1.502 upper=0.498 effort=24 velocity=12 -> lower=-1.5707963 upper=2.1816616 effort=24 velocity=5
- joint right ankle roll: limit lower=0.76 upper=2.76 effort=24 velocity=12 -> lower=-2.268928 upper=-1.2217305 effort=24 velocity=5
- joint right elbow pitch: limit lower=-2.57 upper=-2.569 effort=24 velocity=5 -> lower=1.4486233 upper=5.4454273 effort=24 velocity=5
- joint right hip pitch: limit lower=0.13 upper=2.13 effort=150 velocity=40 -> lower=-4.712389 upper=4.712389 effort=80 velocity=5
- joint right hip roll: limit lower=-1 upper=1 effort=90 velocity=40 -> lower=-3.1415927 upper=0 effort=90 velocity=5
- joint right hip yaw: limit lower=0.07 upper=2.07 effort=90 velocity=40 -> lower=-1.0471976 upper=2.0943951 effort=90 velocity=5
- joint right knee pitch: limit lower=-0.121 upper=1.879 effort=90 velocity=40 -> lower=-4.712389 upper=4.712389 effort=90 velocity=5
- joint right shoulder pitch: limit lower=2.7 upper=2.701 effort=90 velocity=5 -> lower=-3.1415927 upper=3.1415927 effort=90 velocity=5
- joint right shoulder roll: limit lower=-2.57 upper=-2.569 effort=24 velocity=5 -> lower=-4.712389 upper=4.712389 effort=24 velocity=5
- joint right shoulder yaw: limit lower=-1.82 upper=-1.819 effort=90 velocity=5 -> lower=0.97738438 upper=5.3058009 effort=90 velocity=5
- joint right wrist pitch: limit lower=0.251 upper=0.252 effort=24 velocity=5 -> lower=-4.712389 upper=4.712389 effort=24 velocity=5
- joint right wrist roll: limit lower=0 upper=0.001 effort=24 velocity=5 -> lower=-4.712389 upper=4.712389 effort=24 velocity=5
- joint right wrist yaw: limit lower=1.38 upper=1.381 effort=24 velocity=5 -> lower=-4.712389 upper=4.712389 effort=24 velocity=5
- joint torso roll: limit lower=-0.502 upper=-0.501 effort=90 velocity=5 -> lower=-4.3633231 upper=4.3633231 effort=90 velocity=5
