Commit message: updates to the config

File: sim/stompy/robot_fixed.urdf (robot description, URDF)
Before this commit: robot robot_7dof_arm, 139 links, 138 joints
Joints:
- joint left elbow pitch: limit lower=2.07 upper=2.071 effort=24 velocity=5 -> lower=2.07 upper=2.071 effort=0 velocity=0
- joint left shoulder pitch: limit lower=-0.251 upper=-0.25 effort=90 velocity=5 -> lower=-0.251 upper=-0.25 effort=0 velocity=0
- joint left shoulder roll: limit lower=-1.44 upper=-1.439 effort=24 velocity=5 -> lower=-1.44 upper=-1.439 effort=0 velocity=0
- joint left shoulder yaw: limit lower=1.82 upper=1.821 effort=90 velocity=5 -> lower=1.82 upper=1.821 effort=0 velocity=0
- joint left wrist pitch: limit lower=3.33 upper=3.331 effort=24 velocity=5 -> lower=3.33 upper=3.331 effort=0 velocity=0
- joint left wrist roll: limit lower=-2.51 upper=-2.509 effort=24 velocity=5 -> lower=-2.51 upper=-2.509 effort=0 velocity=0
- joint left wrist yaw: limit lower=0.0628 upper=0.0638 effort=24 velocity=5 -> lower=0.0628 upper=0.0638 effort=0 velocity=0
- joint right elbow pitch: limit lower=-2.57 upper=-2.569 effort=24 velocity=5 -> lower=-2.57 upper=-2.569 effort=0 velocity=0
- joint right shoulder pitch: limit lower=2.7 upper=2.701 effort=90 velocity=5 -> lower=2.7 upper=2.701 effort=0 velocity=0
- joint right shoulder roll: limit lower=-2.57 upper=-2.569 effort=24 velocity=5 -> lower=-2.57 upper=-2.569 effort=0 velocity=0
- joint right shoulder yaw: limit lower=-1.82 upper=-1.819 effort=90 velocity=5 -> lower=-1.82 upper=-1.819 effort=0 velocity=0
- joint right wrist pitch: limit lower=0.251 upper=0.252 effort=24 velocity=5 -> lower=0.251 upper=0.252 effort=0 velocity=0
- joint right wrist roll: limit lower=0 upper=0.001 effort=24 velocity=5 -> lower=0 upper=0.001 effort=0 velocity=0
- joint right wrist yaw: limit lower=1.38 upper=1.381 effort=24 velocity=5 -> lower=1.38 upper=1.381 effort=0 velocity=0
- joint torso roll: limit lower=-0.502 upper=-0.501 effort=90 velocity=5 -> lower=-0.502 upper=-0.501 effort=0 velocity=0

Commit message: save more realistic efforts and velocities

File: sim/stompy/robot_fixed.urdf (robot description, URDF)
Before this commit: robot robot_7dof_arm, 139 links, 138 joints
Joints:
- joint left ankle pitch: limit lower=0 upper=2 effort=24 velocity=12 -> lower=0 upper=2 effort=24 velocity=24
- joint left ankle roll: limit lower=0.76 upper=2.76 effort=24 velocity=12 -> lower=0.76 upper=2.76 effort=24 velocity=24
- joint left elbow pitch: limit lower=2.07 upper=2.071 effort=24 velocity=5 -> lower=2.06 upper=2.071 effort=24 velocity=12
- joint left shoulder pitch: limit lower=-0.251 upper=-0.25 effort=90 velocity=5 -> lower=-0.252 upper=-0.25 effort=24 velocity=12
- joint left shoulder roll: limit lower=-1.44 upper=-1.439 effort=24 velocity=5 -> lower=-1.45 upper=-1.439 effort=24 velocity=12
- joint left shoulder yaw: limit lower=1.82 upper=1.821 effort=90 velocity=5 -> lower=1.819 upper=1.821 effort=24 velocity=12
- joint left wrist pitch: limit lower=3.33 upper=3.331 effort=24 velocity=5 -> lower=3.32 upper=3.331 effort=24 velocity=12
- joint left wrist roll: limit lower=-2.51 upper=-2.509 effort=24 velocity=5 -> lower=-2.512 upper=-2.509 effort=24 velocity=12
- joint left wrist yaw: limit lower=0.0628 upper=0.0638 effort=24 velocity=5 -> lower=0.062 upper=0.0638 effort=24 velocity=12
- joint right ankle pitch: limit lower=-1.502 upper=0.498 effort=24 velocity=12 -> lower=-1.502 upper=0.498 effort=24 velocity=24
- joint right ankle roll: limit lower=0.76 upper=2.76 effort=24 velocity=12 -> lower=0.76 upper=2.76 effort=24 velocity=24
- joint right elbow pitch: limit lower=-2.57 upper=-2.569 effort=24 velocity=5 -> lower=-2.58 upper=-2.569 effort=24 velocity=12
- joint right shoulder pitch: limit lower=2.7 upper=2.701 effort=90 velocity=5 -> lower=2.69 upper=2.701 effort=24 velocity=12
- joint right shoulder roll: limit lower=-2.57 upper=-2.569 effort=24 velocity=5 -> lower=-2.58 upper=-2.569 effort=24 velocity=12
- joint right shoulder yaw: limit lower=-1.82 upper=-1.819 effort=90 velocity=5 -> lower=-1.83 upper=-1.819 effort=24 velocity=12
- joint right wrist pitch: limit lower=0.251 upper=0.252 effort=24 velocity=5 -> lower=0.25 upper=0.252 effort=24 velocity=12
- joint right wrist roll: limit lower=0 upper=0.001 effort=24 velocity=5 -> lower=-0.01 upper=0.001 effort=24 velocity=12
- joint right wrist yaw: limit lower=1.38 upper=1.381 effort=24 velocity=5 -> lower=1.37 upper=1.381 effort=24 velocity=12
- joint torso roll: limit lower=-0.502 upper=-0.501 effort=90 velocity=5 -> lower=-0.503 upper=-0.501 effort=150 velocity=12

Commit message: higher velocity works with tgs engine

File: sim/stompy/robot_fixed.urdf (robot description, URDF)
Before this commit: robot robot_7dof_arm, 139 links, 138 joints
Joints:
- joint left ankle pitch: limit lower=0 upper=2 effort=24 velocity=24 -> lower=0 upper=2 effort=24 velocity=150
- joint left ankle roll: limit lower=0.76 upper=2.76 effort=24 velocity=24 -> lower=0.76 upper=2.76 effort=24 velocity=150
- joint left elbow pitch: limit lower=2.06 upper=2.071 effort=24 velocity=12 -> lower=2.06 upper=2.071 effort=24 velocity=150
- joint left hip pitch: limit lower=-0.498 upper=1.502 effort=150 velocity=40 -> lower=-0.498 upper=1.502 effort=150 velocity=150
- joint left hip roll: limit lower=-2.57 upper=-0.57 effort=90 velocity=40 -> lower=-2.57 upper=-0.57 effort=90 velocity=150
- joint left hip yaw: limit lower=-3.07 upper=-1.07 effort=90 velocity=40 -> lower=-3.07 upper=-1.07 effort=90 velocity=150
- joint left knee pitch: limit lower=2.39 upper=4.39 effort=90 velocity=40 -> lower=2.39 upper=4.39 effort=90 velocity=150
- joint left shoulder pitch: limit lower=-0.252 upper=-0.25 effort=24 velocity=12 -> lower=-0.252 upper=-0.25 effort=24 velocity=150
- joint left shoulder roll: limit lower=-1.45 upper=-1.439 effort=24 velocity=12 -> lower=-1.45 upper=-1.439 effort=24 velocity=150
- joint left shoulder yaw: limit lower=1.819 upper=1.821 effort=24 velocity=12 -> lower=1.819 upper=1.821 effort=24 velocity=150
- joint left wrist pitch: limit lower=3.32 upper=3.331 effort=24 velocity=12 -> lower=3.32 upper=3.331 effort=24 velocity=150
- joint left wrist roll: limit lower=-2.512 upper=-2.509 effort=24 velocity=12 -> lower=-2.512 upper=-2.509 effort=24 velocity=150
- joint left wrist yaw: limit lower=0.062 upper=0.0638 effort=24 velocity=12 -> lower=0.062 upper=0.0638 effort=24 velocity=150
- joint right ankle pitch: limit lower=-1.502 upper=0.498 effort=24 velocity=24 -> lower=-1.502 upper=0.498 effort=24 velocity=150
- joint right ankle roll: limit lower=0.76 upper=2.76 effort=24 velocity=24 -> lower=0.76 upper=2.76 effort=24 velocity=150
- joint right elbow pitch: limit lower=-2.58 upper=-2.569 effort=24 velocity=12 -> lower=-2.58 upper=-2.569 effort=24 velocity=150
- joint right hip pitch: limit lower=0.13 upper=2.13 effort=150 velocity=40 -> lower=0.13 upper=2.13 effort=150 velocity=150
- joint right hip roll: limit lower=-1 upper=1 effort=90 velocity=40 -> lower=-1 upper=1 effort=90 velocity=150
- joint right hip yaw: limit lower=0.07 upper=2.07 effort=90 velocity=40 -> lower=0.07 upper=2.07 effort=90 velocity=150
- joint right knee pitch: limit lower=-0.121 upper=1.879 effort=90 velocity=40 -> lower=-0.121 upper=1.879 effort=90 velocity=150
- joint right shoulder pitch: limit lower=2.69 upper=2.701 effort=24 velocity=12 -> lower=2.69 upper=2.701 effort=24 velocity=150
- joint right shoulder roll: limit lower=-2.58 upper=-2.569 effort=24 velocity=12 -> lower=-2.58 upper=-2.569 effort=24 velocity=150
- joint right shoulder yaw: limit lower=-1.83 upper=-1.819 effort=24 velocity=12 -> lower=-1.83 upper=-1.819 effort=24 velocity=150
- joint right wrist pitch: limit lower=0.25 upper=0.252 effort=24 velocity=12 -> lower=0.25 upper=0.252 effort=24 velocity=150
- joint right wrist roll: limit lower=-0.01 upper=0.001 effort=24 velocity=12 -> lower=-0.01 upper=0.001 effort=24 velocity=150
- joint right wrist yaw: limit lower=1.37 upper=1.381 effort=24 velocity=12 -> lower=1.37 upper=1.381 effort=24 velocity=150
- joint torso roll: limit lower=-0.503 upper=-0.501 effort=150 velocity=12 -> lower=-0.503 upper=-0.501 effort=150 velocity=150

Commit message: vaguely fixed full robot

File: sim/stompy/robot_fixed.urdf (robot description, URDF)
Before this commit: robot robot_7dof_arm, 139 links, 138 joints
Joints:
- joint left ankle pitch: limit lower=0 upper=2 effort=24 velocity=150 -> lower=0 upper=2 effort=24 velocity=24
- joint left ankle roll: limit lower=0.76 upper=2.76 effort=24 velocity=150 -> lower=0.76 upper=2.76 effort=24 velocity=24
- joint left elbow pitch: limit lower=2.06 upper=2.071 effort=24 velocity=150 -> lower=2.06 upper=2.071 effort=1 velocity=40
- joint left hip pitch: limit lower=-0.498 upper=1.502 effort=150 velocity=150 -> lower=-0.498 upper=1.502 effort=150 velocity=40
- joint left hip roll: limit lower=-2.57 upper=-0.57 effort=90 velocity=150 -> lower=-2.57 upper=-0.57 effort=90 velocity=40
- joint left hip yaw: limit lower=-3.07 upper=-1.07 effort=90 velocity=150 -> lower=-3.07 upper=-1.07 effort=90 velocity=40
- joint left knee pitch: limit lower=2.39 upper=4.39 effort=90 velocity=150 -> lower=2.39 upper=4.39 effort=90 velocity=40
- joint left shoulder pitch: limit lower=-0.252 upper=-0.25 effort=24 velocity=150 -> lower=-0.252 upper=-0.25 effort=1 velocity=5
- joint left shoulder roll: limit lower=-1.45 upper=-1.439 effort=24 velocity=150 -> lower=-1.45 upper=-1.439 effort=1 velocity=40
- joint left shoulder yaw: limit lower=1.819 upper=1.821 effort=24 velocity=150 -> lower=1.819 upper=1.821 effort=1 velocity=40
- joint left wrist pitch: limit lower=3.32 upper=3.331 effort=24 velocity=150 -> lower=3.32 upper=3.331 effort=1 velocity=40
- joint left wrist roll: limit lower=-2.512 upper=-2.509 effort=24 velocity=150 -> lower=-2.512 upper=-2.509 effort=1 velocity=40
- joint left wrist yaw: limit lower=0.062 upper=0.0638 effort=24 velocity=150 -> lower=0.062 upper=0.0638 effort=1 velocity=40
- joint right ankle pitch: limit lower=-1.502 upper=0.498 effort=24 velocity=150 -> lower=-1.502 upper=0.498 effort=24 velocity=24
- joint right ankle roll: limit lower=0.76 upper=2.76 effort=24 velocity=150 -> lower=0.76 upper=2.76 effort=24 velocity=24
- joint right elbow pitch: limit lower=-2.58 upper=-2.569 effort=24 velocity=150 -> lower=-2.58 upper=-2.569 effort=1 velocity=40
- joint right hip pitch: limit lower=0.13 upper=2.13 effort=150 velocity=150 -> lower=0.13 upper=2.13 effort=150 velocity=40
- joint right hip roll: limit lower=-1 upper=1 effort=90 velocity=150 -> lower=-1 upper=1 effort=90 velocity=40
- joint right hip yaw: limit lower=0.07 upper=2.07 effort=90 velocity=150 -> lower=0.07 upper=2.07 effort=90 velocity=40
- joint right knee pitch: limit lower=-0.121 upper=1.879 effort=90 velocity=150 -> lower=-0.121 upper=1.879 effort=90 velocity=40
- joint right shoulder pitch: limit lower=2.69 upper=2.701 effort=24 velocity=150 -> lower=2.69 upper=2.701 effort=1 velocity=5
- joint right shoulder roll: limit lower=-2.58 upper=-2.569 effort=24 velocity=150 -> lower=-2.58 upper=-2.569 effort=1 velocity=40
- joint right shoulder yaw: limit lower=-1.83 upper=-1.819 effort=24 velocity=150 -> lower=-1.83 upper=-1.819 effort=1 velocity=40
- joint right wrist pitch: limit lower=0.25 upper=0.252 effort=24 velocity=150 -> lower=0.25 upper=0.252 effort=1 velocity=40
- joint right wrist roll: limit lower=-0.01 upper=0.001 effort=24 velocity=150 -> lower=-0.01 upper=0.001 effort=1 velocity=40
- joint right wrist yaw: limit lower=1.37 upper=1.381 effort=24 velocity=150 -> lower=1.37 upper=1.381 effort=1 velocity=40
- joint torso roll: limit lower=-0.503 upper=-0.501 effort=150 velocity=150 -> lower=-0.503 upper=-0.501 effort=1 velocity=40
