Commit message: save changes different knee axes

File: sim/stompy_legs/robot_fixed copy.urdf (robot description, URDF)
Before this commit: robot lower_limbs, 47 links, 46 joints
Joints:
- joint left knee pitch: axis 0 0 1 -> 0 0 -1; limit lower=-2.14 upper=-1.0 effort=90 velocity=40 -> lower=0.5 upper=2.5 effort=90 velocity=40
