Commit message: test different axis for left leg knee

File: sim/stompy_legs/robot.urdf (robot description, URDF)
Before this commit: robot lower_limbs, 47 links, 46 joints
Joints:
- joint left ankle pitch: limit lower=-1.5707963 upper=2.1816616 effort=24 velocity=5 -> lower=-0.8 upper=0.6 effort=24 velocity=24
- joint left ankle roll: limit lower=-2.268928 upper=-1.2217305 effort=24 velocity=5 -> lower=1 upper=2.3 effort=24 velocity=24
- joint left hip pitch: limit lower=-4.712389 upper=4.712389 effort=80 velocity=5 -> lower=0.5 upper=2.69 effort=150 velocity=40
- joint left hip roll: limit lower=-3.1415927 upper=0 effort=90 velocity=5 -> lower=-0.5 upper=0.5 effort=90 velocity=40
- joint left hip yaw: limit lower=-1.0471976 upper=2.0943951 effort=90 velocity=5 -> lower=0.5 upper=1.19 effort=90 velocity=40
- joint left knee pitch: axis 0 0 -1 -> 0 0 1; limit lower=-4.712389 upper=4.712389 effort=90 velocity=5 -> lower=-2.14 upper=0.5 effort=90 velocity=40
- joint right ankle pitch: limit lower=-1.5707963 upper=2.1816616 effort=24 velocity=5 -> lower=0 upper=1.5 effort=24 velocity=24
- joint right ankle roll: limit lower=-2.268928 upper=-1.2217305 effort=24 velocity=5 -> lower=1 upper=2.3 effort=24 velocity=24
- joint right hip pitch: limit lower=-4.712389 upper=4.712389 effort=80 velocity=5 -> lower=-1 upper=1 effort=150 velocity=40
- joint right hip roll: limit lower=-3.1415927 upper=3.1415927 effort=90 velocity=5 -> lower=-2.39 upper=-1 effort=90 velocity=40
- joint right hip yaw: limit lower=-4.712389 upper=4.712389 effort=90 velocity=5 -> lower=-2.6 upper=-1.5 effort=90 velocity=40
- joint right knee pitch: limit lower=-4.712389 upper=4.712389 effort=90 velocity=5 -> lower=2.09 upper=3.2 effort=90 velocity=40

Commit message: walking works sidewise but the damping setup works with mujoco

File: sim/stompy_legs/robot.urdf (robot description, URDF)
Before this commit: robot lower_limbs, 47 links, 46 joints
Joints:
- joint left ankle pitch: limit lower=-0.8 upper=0.6 effort=24 velocity=24 -> lower=-1.5707963 upper=2.1816616 effort=24 velocity=5
- joint left ankle roll: limit lower=1 upper=2.3 effort=24 velocity=24 -> lower=-2.268928 upper=-1.2217305 effort=24 velocity=5
- joint left hip pitch: limit lower=0.5 upper=2.69 effort=150 velocity=40 -> lower=-4.712389 upper=4.712389 effort=80 velocity=5
- joint left hip roll: limit lower=-0.5 upper=0.5 effort=90 velocity=40 -> lower=-3.1415927 upper=0 effort=90 velocity=5
- joint left hip yaw: limit lower=0.5 upper=1.19 effort=90 velocity=40 -> lower=-1.0471976 upper=2.0943951 effort=90 velocity=5
- joint left knee pitch: limit lower=-2.14 upper=0.5 effort=90 velocity=40 -> lower=-4.712389 upper=4.712389 effort=90 velocity=5
- joint right ankle pitch: limit lower=0 upper=1.5 effort=24 velocity=24 -> lower=-1.5707963 upper=2.1816616 effort=24 velocity=5
- joint right ankle roll: limit lower=1 upper=2.3 effort=24 velocity=24 -> lower=-2.268928 upper=-1.2217305 effort=24 velocity=5
- joint right hip pitch: limit lower=-1 upper=1 effort=150 velocity=40 -> lower=-4.712389 upper=4.712389 effort=80 velocity=5
- joint right hip roll: limit lower=-2.39 upper=-1 effort=90 velocity=40 -> lower=-3.1415927 upper=3.1415927 effort=90 velocity=5
- joint right hip yaw: limit lower=-2.6 upper=-1.5 effort=90 velocity=40 -> lower=-4.712389 upper=4.712389 effort=90 velocity=5
- joint right knee pitch: limit lower=2.09 upper=3.2 effort=90 velocity=40 -> lower=-4.712389 upper=4.712389 effort=90 velocity=5

Commit message: Add only_legs setup with different simulators (#32)
* adding only legs sim2sim

---------

Co-authored-by: nathanjzhao <nathanzh@stanford.edu>
Co-authored-by: is2ac2 <wlight@emory.edu>
Co-authored-by: wuallenwu <allenwu.12@outlook.com>
Co-authored-by: Stompy McStompyface <stompy@kscale.dev>
Co-authored-by: WT-MM <wesley.maa@gmail.com>

File: sim/stompy_legs/robot.urdf (robot description, URDF)
Before this commit: robot lower_limbs, 47 links, 46 joints
Joints:
- joint left knee pitch: axis 0 0 -1 -> 0 0 1
