Commit message: latest settings for making legs_only ppo realistic

File: sim/stompy_legs/robot_fixed.urdf (robot description, URDF)
Before this commit: robot lower_limbs, 46 links, 45 joints
Joints:
- joint left ankle pitch: limit lower=0.0 upper=1.13 effort=80 velocity=5 -> lower=-0.3 upper=1.13 effort=80 velocity=5
- joint left knee pitch: limit lower=0.5 upper=2.1 effort=80 velocity=5 -> lower=1 upper=3.1 effort=80 velocity=5
- joint right ankle roll: limit lower=1 upper=2 effort=80 velocity=5 -> lower=1 upper=2.3 effort=80 velocity=5
- joint right knee pitch: limit lower=1.84 upper=3 effort=80 velocity=5 -> lower=1.54 upper=3 effort=80 velocity=5

Commit message: newest walking

File: sim/stompy_legs/robot_fixed.urdf (robot description, URDF)
Before this commit: robot lower_limbs, 46 links, 45 joints
Joints:
- joint left ankle pitch: limit lower=-0.3 upper=1.13 effort=80 velocity=5 -> lower=-0.8 upper=0.6 effort=80 velocity=5
- joint left ankle roll: limit lower=1.3 upper=2 effort=80 velocity=5 -> lower=1 upper=5 effort=80 velocity=5
- joint left hip pitch: limit lower=0.5 upper=2.69 effort=80 velocity=5 -> lower=0.25 upper=2.69 effort=80 velocity=5
- joint left knee pitch: limit lower=1 upper=3.1 effort=80 velocity=5 -> lower=0.5 upper=2.5 effort=80 velocity=5
- joint right ankle pitch: limit lower=-0.5 upper=0.94 effort=80 velocity=5 -> lower=0 upper=1.5 effort=80 velocity=5
- joint right hip pitch: limit lower=-1 upper=1 effort=80 velocity=5 -> lower=-1 upper=1.25 effort=80 velocity=5
- joint right knee pitch: limit lower=1.54 upper=3 effort=80 velocity=5 -> lower=1.54 upper=3.5 effort=80 velocity=5

Commit message: saving setup current

File: sim/stompy_legs/robot_fixed.urdf (robot description, URDF)
Before this commit: robot lower_limbs, 46 links, 45 joints
Joints:
- joint left ankle pitch: limit lower=-0.3 upper=1.13 effort=80 velocity=5 -> lower=-0.8 upper=0.6 effort=80 velocity=5
- joint left ankle roll: limit lower=1.3 upper=2 effort=80 velocity=5 -> lower=1 upper=5 effort=80 velocity=5
- joint left knee pitch: limit lower=1 upper=3.1 effort=80 velocity=5 -> lower=0.5 upper=2.5 effort=80 velocity=5
- joint right ankle pitch: limit lower=-0.5 upper=0.94 effort=80 velocity=5 -> lower=0 upper=1.5 effort=80 velocity=5

Commit message: update setup, fix dof pos

File: sim/stompy_legs/robot_fixed.urdf (robot description, URDF)
Before this commit: robot lower_limbs, 46 links, 45 joints
Joints:
- joint left ankle pitch: limit lower=-0.8 upper=0.6 effort=80 velocity=5 -> lower=-0.8 upper=0.6 effort=80 velocity=2.25
- joint left ankle roll: limit lower=1 upper=5 effort=80 velocity=5 -> lower=1 upper=5 effort=80 velocity=2.25
- joint left hip pitch: limit lower=0.5 upper=2.69 effort=80 velocity=5 -> lower=0.5 upper=2.69 effort=80 velocity=2.25
- joint left hip roll: limit lower=-0.5 upper=0.5 effort=80 velocity=5 -> lower=-0.5 upper=0.5 effort=80 velocity=2.25
- joint left hip yaw: limit lower=0.5 upper=1.19 effort=80 velocity=5 -> lower=0.5 upper=1.19 effort=80 velocity=2.25
- joint left knee pitch: limit lower=0.5 upper=2.5 effort=80 velocity=5 -> lower=0.5 upper=2.5 effort=80 velocity=2.25
- joint right ankle pitch: limit lower=0 upper=1.5 effort=80 velocity=5 -> lower=0 upper=1.5 effort=80 velocity=2.25
- joint right ankle roll: limit lower=1 upper=2.3 effort=80 velocity=5 -> lower=1 upper=2.3 effort=80 velocity=2.25
- joint right hip pitch: limit lower=-1 upper=1 effort=80 velocity=5 -> lower=-1 upper=1 effort=80 velocity=2.25
- joint right hip roll: limit lower=-2.39 upper=-1 effort=80 velocity=5 -> lower=-2.39 upper=-1 effort=80 velocity=2.25
- joint right hip yaw: limit lower=-2.2 upper=-1 effort=80 velocity=5 -> lower=-2.2 upper=-1 effort=80 velocity=2.25
- joint right knee pitch: limit lower=1.54 upper=3 effort=80 velocity=5 -> lower=1.54 upper=3 effort=80 velocity=2.25

Commit message: add realisitc values to the urdf but the sim behaves wrongly

File: sim/stompy_legs/robot_fixed.urdf (robot description, URDF)
Before this commit: robot lower_limbs, 46 links, 45 joints
Joints:
- joint left ankle pitch: limit lower=-0.8 upper=0.6 effort=80 velocity=2.25 -> lower=-0.8 upper=0.6 effort=24 velocity=2.4
- joint left ankle roll: limit lower=1 upper=5 effort=80 velocity=2.25 -> lower=1 upper=2.3 effort=24 velocity=2.4
- joint left hip pitch: limit lower=0.5 upper=2.69 effort=80 velocity=2.25 -> lower=0.5 upper=2.69 effort=90 velocity=9
- joint left hip roll: limit lower=-0.5 upper=0.5 effort=80 velocity=2.25 -> lower=-0.5 upper=0.5 effort=90 velocity=9
- joint left hip yaw: limit lower=0.5 upper=1.19 effort=80 velocity=2.25 -> lower=0.5 upper=1.19 effort=90 velocity=9
- joint left knee pitch: limit lower=0.5 upper=2.5 effort=80 velocity=2.25 -> lower=0.5 upper=2.5 effort=90 velocity=9
- joint right ankle pitch: limit lower=0 upper=1.5 effort=80 velocity=2.25 -> lower=0 upper=1.5 effort=24 velocity=2.4
- joint right ankle roll: limit lower=1 upper=2.3 effort=80 velocity=2.25 -> lower=1 upper=2.3 effort=24 velocity=2.4
- joint right hip pitch: limit lower=-1 upper=1 effort=80 velocity=2.25 -> lower=-1 upper=1 effort=90 velocity=9
- joint right hip roll: limit lower=-2.39 upper=-1 effort=80 velocity=2.25 -> lower=-2.39 upper=-1 effort=90 velocity=9
- joint right hip yaw: limit lower=-2.2 upper=-1 effort=80 velocity=2.25 -> lower=-2.2 upper=-1 effort=90 velocity=9
- joint right knee pitch: limit lower=1.54 upper=3 effort=80 velocity=2.25 -> lower=1.54 upper=3 effort=90 velocity=9

Commit message: save last changes for allen

File: sim/stompy_legs/robot_fixed.urdf (robot description, URDF)
Before this commit: robot lower_limbs, 46 links, 45 joints
Joints:
- joint left ankle pitch: limit lower=-0.8 upper=0.6 effort=24 velocity=2.4 -> lower=-0.8 upper=0.6 effort=24 velocity=40
- joint left ankle roll: limit lower=1 upper=2.3 effort=24 velocity=2.4 -> lower=1 upper=2.3 effort=24 velocity=40
- joint left hip pitch: limit lower=0.5 upper=2.69 effort=90 velocity=9 -> lower=0.5 upper=2.69 effort=150 velocity=25
- joint left hip roll: limit lower=-0.5 upper=0.5 effort=90 velocity=9 -> lower=-0.5 upper=0.5 effort=90 velocity=40
- joint left hip yaw: limit lower=0.5 upper=1.19 effort=90 velocity=9 -> lower=0.5 upper=1.19 effort=90 velocity=40
- joint left knee pitch: limit lower=0.5 upper=2.5 effort=90 velocity=9 -> lower=0.5 upper=2.5 effort=90 velocity=40
- joint right ankle pitch: limit lower=0 upper=1.5 effort=24 velocity=2.4 -> lower=0 upper=1.5 effort=24 velocity=40
- joint right ankle roll: limit lower=1 upper=2.3 effort=24 velocity=2.4 -> lower=1 upper=2.3 effort=24 velocity=40
- joint right hip pitch: limit lower=-1 upper=1 effort=90 velocity=9 -> lower=-1 upper=1 effort=150 velocity=25
- joint right hip roll: limit lower=-2.39 upper=-1 effort=90 velocity=9 -> lower=-2.39 upper=-1 effort=90 velocity=40
- joint right hip yaw: limit lower=-2.2 upper=-1 effort=90 velocity=9 -> lower=-2.2 upper=-1 effort=90 velocity=40
- joint right knee pitch: limit lower=1.54 upper=3 effort=90 velocity=9 -> lower=1.54 upper=3 effort=90 velocity=40

Commit message: update legs joints and artifacts

File: sim/stompy_legs/robot_fixed.urdf (robot description, URDF)
Before this commit: robot lower_limbs, 47 links, 46 joints
Joints:
- joint left ankle pitch: axis 0 0 -1 -> 0 0 1; limit lower=-0.8 upper=0.6 effort=24 velocity=24 -> lower=-0.827 upper=1.173 effort=24 velocity=24
- joint left ankle roll: limit lower=1 upper=2.3 effort=24 velocity=24 -> lower=0.75 upper=2.75 effort=24 velocity=24
- joint left hip pitch: axis 0 0 -1 -> 0 0 1; limit lower=0.5 upper=2.69 effort=150 velocity=40 -> lower=-2.2 upper=-0.2 effort=150 velocity=40
- joint left hip roll: limit lower=-0.5 upper=0.5 effort=90 velocity=40 -> lower=-1.03 upper=0.97 effort=90 velocity=40
- joint left hip yaw: limit lower=0.5 upper=1.19 effort=90 velocity=40 -> lower=0.6 upper=1.2 effort=90 velocity=40
- joint left knee pitch: limit lower=-2.14 upper=-1.0 effort=90 velocity=40 -> lower=-2.27 upper=-0.27 effort=90 velocity=40
- joint right ankle pitch: limit lower=0 upper=1.5 effort=24 velocity=24 -> lower=-0.258 upper=1.742 effort=24 velocity=24
- joint right ankle roll: limit lower=1 upper=2.3 effort=24 velocity=24 -> lower=0.69 upper=2.69 effort=24 velocity=24
- joint right hip pitch: limit lower=-1 upper=1 effort=150 velocity=40 -> lower=-0.58 upper=1.42 effort=150 velocity=40
- joint right hip roll: limit lower=-2.39 upper=-1 effort=90 velocity=40 -> lower=-2.65 upper=-0.65 effort=90 velocity=40
- joint right hip yaw: limit lower=-2.6 upper=-1.5 effort=90 velocity=40 -> lower=-2.2 upper=-1.6 effort=90 velocity=40
- joint right knee pitch: axis 0 0 -1 -> 0 0 1; limit lower=2.09 upper=3.2 effort=90 velocity=40 -> lower=2.3 upper=4.3 effort=90 velocity=40
