Commit message: fixing merge

File: sim/h1_2/h1_2_full.urdf (robot description, URDF)
Before this commit: robot h1_5, 56 links, 55 joints
Links:
- link L_hand_base_link: geometry collision mesh filename=meshes/L_hand_base_link.STL; visual mesh filename=meshes/L_hand_base_link.STL
- link L_index_intermediate: geometry collision mesh filename=meshes/link16_L.STL; visual mesh filename=meshes/link16_L.STL
- link L_index_proximal: geometry collision mesh filename=meshes/link15_L.STL; visual mesh filename=meshes/link15_L.STL
- link L_middle_intermediate: geometry collision mesh filename=meshes/link18_L.STL; visual mesh filename=meshes/link18_L.STL
- link L_middle_proximal: geometry collision mesh filename=meshes/link17_L.STL; visual mesh filename=meshes/link17_L.STL
- link L_pinky_intermediate: geometry collision mesh filename=meshes/link22_L.STL; visual mesh filename=meshes/link22_L.STL
- link L_pinky_proximal: geometry collision mesh filename=meshes/link21_L.STL; visual mesh filename=meshes/link21_L.STL
- link L_ring_intermediate: geometry collision mesh filename=meshes/link20_L.STL; visual mesh filename=meshes/link20_L.STL
- link L_ring_proximal: geometry collision mesh filename=meshes/link19_L.STL; visual mesh filename=meshes/link19_L.STL
- link L_thumb_distal: geometry collision mesh filename=meshes/link14_L.STL; visual mesh filename=meshes/link14_L.STL
- link L_thumb_intermediate: geometry collision mesh filename=meshes/link13_L.STL; visual mesh filename=meshes/link13_L.STL
- link L_thumb_proximal: geometry collision mesh filename=meshes/link12_L.STL; visual mesh filename=meshes/link12_L.STL
- link L_thumb_proximal_base: geometry collision mesh filename=meshes/link11_L.STL; visual mesh filename=meshes/link11_L.STL
- link R_hand_base_link: geometry collision mesh filename=meshes/R_hand_base_link.STL; visual mesh filename=meshes/R_hand_base_link.STL
- link R_index_intermediate: geometry collision mesh filename=meshes/link16_R.STL; visual mesh filename=meshes/link16_R.STL
- link R_index_proximal: geometry collision mesh filename=meshes/link15_R.STL; visual mesh filename=meshes/link15_R.STL
- link R_middle_intermediate: geometry collision mesh filename=meshes/link18_R.STL; visual mesh filename=meshes/link18_R.STL
- link R_middle_proximal: geometry collision mesh filename=meshes/link17_R.STL; visual mesh filename=meshes/link17_R.STL
- link R_pinky_intermediate: geometry collision mesh filename=meshes/link22_R.STL; visual mesh filename=meshes/link22_R.STL
- link R_pinky_proximal: geometry collision mesh filename=meshes/link21_R.STL; visual mesh filename=meshes/link21_R.STL
- link R_ring_intermediate: geometry collision mesh filename=meshes/link20_R.STL; visual mesh filename=meshes/link20_R.STL
- link R_ring_proximal: geometry collision mesh filename=meshes/link19_R.STL; visual mesh filename=meshes/link19_R.STL
- link R_thumb_distal: geometry collision mesh filename=meshes/link14_R.STL; visual mesh filename=meshes/link14_R.STL
- link R_thumb_intermediate: geometry collision mesh filename=meshes/link13_R.STL; visual mesh filename=meshes/link13_R.STL
- link R_thumb_proximal: geometry collision mesh filename=meshes/link12_R.STL; visual mesh filename=meshes/link12_R.STL
- link R_thumb_proximal_base: geometry collision mesh filename=meshes/link11_R.STL; visual mesh filename=meshes/link11_R.STL
- link left_ankle_pitch_link: geometry collision mesh filename=meshes/left_ankle_pitch_link.STL; visual mesh filename=meshes/left_ankle_pitch_link.STL
- link left_ankle_roll_link: geometry collision mesh filename=meshes/left_ankle_roll_link.STL; visual mesh filename=meshes/left_ankle_roll_link.STL
- link left_elbow_pitch_link: geometry collision mesh filename=meshes/left_elbow_pitch_link.STL; visual mesh filename=meshes/left_elbow_pitch_link.STL
- link left_elbow_roll_link: geometry collision mesh filename=meshes/left_elbow_roll_link.STL; visual mesh filename=meshes/left_elbow_roll_link.STL
- link left_hip_pitch_link: geometry collision cylinder length=0.2 radius=0.02; visual mesh filename=meshes/left_hip_pitch_link.STL
- link left_hip_roll_link: geometry collision cylinder length=0.01 radius=0.02; visual mesh filename=meshes/left_hip_roll_link.STL
- link left_hip_yaw_link: geometry collision cylinder length=0.02 radius=0.01; visual mesh filename=meshes/left_hip_yaw_link.STL
- link left_shoulder_pitch_link: geometry collision mesh filename=meshes/left_shoulder_pitch_link.STL; visual mesh filename=meshes/left_shoulder_pitch_link.STL
- link left_shoulder_roll_link: geometry collision mesh filename=meshes/left_shoulder_roll_link.STL; visual mesh filename=meshes/left_shoulder_roll_link.STL
- link left_shoulder_yaw_link: geometry collision mesh filename=meshes/left_shoulder_yaw_link.STL; visual mesh filename=meshes/left_shoulder_yaw_link.STL
- link left_wrist_pitch_link: geometry collision mesh filename=meshes/left_wrist_pitch_link.STL; visual mesh filename=meshes/left_wrist_pitch_link.STL
- link pelvis: geometry collision sphere radius=0.05; visual mesh filename=meshes/pelvis.STL
- link right_ankle_pitch_link: geometry collision mesh filename=meshes/right_ankle_pitch_link.STL; visual mesh filename=meshes/right_ankle_pitch_link.STL
- link right_ankle_roll_link: geometry collision mesh filename=meshes/right_ankle_roll_link.STL; visual mesh filename=meshes/right_ankle_roll_link.STL
- link right_elbow_pitch_link: geometry collision mesh filename=meshes/right_elbow_pitch_link.STL; visual mesh filename=meshes/right_elbow_pitch_link.STL
- link right_elbow_roll_link: geometry collision mesh filename=meshes/right_elbow_roll_link.STL; visual mesh filename=meshes/right_elbow_roll_link.STL
- link right_hip_pitch_link: geometry collision cylinder length=0.2 radius=0.02; visual mesh filename=meshes/right_hip_pitch_link.STL
- link right_hip_roll_link: geometry collision cylinder length=0.01 radius=0.02; visual mesh filename=meshes/right_hip_roll_link.STL
- link right_hip_yaw_link: geometry collision cylinder length=0.02 radius=0.01; visual mesh filename=meshes/right_hip_yaw_link.STL
- link right_shoulder_pitch_link: geometry collision mesh filename=meshes/right_shoulder_pitch_link.STL; visual mesh filename=meshes/right_shoulder_pitch_link.STL
- link right_shoulder_roll_link: geometry collision mesh filename=meshes/right_shoulder_roll_link.STL; visual mesh filename=meshes/right_shoulder_roll_link.STL
- link right_shoulder_yaw_link: geometry collision mesh filename=meshes/right_shoulder_yaw_link.STL; visual mesh filename=meshes/right_shoulder_yaw_link.STL
- link right_wrist_pitch_link: geometry collision mesh filename=meshes/right_wrist_pitch_link.STL; visual mesh filename=meshes/right_wrist_pitch_link.STL
Joints:
- joint L_index_intermediate_joint: type fixed -> revolute
- joint L_index_proximal_joint: type fixed -> revolute
- joint L_middle_intermediate_joint: type fixed -> revolute
- joint L_middle_proximal_joint: type fixed -> revolute
- joint L_pinky_intermediate_joint: type fixed -> revolute
- joint L_pinky_proximal_joint: type fixed -> revolute
- joint L_ring_intermediate_joint: type fixed -> revolute
- joint L_ring_proximal_joint: type fixed -> revolute
- joint L_thumb_distal_joint: type fixed -> revolute
- joint L_thumb_intermediate_joint: type fixed -> revolute
- joint L_thumb_proximal_pitch_joint: type fixed -> revolute
- joint L_thumb_proximal_yaw_joint: type fixed -> revolute
- joint R_index_intermediate_joint: type fixed -> revolute
- joint R_index_proximal_joint: type fixed -> revolute
- joint R_middle_intermediate_joint: type fixed -> revolute
- joint R_middle_proximal_joint: type fixed -> revolute
- joint R_pinky_intermediate_joint: type fixed -> revolute
- joint R_pinky_proximal_joint: type fixed -> revolute
- joint R_ring_intermediate_joint: type fixed -> revolute
- joint R_ring_proximal_joint: type fixed -> revolute
- joint R_thumb_distal_joint: type fixed -> revolute
- joint R_thumb_intermediate_joint: type fixed -> revolute
- joint R_thumb_proximal_pitch_joint: type fixed -> revolute
- joint R_thumb_proximal_yaw_joint: type fixed -> revolute
- joint left_elbow_roll_joint: type fixed -> revolute
- joint left_wrist_pitch_joint: type fixed -> revolute
- joint left_wrist_yaw_joint: type fixed -> revolute
- joint right_elbow_roll_joint: type fixed -> revolute
- joint right_wrist_pitch_joint: type fixed -> revolute
- joint right_wrist_yaw_joint: type fixed -> revolute
