Commit message: finalized g1

File: sim/g1/robot_fixed.urdf (robot description, URDF)
Before this commit: robot g1, 44 links, 43 joints
Links:
- link head_link: geometry collision mesh filename=./meshes/head_link.STL; visual mesh filename=./meshes/head_link.STL
- link left_ankle_pitch_link: geometry collision mesh filename=./meshes/left_ankle_pitch_link.STL; visual mesh filename=./meshes/left_ankle_pitch_link.STL
- link left_ankle_roll_link: geometry collision mesh filename=./meshes/left_ankle_roll_link.STL; visual mesh filename=./meshes/left_ankle_roll_link.STL
- link left_elbow_pitch_link: geometry collision mesh filename=./meshes/left_elbow_pitch_link.STL; visual mesh filename=./meshes/left_elbow_pitch_link.STL
- link left_elbow_roll_link: geometry collision mesh filename=./meshes/left_elbow_roll_link.STL; visual mesh filename=./meshes/left_elbow_roll_link.STL
- link left_five_link: geometry collision mesh filename=./meshes/left_five_link.STL; visual mesh filename=./meshes/left_five_link.STL
- link left_four_link: geometry collision mesh filename=./meshes/left_four_link.STL; visual mesh filename=./meshes/left_four_link.STL
- link left_hip_pitch_link: geometry collision mesh filename=./meshes/left_hip_pitch_link.STL; visual mesh filename=./meshes/left_hip_pitch_link.STL
- link left_hip_roll_link: geometry collision mesh filename=./meshes/left_hip_roll_link.STL; visual mesh filename=./meshes/left_hip_roll_link.STL
- link left_hip_yaw_link: geometry collision mesh filename=./meshes/left_hip_yaw_link.STL; visual mesh filename=./meshes/left_hip_yaw_link.STL
- link left_knee_link: geometry collision cylinder length=0.15 radius=0.015; visual mesh filename=./meshes/left_knee_link.STL
- link left_one_link: geometry collision box size=0.02 0.03 0.02; visual mesh filename=./meshes/left_one_link.STL
- link left_palm_link: geometry collision mesh filename=./meshes/left_palm_link.STL; visual mesh filename=./meshes/left_palm_link.STL
- link left_shoulder_pitch_link: geometry collision mesh filename=./meshes/left_shoulder_pitch_link.STL; visual mesh filename=./meshes/left_shoulder_pitch_link.STL
- link left_shoulder_roll_link: geometry collision cylinder length=0.03 radius=0.03; visual mesh filename=./meshes/left_shoulder_roll_link.STL
- link left_shoulder_yaw_link: geometry collision mesh filename=./meshes/left_shoulder_yaw_link.STL; visual mesh filename=./meshes/left_shoulder_yaw_link.STL
- link left_six_link: geometry collision mesh filename=./meshes/left_six_link.STL; visual mesh filename=./meshes/left_six_link.STL
- link left_three_link: geometry collision mesh filename=./meshes/left_three_link.STL; visual mesh filename=./meshes/left_three_link.STL
- link left_two_link: geometry collision mesh filename=./meshes/left_two_link.STL; visual mesh filename=./meshes/left_two_link.STL
- link left_zero_link: geometry visual mesh filename=./meshes/left_zero_link.STL
- link logo_link: geometry collision mesh filename=./meshes/logo_link.STL; visual mesh filename=./meshes/logo_link.STL
- link pelvis: geometry collision mesh filename=./meshes/pelvis.STL; visual mesh filename=./meshes/pelvis.STL
- link pelvis_contour_link: geometry visual mesh filename=./meshes/pelvis_contour_link.STL
- link right_ankle_pitch_link: geometry collision mesh filename=./meshes/right_ankle_pitch_link.STL; visual mesh filename=./meshes/right_ankle_pitch_link.STL
- link right_ankle_roll_link: geometry collision mesh filename=./meshes/right_ankle_roll_link.STL; visual mesh filename=./meshes/right_ankle_roll_link.STL
- link right_elbow_pitch_link: geometry collision mesh filename=./meshes/right_elbow_pitch_link.STL; visual mesh filename=./meshes/right_elbow_pitch_link.STL
- link right_elbow_roll_link: geometry collision mesh filename=./meshes/right_elbow_roll_link.STL; visual mesh filename=./meshes/right_elbow_roll_link.STL
- link right_five_link: geometry collision mesh filename=./meshes/right_five_link.STL; visual mesh filename=./meshes/right_five_link.STL
- link right_four_link: geometry collision mesh filename=./meshes/right_four_link.STL; visual mesh filename=./meshes/right_four_link.STL
- link right_hip_pitch_link: geometry collision mesh filename=./meshes/right_hip_pitch_link.STL; visual mesh filename=./meshes/right_hip_pitch_link.STL
- link right_hip_roll_link: geometry collision mesh filename=./meshes/right_hip_roll_link.STL; visual mesh filename=./meshes/right_hip_roll_link.STL
- link right_hip_yaw_link: geometry collision mesh filename=./meshes/right_hip_yaw_link.STL; visual mesh filename=./meshes/right_hip_yaw_link.STL
- link right_knee_link: geometry collision cylinder length=0.15 radius=0.015; visual mesh filename=./meshes/right_knee_link.STL
- link right_one_link: geometry collision box size=0.02 0.03 0.02; visual mesh filename=./meshes/right_one_link.STL
- link right_palm_link: geometry collision mesh filename=./meshes/right_palm_link.STL; visual mesh filename=./meshes/right_palm_link.STL
- link right_shoulder_pitch_link: geometry collision mesh filename=./meshes/right_shoulder_pitch_link.STL; visual mesh filename=./meshes/right_shoulder_pitch_link.STL
- link right_shoulder_roll_link: geometry collision cylinder length=0.03 radius=0.03; visual mesh filename=./meshes/right_shoulder_roll_link.STL
- link right_shoulder_yaw_link: geometry collision mesh filename=./meshes/right_shoulder_yaw_link.STL; visual mesh filename=./meshes/right_shoulder_yaw_link.STL
- link right_six_link: geometry collision mesh filename=./meshes/right_six_link.STL; visual mesh filename=./meshes/right_six_link.STL
- link right_three_link: geometry collision mesh filename=./meshes/right_three_link.STL; visual mesh filename=./meshes/right_three_link.STL
- link right_two_link: geometry collision mesh filename=./meshes/right_two_link.STL; visual mesh filename=./meshes/right_two_link.STL
- link right_zero_link: geometry visual mesh filename=./meshes/right_zero_link.STL
- link torso_link: geometry collision mesh filename=./meshes/torso_link.STL; visual mesh filename=./meshes/torso_link.STL
