Commit message: added squatting position

File: sim/stompymini/robot_fixed.urdf (robot description, URDF)
Before this commit: robot full_assembly, 253 links, 252 joints
Joints:
- joint left elbow pitch: limit lower=0.2 upper=2.2 effort=17 velocity=40 -> lower=1.2 upper=1.201 effort=17 velocity=40
- joint left hip pitch: limit lower=-1.06 upper=0.94 effort=120 velocity=40 -> lower=-1.28 upper=0.72 effort=120 velocity=40
- joint left knee pitch: limit lower=-1 upper=1 effort=120 velocity=40 -> lower=0 upper=2 effort=120 velocity=40
- joint left shoulder pitch: limit lower=-2.02 upper=-0.02 effort=120 velocity=40 -> lower=-1.02 upper=-1.019 effort=120 velocity=40
- joint left shoulder roll: limit lower=-4.24 upper=-2.24 effort=17 velocity=40 -> lower=-3.24 upper=-3.239 effort=17 velocity=40
- joint left shoulder yaw: limit lower=0.38 upper=2.38 effort=17 velocity=40 -> lower=1.38 upper=1.381 effort=17 velocity=40
- joint left wrist roll: limit lower=-1 upper=1 effort=17 velocity=40 -> lower=0 upper=0.001 effort=17 velocity=40
- joint right elbow pitch: limit lower=0.32 upper=2.32 effort=17 velocity=40 -> lower=1.32 upper=1.321 effort=17 velocity=40
- joint right hip pitch: limit lower=2.06 upper=4.06 effort=120 velocity=40 -> lower=2.55 upper=4.55 effort=120 velocity=40
- joint right knee pitch: limit lower=-1 upper=1 effort=120 velocity=40 -> lower=-2 upper=0 effort=120 velocity=40
- joint right shoulder pitch: limit lower=2.12 upper=4.12 effort=120 velocity=40 -> lower=3.12 upper=3.121 effort=120 velocity=40
- joint right shoulder roll: limit lower=-2.38 upper=-0.38 effort=17 velocity=40 -> lower=-1.38 upper=-1.379 effort=17 velocity=40
- joint right shoulder yaw: limit lower=-2.98 upper=-0.98 effort=17 velocity=40 -> lower=-1.98 upper=-1.979 effort=17 velocity=40
- joint right wrist roll: limit lower=-1 upper=1 effort=17 velocity=40 -> lower=0 upper=0.001 effort=17 velocity=40
