Commit message: fix mini so it walks and stops spinning (#49)
* added squatting position

* stompy no longer flies

* clean up play, add h5py import

* update some more env stuff

* lint

File: sim/stompymini/robot_fixed.urdf (robot description, URDF)
Before this commit: robot full_assembly, 253 links, 252 joints
Links:
- link link_lower_half_assembly_1_hip_assembly_1_hip_left_1: geometry visual mesh filename=./meshes/lower_half_assembly_1_hip_assembly_1_hip_left_1_si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
- link link_lower_half_assembly_1_hip_assembly_1_hip_left_2: geometry visual mesh filename=./meshes/lower_half_assembly_1_hip_assembly_1_hip_left_2_si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
- link link_lower_half_assembly_1_hip_assembly_1_robstride_04_mock_1_rs_04_rotor_1: geometry visual mesh filename=./meshes/lower_half_assembly_1_hip_assembly_1_robstride_04_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
- link link_lower_half_assembly_1_hip_assembly_1_robstride_04_mock_1_rs_04_stator_1: geometry visual mesh filename=./meshes/lower_half_assembly_1_hip_assembly_1_robstride_04_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
- link link_lower_half_assembly_1_hip_assembly_1_robstride_04_mock_2_rs_04_rotor_1: geometry visual mesh filename=./meshes/lower_half_assembly_1_hip_assembly_1_robstride_04_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
- link link_lower_half_assembly_1_hip_assembly_1_robstride_04_mock_2_rs_04_stator_1: geometry visual mesh filename=./meshes/lower_half_assembly_1_hip_assembly_1_robstride_04_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
- link link_lower_half_assembly_1_hip_assembly_1_washer_m4_1: geometry visual mesh filename=./meshes/lower_half_assembly_1_hip_assembly_1_washer_m4_1_s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
- link link_lower_half_assembly_1_hip_assembly_1_washer_m4_10: geometry visual mesh filename=./meshes/lower_half_assembly_1_hip_assembly_1_washer_m4_10_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
- link link_lower_half_assembly_1_hip_assembly_1_washer_m4_11: geometry visual mesh filename=./meshes/lower_half_assembly_1_hip_assembly_1_washer_m4_11_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
- link link_lower_half_assembly_1_hip_assembly_1_washer_m4_12: geometry visual mesh filename=./meshes/lower_half_assembly_1_hip_assembly_1_washer_m4_12_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
- link link_lower_half_assembly_1_hip_assembly_1_washer_m4_2: geometry visual mesh filename=./meshes/lower_half_assembly_1_hip_assembly_1_washer_m4_2_s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
- link link_lower_half_assembly_1_hip_assembly_1_washer_m4_3: geometry visual mesh filename=./meshes/lower_half_assembly_1_hip_assembly_1_washer_m4_3_s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
- link link_lower_half_assembly_1_hip_assembly_1_washer_m4_4: geometry visual mesh filename=./meshes/lower_half_assembly_1_hip_assembly_1_washer_m4_4_s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
- link link_lower_half_assembly_1_hip_assembly_1_washer_m4_5: geometry visual mesh filename=./meshes/lower_half_assembly_1_hip_assembly_1_washer_m4_5_s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
- link link_lower_half_assembly_1_hip_assembly_1_washer_m4_6: geometry visual mesh filename=./meshes/lower_half_assembly_1_hip_assembly_1_washer_m4_6_s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
- link link_lower_half_assembly_1_hip_assembly_1_washer_m4_7: geometry visual mesh filename=./meshes/lower_half_assembly_1_hip_assembly_1_washer_m4_7_s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
- link link_lower_half_assembly_1_hip_assembly_1_washer_m4_8: geometry visual mesh filename=./meshes/lower_half_assembly_1_hip_assembly_1_washer_m4_8_s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
- link link_lower_half_assembly_1_hip_assembly_1_washer_m4_9: geometry visual mesh filename=./meshes/lower_half_assembly_1_hip_assembly_1_washer_m4_9_s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
- link link_lower_half_assembly_1_left_leg_1_7806k63_1: geometry visual mesh filename=./meshes/lower_half_assembly_1_left_leg_1_7806k63_1_simple.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
- link link_lower_half_assembly_1_left_leg_1_7806k63_2: geometry visual mesh filename=./meshes/lower_half_assembly_1_left_leg_1_7806k63_2_simple.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
- link link_lower_half_assembly_1_left_leg_1_7806k63_4: geometry visual mesh filename=./meshes/lower_half_assembly_1_left_leg_1_7806k63_4_simple.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
- link link_lower_half_assembly_1_left_leg_1_calf_left_inner_1: geometry visual mesh filename=./meshes/lower_half_assembly_1_left_leg_1_calf_left_inner_1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
- link link_lower_half_assembly_1_left_leg_1_calf_left_outer_1: geometry visual mesh filename=./meshes/lower_half_assembly_1_left_leg_1_calf_left_outer_1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
- link link_lower_half_assembly_1_left_leg_1_foot_left_inner_1: geometry visual mesh filename=./meshes/lower_half_assembly_1_left_leg_1_foot_left_inner_1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
- link link_lower_half_assembly_1_left_leg_1_foot_left_outter_1: geometry visual mesh filename=./meshes/lower_half_assembly_1_left_leg_1_foot_left_outter_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
- link link_lower_half_assembly_1_left_leg_1_hip_pitch_left_1: geometry visual mesh filename=./meshes/lower_half_assembly_1_left_leg_1_hip_pitch_left_1_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
- link link_lower_half_assembly_1_left_leg_1_hip_pitch_support_1: geometry visual mesh filename=./meshes/lower_half_assembly_1_left_leg_1_hip_pitch_support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
- link link_lower_half_assembly_1_left_leg_1_hip_roll_left_rear_1: geometry visual mesh filename=./meshes/lower_half_assembly_1_left_leg_1_hip_roll_left_rea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
- link link_lower_half_assembly_1_left_leg_1_knee_left_1: geometry visual mesh filename=./meshes/lower_half_assembly_1_left_leg_1_knee_left_1_simpl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
- link link_lower_half_assembly_1_left_leg_1_robstride_01_mock_1_rs_01_rotor_1: geometry visual mesh filename=./meshes/lower_half_assembly_1_left_leg_1_robstride_01_mock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
- link link_lower_half_assembly_1_left_leg_1_robstride_01_mock_1_rs_01_stator_1: geometry visual mesh filename=./meshes/lower_half_assembly_1_left_leg_1_robstride_01_mock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
- link link_lower_half_assembly_1_left_leg_1_robstride_01_mock_2_rs_01_rotor_1: geometry visual mesh filename=./meshes/lower_half_assembly_1_left_leg_1_robstride_01_mock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
- link link_lower_half_assembly_1_left_leg_1_robstride_01_mock_2_rs_01_stator_1: geometry visual mesh filename=./meshes/lower_half_assembly_1_left_leg_1_robstride_01_mock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
- link link_lower_half_assembly_1_left_leg_1_robstride_04_mock_1_rs_04_rotor_1: geometry visual mesh filename=./meshes/lower_half_assembly_1_left_leg_1_robstride_04_mock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
- link link_lower_half_assembly_1_left_leg_1_robstride_04_mock_1_rs_04_stator_1: geometry visual mesh filename=./meshes/lower_half_assembly_1_left_leg_1_robstride_04_mock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
- link link_lower_half_assembly_1_left_leg_1_robstride_04_mock_2_rs_04_rotor_1: geometry visual mesh filename=./meshes/lower_half_assembly_1_left_leg_1_robstride_04_mock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
- link link_lower_half_assembly_1_left_leg_1_robstride_04_mock_2_rs_04_stator_1: geometry visual mesh filename=./meshes/lower_half_assembly_1_left_leg_1_robstride_04_mock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
- link link_lower_half_assembly_1_left_leg_1_washer_m3_13: geometry visual mesh filename=./meshes/lower_half_assembly_1_left_leg_1_washer_m3_13_simp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
- link link_lower_half_assembly_1_left_leg_1_washer_m3_14: geometry visual mesh filename=./meshes/lower_half_assembly_1_left_leg_1_washer_m3_14_simp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
- link link_lower_half_assembly_1_left_leg_1_washer_m3_25: geometry visual mesh filename=./meshes/lower_half_assembly_1_left_leg_1_washer_m3_25_simp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
- link link_lower_half_assembly_1_left_leg_1_washer_m4_10: geometry visual mesh filename=./meshes/lower_half_assembly_1_left_leg_1_washer_m4_10_simp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
- link link_lower_half_assembly_1_left_leg_1_washer_m4_11: geometry visual mesh filename=./meshes/lower_half_assembly_1_left_leg_1_washer_m4_11_simp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
- link link_lower_half_assembly_1_left_leg_1_washer_m4_12: geometry visual mesh filename=./meshes/lower_half_assembly_1_left_leg_1_washer_m4_12_simp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
- link link_lower_half_assembly_1_left_leg_1_washer_m4_19: geometry visual mesh filename=./meshes/lower_half_assembly_1_left_leg_1_washer_m4_19_simp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
- link link_lower_half_assembly_1_left_leg_1_washer_m4_24: geometry visual mesh filename=./meshes/lower_half_assembly_1_left_leg_1_washer_m4_24_simp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
- link link_lower_half_assembly_1_left_leg_1_washer_m4_7: geometry visual mesh filename=./meshes/lower_half_assembly_1_left_leg_1_washer_m4_7_simpl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
- link link_lower_half_assembly_1_left_leg_1_washer_m4_8: geometry visual mesh filename=./meshes/lower_half_assembly_1_left_leg_1_washer_m4_8_simpl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
- link link_lower_half_assembly_1_left_leg_1_washer_m4_9: geometry visual mesh filename=./meshes/lower_half_assembly_1_left_leg_1_washer_m4_9_simpl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
- link link_lower_half_assembly_1_left_leg_1_washer_m5_1: geometry visual mesh filename=./meshes/lower_half_assembly_1_left_leg_1_washer_m5_1_simpl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
- link link_lower_half_assembly_1_left_leg_1_washer_m5_2: geometry visual mesh filename=./meshes/lower_half_assembly_1_left_leg_1_washer_m5_2_simpl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
- link link_lower_half_assembly_1_left_leg_1_washer_m5_3: geometry visual mesh filename=./meshes/lower_half_assembly_1_left_leg_1_washer_m5_3_simpl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
- link link_lower_half_assembly_1_left_leg_1_washer_m5_4: geometry visual mesh filename=./meshes/lower_half_assembly_1_left_leg_1_washer_m5_4_simpl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
- link link_lower_half_assembly_1_left_leg_1_washer_m5_5: geometry visual mesh filename=./meshes/lower_half_assembly_1_left_leg_1_washer_m5_5_simpl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
- link link_lower_half_assembly_1_left_leg_1_washer_m5_6: geometry visual mesh filename=./meshes/lower_half_assembly_1_left_leg_1_washer_m5_6_simpl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
- link link_lower_half_assembly_1_right_leg_1_7806k63_1: geometry visual mesh filename=./meshes/lower_half_assembly_1_right_leg_1_7806k63_1_simple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
- link link_lower_half_assembly_1_right_leg_1_7806k63_2: geometry visual mesh filename=./meshes/lower_half_assembly_1_right_leg_1_7806k63_2_simple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
- link link_lower_half_assembly_1_right_leg_1_7806k63_3: geometry visual mesh filename=./meshes/lower_half_assembly_1_right_leg_1_7806k63_3_simple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
- link link_lower_half_assembly_1_right_leg_1_calf_right_inner_1: geometry visual mesh filename=./meshes/lower_half_assembly_1_right_leg_1_calf_right_inner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
- link link_lower_half_assembly_1_right_leg_1_calf_right_outer_1: geometry visual mesh filename=./meshes/lower_half_assembly_1_right_leg_1_calf_right_outer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
- link link_lower_half_assembly_1_right_leg_1_foot_right_inner_1: geometry visual mesh filename=./meshes/lower_half_assembly_1_right_leg_1_foot_right_inner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
- link link_lower_half_assembly_1_right_leg_1_foot_right_outter_1: geometry visual mesh filename=./meshes/lower_half_assembly_1_right_leg_1_foot_right_outte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
- link link_lower_half_assembly_1_right_leg_1_hip_pitch_right_1: geometry visual mesh filename=./meshes/lower_half_assembly_1_right_leg_1_hip_pitch_right_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
- link link_lower_half_assembly_1_right_leg_1_hip_pitch_support_1: geometry visual mesh filename=./meshes/lower_half_assembly_1_right_leg_1_hip_pitch_suppor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
- link link_lower_half_assembly_1_right_leg_1_hip_roll_right_rear_1: geometry visual mesh filename=./meshes/lower_half_assembly_1_right_leg_1_hip_roll_right_r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
- link link_lower_half_assembly_1_right_leg_1_knee_right_1: geometry visual mesh filename=./meshes/lower_half_assembly_1_right_leg_1_knee_right_1_sim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
- link link_lower_half_assembly_1_right_leg_1_robstride_01_mock_1_rs_01_rotor_1: geometry visual mesh filename=./meshes/lower_half_assembly_1_right_leg_1_robstride_01_moc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
- link link_lower_half_assembly_1_right_leg_1_robstride_01_mock_1_rs_01_stator_1: geometry visual mesh filename=./meshes/lower_half_assembly_1_right_leg_1_robstride_01_moc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
- link link_lower_half_assembly_1_right_leg_1_robstride_01_mock_2_rs_01_rotor_1: geometry visual mesh filename=./meshes/lower_half_assembly_1_right_leg_1_robstride_01_moc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
- link link_lower_half_assembly_1_right_leg_1_robstride_01_mock_2_rs_01_stator_1: geometry visual mesh filename=./meshes/lower_half_assembly_1_right_leg_1_robstride_01_moc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
- link link_lower_half_assembly_1_right_leg_1_robstride_04_mock_1_rs_04_rotor_1: geometry visual mesh filename=./meshes/lower_half_assembly_1_right_leg_1_robstride_04_moc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
- link link_lower_half_assembly_1_right_leg_1_robstride_04_mock_1_rs_04_stator_1: geometry visual mesh filename=./meshes/lower_half_assembly_1_right_leg_1_robstride_04_moc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
- link link_lower_half_assembly_1_right_leg_1_robstride_04_mock_2_rs_04_rotor_1: geometry visual mesh filename=./meshes/lower_half_assembly_1_right_leg_1_robstride_04_moc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
- link link_lower_half_assembly_1_right_leg_1_robstride_04_mock_2_rs_04_stator_1: geometry visual mesh filename=./meshes/lower_half_assembly_1_right_leg_1_robstride_04_moc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
- link link_lower_half_assembly_1_right_leg_1_washer_m3_10: geometry visual mesh filename=./meshes/lower_half_assembly_1_right_leg_1_washer_m3_10_sim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
- link link_lower_half_assembly_1_right_leg_1_washer_m3_7: geometry visual mesh filename=./meshes/lower_half_assembly_1_right_leg_1_washer_m3_7_simp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
- link link_lower_half_assembly_1_right_leg_1_washer_m3_9: geometry visual mesh filename=./meshes/lower_half_assembly_1_right_leg_1_washer_m3_9_simp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
- link link_lower_half_assembly_1_right_leg_1_washer_m4_1: geometry visual mesh filename=./meshes/lower_half_assembly_1_right_leg_1_washer_m4_1_simp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
- link link_lower_half_assembly_1_right_leg_1_washer_m4_2: geometry visual mesh filename=./meshes/lower_half_assembly_1_right_leg_1_washer_m4_2_simp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
- link link_lower_half_assembly_1_right_leg_1_washer_m4_3: geometry visual mesh filename=./meshes/lower_half_assembly_1_right_leg_1_washer_m4_3_simp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
- link link_lower_half_assembly_1_right_leg_1_washer_m4_4: geometry visual mesh filename=./meshes/lower_half_assembly_1_right_leg_1_washer_m4_4_simp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
- link link_lower_half_assembly_1_right_leg_1_washer_m4_5: geometry visual mesh filename=./meshes/lower_half_assembly_1_right_leg_1_washer_m4_5_simp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
- link link_lower_half_assembly_1_right_leg_1_washer_m4_6: geometry visual mesh filename=./meshes/lower_half_assembly_1_right_leg_1_washer_m4_6_simp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
- link link_lower_half_assembly_1_right_leg_1_washer_m4_8: geometry visual mesh filename=./meshes/lower_half_assembly_1_right_leg_1_washer_m4_8_simp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
- link link_upper_half_assembly_1_36v_battery_1: geometry visual mesh filename=./meshes/upper_half_assembly_1_36v_battery_1_simple.stl
- link link_upper_half_assembly_1_back_plate_lower_section_1: geometry visual mesh filename=./meshes/upper_half_assembly_1_back_plate_lower_section_1_s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
- link link_upper_half_assembly_1_back_plate_upper_section_2: geometry visual mesh filename=./meshes/upper_half_assembly_1_back_plate_upper_section_2_s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
- link link_upper_half_assembly_1_breadboard_1: geometry visual mesh filename=./meshes/upper_half_assembly_1_breadboard_1_simple.stl
- link link_upper_half_assembly_1_ethercat_with_board_1: geometry visual mesh filename=./meshes/upper_half_assembly_1_ethercat_with_board_1_simple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
- link link_upper_half_assembly_1_front_plate_bottom_section_1: geometry visual mesh filename=./meshes/upper_half_assembly_1_front_plate_bottom_section_1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
- link link_upper_half_assembly_1_front_plate_top_section_1: geometry visual mesh filename=./meshes/upper_half_assembly_1_front_plate_top_section_1_si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
- link link_upper_half_assembly_1_head_assembly_1_camera_1_board_1: geometry visual mesh filename=./meshes/upper_half_assembly_1_head_assembly_1_camera_1_boa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
- link link_upper_half_assembly_1_head_assembly_1_camera_1_lens_1: geometry visual mesh filename=./meshes/upper_half_assembly_1_head_assembly_1_camera_1_len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
- link link_upper_half_assembly_1_head_assembly_1_camera_2_board_1: geometry visual mesh filename=./meshes/upper_half_assembly_1_head_assembly_1_camera_2_boa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
- link link_upper_half_assembly_1_head_assembly_1_camera_2_lens_1: geometry visual mesh filename=./meshes/upper_half_assembly_1_head_assembly_1_camera_2_len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
- link link_upper_half_assembly_1_head_assembly_1_camera_mount_1: geometry visual mesh filename=./meshes/upper_half_assembly_1_head_assembly_1_camera_mount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
- link link_upper_half_assembly_1_head_assembly_1_head_inner_1: geometry visual mesh filename=./meshes/upper_half_assembly_1_head_assembly_1_head_inner_1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
- link link_upper_half_assembly_1_head_assembly_1_head_outter_1: geometry visual mesh filename=./meshes/upper_half_assembly_1_head_assembly_1_head_outter_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
- link link_upper_half_assembly_1_head_assembly_1_neck_1: geometry visual mesh filename=./meshes/upper_half_assembly_1_head_assembly_1_neck_1_simpl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
- link link_upper_half_assembly_1_left_arm_1_left_arm_part_1a_1: geometry visual mesh filename=./meshes/upper_half_assembly_1_left_arm_1_left_arm_part_1a_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
- link link_upper_half_assembly_1_left_arm_1_left_arm_part_1b_1: geometry visual mesh filename=./meshes/upper_half_assembly_1_left_arm_1_left_arm_part_1b_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
- link link_upper_half_assembly_1_left_arm_1_left_arm_part_2a_1: geometry visual mesh filename=./meshes/upper_half_assembly_1_left_arm_1_left_arm_part_2a_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
- link link_upper_half_assembly_1_left_arm_1_left_arm_part_2b_1: geometry visual mesh filename=./meshes/upper_half_assembly_1_left_arm_1_left_arm_part_2b_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
- link link_upper_half_assembly_1_left_arm_1_left_arm_part_3a_1: geometry visual mesh filename=./meshes/upper_half_assembly_1_left_arm_1_left_arm_part_3a_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
- link link_upper_half_assembly_1_left_arm_1_left_arm_part_3b_1: geometry visual mesh filename=./meshes/upper_half_assembly_1_left_arm_1_left_arm_part_3b_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
- link link_upper_half_assembly_1_left_arm_1_robstride_01_mock_1_rs_01_rotor_1: geometry visual mesh filename=./meshes/upper_half_assembly_1_left_arm_1_robstride_01_mock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
- link link_upper_half_assembly_1_left_arm_1_robstride_01_mock_1_rs_01_stator_1: geometry visual mesh filename=./meshes/upper_half_assembly_1_left_arm_1_robstride_01_mock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
- link link_upper_half_assembly_1_left_arm_1_robstride_01_mock_2_rs_01_rotor_1: geometry visual mesh filename=./meshes/upper_half_assembly_1_left_arm_1_robstride_01_mock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
- link link_upper_half_assembly_1_left_arm_1_robstride_01_mock_2_rs_01_stator_1: geometry visual mesh filename=./meshes/upper_half_assembly_1_left_arm_1_robstride_01_mock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
- link link_upper_half_assembly_1_left_arm_1_robstride_01_mock_3_rs_01_rotor_1: geometry visual mesh filename=./meshes/upper_half_assembly_1_left_arm_1_robstride_01_mock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
- link link_upper_half_assembly_1_left_arm_1_robstride_01_mock_3_rs_01_stator_1: geometry visual mesh filename=./meshes/upper_half_assembly_1_left_arm_1_robstride_01_mock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
- link link_upper_half_assembly_1_left_arm_1_robstride_01_mock_4_rs_01_rotor_1: geometry visual mesh filename=./meshes/upper_half_assembly_1_left_arm_1_robstride_01_mock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
- link link_upper_half_assembly_1_left_arm_1_robstride_01_mock_4_rs_01_stator_1: geometry visual mesh filename=./meshes/upper_half_assembly_1_left_arm_1_robstride_01_mock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
- link link_upper_half_assembly_1_left_arm_1_shoulder_1: geometry visual mesh filename=./meshes/upper_half_assembly_1_left_arm_1_shoulder_1_simple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
- link link_upper_half_assembly_1_left_arm_1_stub_1: geometry visual mesh filename=./meshes/upper_half_assembly_1_left_arm_1_stub_1_simple.stl
- link link_upper_half_assembly_1_left_arm_1_washer_m4_1: geometry visual mesh filename=./meshes/upper_half_assembly_1_left_arm_1_washer_m4_1_simpl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
- link link_upper_half_assembly_1_left_arm_1_washer_m4_10: geometry visual mesh filename=./meshes/upper_half_assembly_1_left_arm_1_washer_m4_10_simp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
- link link_upper_half_assembly_1_left_arm_1_washer_m4_11: geometry visual mesh filename=./meshes/upper_half_assembly_1_left_arm_1_washer_m4_11_simp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
- link link_upper_half_assembly_1_left_arm_1_washer_m4_12: geometry visual mesh filename=./meshes/upper_half_assembly_1_left_arm_1_washer_m4_12_simp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
- link link_upper_half_assembly_1_left_arm_1_washer_m4_13: geometry visual mesh filename=./meshes/upper_half_assembly_1_left_arm_1_washer_m4_13_simp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
- link link_upper_half_assembly_1_left_arm_1_washer_m4_14: geometry visual mesh filename=./meshes/upper_half_assembly_1_left_arm_1_washer_m4_14_simp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
- link link_upper_half_assembly_1_left_arm_1_washer_m4_15: geometry visual mesh filename=./meshes/upper_half_assembly_1_left_arm_1_washer_m4_15_simp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
- link link_upper_half_assembly_1_left_arm_1_washer_m4_16: geometry visual mesh filename=./meshes/upper_half_assembly_1_left_arm_1_washer_m4_16_simp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
- link link_upper_half_assembly_1_left_arm_1_washer_m4_17: geometry visual mesh filename=./meshes/upper_half_assembly_1_left_arm_1_washer_m4_17_simp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
- link link_upper_half_assembly_1_left_arm_1_washer_m4_18: geometry visual mesh filename=./meshes/upper_half_assembly_1_left_arm_1_washer_m4_18_simp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
- link link_upper_half_assembly_1_left_arm_1_washer_m4_19: geometry visual mesh filename=./meshes/upper_half_assembly_1_left_arm_1_washer_m4_19_simp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
- link link_upper_half_assembly_1_left_arm_1_washer_m4_2: geometry visual mesh filename=./meshes/upper_half_assembly_1_left_arm_1_washer_m4_2_simpl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
- link link_upper_half_assembly_1_left_arm_1_washer_m4_20: geometry visual mesh filename=./meshes/upper_half_assembly_1_left_arm_1_washer_m4_20_simp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
- link link_upper_half_assembly_1_left_arm_1_washer_m4_21: geometry visual mesh filename=./meshes/upper_half_assembly_1_left_arm_1_washer_m4_21_simp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
- link link_upper_half_assembly_1_left_arm_1_washer_m4_22: geometry visual mesh filename=./meshes/upper_half_assembly_1_left_arm_1_washer_m4_22_simp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
- link link_upper_half_assembly_1_left_arm_1_washer_m4_23: geometry visual mesh filename=./meshes/upper_half_assembly_1_left_arm_1_washer_m4_23_simp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
- link link_upper_half_assembly_1_left_arm_1_washer_m4_24: geometry visual mesh filename=./meshes/upper_half_assembly_1_left_arm_1_washer_m4_24_simp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
- link link_upper_half_assembly_1_left_arm_1_washer_m4_25: geometry visual mesh filename=./meshes/upper_half_assembly_1_left_arm_1_washer_m4_25_simp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
- link link_upper_half_assembly_1_left_arm_1_washer_m4_26: geometry visual mesh filename=./meshes/upper_half_assembly_1_left_arm_1_washer_m4_26_simp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
- link link_upper_half_assembly_1_left_arm_1_washer_m4_27: geometry visual mesh filename=./meshes/upper_half_assembly_1_left_arm_1_washer_m4_27_simp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
- link link_upper_half_assembly_1_left_arm_1_washer_m4_28: geometry visual mesh filename=./meshes/upper_half_assembly_1_left_arm_1_washer_m4_28_simp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
- link link_upper_half_assembly_1_left_arm_1_washer_m4_29: geometry visual mesh filename=./meshes/upper_half_assembly_1_left_arm_1_washer_m4_29_simp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
- link link_upper_half_assembly_1_left_arm_1_washer_m4_3: geometry visual mesh filename=./meshes/upper_half_assembly_1_left_arm_1_washer_m4_3_simpl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
- link link_upper_half_assembly_1_left_arm_1_washer_m4_30: geometry visual mesh filename=./meshes/upper_half_assembly_1_left_arm_1_washer_m4_30_simp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
- link link_upper_half_assembly_1_left_arm_1_washer_m4_31: geometry visual mesh filename=./meshes/upper_half_assembly_1_left_arm_1_washer_m4_31_simp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
- link link_upper_half_assembly_1_left_arm_1_washer_m4_4: geometry visual mesh filename=./meshes/upper_half_assembly_1_left_arm_1_washer_m4_4_simpl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
- link link_upper_half_assembly_1_left_arm_1_washer_m4_5: geometry visual mesh filename=./meshes/upper_half_assembly_1_left_arm_1_washer_m4_5_simpl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
- link link_upper_half_assembly_1_left_arm_1_washer_m4_6: geometry visual mesh filename=./meshes/upper_half_assembly_1_left_arm_1_washer_m4_6_simpl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
- link link_upper_half_assembly_1_left_arm_1_washer_m4_7: geometry visual mesh filename=./meshes/upper_half_assembly_1_left_arm_1_washer_m4_7_simpl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
- link link_upper_half_assembly_1_left_arm_1_washer_m4_8: geometry visual mesh filename=./meshes/upper_half_assembly_1_left_arm_1_washer_m4_8_simpl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
- link link_upper_half_assembly_1_left_arm_1_washer_m4_9: geometry visual mesh filename=./meshes/upper_half_assembly_1_left_arm_1_washer_m4_9_simpl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
- link link_upper_half_assembly_1_main_case_section_1: geometry visual mesh filename=./meshes/upper_half_assembly_1_main_case_section_1_simple.s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
- link link_upper_half_assembly_1_open_cascade_step_translator_7.5_1.1.1_1: geometry visual mesh filename=./meshes/upper_half_assembly_1_open_cascade_step_translator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
- link link_upper_half_assembly_1_orin_nano_1: geometry visual mesh filename=./meshes/upper_half_assembly_1_orin_nano_1_simple.stl
- link link_upper_half_assembly_1_part_1_2: geometry visual mesh filename=./meshes/upper_half_assembly_1_part_1_2_simple.stl
- link link_upper_half_assembly_1_removable_cap_1: geometry visual mesh filename=./meshes/upper_half_assembly_1_removable_cap_1_simple.stl
- link link_upper_half_assembly_1_right_arm_1_right_arm_part_1a_1: geometry visual mesh filename=./meshes/upper_half_assembly_1_right_arm_1_right_arm_part_1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
- link link_upper_half_assembly_1_right_arm_1_right_arm_part_1b_1: geometry visual mesh filename=./meshes/upper_half_assembly_1_right_arm_1_right_arm_part_1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
- link link_upper_half_assembly_1_right_arm_1_right_arm_part_2a_1: geometry visual mesh filename=./meshes/upper_half_assembly_1_right_arm_1_right_arm_part_2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
- link link_upper_half_assembly_1_right_arm_1_right_arm_part_3a_1: geometry visual mesh filename=./meshes/upper_half_assembly_1_right_arm_1_right_arm_part_3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
- link link_upper_half_assembly_1_right_arm_1_right_arm_part_3b_1: geometry visual mesh filename=./meshes/upper_half_assembly_1_right_arm_1_right_arm_part_3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
- link link_upper_half_assembly_1_right_arm_1_rightt_arm_part_2b_1: geometry visual mesh filename=./meshes/upper_half_assembly_1_right_arm_1_rightt_arm_part_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
- link link_upper_half_assembly_1_right_arm_1_robstride_01_mock_1_rs_01_rotor_1: geometry visual mesh filename=./meshes/upper_half_assembly_1_right_arm_1_robstride_01_moc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
- link link_upper_half_assembly_1_right_arm_1_robstride_01_mock_1_rs_01_stator_1: geometry visual mesh filename=./meshes/upper_half_assembly_1_right_arm_1_robstride_01_moc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
- link link_upper_half_assembly_1_right_arm_1_robstride_01_mock_2_rs_01_rotor_1: geometry visual mesh filename=./meshes/upper_half_assembly_1_right_arm_1_robstride_01_moc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
- link link_upper_half_assembly_1_right_arm_1_robstride_01_mock_2_rs_01_stator_1: geometry visual mesh filename=./meshes/upper_half_assembly_1_right_arm_1_robstride_01_moc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
- link link_upper_half_assembly_1_right_arm_1_robstride_01_mock_3_rs_01_rotor_1: geometry visual mesh filename=./meshes/upper_half_assembly_1_right_arm_1_robstride_01_moc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
- link link_upper_half_assembly_1_right_arm_1_robstride_01_mock_3_rs_01_stator_1: geometry visual mesh filename=./meshes/upper_half_assembly_1_right_arm_1_robstride_01_moc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
- link link_upper_half_assembly_1_right_arm_1_robstride_01_mock_4_rs_01_rotor_1: geometry visual mesh filename=./meshes/upper_half_assembly_1_right_arm_1_robstride_01_moc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
- link link_upper_half_assembly_1_right_arm_1_robstride_01_mock_4_rs_01_stator_1: geometry visual mesh filename=./meshes/upper_half_assembly_1_right_arm_1_robstride_01_moc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
- link link_upper_half_assembly_1_right_arm_1_shoulder_1: geometry visual mesh filename=./meshes/upper_half_assembly_1_right_arm_1_shoulder_1_simpl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
- link link_upper_half_assembly_1_right_arm_1_stub_1: geometry visual mesh filename=./meshes/upper_half_assembly_1_right_arm_1_stub_1_simple.stl
- link link_upper_half_assembly_1_right_arm_1_washer_m4_1: geometry visual mesh filename=./meshes/upper_half_assembly_1_right_arm_1_washer_m4_1_simp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
- link link_upper_half_assembly_1_right_arm_1_washer_m4_10: geometry visual mesh filename=./meshes/upper_half_assembly_1_right_arm_1_washer_m4_10_sim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
- link link_upper_half_assembly_1_right_arm_1_washer_m4_11: geometry visual mesh filename=./meshes/upper_half_assembly_1_right_arm_1_washer_m4_11_sim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
- link link_upper_half_assembly_1_right_arm_1_washer_m4_12: geometry visual mesh filename=./meshes/upper_half_assembly_1_right_arm_1_washer_m4_12_sim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
- link link_upper_half_assembly_1_right_arm_1_washer_m4_13: geometry visual mesh filename=./meshes/upper_half_assembly_1_right_arm_1_washer_m4_13_sim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
- link link_upper_half_assembly_1_right_arm_1_washer_m4_14: geometry visual mesh filename=./meshes/upper_half_assembly_1_right_arm_1_washer_m4_14_sim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
- link link_upper_half_assembly_1_right_arm_1_washer_m4_15: geometry visual mesh filename=./meshes/upper_half_assembly_1_right_arm_1_washer_m4_15_sim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
- link link_upper_half_assembly_1_right_arm_1_washer_m4_16: geometry visual mesh filename=./meshes/upper_half_assembly_1_right_arm_1_washer_m4_16_sim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
- link link_upper_half_assembly_1_right_arm_1_washer_m4_17: geometry visual mesh filename=./meshes/upper_half_assembly_1_right_arm_1_washer_m4_17_sim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
- link link_upper_half_assembly_1_right_arm_1_washer_m4_18: geometry visual mesh filename=./meshes/upper_half_assembly_1_right_arm_1_washer_m4_18_sim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
- link link_upper_half_assembly_1_right_arm_1_washer_m4_19: geometry visual mesh filename=./meshes/upper_half_assembly_1_right_arm_1_washer_m4_19_sim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
- link link_upper_half_assembly_1_right_arm_1_washer_m4_2: geometry visual mesh filename=./meshes/upper_half_assembly_1_right_arm_1_washer_m4_2_simp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
- link link_upper_half_assembly_1_right_arm_1_washer_m4_20: geometry visual mesh filename=./meshes/upper_half_assembly_1_right_arm_1_washer_m4_20_sim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
- link link_upper_half_assembly_1_right_arm_1_washer_m4_21: geometry visual mesh filename=./meshes/upper_half_assembly_1_right_arm_1_washer_m4_21_sim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
- link link_upper_half_assembly_1_right_arm_1_washer_m4_22: geometry visual mesh filename=./meshes/upper_half_assembly_1_right_arm_1_washer_m4_22_sim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
- link link_upper_half_assembly_1_right_arm_1_washer_m4_23: geometry visual mesh filename=./meshes/upper_half_assembly_1_right_arm_1_washer_m4_23_sim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
- link link_upper_half_assembly_1_right_arm_1_washer_m4_24: geometry visual mesh filename=./meshes/upper_half_assembly_1_right_arm_1_washer_m4_24_sim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
- link link_upper_half_assembly_1_right_arm_1_washer_m4_25: geometry visual mesh filename=./meshes/upper_half_assembly_1_right_arm_1_washer_m4_25_sim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
- link link_upper_half_assembly_1_right_arm_1_washer_m4_26: geometry visual mesh filename=./meshes/upper_half_assembly_1_right_arm_1_washer_m4_26_sim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
- link link_upper_half_assembly_1_right_arm_1_washer_m4_27: geometry visual mesh filename=./meshes/upper_half_assembly_1_right_arm_1_washer_m4_27_sim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
- link link_upper_half_assembly_1_right_arm_1_washer_m4_28: geometry visual mesh filename=./meshes/upper_half_assembly_1_right_arm_1_washer_m4_28_sim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
- link link_upper_half_assembly_1_right_arm_1_washer_m4_29: geometry visual mesh filename=./meshes/upper_half_assembly_1_right_arm_1_washer_m4_29_sim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
- link link_upper_half_assembly_1_right_arm_1_washer_m4_3: geometry visual mesh filename=./meshes/upper_half_assembly_1_right_arm_1_washer_m4_3_simp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
- link link_upper_half_assembly_1_right_arm_1_washer_m4_30: geometry visual mesh filename=./meshes/upper_half_assembly_1_right_arm_1_washer_m4_30_sim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
- link link_upper_half_assembly_1_right_arm_1_washer_m4_31: geometry visual mesh filename=./meshes/upper_half_assembly_1_right_arm_1_washer_m4_31_sim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
- link link_upper_half_assembly_1_right_arm_1_washer_m4_32: geometry visual mesh filename=./meshes/upper_half_assembly_1_right_arm_1_washer_m4_32_sim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
- link link_upper_half_assembly_1_right_arm_1_washer_m4_4: geometry visual mesh filename=./meshes/upper_half_assembly_1_right_arm_1_washer_m4_4_simp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
- link link_upper_half_assembly_1_right_arm_1_washer_m4_5: geometry visual mesh filename=./meshes/upper_half_assembly_1_right_arm_1_washer_m4_5_simp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
- link link_upper_half_assembly_1_right_arm_1_washer_m4_6: geometry visual mesh filename=./meshes/upper_half_assembly_1_right_arm_1_washer_m4_6_simp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
- link link_upper_half_assembly_1_right_arm_1_washer_m4_7: geometry visual mesh filename=./meshes/upper_half_assembly_1_right_arm_1_washer_m4_7_simp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
- link link_upper_half_assembly_1_right_arm_1_washer_m4_8: geometry visual mesh filename=./meshes/upper_half_assembly_1_right_arm_1_washer_m4_8_simp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
- link link_upper_half_assembly_1_right_arm_1_washer_m4_9: geometry visual mesh filename=./meshes/upper_half_assembly_1_right_arm_1_washer_m4_9_simp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
- link link_upper_half_assembly_1_robot_side_connector_1: geometry visual mesh filename=./meshes/upper_half_assembly_1_robot_side_connector_1_simpl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
- link link_upper_half_assembly_1_robstride_04_mock_1_rs_04_rotor_1: geometry visual mesh filename=./meshes/upper_half_assembly_1_robstride_04_mock_1_rs_04_ro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
- link link_upper_half_assembly_1_robstride_04_mock_1_rs_04_stator_1: geometry visual mesh filename=./meshes/upper_half_assembly_1_robstride_04_mock_1_rs_04_st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
- link link_upper_half_assembly_1_robstride_04_mock_2_rs_04_rotor_1: geometry visual mesh filename=./meshes/upper_half_assembly_1_robstride_04_mock_2_rs_04_ro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
- link link_upper_half_assembly_1_robstride_04_mock_2_rs_04_stator_1: geometry visual mesh filename=./meshes/upper_half_assembly_1_robstride_04_mock_2_rs_04_st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
- link link_upper_half_assembly_1_standoff_1: geometry visual mesh filename=./meshes/upper_half_assembly_1_standoff_1_simple.stl
- link link_upper_half_assembly_1_standoff_10: geometry visual mesh filename=./meshes/upper_half_assembly_1_standoff_10_simple.stl
- link link_upper_half_assembly_1_standoff_11: geometry visual mesh filename=./meshes/upper_half_assembly_1_standoff_11_simple.stl
- link link_upper_half_assembly_1_standoff_12: geometry visual mesh filename=./meshes/upper_half_assembly_1_standoff_12_simple.stl
- link link_upper_half_assembly_1_standoff_2: geometry visual mesh filename=./meshes/upper_half_assembly_1_standoff_2_simple.stl
- link link_upper_half_assembly_1_standoff_3: geometry visual mesh filename=./meshes/upper_half_assembly_1_standoff_3_simple.stl
- link link_upper_half_assembly_1_standoff_4: geometry visual mesh filename=./meshes/upper_half_assembly_1_standoff_4_simple.stl
- link link_upper_half_assembly_1_standoff_5: geometry visual mesh filename=./meshes/upper_half_assembly_1_standoff_5_simple.stl
- link link_upper_half_assembly_1_standoff_6: geometry visual mesh filename=./meshes/upper_half_assembly_1_standoff_6_simple.stl
- link link_upper_half_assembly_1_standoff_7: geometry visual mesh filename=./meshes/upper_half_assembly_1_standoff_7_simple.stl
- link link_upper_half_assembly_1_standoff_8: geometry visual mesh filename=./meshes/upper_half_assembly_1_standoff_8_simple.stl
- link link_upper_half_assembly_1_standoff_9: geometry visual mesh filename=./meshes/upper_half_assembly_1_standoff_9_simple.stl
- link link_upper_half_assembly_1_torso_bottom_half_1: geometry visual mesh filename=./meshes/upper_half_assembly_1_torso_bottom_half_1_simple.s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
- link link_upper_half_assembly_1_torso_bottom_half_2: geometry visual mesh filename=./meshes/upper_half_assembly_1_torso_bottom_half_2_simple.s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
- link link_upper_half_assembly_1_torso_top_half_2: geometry visual mesh filename=./meshes/upper_half_assembly_1_torso_top_half_2_simple.stl
- link link_upper_half_assembly_1_torso_top_left_1: geometry visual mesh filename=./meshes/upper_half_assembly_1_torso_top_left_1_simple.stl
- link link_upper_half_assembly_1_washer_m4_10: geometry visual mesh filename=./meshes/upper_half_assembly_1_washer_m4_10_simple.stl
- link link_upper_half_assembly_1_washer_m4_11: geometry visual mesh filename=./meshes/upper_half_assembly_1_washer_m4_11_simple.stl
- link link_upper_half_assembly_1_washer_m4_12: geometry visual mesh filename=./meshes/upper_half_assembly_1_washer_m4_12_simple.stl
- link link_upper_half_assembly_1_washer_m4_13: geometry visual mesh filename=./meshes/upper_half_assembly_1_washer_m4_13_simple.stl
- link link_upper_half_assembly_1_washer_m4_14: geometry visual mesh filename=./meshes/upper_half_assembly_1_washer_m4_14_simple.stl
- link link_upper_half_assembly_1_washer_m4_15: geometry visual mesh filename=./meshes/upper_half_assembly_1_washer_m4_15_simple.stl
- link link_upper_half_assembly_1_washer_m4_16: geometry visual mesh filename=./meshes/upper_half_assembly_1_washer_m4_16_simple.stl
- link link_upper_half_assembly_1_washer_m4_17: geometry visual mesh filename=./meshes/upper_half_assembly_1_washer_m4_17_simple.stl
- link link_upper_half_assembly_1_washer_m4_18: geometry visual mesh filename=./meshes/upper_half_assembly_1_washer_m4_18_simple.stl
- link link_upper_half_assembly_1_washer_m4_19: geometry visual mesh filename=./meshes/upper_half_assembly_1_washer_m4_19_simple.stl
- link link_upper_half_assembly_1_washer_m4_20: geometry visual mesh filename=./meshes/upper_half_assembly_1_washer_m4_20_simple.stl
- link link_upper_half_assembly_1_washer_m4_21: geometry visual mesh filename=./meshes/upper_half_assembly_1_washer_m4_21_simple.stl
- link link_upper_half_assembly_1_washer_m4_22: geometry visual mesh filename=./meshes/upper_half_assembly_1_washer_m4_22_simple.stl
- link link_upper_half_assembly_1_washer_m4_23: geometry visual mesh filename=./meshes/upper_half_assembly_1_washer_m4_23_simple.stl
- link link_upper_half_assembly_1_washer_m4_24: geometry visual mesh filename=./meshes/upper_half_assembly_1_washer_m4_24_simple.stl
- link link_upper_half_assembly_1_washer_m4_25: geometry visual mesh filename=./meshes/upper_half_assembly_1_washer_m4_25_simple.stl
- link link_upper_half_assembly_1_washer_m4_26: geometry visual mesh filename=./meshes/upper_half_assembly_1_washer_m4_26_simple.stl
- link link_upper_half_assembly_1_washer_m4_27: geometry visual mesh filename=./meshes/upper_half_assembly_1_washer_m4_27_simple.stl
- link link_upper_half_assembly_1_washer_m4_28: geometry visual mesh filename=./meshes/upper_half_assembly_1_washer_m4_28_simple.stl
- link link_upper_half_assembly_1_washer_m4_29: geometry visual mesh filename=./meshes/upper_half_assembly_1_washer_m4_29_simple.stl
- link link_upper_half_assembly_1_washer_m4_3: geometry visual mesh filename=./meshes/upper_half_assembly_1_washer_m4_3_simple.stl
- link link_upper_half_assembly_1_washer_m4_30: geometry visual mesh filename=./meshes/upper_half_assembly_1_washer_m4_30_simple.stl
- link link_upper_half_assembly_1_washer_m4_31: geometry visual mesh filename=./meshes/upper_half_assembly_1_washer_m4_31_simple.stl
- link link_upper_half_assembly_1_washer_m4_32: geometry visual mesh filename=./meshes/upper_half_assembly_1_washer_m4_32_simple.stl
- link link_upper_half_assembly_1_washer_m4_33: geometry visual mesh filename=./meshes/upper_half_assembly_1_washer_m4_33_simple.stl
- link link_upper_half_assembly_1_washer_m4_34: geometry visual mesh filename=./meshes/upper_half_assembly_1_washer_m4_34_simple.stl
- link link_upper_half_assembly_1_washer_m4_4: geometry visual mesh filename=./meshes/upper_half_assembly_1_washer_m4_4_simple.stl
- link link_upper_half_assembly_1_washer_m4_5: geometry visual mesh filename=./meshes/upper_half_assembly_1_washer_m4_5_simple.stl
- link link_upper_half_assembly_1_washer_m4_6: geometry visual mesh filename=./meshes/upper_half_assembly_1_washer_m4_6_simple.stl
- link link_upper_half_assembly_1_washer_m4_7: geometry visual mesh filename=./meshes/upper_half_assembly_1_washer_m4_7_simple.stl
- link link_upper_half_assembly_1_washer_m4_8: geometry visual mesh filename=./meshes/upper_half_assembly_1_washer_m4_8_simple.stl
- link link_upper_half_assembly_1_washer_m4_9: geometry visual mesh filename=./meshes/upper_half_assembly_1_washer_m4_9_simple.stl
Joints:
- joint left elbow pitch: limit lower=0.2 upper=2.2 effort=17 velocity=40 -> lower=1.2 upper=1.201 effort=17 velocity=40
- joint left hip pitch: limit lower=-1.06 upper=0.94 effort=120 velocity=40 -> lower=-1.28 upper=0.72 effort=120 velocity=40
- joint left knee pitch: limit lower=-1 upper=1 effort=120 velocity=40 -> lower=0 upper=2 effort=120 velocity=40
- joint left shoulder pitch: limit lower=-2.02 upper=-0.02 effort=120 velocity=40 -> lower=-1.02 upper=-1.019 effort=120 velocity=40
- joint left shoulder roll: limit lower=-4.24 upper=-2.24 effort=17 velocity=40 -> lower=-3.24 upper=-3.239 effort=17 velocity=40
- joint left shoulder yaw: limit lower=0.38 upper=2.38 effort=17 velocity=40 -> lower=1.38 upper=1.381 effort=17 velocity=40
- joint left wrist roll: limit lower=-1 upper=1 effort=17 velocity=40 -> lower=0 upper=0.001 effort=17 velocity=40
- joint right elbow pitch: limit lower=0.32 upper=2.32 effort=17 velocity=40 -> lower=1.32 upper=1.321 effort=17 velocity=40
- joint right hip pitch: limit lower=2.06 upper=4.06 effort=120 velocity=40 -> lower=2.55 upper=4.55 effort=120 velocity=40
- joint right knee pitch: limit lower=-1 upper=1 effort=120 velocity=40 -> lower=-2 upper=0 effort=120 velocity=40
- joint right shoulder pitch: limit lower=2.12 upper=4.12 effort=120 velocity=40 -> lower=3.12 upper=3.121 effort=120 velocity=40
- joint right shoulder roll: limit lower=-2.38 upper=-0.38 effort=17 velocity=40 -> lower=-1.38 upper=-1.379 effort=17 velocity=40
- joint right shoulder yaw: limit lower=-2.98 upper=-0.98 effort=17 velocity=40 -> lower=-1.98 upper=-1.979 effort=17 velocity=40
- joint right wrist roll: limit lower=-1 upper=1 effort=17 velocity=40 -> lower=0 upper=0.001 effort=17 velocity=40
