Commit message: added logging

File: sim/stompymini/robot_fixed.urdf (robot description, URDF)
Before this commit: robot full_assembly, 253 links, 252 joints
Joints:
- joint left ankle pitch: limit lower=-2.62 upper=-0.62 effort=17 velocity=40 -> lower=-2.74 upper=-0.74 effort=17 velocity=40
- joint left hip pitch: limit lower=-1.28 upper=0.72 effort=120 velocity=40 -> lower=-1.087 upper=0.913 effort=120 velocity=40
- joint left hip roll: limit lower=0.5 upper=2.5 effort=17 velocity=40 -> lower=0.62 upper=2.62 effort=17 velocity=40
- joint left hip yaw: limit lower=0.62 upper=2.62 effort=120 velocity=40 -> lower=0.55 upper=2.55 effort=120 velocity=40
- joint left knee pitch: limit lower=0 upper=2 effort=120 velocity=40 -> lower=-0.8 upper=1.2 effort=120 velocity=40
- joint left shoulder pitch: limit lower=-1.02 upper=-1.019 effort=120 velocity=40 -> lower=-1.03 upper=-1.009 effort=120 velocity=40
- joint right ankle pitch: limit lower=-0.58 upper=1.42 effort=17 velocity=40 -> lower=-0.83 upper=1.17 effort=17 velocity=40
- joint right hip pitch: limit lower=2.55 upper=4.55 effort=120 velocity=40 -> lower=2.25 upper=4.25 effort=120 velocity=40
- joint right hip roll: limit lower=2.18 upper=4.18 effort=17 velocity=40 -> lower=2.24 upper=4.24 effort=17 velocity=40
- joint right hip yaw: limit lower=2.24 upper=4.24 effort=120 velocity=40 -> lower=2.08 upper=4.08 effort=120 velocity=40
- joint right knee pitch: limit lower=-2 upper=0 effort=120 velocity=40 -> lower=-1.24 upper=0.76 effort=120 velocity=40
