Commit message: dora env and config updates

File: sim/dora/robot_fixed.urdf (robot description, URDF)
Before this commit: robot Dora2_yin, 21 links, 20 joints
Joints:
- joint left ankle pitch: limit lower=-0.28 upper=1.08 effort=27 velocity=100 -> lower=-1.28 upper=1.08 effort=27 velocity=100
- joint right ankle pitch: limit lower=-0.28 upper=1.08 effort=27 velocity=100 -> lower=-1.28 upper=1.08 effort=27 velocity=100
