Commit message: adjustments

File: sim/resources/xbot/robot_fixed.urdf (robot description, URDF)
Before this commit: robot XBot-L, 91 links, 90 joints
Links:
- link base_link: geometry collision box size=0.4 0.4 0.4; visual mesh filename=meshes/base_link.STL
- link left_ankle_pitch_link: geometry visual mesh filename=meshes/left_ankle_pitch_link.STL
- link left_ankle_pitch_linkage1_link: geometry visual mesh filename=meshes/left_ankle_pitch_linkage1_link.STL
- link left_ankle_pitch_linkage2_link: geometry visual mesh filename=meshes/left_ankle_pitch_linkage2_link.STL
- link left_ankle_pitch_motor1_link: geometry visual mesh filename=meshes/left_ankle_pitch_motor1_link.STL
- link left_ankle_pitch_motor2_link: geometry visual mesh filename=meshes/left_ankle_pitch_motor2_link.STL
- link left_ankle_roll_link: geometry collision mesh filename=meshes/left_ankle_roll_link.STL; visual mesh filename=meshes/left_ankle_roll_link.STL
- link left_arm_base_link: geometry collision mesh filename=meshes/left_arm_base_link.STL; visual mesh filename=meshes/left_arm_base_link.STL
- link left_arm_yaw_link: geometry collision mesh filename=meshes/left_arm_yaw_link.STL; visual mesh filename=meshes/left_arm_yaw_link.STL
- link left_elbow_pitch_link: geometry collision mesh filename=meshes/left_elbow_pitch_link.STL; visual mesh filename=meshes/left_elbow_pitch_link.STL
- link left_elbow_yaw_link: geometry collision mesh filename=meshes/left_elbow_yaw_link.STL; visual mesh filename=meshes/left_elbow_yaw_link.STL
- link left_foot_ee_link: geometry visual mesh filename=meshes/left_foot_ee_link.STL
- link left_hand_ee_link: geometry collision mesh filename=meshes/left_hand_ee_link.STL; visual mesh filename=meshes/left_hand_ee_link.STL
- link left_hand_index_rota_link1: geometry collision mesh filename=meshes/left_hand_index_rota_link1.STL; visual mesh filename=meshes/left_hand_index_rota_link1.STL
- link left_hand_index_rota_link2: geometry collision mesh filename=meshes/left_hand_index_rota_link2.STL; visual mesh filename=meshes/left_hand_index_rota_link2.STL
- link left_hand_index_tip: geometry collision mesh filename=meshes/left_hand_index_tip.STL; visual mesh filename=meshes/left_hand_index_tip.STL
- link left_hand_link: geometry collision mesh filename=meshes/left_hand_link.STL; visual mesh filename=meshes/left_hand_link.STL
- link left_hand_mid_link1: geometry collision mesh filename=meshes/left_hand_mid_link1.STL; visual mesh filename=meshes/left_hand_mid_link1.STL
- link left_hand_mid_link2: geometry collision mesh filename=meshes/left_hand_mid_link2.STL; visual mesh filename=meshes/left_hand_mid_link2.STL
- link left_hand_mid_tip: geometry collision mesh filename=meshes/left_hand_mid_tip.STL; visual mesh filename=meshes/left_hand_mid_tip.STL
- link left_hand_pinky_link1: geometry collision mesh filename=meshes/left_hand_pinky_link1.STL; visual mesh filename=meshes/left_hand_pinky_link1.STL
- link left_hand_pinky_link2: geometry collision mesh filename=meshes/left_hand_pinky_link2.STL; visual mesh filename=meshes/left_hand_pinky_link2.STL
- link left_hand_pinky_tip: geometry collision mesh filename=meshes/left_hand_pinky_tip.STL; visual mesh filename=meshes/left_hand_pinky_tip.STL
- link left_hand_ring_link1: geometry collision mesh filename=meshes/left_hand_ring_link1.STL; visual mesh filename=meshes/left_hand_ring_link1.STL
- link left_hand_ring_link2: geometry collision mesh filename=meshes/left_hand_ring_link2.STL; visual mesh filename=meshes/left_hand_ring_link2.STL
- link left_hand_ring_tip: geometry collision mesh filename=meshes/left_hand_ring_tip.STL; visual mesh filename=meshes/left_hand_ring_tip.STL
- link left_hand_thumb_bend_link: geometry collision mesh filename=meshes/left_hand_thumb_bend_link.STL; visual mesh filename=meshes/left_hand_thumb_bend_link.STL
- link left_hand_thumb_rota_link1: geometry collision mesh filename=meshes/left_hand_thumb_rota_link1.STL; visual mesh filename=meshes/left_hand_thumb_rota_link1.STL
- link left_hand_thumb_rota_link2: geometry collision mesh filename=meshes/left_hand_thumb_rota_link2.STL; visual mesh filename=meshes/left_hand_thumb_rota_link2.STL
- link left_hand_thumb_tip: geometry collision mesh filename=meshes/left_hand_thumb_tip.STL; visual mesh filename=meshes/left_hand_thumb_tip.STL
- link left_knee_link: geometry collision mesh filename=meshes/left_knee_link.STL; visual mesh filename=meshes/left_knee_link.STL
- link left_knee_linkage_link: geometry visual mesh filename=meshes/left_knee_linkage_link.STL
- link left_knee_motor_link: geometry visual mesh filename=meshes/left_knee_motor_link.STL
- link left_leg_pitch_link: geometry collision mesh filename=meshes/left_leg_pitch_link.STL; visual mesh filename=meshes/left_leg_pitch_link.STL
- link left_leg_roll_link: geometry visual mesh filename=meshes/left_leg_roll_link.STL
- link left_leg_yaw_link: geometry visual mesh filename=meshes/left_leg_yaw_link.STL
- link left_shoulder_pitch_link: geometry collision mesh filename=meshes/left_shoulder_pitch_link.STL; visual mesh filename=meshes/left_shoulder_pitch_link.STL
- link left_shoulder_roll_link: geometry collision mesh filename=meshes/left_shoulder_roll_link.STL; visual mesh filename=meshes/left_shoulder_roll_link.STL
- link left_wrist_roll_link: geometry collision mesh filename=meshes/left_wrist_roll_link.STL; visual mesh filename=meshes/left_wrist_roll_link.STL
- link left_wrist_yaw_link: geometry visual mesh filename=meshes/left_wrist_yaw_link.STL
- link neck_base_link: geometry collision mesh filename=meshes/neck_base_link.STL; visual mesh filename=meshes/neck_base_link.STL
- link neck_pitch_link: geometry collision mesh filename=meshes/neck_pitch_link.STL; visual mesh filename=meshes/neck_pitch_link.STL
- link neck_yaw_link: geometry collision mesh filename=meshes/neck_yaw_link.STL; visual mesh filename=meshes/neck_yaw_link.STL
- link realsense_link: geometry collision mesh filename=meshes/realsense_link.STL; visual mesh filename=meshes/realsense_link.STL
- link right_ankle_pitch_link: geometry visual mesh filename=meshes/right_ankle_pitch_link.STL
- link right_ankle_pitch_linkage1_link: geometry visual mesh filename=meshes/right_ankle_pitch_linkage1_link.STL
- link right_ankle_pitch_linkage2_link: geometry visual mesh filename=meshes/right_ankle_pitch_linkage2_link.STL
- link right_ankle_pitch_motor1_link: geometry visual mesh filename=meshes/right_ankle_pitch_motor1_link.STL
- link right_ankle_pitch_motor2_link: geometry visual mesh filename=meshes/right_ankle_pitch_motor2_link.STL
- link right_ankle_roll_link: geometry collision mesh filename=meshes/right_ankle_roll_link.STL; visual mesh filename=meshes/right_ankle_roll_link.STL
- link right_arm_base_link: geometry collision mesh filename=meshes/right_arm_base_link.STL; visual mesh filename=meshes/right_arm_base_link.STL
- link right_arm_yaw_link: geometry collision mesh filename=meshes/right_arm_yaw_link.STL; visual mesh filename=meshes/right_arm_yaw_link.STL
- link right_elbow_pitch_link: geometry collision mesh filename=meshes/right_elbow_pitch_link.STL; visual mesh filename=meshes/right_elbow_pitch_link.STL
- link right_elbow_yaw_link: geometry collision mesh filename=meshes/right_elbow_yaw_link.STL; visual mesh filename=meshes/right_elbow_yaw_link.STL
- link right_foot_ee_link: geometry visual mesh filename=meshes/right_foot_ee_link.STL
- link right_hand_ee_link: geometry collision mesh filename=meshes/right_hand_ee_link.STL; visual mesh filename=meshes/right_hand_ee_link.STL
- link right_hand_index_rota_link1: geometry collision mesh filename=meshes/right_hand_index_rota_link1.STL; visual mesh filename=meshes/right_hand_index_rota_link1.STL
- link right_hand_index_rota_link2: geometry collision mesh filename=meshes/right_hand_index_rota_link2.STL; visual mesh filename=meshes/right_hand_index_rota_link2.STL
- link right_hand_index_tip: geometry collision mesh filename=meshes/right_hand_index_tip.STL; visual mesh filename=meshes/right_hand_index_tip.STL
- link right_hand_link: geometry collision mesh filename=meshes/right_hand_link.STL; visual mesh filename=meshes/right_hand_link.STL
- link right_hand_mid_link1: geometry collision mesh filename=meshes/right_hand_mid_link1.STL; visual mesh filename=meshes/right_hand_mid_link1.STL
- link right_hand_mid_link2: geometry collision mesh filename=meshes/right_hand_mid_link2.STL; visual mesh filename=meshes/right_hand_mid_link2.STL
- link right_hand_mid_tip: geometry collision mesh filename=meshes/right_hand_mid_tip.STL; visual mesh filename=meshes/right_hand_mid_tip.STL
- link right_hand_pinky_link1: geometry collision mesh filename=meshes/right_hand_pinky_link1.STL; visual mesh filename=meshes/right_hand_pinky_link1.STL
- link right_hand_pinky_link2: geometry collision mesh filename=meshes/right_hand_pinky_link2.STL; visual mesh filename=meshes/right_hand_pinky_link2.STL
- link right_hand_pinky_tip: geometry collision mesh filename=meshes/right_hand_pinky_tip.STL; visual mesh filename=meshes/right_hand_pinky_tip.STL
- link right_hand_ring_link1: geometry collision mesh filename=meshes/right_hand_ring_link1.STL; visual mesh filename=meshes/right_hand_ring_link1.STL
- link right_hand_ring_link2: geometry collision mesh filename=meshes/right_hand_ring_link2.STL; visual mesh filename=meshes/right_hand_ring_link2.STL
- link right_hand_ring_tip: geometry collision mesh filename=meshes/right_hand_ring_tip.STL; visual mesh filename=meshes/right_hand_ring_tip.STL
- link right_hand_thumb_bend_link: geometry collision mesh filename=meshes/right_hand_thumb_bend_link.STL; visual mesh filename=meshes/right_hand_thumb_bend_link.STL
- link right_hand_thumb_rota_link1: geometry collision mesh filename=meshes/right_hand_thumb_rota_link1.STL; visual mesh filename=meshes/right_hand_thumb_rota_link1.STL
- link right_hand_thumb_rota_link2: geometry collision mesh filename=meshes/right_hand_thumb_rota_link2.STL; visual mesh filename=meshes/right_hand_thumb_rota_link2.STL
- link right_hand_thumb_rota_tip: geometry collision mesh filename=meshes/right_hand_thumb_rota_tip.STL; visual mesh filename=meshes/right_hand_thumb_rota_tip.STL
- link right_knee_link: geometry collision mesh filename=meshes/right_knee_link.STL; visual mesh filename=meshes/right_knee_link.STL
- link right_knee_linkage_link: geometry visual mesh filename=meshes/right_knee_linkage_link.STL
- link right_knee_motor_link: geometry visual mesh filename=meshes/right_knee_motor_link.STL
- link right_leg_pitch_link: geometry collision mesh filename=meshes/right_leg_pitch_link.STL; visual mesh filename=meshes/right_leg_pitch_link.STL
- link right_leg_roll_link: geometry visual mesh filename=meshes/right_leg_roll_link.STL
- link right_leg_yaw_link: geometry visual mesh filename=meshes/right_leg_yaw_link.STL
- link right_shoulder_pitch_link: geometry collision mesh filename=meshes/right_shoulder_pitch_link.STL; visual mesh filename=meshes/right_shoulder_pitch_link.STL
- link right_shoulder_roll_link: geometry collision mesh filename=meshes/right_shoulder_roll_link.STL; visual mesh filename=meshes/right_shoulder_roll_link.STL
- link right_wrist_roll_link: geometry collision mesh filename=meshes/right_wrist_roll_link.STL; visual mesh filename=meshes/right_wrist_roll_link.STL
- link right_wrist_yaw_link: geometry visual mesh filename=meshes/right_wrist_yaw_link.STL
- link waist_roll_link: geometry visual mesh filename=meshes/waist_roll_link.STL
- link waist_yaw_link: geometry visual mesh filename=meshes/waist_yaw_link.STL
