Commit message: add fixed position

File: sim/resources/stompy/robot_fixed.urdf (robot description, URDF)
Before this commit: robot robot, 20 links, 19 joints
Joints:
- joint L_ankle_y: limit lower=-0.698 upper=0.698 effort=17 velocity=0 -> lower=-0.698 upper=0.698 effort=17 velocity=5
- joint L_elbow_x: type revolute -> fixed
- joint L_hip_x: limit lower=-0.523 upper=2.093 effort=60 velocity=0 -> lower=-0.523 upper=2.093 effort=60 velocity=5
- joint L_hip_y: limit lower=-3.14 upper=3.14 effort=120 velocity=0 -> lower=-3.14 upper=3.14 effort=120 velocity=5
- joint L_hip_z: limit lower=-3.14 upper=3.14 effort=60 velocity=0 -> lower=-3.14 upper=3.14 effort=60 velocity=5
- joint L_knee: limit lower=-1.919 upper=1.919 effort=120 velocity=0 -> lower=-1.919 upper=1.919 effort=120 velocity=5
- joint L_shoulder_x: type revolute -> fixed
- joint L_shoulder_y: type revolute -> fixed
- joint L_shoulder_z: type revolute -> fixed
- joint R_ankle_y: limit lower=-0.698 upper=0.698 effort=17 velocity=0 -> lower=-0.698 upper=0.698 effort=17 velocity=5
- joint R_elbow_x: type revolute -> fixed
- joint R_hip_x: limit lower=-2.093 upper=0.523 effort=60 velocity=0 -> lower=-2.093 upper=0.523 effort=60 velocity=5
- joint R_hip_y: limit lower=-3.14 upper=3.14 effort=120 velocity=0 -> lower=-3.14 upper=3.14 effort=120 velocity=5
- joint R_hip_z: limit lower=-3.14 upper=3.14 effort=60 velocity=0 -> lower=-3.14 upper=3.14 effort=60 velocity=5
- joint R_knee: limit lower=-1.919 upper=1.919 effort=120 velocity=0 -> lower=-1.919 upper=1.919 effort=120 velocity=5
- joint R_shoulder_x: type revolute -> fixed
- joint R_shoulder_y: type revolute -> fixed
- joint R_shoulder_z: type revolute -> fixed

Commit message: redner the setup

File: sim/resources/stompy/robot_fixed.urdf (robot description, URDF)
Before this commit: robot robot, 20 links, 19 joints
Joints:
- joint L_ankle_y: limit lower=-0.698 upper=0.698 effort=17 velocity=0 -> lower=-0.698 upper=0.698 effort=17 velocity=5; type fixed -> revolute
- joint L_hip_x: limit lower=-0.523 upper=2.093 effort=60 velocity=0 -> lower=-0.523 upper=2.093 effort=60 velocity=5; type fixed -> revolute
- joint L_hip_y: limit lower=-3.14 upper=3.14 effort=120 velocity=0 -> lower=-3.14 upper=3.14 effort=120 velocity=5; type fixed -> revolute
- joint L_hip_z: limit lower=-3.14 upper=3.14 effort=60 velocity=0 -> lower=-3.14 upper=3.14 effort=60 velocity=5; type fixed -> revolute
- joint L_knee: limit lower=-1.919 upper=1.919 effort=120 velocity=0 -> lower=-1.919 upper=1.919 effort=120 velocity=5; type fixed -> revolute
- joint R_ankle_y: limit lower=-0.698 upper=0.698 effort=17 velocity=0 -> lower=-0.698 upper=0.698 effort=17 velocity=5; type fixed -> revolute
- joint R_hip_x: limit lower=-2.093 upper=0.523 effort=60 velocity=0 -> lower=-2.093 upper=0.523 effort=60 velocity=5; type fixed -> revolute
- joint R_hip_y: limit lower=-3.14 upper=3.14 effort=120 velocity=0 -> lower=-3.14 upper=3.14 effort=120 velocity=5; type fixed -> revolute
- joint R_hip_z: limit lower=-3.14 upper=3.14 effort=60 velocity=0 -> lower=-3.14 upper=3.14 effort=60 velocity=5; type fixed -> revolute
- joint R_knee: limit lower=-1.919 upper=1.919 effort=120 velocity=0 -> lower=-1.919 upper=1.919 effort=120 velocity=5; type fixed -> revolute
