Commit message: logic works with the new setup

File: sim/resources/stompymini/robot.urdf (robot description, URDF)
Before this commit: robot full_assembly, 23 links, 22 joints
Joints:
- removed joint right wrist roll
- added joint right hand roll: type revolute, parent RS_01_Rotor_8, child RS_01_Rotor_10, origin xyz=3.529497187571007e-08 -0.07449999902199926 -0.012501018201999262 rpy=-1.5707963071795865 1.5707963 0.0, axis 0 0 1, limit lower=-4.712389 upper=3.1415927 effort=80 velocity=5

File: sim/resources/stompymini/robot_fixed.urdf (robot description, URDF)
Before this commit: robot full_assembly, 23 links, 22 joints
Joints:
- removed joint right wrist roll
- added joint right hand roll: type revolute, parent RS_01_Rotor_8, child RS_01_Rotor_10, origin xyz=3.529497187571007e-08 -0.07449999902199926 -0.012501018201999262 rpy=-1.5707963071795865 1.5707963 0.0, axis 0 0 1, limit lower=-0.501 upper=0.501 effort=17 velocity=40
- joint left ankle pitch: limit lower=1.4 upper=2.2 effort=17 velocity=40 -> lower=0.9 upper=2.7 effort=17 velocity=40
- joint left elbow pitch: limit lower=-1.56 upper=-1.58 effort=17 velocity=40 -> lower=-2.06 upper=-1.08 effort=17 velocity=40
- joint left hand gripper: limit lower=0 upper=1.57 effort=17 velocity=40 -> lower=-0.5 upper=2.07 effort=17 velocity=40
- joint left hand roll: limit lower=-3.1415927 upper=0 effort=80 velocity=5 -> lower=-2.06 upper=-1.08 effort=17 velocity=40; type fixed -> revolute
- joint left hip pitch: limit lower=-1.14 upper=1.14 effort=120 velocity=40 -> lower=-1.64 upper=1.64 effort=120 velocity=40
- joint left hip roll: limit lower=-3.5 upper=0.5 effort=17 velocity=40 -> lower=-4.0 upper=1.0 effort=17 velocity=40
- joint left hip yaw: limit lower=3.14 upper=5.14 effort=120 velocity=40 -> lower=2.64 upper=5.64 effort=120 velocity=40
- joint left knee pitch: limit lower=-2 upper=0 effort=120 velocity=40 -> lower=-2.5 upper=0.5 effort=120 velocity=40
- joint left shoulder pitch: limit lower=2.54 upper=2.56 effort=120 velocity=40 -> lower=2.04 upper=3.06 effort=120 velocity=40
- joint left shoulder roll: limit lower=3.13 upper=3.14 effort=17 velocity=40 -> lower=2.63 upper=3.64 effort=17 velocity=40
- joint left shoulder yaw: limit lower=1.56 upper=1.58 effort=17 velocity=40 -> lower=-1 upper=2 effort=17 velocity=40
- joint right ankle pitch: limit lower=-1.0 upper=1 effort=17 velocity=40 -> lower=-1.5 upper=0.7 effort=17 velocity=40
- joint right elbow pitch: limit lower=-3.319 upper=3.321 effort=17 velocity=40 -> lower=-3.819 upper=3.821 effort=17 velocity=40
- joint right hand gripper: limit lower=0 upper=1.57 effort=17 velocity=40 -> lower=-0.5 upper=2.07 effort=17 velocity=40
- joint right hip pitch: limit lower=0.55 upper=3.55 effort=120 velocity=40 -> lower=0.05 upper=4.05 effort=120 velocity=40
- joint right hip roll: limit lower=0 upper=3.24 effort=17 velocity=40 -> lower=2.25 upper=4.49 effort=17 velocity=40
- joint right hip yaw: limit lower=2.24 upper=4.24 effort=120 velocity=40 -> lower=1.74 upper=4.74 effort=120 velocity=40
- joint right knee pitch: limit lower=0 upper=2 effort=120 velocity=40 -> lower=-0.5 upper=2.5 effort=120 velocity=40
- joint right shoulder pitch: limit lower=3.119 upper=3.121 effort=120 velocity=40 -> lower=2.619 upper=3.621 effort=120 velocity=40
- joint right shoulder roll: limit lower=-1.381 upper=-1.979 effort=17 velocity=40 -> lower=-1.881 upper=-1.479 effort=17 velocity=40
- joint right shoulder yaw: limit lower=1.981 upper=1.979 effort=17 velocity=40 -> lower=-1.481 upper=1 effort=17 velocity=40
