Commit message: fix pd and urdf effort vel issues for flying quad

File: sim/resources/quadruped/robot.urdf (robot description, URDF)
Before this commit: robot quadruped, 9 links, 8 joints
Joints:
- joint Left_Elbow_Pitch: limit lower=-1.3962634 upper=1.3962634 effort=80 velocity=5 -> lower=-1.3962634 upper=1.3962634 effort=24 velocity=30
- joint Left_Hip_Pitch: limit lower=0 upper=1.5707963 effort=80 velocity=5 -> lower=0 upper=1.5707963 effort=24 velocity=30
- joint Left_Knee_Pitch: limit lower=-1.3962634 upper=1.3962634 effort=80 velocity=5 -> lower=-1.3962634 upper=1.3962634 effort=24 velocity=30
- joint Left_Shoulder_Pitch: limit lower=0 upper=1.2217305 effort=80 velocity=5 -> lower=0 upper=1.2217305 effort=24 velocity=30
- joint Right_Elbow_Pitch: limit lower=-1.3962634 upper=1.3962634 effort=80 velocity=5 -> lower=-1.3962634 upper=1.3962634 effort=24 velocity=30
- joint Right_Hip_Pitch: limit lower=0 upper=1.5707963 effort=80 velocity=5 -> lower=0 upper=1.5707963 effort=24 velocity=30
- joint Right_Knee_Pitch: limit lower=-1.3962634 upper=1.3962634 effort=80 velocity=5 -> lower=-1.3962634 upper=1.3962634 effort=24 velocity=30
- joint Right_Shoulder_Pitch: limit lower=0 upper=1.2217305 effort=80 velocity=5 -> lower=0 upper=1.2217305 effort=24 velocity=30
