Commit message: add arm joints

File: sim/resources/stompymicro/robot_fixed.urdf (robot description, URDF)
Before this commit: robot tla_v02_legs, 12 links, 11 joints
Links:
- added link DRIVING_ROTOR_PLATE_11, mass 0.0704091068; collision mesh filename=meshes/DRIVING_ROTOR_PLATE_11.stl; visual mesh filename=meshes/DRIVING_ROTOR_PLATE_11.stl
- added link DRIVING_ROTOR_PLATE_12, mass 0.0704091068; collision mesh filename=meshes/DRIVING_ROTOR_PLATE_12.stl; visual mesh filename=meshes/DRIVING_ROTOR_PLATE_12.stl
- added link DRIVING_ROTOR_PLATE_13, mass 0.0450552098; collision mesh filename=meshes/DRIVING_ROTOR_PLATE_13.stl; visual mesh filename=meshes/DRIVING_ROTOR_PLATE_13.stl
- added link DRIVING_ROTOR_PLATE_14, mass 0.0450744538; collision mesh filename=meshes/DRIVING_ROTOR_PLATE_14.stl; visual mesh filename=meshes/DRIVING_ROTOR_PLATE_14.stl
- added link LX-16A, mass 0.1093848811; collision mesh filename=meshes/LX-16A.stl; visual mesh filename=meshes/LX-16A.stl
- added link LX-16A_2, mass 0.1093848811; collision mesh filename=meshes/LX-16A_2.stl; visual mesh filename=meshes/LX-16A_2.stl
- link Base_Motor_Mount: mass 0.135498239 -> 0.987160788
- link DRIVING_ROTOR_PLATE_10: mass 0.0450744538 -> 0.0598570834
- link DRIVING_ROTOR_PLATE_3: mass 0.19605975280000001 -> 0.0295473156
- link DRIVING_ROTOR_PLATE_4: mass 0.19605975280000001 -> 0.0295473156
- link DRIVING_ROTOR_PLATE_5: mass 0.0598570834 -> 0.19605975280000001
- link DRIVING_ROTOR_PLATE_6: mass 0.0598570834 -> 0.19605975280000001
- link DRIVING_ROTOR_PLATE_7: mass 0.0704091068 -> 0.0385277488
- link DRIVING_ROTOR_PLATE_8: mass 0.0704091068 -> 0.0385277488
- link DRIVING_ROTOR_PLATE_9: mass 0.0450552098 -> 0.0598570834
Joints:
- added joint Bicep: type revolute, parent DRIVING_ROTOR_PLATE_4, child LX-16A_2, origin xyz=0.018273437430571058 0.01494999951036515 0.029393121151926025 rpy=-1.570796253589793 1.5707962732050307 0.0, axis 0 0 1, limit lower=-1.5707963 upper=1.5707963 effort=80 velocity=5
- added joint Left_Shoulder: type revolute, parent Base_Motor_Mount, child DRIVING_ROTOR_PLATE_4, origin xyz=-0.07131383054661666 -0.023482764740008488 0.10812717280524366 rpy=-3.141592653589792 1.5707962732050302 0.0, axis 0 0 -1, limit lower=-1.5707963 upper=1.5707963 effort=80 velocity=5
- added joint Shoulder: type revolute, parent Base_Motor_Mount, child DRIVING_ROTOR_PLATE_3, origin xyz=0.07131383054661666 -0.023482764740008488 0.10812717280524366 rpy=-3.141592653589792 -1.5707962732050302 0.0, axis 0 0 -1, limit lower=-1.5707963 upper=1.5707963 effort=80 velocity=5
- added joint Shoulder_2: type revolute, parent DRIVING_ROTOR_PLATE_3, child LX-16A, origin xyz=-0.018273437468083912 0.01634999951036515 0.029393121151926025 rpy=-1.5707962535897932 -1.5707962732050302 0.0, axis 0 0 1, limit lower=-1.5707963 upper=1.5707963 effort=80 velocity=5
- added joint Shoulder_3: type revolute, parent LX-16A, child DRIVING_ROTOR_PLATE_7, origin xyz=-1.4993347535741108e-10 -0.07020000022229234 0.0 rpy=0.0 0.0 -3.14159264, axis 0 0 -1, limit lower=-1.5707963 upper=1.5707963 effort=80 velocity=5
- added joint Shoulder_4: type revolute, parent LX-16A_2, child DRIVING_ROTOR_PLATE_8, origin xyz=-1.5347855347735972e-09 -0.0702000019724337 -1.7232110183229565e-09 rpy=0.0 -2.220446049250313e-15 3.1415926071795868, axis 0 0 -1, limit lower=-1.5707963 upper=1.5707963 effort=80 velocity=5
- joint Foot_rotate: child DRIVING_ROTOR_PLATE_9 -> DRIVING_ROTOR_PLATE_13; parent DRIVING_ROTOR_PLATE_7 -> DRIVING_ROTOR_PLATE_11
- joint Foot_rotate_2: child DRIVING_ROTOR_PLATE_10 -> DRIVING_ROTOR_PLATE_14; parent DRIVING_ROTOR_PLATE_8 -> DRIVING_ROTOR_PLATE_12
- joint Hip_Lift_Joint_Limit: child DRIVING_ROTOR_PLATE_3 -> DRIVING_ROTOR_PLATE_5
- joint Hip_Lift_Joint_Limit_2: child DRIVING_ROTOR_PLATE_4 -> DRIVING_ROTOR_PLATE_6
- joint Hip_Pitch_Left: origin xyz=-0.04131383163080649 -0.024183361086076917 -0.0037431400080385063 rpy=-3.1415926071795863 1.5707963 0.0 -> xyz=-0.0428138310841906 -0.023482760616461606 -0.004372827248230849 rpy=-3.1415926071795863 1.5707963 0.0
- joint Hip_Pitch_Right: origin xyz=0.04131383163080649 -0.024183361086076917 -0.0037431400080385063 rpy=-3.1415926071795863 -1.5707963 0.0 -> xyz=0.0413138310841906 -0.023482760686076916 -0.004372827208038505 rpy=-3.1415926071795863 -1.5707963 0.0
- joint Knee_Rotate: child DRIVING_ROTOR_PLATE_7 -> DRIVING_ROTOR_PLATE_11; parent DRIVING_ROTOR_PLATE_5 -> DRIVING_ROTOR_PLATE_9
- joint Knee_Rotate_2: child DRIVING_ROTOR_PLATE_8 -> DRIVING_ROTOR_PLATE_12; parent DRIVING_ROTOR_PLATE_6 -> DRIVING_ROTOR_PLATE_10
- joint Thigh_Rotate: child DRIVING_ROTOR_PLATE_5 -> DRIVING_ROTOR_PLATE_9; origin xyz=-2.4481384211516577e-09 0.05275000029180242 -0.00700000245617689 rpy=1.5707963999999994 6.661338147750939e-16 -3.1415926071795863 -> xyz=-2.44813840727387e-09 0.05275000029180242 -0.0070000024561768966 rpy=1.5707963999999994 0.0 -3.1415926071795863; parent DRIVING_ROTOR_PLATE_3 -> DRIVING_ROTOR_PLATE_5
- joint Thigh_Rotate_2: child DRIVING_ROTOR_PLATE_6 -> DRIVING_ROTOR_PLATE_10; origin xyz=-2.4481384211516577e-09 0.05275000029180242 -0.00700000245617689 rpy=1.5707963999999994 6.661338147750939e-16 -3.1415926071795863 -> xyz=-2.44813840727387e-09 0.05275000029180242 -0.0070000024561768966 rpy=1.5707963999999994 0.0 -3.1415926071795863; parent DRIVING_ROTOR_PLATE_4 -> DRIVING_ROTOR_PLATE_6

Commit message: fixed urdf

File: sim/resources/stompymicro/robot_fixed.urdf (robot description, URDF)
Before this commit: robot torso, 18 links, 17 joints
Joints:
- removed joint Bicep
- removed joint Foot_rotate
- removed joint Foot_rotate_2
- removed joint Hip_Lift_Joint_Limit
- removed joint Hip_Lift_Joint_Limit_2
- removed joint Hip_Pitch_Left
- removed joint Hip_Pitch_Right
- removed joint Knee_Rotate
- removed joint Knee_Rotate_2
- removed joint Left_Shoulder
- removed joint Shoulder
- removed joint Shoulder_2
- removed joint Shoulder_3
- removed joint Shoulder_4
- removed joint Thigh_Rotate
- removed joint Thigh_Rotate_2
- added joint left_ankle_pitch: type revolute, parent DRIVING_ROTOR_PLATE_12, child DRIVING_ROTOR_PLATE_14, origin xyz=-1.204344863420248e-09 0.0552000002775737 -0.00031912410434488224 rpy=4.963083675318156e-23 -2.220446049250313e-15 4.998164106755064e-23, axis 0 0 -1, limit lower=-1.5707963 upper=1.5707963 effort=80 velocity=5
- added joint left_elbow_yaw: type revolute, parent LX-16A_2, child DRIVING_ROTOR_PLATE_8, origin xyz=-1.5347855347735972e-09 -0.0702000019724337 -1.7232110183229565e-09 rpy=0.0 -2.220446049250313e-15 3.1415926071795868, axis 0 0 -1, limit lower=-1.5707963 upper=1.5707963 effort=80 velocity=5
- added joint left_hip_pitch: type revolute, parent Base_Motor_Mount, child DRIVING_ROTOR_PLATE_2, origin xyz=0.0413138310841906 -0.023482760686076916 -0.004372827208038505 rpy=-3.1415926071795863 -1.5707963 0.0, axis 0 0 -1, limit lower=-1.5707963 upper=1.5707963 effort=80 velocity=5
- added joint left_hip_roll: type revolute, parent DRIVING_ROTOR_PLATE_5, child DRIVING_ROTOR_PLATE_9, origin xyz=-2.44813840727387e-09 0.05275000029180242 -0.0070000024561768966 rpy=1.5707963999999994 0.0 -3.1415926071795863, axis 0 0 -1, limit lower=-0.52359878 upper=0.52359878 effort=80 velocity=5
- added joint left_hip_yaw: type revolute, parent DRIVING_ROTOR_PLATE_2, child DRIVING_ROTOR_PLATE_6, origin xyz=-0.007400000327569208 0.016949999801717745 0.02285000258156657 rpy=-1.5707963071795867 1.5707963196152375 0.0, axis 0 0 -1, limit lower=-1.5707963 upper=0.087266463 effort=80 velocity=5
- added joint left_knee_pitch: type revolute, parent DRIVING_ROTOR_PLATE_10, child DRIVING_ROTOR_PLATE_12, origin xyz=-0.01623087751044281 1.0229889869234343e-09 0.04169999999196149 rpy=1.5707963535897935 -4.641020678874952e-08 -1.5707963071795867, axis 0 0 -1, limit lower=-1.5707963 upper=1.5707963 effort=80 velocity=5
- added joint left_shoulder_pitch: type revolute, parent Base_Motor_Mount, child DRIVING_ROTOR_PLATE_3, origin xyz=0.07131383054661666 -0.023482764740008488 0.10812717280524366 rpy=-3.141592653589792 -1.5707962732050302 0.0, axis 0 0 -1, limit lower=-1.5707963 upper=1.5707963 effort=80 velocity=5
- added joint left_shoulder_yaw: type revolute, parent DRIVING_ROTOR_PLATE_3, child LX-16A, origin xyz=-0.018273437468083912 0.01634999951036515 0.029393121151926025 rpy=-1.5707962535897932 -1.5707962732050302 0.0, axis 0 0 1, limit lower=-1.5707963 upper=1.5707963 effort=80 velocity=5
- added joint right_ankle_pitch: type revolute, parent DRIVING_ROTOR_PLATE_11, child DRIVING_ROTOR_PLATE_13, origin xyz=-1.204344863420248e-09 0.0552000002775737 -0.00031912410434488224 rpy=4.963083675318156e-23 -2.220446049250313e-15 4.998164106755064e-23, axis 0 0 -1, limit lower=-1.5707963 upper=1.5707963 effort=80 velocity=5
- added joint right_elbow_yaw: type revolute, parent LX-16A, child DRIVING_ROTOR_PLATE_7, origin xyz=-1.4993347535741108e-10 -0.07020000022229234 0.0 rpy=0.0 0.0 -3.14159264, axis 0 0 -1, limit lower=-1.5707963 upper=1.5707963 effort=80 velocity=5
- added joint right_hip_pitch: type revolute, parent Base_Motor_Mount, child DRIVING_ROTOR_PLATE, origin xyz=-0.0428138310841906 -0.023482760616461606 -0.004372827248230849 rpy=-3.1415926071795863 1.5707963 0.0, axis 0 0 -1, limit lower=-1.5707963 upper=1.5707963 effort=80 velocity=5
- added joint right_hip_roll: type revolute, parent DRIVING_ROTOR_PLATE_6, child DRIVING_ROTOR_PLATE_10, origin xyz=-2.44813840727387e-09 0.05275000029180242 -0.0070000024561768966 rpy=1.5707963999999994 0.0 -3.1415926071795863, axis 0 0 -1, limit lower=-0.52359878 upper=0.52359878 effort=80 velocity=5
- added joint right_hip_yaw: type revolute, parent DRIVING_ROTOR_PLATE, child DRIVING_ROTOR_PLATE_5, origin xyz=0.007399999685828183 0.016450000198282227 0.02284999703643316 rpy=-1.5707962535897932 -1.570796273205031 0.0, axis 0 0 -1, limit lower=-0.087266463 upper=1.5707963 effort=80 velocity=5
- added joint right_knee_pitch: type revolute, parent DRIVING_ROTOR_PLATE_9, child DRIVING_ROTOR_PLATE_11, origin xyz=0.01623087751044278 -1.7762673623633596e-09 0.04169999999196149 rpy=1.5707963535897942 -4.6410206566704915e-08 1.5707963000000003, axis 0 0 -1, limit lower=-1.5707963 upper=1.5707963 effort=80 velocity=5
- added joint right_shoulder_pitch: type revolute, parent Base_Motor_Mount, child DRIVING_ROTOR_PLATE_4, origin xyz=-0.07131383054661666 -0.023482764740008488 0.10812717280524366 rpy=-3.141592653589792 1.5707962732050302 0.0, axis 0 0 -1, limit lower=-1.5707963 upper=1.5707963 effort=80 velocity=5
- added joint right_shoulder_yaw: type revolute, parent DRIVING_ROTOR_PLATE_4, child LX-16A_2, origin xyz=0.018273437430571058 0.01494999951036515 0.029393121151926025 rpy=-1.570796253589793 1.5707962732050307 0.0, axis 0 0 1, limit lower=-1.5707963 upper=1.5707963 effort=80 velocity=5

Commit message: added full body

File: sim/resources/stompymicro/robot_fixed.urdf (robot description, URDF)
Before this commit: robot torso, 18 links, 17 joints
Links:
- link DRIVING_ROTOR_PLATE: mass 0.06789254880000001 -> 0.0679127138
- link DRIVING_ROTOR_PLATE_13: mass 0.0450552098 -> 0.0450744538
- link DRIVING_ROTOR_PLATE_14: mass 0.0450744538 -> 0.0450552098
- link DRIVING_ROTOR_PLATE_2: mass 0.0679127138 -> 0.06789254880000001
Joints:
- joint left_ankle_pitch: child DRIVING_ROTOR_PLATE_14 -> DRIVING_ROTOR_PLATE_13; parent DRIVING_ROTOR_PLATE_12 -> DRIVING_ROTOR_PLATE_11
- joint left_elbow_yaw: child DRIVING_ROTOR_PLATE_8 -> DRIVING_ROTOR_PLATE_7; origin xyz=-1.5347855347735972e-09 -0.0702000019724337 -1.7232110183229565e-09 rpy=0.0 -2.220446049250313e-15 3.1415926071795868 -> xyz=-1.4993347535741108e-10 -0.07020000022229234 0.0 rpy=0.0 0.0 -3.14159264; parent LX-16A_2 -> LX-16A
- joint left_hip_pitch: child DRIVING_ROTOR_PLATE_2 -> DRIVING_ROTOR_PLATE
- joint left_hip_yaw: child DRIVING_ROTOR_PLATE_6 -> DRIVING_ROTOR_PLATE_5; parent DRIVING_ROTOR_PLATE_2 -> DRIVING_ROTOR_PLATE
- joint left_knee_pitch: child DRIVING_ROTOR_PLATE_12 -> DRIVING_ROTOR_PLATE_11; parent DRIVING_ROTOR_PLATE_10 -> DRIVING_ROTOR_PLATE_9
- joint right_ankle_pitch: child DRIVING_ROTOR_PLATE_13 -> DRIVING_ROTOR_PLATE_14; parent DRIVING_ROTOR_PLATE_11 -> DRIVING_ROTOR_PLATE_12
- joint right_elbow_yaw: child DRIVING_ROTOR_PLATE_7 -> DRIVING_ROTOR_PLATE_8; origin xyz=-1.4993347535741108e-10 -0.07020000022229234 0.0 rpy=0.0 0.0 -3.14159264 -> xyz=-1.5347855347735972e-09 -0.0702000019724337 -1.7232110183229565e-09 rpy=0.0 -2.220446049250313e-15 3.1415926071795868; parent LX-16A -> LX-16A_2
- joint right_hip_pitch: child DRIVING_ROTOR_PLATE -> DRIVING_ROTOR_PLATE_2; origin xyz=-0.0428138310841906 -0.023482760616461606 -0.004372827248230849 rpy=-3.1415926071795863 1.5707963 0.0 -> xyz=-0.04131383051044278 -0.023482760691961528 -0.004372827208038465 rpy=-3.1415925803846902 1.570796288901191 0.0
- joint right_hip_yaw: child DRIVING_ROTOR_PLATE_5 -> DRIVING_ROTOR_PLATE_6; parent DRIVING_ROTOR_PLATE -> DRIVING_ROTOR_PLATE_2
- joint right_knee_pitch: child DRIVING_ROTOR_PLATE_11 -> DRIVING_ROTOR_PLATE_12; parent DRIVING_ROTOR_PLATE_9 -> DRIVING_ROTOR_PLATE_10

Commit message: adjust parameters in urdf

File: sim/resources/stompymicro/robot_fixed.urdf (robot description, URDF)
Before this commit: robot torso, 18 links, 17 joints
Joints:
- joint left_ankle_pitch: limit lower=-1.5707963 upper=1.5707963 effort=80 velocity=5 -> lower=-1.5707963 upper=1.5707963 effort=1 velocity=20
- joint left_elbow_yaw: limit lower=-1.5707963 upper=1.5707963 effort=80 velocity=5 -> lower=-1.5707963 upper=1.5707963 effort=1 velocity=20
- joint left_hip_pitch: limit lower=-1.5707963 upper=1.5707963 effort=80 velocity=5 -> lower=-1.5707963 upper=1.5707963 effort=1 velocity=20
- joint left_hip_roll: limit lower=-0.52359878 upper=0.52359878 effort=80 velocity=5 -> lower=-0.52359878 upper=0.52359878 effort=1 velocity=20
- joint left_hip_yaw: limit lower=-1.5707963 upper=0.087266463 effort=80 velocity=5 -> lower=-1.5707963 upper=0.087266463 effort=1 velocity=20
- joint left_knee_pitch: limit lower=-1.5707963 upper=1.5707963 effort=80 velocity=5 -> lower=-1.5707963 upper=1.5707963 effort=1 velocity=20
- joint left_shoulder_pitch: limit lower=-1.5707963 upper=1.5707963 effort=80 velocity=5 -> lower=-1.5707963 upper=1.5707963 effort=1 velocity=20
- joint left_shoulder_yaw: limit lower=-1.5707963 upper=1.5707963 effort=80 velocity=5 -> lower=-1.5707963 upper=1.5707963 effort=1 velocity=20
- joint right_ankle_pitch: limit lower=-1.5707963 upper=1.5707963 effort=80 velocity=5 -> lower=-1.5707963 upper=1.5707963 effort=1 velocity=20
- joint right_elbow_yaw: limit lower=-1.5707963 upper=1.5707963 effort=80 velocity=5 -> lower=-1.5707963 upper=1.5707963 effort=1 velocity=20
- joint right_hip_pitch: limit lower=-1.5707963 upper=1.5707963 effort=80 velocity=5 -> lower=-1.5707963 upper=1.5707963 effort=1 velocity=20
- joint right_hip_roll: limit lower=-0.52359878 upper=0.52359878 effort=80 velocity=5 -> lower=-0.52359878 upper=0.52359878 effort=1 velocity=20
- joint right_hip_yaw: limit lower=-0.087266463 upper=1.5707963 effort=80 velocity=5 -> lower=-0.087266463 upper=1.5707963 effort=1 velocity=20
- joint right_knee_pitch: limit lower=-1.5707963 upper=1.5707963 effort=80 velocity=5 -> lower=-1.5707963 upper=1.5707963 effort=1 velocity=20
- joint right_shoulder_pitch: limit lower=-1.5707963 upper=1.5707963 effort=80 velocity=5 -> lower=-1.5707963 upper=1.5707963 effort=1 velocity=20
- joint right_shoulder_yaw: limit lower=-1.5707963 upper=1.5707963 effort=80 velocity=5 -> lower=-1.5707963 upper=1.5707963 effort=1 velocity=20

Commit message: update the config and fixed arms

File: sim/resources/stompymicro/robot_fixed.urdf (robot description, URDF)
Before this commit: robot torso, 18 links, 17 joints
Joints:
- joint left_elbow_yaw: type revolute -> fixed
- joint left_shoulder_pitch: type revolute -> fixed
- joint left_shoulder_yaw: type revolute -> fixed
- joint right_elbow_yaw: type revolute -> fixed
- joint right_shoulder_pitch: type revolute -> fixed
- joint right_shoulder_yaw: type revolute -> fixed

Commit message: stompy micro - adjust parameters in urdf (#89)
* adjust parameters in urdf

* update to the reward default

* all actuators work now

* update the termination joints

* latest setup

* update the config and fixed arms

* saving more robust setup

File: sim/resources/stompymicro/robot_fixed.urdf (robot description, URDF)
Before this commit: robot torso, 18 links, 17 joints
Joints:
- joint left_ankle_pitch: limit lower=-1.5707963 upper=1.5707963 effort=80 velocity=5 -> lower=-1.5707963 upper=1.5707963 effort=1 velocity=20
- joint left_elbow_yaw: limit lower=-1.5707963 upper=1.5707963 effort=80 velocity=5 -> lower=-1.5707963 upper=1.5707963 effort=1 velocity=20; type revolute -> fixed
- joint left_hip_pitch: limit lower=-1.5707963 upper=1.5707963 effort=80 velocity=5 -> lower=-1.5707963 upper=1.5707963 effort=1 velocity=20
- joint left_hip_roll: limit lower=-0.52359878 upper=0.52359878 effort=80 velocity=5 -> lower=-0.52359878 upper=0.52359878 effort=1 velocity=20
- joint left_hip_yaw: limit lower=-1.5707963 upper=0.087266463 effort=80 velocity=5 -> lower=-1.5707963 upper=0.087266463 effort=1 velocity=20
- joint left_knee_pitch: limit lower=-1.5707963 upper=1.5707963 effort=80 velocity=5 -> lower=-1.5707963 upper=1.5707963 effort=1 velocity=20
- joint left_shoulder_pitch: limit lower=-1.5707963 upper=1.5707963 effort=80 velocity=5 -> lower=-1.5707963 upper=1.5707963 effort=1 velocity=20; type revolute -> fixed
- joint left_shoulder_yaw: limit lower=-1.5707963 upper=1.5707963 effort=80 velocity=5 -> lower=-1.5707963 upper=1.5707963 effort=1 velocity=20; type revolute -> fixed
- joint right_ankle_pitch: limit lower=-1.5707963 upper=1.5707963 effort=80 velocity=5 -> lower=-1.5707963 upper=1.5707963 effort=1 velocity=20
- joint right_elbow_yaw: limit lower=-1.5707963 upper=1.5707963 effort=80 velocity=5 -> lower=-1.5707963 upper=1.5707963 effort=1 velocity=20; type revolute -> fixed
- joint right_hip_pitch: limit lower=-1.5707963 upper=1.5707963 effort=80 velocity=5 -> lower=-1.5707963 upper=1.5707963 effort=1 velocity=20
- joint right_hip_roll: limit lower=-0.52359878 upper=0.52359878 effort=80 velocity=5 -> lower=-0.52359878 upper=0.52359878 effort=1 velocity=20
- joint right_hip_yaw: limit lower=-0.087266463 upper=1.5707963 effort=80 velocity=5 -> lower=-0.087266463 upper=1.5707963 effort=1 velocity=20
- joint right_knee_pitch: limit lower=-1.5707963 upper=1.5707963 effort=80 velocity=5 -> lower=-1.5707963 upper=1.5707963 effort=1 velocity=20
- joint right_shoulder_pitch: limit lower=-1.5707963 upper=1.5707963 effort=80 velocity=5 -> lower=-1.5707963 upper=1.5707963 effort=1 velocity=20; type revolute -> fixed
- joint right_shoulder_yaw: limit lower=-1.5707963 upper=1.5707963 effort=80 velocity=5 -> lower=-1.5707963 upper=1.5707963 effort=1 velocity=20; type revolute -> fixed
