Commit message: urdf for V0.3.1

File: sim/resources/stompymicro/robot_fixed.urdf (robot description, URDF)
Before this commit: robot torso, 18 links, 17 joints
Links:
- removed link Base_Motor_Mount
- removed link DRIVING_ROTOR_PLATE
- removed link DRIVING_ROTOR_PLATE_10
- removed link DRIVING_ROTOR_PLATE_11
- removed link DRIVING_ROTOR_PLATE_12
- removed link DRIVING_ROTOR_PLATE_13
- removed link DRIVING_ROTOR_PLATE_14
- removed link DRIVING_ROTOR_PLATE_2
- removed link DRIVING_ROTOR_PLATE_3
- removed link DRIVING_ROTOR_PLATE_4
- removed link DRIVING_ROTOR_PLATE_5
- removed link DRIVING_ROTOR_PLATE_6
- removed link DRIVING_ROTOR_PLATE_7
- removed link DRIVING_ROTOR_PLATE_8
- removed link DRIVING_ROTOR_PLATE_9
- removed link LX-16A
- removed link LX-16A_2
- added link Left_Hand, mass 0.075184887; collision mesh filename=meshes/Left_Hand.stl; visual mesh filename=meshes/Left_Hand.stl
- added link Torso, mass 1.5697539312; collision mesh filename=meshes/Torso.stl; visual mesh filename=meshes/Torso.stl
- added link ankle_pitch_left, mass 0.109625115; collision mesh filename=meshes/ankle_pitch_left.stl; visual mesh filename=meshes/ankle_pitch_left.stl
- added link ankle_pitch_right, mass 0.109625116; collision mesh filename=meshes/ankle_pitch_right.stl; visual mesh filename=meshes/ankle_pitch_right.stl
- added link foot_left, mass 0.04062216; collision mesh filename=meshes/foot_left.stl; visual mesh filename=meshes/foot_left.stl
- added link foot_right, mass 0.040622158; collision mesh filename=meshes/foot_right.stl; visual mesh filename=meshes/foot_right.stl
- added link hand_right, mass 0.075183656; collision mesh filename=meshes/hand_right.stl; visual mesh filename=meshes/hand_right.stl
- added link hip_roll_left, mass 0.111293526; collision mesh filename=meshes/hip_roll_left.stl; visual mesh filename=meshes/hip_roll_left.stl
- added link hip_roll_right, mass 0.111293388; collision mesh filename=meshes/hip_roll_right.stl; visual mesh filename=meshes/hip_roll_right.stl
- added link hip_yaw_left, mass 0.103201904; collision mesh filename=meshes/hip_yaw_left.stl; visual mesh filename=meshes/hip_yaw_left.stl
- added link hip_yaw_right, mass 0.10319577099999999; collision mesh filename=meshes/hip_yaw_right.stl; visual mesh filename=meshes/hip_yaw_right.stl
- added link knee_pitch_right, mass 0.11061241299999999; collision mesh filename=meshes/knee_pitch_right.stl; visual mesh filename=meshes/knee_pitch_right.stl
- added link knee_pitch_right_2, mass 0.11061241299999999; collision mesh filename=meshes/knee_pitch_right_2.stl; visual mesh filename=meshes/knee_pitch_right_2.stl
- added link left_shoulder_yaw_motor, mass 0.171459652; collision mesh filename=meshes/left_shoulder_yaw_motor.stl; visual mesh filename=meshes/left_shoulder_yaw_motor.stl
- added link right_shoulder_yaw_motor, mass 0.17145988099999998; collision mesh filename=meshes/right_shoulder_yaw_motor.stl; visual mesh filename=meshes/right_shoulder_yaw_motor.stl
- added link shoulder_yaw_left, mass 0.040363129; collision mesh filename=meshes/shoulder_yaw_left.stl; visual mesh filename=meshes/shoulder_yaw_left.stl
- added link shoulder_yaw_right, mass 0.040362728; collision mesh filename=meshes/shoulder_yaw_right.stl; visual mesh filename=meshes/shoulder_yaw_right.stl
Joints:
- joint floating_base: child Base_Motor_Mount -> Torso
- joint left_ankle_pitch: axis 0 0 -1 -> 0 0 1; child DRIVING_ROTOR_PLATE_13 -> foot_left; limit lower=-1.5707963 upper=1.5707963 effort=1 velocity=20 -> lower=-1.0471976 upper=1.0471976 effort=80 velocity=5; origin xyz=-1.204344863420248e-09 0.0552000002775737 -0.00031912410434488224 rpy=4.963083675318156e-23 -2.220446049250313e-15 4.998164106755064e-23 -> xyz=1.3458959276929638e-09 0.05646999986991183 -0.0004500036541040392 rpy=-3.1415926071795863 2.220446049250313e-15 -9.282041313340983e-08; parent DRIVING_ROTOR_PLATE_11 -> ankle_pitch_left
- joint left_elbow_yaw: axis 0 0 -1 -> 0 0 1; child DRIVING_ROTOR_PLATE_7 -> hand_right; limit lower=-1.5707963 upper=1.5707963 effort=1 velocity=20 -> lower=-1.2217305 upper=1.2217305 effort=80 velocity=5; origin xyz=-1.4993347535741108e-10 -0.07020000022229234 0.0 rpy=0.0 0.0 -3.14159264 -> xyz=0.03000311710160605 -0.06434189183411612 -0.0002500013458960012 rpy=-3.141592607179586 -2.220446049250313e-16 0.43633231000000006; parent LX-16A -> left_shoulder_yaw_motor; type fixed -> revolute
- joint left_hip_pitch: child DRIVING_ROTOR_PLATE -> hip_yaw_left; limit lower=-1.5707963 upper=1.5707963 effort=1 velocity=20 -> lower=-1.5707963 upper=1.5707963 effort=80 velocity=5; origin xyz=0.0413138310841906 -0.023482760686076916 -0.004372827208038505 rpy=-3.1415926071795863 -1.5707963 0.0 -> xyz=0.04566353964830031 -0.0003355550191209561 -0.09694671547403086 rpy=1.5707963535897942 -4.6410206566704915e-08 1.5707963000000003; parent Base_Motor_Mount -> Torso
- joint left_hip_roll: axis 0 0 -1 -> 0 0 1; child DRIVING_ROTOR_PLATE_9 -> knee_pitch_right_2; limit lower=-0.52359878 upper=0.52359878 effort=1 velocity=20 -> lower=-0.78539816 upper=0.78539816 effort=80 velocity=5; origin xyz=-2.44813840727387e-09 0.05275000029180242 -0.0070000024561768966 rpy=1.5707963999999994 0.0 -3.1415926071795863 -> xyz=0.0 0.06776001212246713 0.014999999060838654 rpy=1.5707963 0.0 0.0; parent DRIVING_ROTOR_PLATE_5 -> hip_roll_left
- joint left_hip_yaw: axis 0 0 -1 -> 0 0 1; child DRIVING_ROTOR_PLATE_5 -> hip_roll_left; limit lower=-1.5707963 upper=0.087266463 effort=1 velocity=20 -> lower=-1.5707963 upper=0.087266463 effort=80 velocity=5; origin xyz=-0.007400000327569208 0.016949999801717745 0.02285000258156657 rpy=-1.5707963071795867 1.5707963196152375 0.0 -> xyz=-0.02550000297464769 -0.0025000010000000017 0.01936000008172467 rpy=-3.1415926071795863 -1.5707963 0.0; parent DRIVING_ROTOR_PLATE -> hip_yaw_left
- joint left_knee_pitch: child DRIVING_ROTOR_PLATE_11 -> ankle_pitch_left; limit lower=-1.5707963 upper=1.5707963 effort=1 velocity=20 -> lower=-1.0471976 upper=1.0471976 effort=80 velocity=5; origin xyz=-0.01623087751044281 1.0229889869234343e-09 0.04169999999196149 rpy=1.5707963535897935 -4.641020678874952e-08 -1.5707963071795867 -> xyz=-0.018775013847819433 9.3916133203642e-10 -0.04596000193916135 rpy=-1.5707963071795865 0.0 1.5707963000000003; parent DRIVING_ROTOR_PLATE_9 -> knee_pitch_right_2
- joint left_shoulder_pitch: axis 0 0 -1 -> 0 0 1; child DRIVING_ROTOR_PLATE_3 -> shoulder_yaw_left; limit lower=-1.5707963 upper=1.5707963 effort=1 velocity=20 -> lower=-1.5707963 upper=1.5707963 effort=80 velocity=5; origin xyz=0.07131383054661666 -0.023482764740008488 0.10812717280524366 rpy=-3.141592653589792 -1.5707962732050302 0.0 -> xyz=0.0781635406483003 -0.0003355560817246521 0.04305329008172466 rpy=-1.5707963071795865 0.0 1.5707963000000003; parent Base_Motor_Mount -> Torso; type fixed -> revolute
- joint left_shoulder_yaw: child LX-16A -> left_shoulder_yaw_motor; limit lower=-1.5707963 upper=1.5707963 effort=1 velocity=20 -> lower=-1.5707963 upper=1.5707963 effort=80 velocity=5; origin xyz=-0.018273437468083912 0.01634999951036515 0.029393121151926025 rpy=-1.5707962535897932 -1.5707962732050302 0.0 -> xyz=-0.018825 0.01629921 -0.03 rpy=3.1415927 1.5707963 0; parent DRIVING_ROTOR_PLATE_3 -> shoulder_yaw_left; type fixed -> revolute
- joint right_ankle_pitch: child DRIVING_ROTOR_PLATE_14 -> foot_right; limit lower=-1.5707963 upper=1.5707963 effort=1 velocity=20 -> lower=-1.0471976 upper=1.0471976 effort=80 velocity=5; origin xyz=-1.204344863420248e-09 0.0552000002775737 -0.00031912410434488224 rpy=4.963083675318156e-23 -2.220446049250313e-15 4.998164106755064e-23 -> xyz=0.0 0.060220001 -1.3000000000096268e-08 rpy=-3.1415926071795863 0.0 0.0; parent DRIVING_ROTOR_PLATE_12 -> ankle_pitch_right
- joint right_elbow_yaw: axis 0 0 -1 -> 0 0 1; child DRIVING_ROTOR_PLATE_8 -> Left_Hand; limit lower=-1.5707963 upper=1.5707963 effort=1 velocity=20 -> lower=-1.2217305 upper=1.2217305 effort=80 velocity=5; origin xyz=-1.5347855347735972e-09 -0.0702000019724337 -1.7232110183229565e-09 rpy=0.0 -2.220446049250313e-15 3.1415926071795868 -> xyz=-0.03000311610855749 0.06434189253104221 0.00025000101875458525 rpy=8.847213864293657e-08 -1.9613800805728943e-08 0.4363323099999996; parent LX-16A_2 -> right_shoulder_yaw_motor; type fixed -> revolute
- joint right_hip_pitch: child DRIVING_ROTOR_PLATE_2 -> hip_yaw_right; limit lower=-1.5707963 upper=1.5707963 effort=1 velocity=20 -> lower=-1.5707963 upper=1.5707963 effort=80 velocity=5; origin xyz=-0.04131383051044278 -0.023482760691961528 -0.004372827208038465 rpy=-3.1415925803846902 1.570796288901191 0.0 -> xyz=-0.04563646320240432 -0.00033555485567163604 -0.09694671547403086 rpy=-1.570796353589792 -4.6410206566704915e-08 1.5707963000000003; parent Base_Motor_Mount -> Torso
- joint right_hip_roll: axis 0 0 -1 -> 0 0 1; child DRIVING_ROTOR_PLATE_10 -> knee_pitch_right; limit lower=-0.52359878 upper=0.52359878 effort=1 velocity=20 -> lower=-0.78539816 upper=0.78539816 effort=80 velocity=5; origin xyz=-2.44813840727387e-09 0.05275000029180242 -0.0070000024561768966 rpy=1.5707963999999994 0.0 -3.1415926071795863 -> xyz=0.0 0.06776001387753285 0.015000000939161373 rpy=1.5707963999999996 0.0 0.0; parent DRIVING_ROTOR_PLATE_6 -> hip_roll_right
- joint right_hip_yaw: axis 0 0 -1 -> 0 0 1; child DRIVING_ROTOR_PLATE_6 -> hip_roll_right; limit lower=-0.087266463 upper=1.5707963 effort=1 velocity=20 -> lower=-0.087266463 upper=1.5707963 effort=80 velocity=5; origin xyz=0.007399999685828183 0.016450000198282227 0.02284999703643316 rpy=-1.5707962535897932 -1.570796273205031 0.0 -> xyz=-0.02550000162875169 0.0025000011415515153 0.019359999918275368 rpy=9.282041333256968e-08 1.5707963000000005 0.0; parent DRIVING_ROTOR_PLATE_2 -> hip_yaw_right
- joint right_knee_pitch: axis 0 0 -1 -> 0 0 1; child DRIVING_ROTOR_PLATE_12 -> ankle_pitch_right; limit lower=-1.5707963 upper=1.5707963 effort=1 velocity=20 -> lower=-1.0471976 upper=1.0471976 effort=80 velocity=5; origin xyz=0.01623087751044278 -1.7762673623633596e-09 0.04169999999196149 rpy=1.5707963535897942 -4.6410206566704915e-08 1.5707963000000003 -> xyz=0.01882501239711481 -9.39161338975314e-10 -0.04221000153916135 rpy=-1.5707963 0.0 1.5707963; parent DRIVING_ROTOR_PLATE_10 -> knee_pitch_right
- joint right_shoulder_pitch: axis 0 0 -1 -> 0 0 1; child DRIVING_ROTOR_PLATE_4 -> shoulder_yaw_right; limit lower=-1.5707963 upper=1.5707963 effort=1 velocity=20 -> lower=-1.5707963 upper=1.5707963 effort=80 velocity=5; origin xyz=-0.07131383054661666 -0.023482764740008488 0.10812717280524366 rpy=-3.141592653589792 1.5707962732050302 0.0 -> xyz=-0.07813646375169968 -0.0003355559182753147 0.04305328991827533 rpy=1.5707963 2.220446049250313e-16 1.5707963; parent Base_Motor_Mount -> Torso; type fixed -> revolute
- joint right_shoulder_yaw: axis 0 0 1 -> 0 0 -1; child LX-16A_2 -> right_shoulder_yaw_motor; limit lower=-1.5707963 upper=1.5707963 effort=1 velocity=20 -> lower=-1.5707963 upper=1.5707963 effort=80 velocity=5; origin xyz=0.018273437430571058 0.01494999951036515 0.029393121151926025 rpy=-1.570796253589793 1.5707962732050307 0.0 -> xyz=-0.018825 -0.01629921 -0.03 rpy=3.1415927 -1.5707963 0; parent DRIVING_ROTOR_PLATE_4 -> shoulder_yaw_right; type fixed -> revolute

Commit message: update joint config

File: sim/resources/stompymicro/robot_fixed.urdf (robot description, URDF)
Before this commit: robot opus, 18 links, 17 joints
Joints:
- joint left_ankle_pitch: limit lower=-1.0471976 upper=1.0471976 effort=80 velocity=5 -> lower=-1.0471976 upper=1.0471976 effort=1 velocity=20
- joint left_elbow_yaw: limit lower=-1.2217305 upper=1.2217305 effort=80 velocity=5 -> lower=-1.2217305 upper=1.2217305 effort=1 velocity=20
- joint left_hip_pitch: limit lower=-1.5707963 upper=1.5707963 effort=80 velocity=5 -> lower=-1.5707963 upper=1.5707963 effort=1 velocity=20
- joint left_hip_roll: limit lower=-0.78539816 upper=0.78539816 effort=80 velocity=5 -> lower=-0.78539816 upper=0.78539816 effort=1 velocity=20
- joint left_hip_yaw: limit lower=-1.5707963 upper=0.087266463 effort=80 velocity=5 -> lower=-1.5707963 upper=0.087266463 effort=1 velocity=20
- joint left_knee_pitch: limit lower=-1.0471976 upper=1.0471976 effort=80 velocity=5 -> lower=-1.0471976 upper=1.0471976 effort=1 velocity=20
- joint left_shoulder_pitch: limit lower=-1.5707963 upper=1.5707963 effort=80 velocity=5 -> lower=-1.5707963 upper=1.5707963 effort=1 velocity=20
- joint left_shoulder_yaw: limit lower=-1.5707963 upper=1.5707963 effort=80 velocity=5 -> lower=-1.5707963 upper=1.5707963 effort=1 velocity=20
- joint right_ankle_pitch: limit lower=-1.0471976 upper=1.0471976 effort=80 velocity=5 -> lower=-1.0471976 upper=1.0471976 effort=1 velocity=20
- joint right_elbow_yaw: limit lower=-1.2217305 upper=1.2217305 effort=80 velocity=5 -> lower=-1.2217305 upper=1.2217305 effort=1 velocity=20
- joint right_hip_pitch: limit lower=-1.5707963 upper=1.5707963 effort=80 velocity=5 -> lower=-1.5707963 upper=1.5707963 effort=1 velocity=20
- joint right_hip_roll: limit lower=-0.78539816 upper=0.78539816 effort=80 velocity=5 -> lower=-0.78539816 upper=0.78539816 effort=1 velocity=20
- joint right_hip_yaw: limit lower=-0.087266463 upper=1.5707963 effort=80 velocity=5 -> lower=-0.087266463 upper=1.5707963 effort=1 velocity=20
- joint right_knee_pitch: limit lower=-1.0471976 upper=1.0471976 effort=80 velocity=5 -> lower=-1.0471976 upper=1.0471976 effort=1 velocity=20
- joint right_shoulder_pitch: limit lower=-1.5707963 upper=1.5707963 effort=80 velocity=5 -> lower=-1.5707963 upper=1.5707963 effort=1 velocity=20
- joint right_shoulder_yaw: limit lower=-1.5707963 upper=1.5707963 effort=80 velocity=5 -> lower=-1.5707963 upper=1.5707963 effort=1 velocity=20

Commit message: updated joint

File: sim/resources/stompymicro/robot_fixed.urdf (robot description, URDF)
Before this commit: robot opus, 18 links, 17 joints
Joints:
- joint left_ankle_pitch: limit lower=-1.0471976 upper=1.0471976 effort=1 velocity=20 -> lower=-1.0471976 upper=1.0471976 effort=1 velocity=10
- joint left_hip_pitch: limit lower=-1.5707963 upper=1.5707963 effort=1 velocity=20 -> lower=-1.5707963 upper=1.5707963 effort=1 velocity=10
- joint left_hip_roll: limit lower=-0.78539816 upper=0.78539816 effort=1 velocity=20 -> lower=-0.78539816 upper=0.78539816 effort=1 velocity=10
- joint left_hip_yaw: limit lower=-1.5707963 upper=0.087266463 effort=1 velocity=20 -> lower=-1.5707963 upper=0.087266463 effort=1 velocity=10
- joint left_knee_pitch: limit lower=-1.0471976 upper=1.0471976 effort=1 velocity=20 -> lower=0 upper=1.0471976 effort=1 velocity=10
- joint right_ankle_pitch: limit lower=-1.0471976 upper=1.0471976 effort=1 velocity=20 -> lower=-1.0471976 upper=1.0471976 effort=1 velocity=10
- joint right_hip_pitch: limit lower=-1.5707963 upper=1.5707963 effort=1 velocity=20 -> lower=-1.5707963 upper=1.5707963 effort=1 velocity=10
- joint right_hip_roll: limit lower=-0.78539816 upper=0.78539816 effort=1 velocity=20 -> lower=-0.78539816 upper=0.78539816 effort=1 velocity=10
- joint right_hip_yaw: limit lower=-0.087266463 upper=1.5707963 effort=1 velocity=20 -> lower=-0.087266463 upper=1.5707963 effort=1 velocity=10
- joint right_knee_pitch: limit lower=-1.0471976 upper=1.0471976 effort=1 velocity=20 -> lower=-1.0471976 upper=0 effort=1 velocity=10
