Commit message: updated urdf

File: sim/resources/stompymicro/robot.urdf (robot description, URDF)
Before this commit: robot opus, 18 links, 17 joints
Links:
- removed link Left_Hand
- removed link ankle_pitch_left
- removed link ankle_pitch_right
- removed link hand_right
- removed link knee_pitch_right_2
- removed link shoulder_yaw_left
- removed link shoulder_yaw_right
- added link knee_pitch_left, mass 0.017415556; collision mesh filename=meshes/knee_pitch_left.stl; visual mesh filename=meshes/knee_pitch_left.stl
- added link left_hand, mass 0.057634594; collision mesh filename=meshes/left_hand.stl; visual mesh filename=meshes/left_hand.stl
- added link left_knee_pitch_motor, mass 0.164074011; collision mesh filename=meshes/left_knee_pitch_motor.stl; visual mesh filename=meshes/left_knee_pitch_motor.stl
- added link left_shoulder_yaw_2, mass 0.033295444; collision mesh filename=meshes/left_shoulder_yaw.stl; visual mesh filename=meshes/left_shoulder_yaw.stl
- added link right_hand, mass 0.057633913; collision mesh filename=meshes/right_hand.stl; visual mesh filename=meshes/right_hand.stl
- added link right_knee_pitch_motor, mass 0.164074011; collision mesh filename=meshes/right_knee_pitch_motor.stl; visual mesh filename=meshes/right_knee_pitch_motor.stl
- added link right_shoulder_yaw_2, mass 0.033295451; collision mesh filename=meshes/right_shoulder_yaw.stl; visual mesh filename=meshes/right_shoulder_yaw.stl
- link Torso: mass 1.5697539312 -> 1.4248854441999999
- link foot_left: mass 0.04062216 -> 0.074314614
- link foot_right: mass 0.040622158 -> 0.074314817
- link hip_roll_left: mass 0.111293526 -> 0.099288915
- link hip_roll_right: mass 0.111293388 -> 0.09928883999999999
- link hip_yaw_left: mass 0.103201904 -> 0.093205265
- link hip_yaw_right: mass 0.10319577099999999 -> 0.093205286
- link knee_pitch_right: mass 0.11061241299999999 -> 0.017415406
- link left_shoulder_yaw_motor: mass 0.171459652 -> 0.161287862
- link right_shoulder_yaw_motor: mass 0.17145988099999998 -> 0.16128786299999998
Joints:
- removed joint right_elbow_yaw
- added joint righ_elbow_yaw: type revolute, parent right_shoulder_yaw_motor, child right_hand, origin xyz=-0.030003116165437632 -0.06434189265302206 -0.00015000392836930906 rpy=3.141592518707449 -1.961380480253183e-08 2.7052603000000013, axis 0 0 1, limit lower=-1.5707963 upper=1.5707963 effort=80 velocity=5
- joint left_ankle_pitch: limit lower=-1.0471976 upper=1.0471976 effort=1 velocity=20 -> lower=-1.5707963 upper=1.5707963 effort=80 velocity=5; origin xyz=1.3458959276929638e-09 0.05646999986991183 -0.0004500036541040392 rpy=-3.1415926071795863 2.220446049250313e-15 -9.282041313340983e-08 -> xyz=0.0 -0.07771999985844844 -0.000499991045895997 rpy=9.282041357749903e-08 0.0 0.0; parent ankle_pitch_left -> left_knee_pitch_motor
- joint left_elbow_yaw: child hand_right -> left_hand; limit lower=-1.2217305 upper=1.2217305 effort=1 velocity=20 -> lower=-1.5707963 upper=1.5707963 effort=80 velocity=5; origin xyz=0.03000311710160605 -0.06434189183411612 -0.0002500013458960012 rpy=-3.141592607179586 -2.220446049250313e-16 0.43633231000000006 -> xyz=0.03000311710160605 -0.06434189183411612 -0.00015000134589600138 rpy=3.1415926071795863 -1.7763568394002505e-15 -2.70526039
- joint left_hip_pitch: limit lower=-1.5707963 upper=1.5707963 effort=1 velocity=20 -> lower=-1.5707963 upper=1.5707963 effort=80 velocity=5; origin xyz=0.04566353964830031 -0.0003355550191209561 -0.09694671547403086 rpy=1.5707963535897942 -4.6410206566704915e-08 1.5707963000000003 -> xyz=0.045549819648300315 -0.0003268960191209584 -0.10384882247403085 rpy=1.5707963535897942 -4.6410206566704915e-08 1.5707963000000003
- joint left_hip_roll: axis 0 0 1 -> 0 0 -1; child knee_pitch_right_2 -> knee_pitch_right; limit lower=-0.78539816 upper=0.78539816 effort=1 velocity=20 -> lower=-0.78539816 upper=0.78539816 effort=80 velocity=5; origin xyz=0.0 0.06776001212246713 0.014999999060838654 rpy=1.5707963 0.0 0.0 -> xyz=0.0 0.06776001212246713 0.014999999060838654 rpy=-1.5707963071795865 0.0 0.0
- joint left_hip_yaw: limit lower=-1.5707963 upper=0.087266463 effort=1 velocity=20 -> lower=-1.5707963 upper=0.087266463 effort=80 velocity=5; origin xyz=-0.02550000297464769 -0.0025000010000000017 0.01936000008172467 rpy=-3.1415926071795863 -1.5707963 0.0 -> xyz=-0.02550000297464769 -0.012500001 0.01936000008172467 rpy=-3.1415926071795863 -1.5707963 0.0
- joint left_knee_pitch: child ankle_pitch_left -> left_knee_pitch_motor; limit lower=-1.0471976 upper=1.0471976 effort=1 velocity=20 -> lower=-1.5707963 upper=1.5707963 effort=80 velocity=5; origin xyz=-0.018775013847819433 9.3916133203642e-10 -0.04596000193916135 rpy=-1.5707963071795865 0.0 1.5707963000000003 -> xyz=-0.018825 0 0.02221 rpy=-1.5707963 0 -1.5707963; parent knee_pitch_right_2 -> knee_pitch_right
- joint left_shoulder_pitch: child shoulder_yaw_left -> left_shoulder_yaw_2; limit lower=-1.5707963 upper=1.5707963 effort=1 velocity=20 -> lower=-1.7453293 upper=1.7453293 effort=80 velocity=5; origin xyz=0.0781635406483003 -0.0003355560817246521 0.04305329008172466 rpy=-1.5707963071795865 0.0 1.5707963000000003 -> xyz=0.07804981964830031 -0.0003268980817246539 0.04615118308172467 rpy=-1.5707963071795865 0.0 1.5707963000000003
- joint left_shoulder_yaw: limit lower=-1.5707963 upper=1.5707963 effort=1 velocity=20 -> lower=-0.43633231 upper=1.5707963 effort=80 velocity=5; parent shoulder_yaw_left -> left_shoulder_yaw_2
- joint right_ankle_pitch: axis 0 0 -1 -> 0 0 1; limit lower=-1.0471976 upper=1.0471976 effort=1 velocity=20 -> lower=-1.5707963 upper=1.5707963 effort=80 velocity=5; origin xyz=0.0 0.060220001 -1.3000000000096268e-08 rpy=-3.1415926071795863 0.0 0.0 -> xyz=0.0 0.07772000162667812 2.0870670330852548e-09 rpy=9.282041357749903e-08 0.0 0.0; parent ankle_pitch_right -> right_knee_pitch_motor
- joint right_hip_pitch: limit lower=-1.5707963 upper=1.5707963 effort=1 velocity=20 -> lower=-1.5707963 upper=1.5707963 effort=80 velocity=5; origin xyz=-0.04563646320240432 -0.00033555485567163604 -0.09694671547403086 rpy=-1.570796353589792 -4.6410206566704915e-08 1.5707963000000003 -> xyz=-0.045750183202404315 -0.00032689585567163837 -0.10384882247403085 rpy=-1.570796353589792 -4.6410206566704915e-08 1.5707963000000003
- joint right_hip_roll: axis 0 0 1 -> 0 0 -1; child knee_pitch_right -> knee_pitch_left; limit lower=-0.78539816 upper=0.78539816 effort=1 velocity=20 -> lower=-0.78539816 upper=0.78539816 effort=80 velocity=5; origin xyz=0.0 0.06776001387753285 0.015000000939161373 rpy=1.5707963999999996 0.0 0.0 -> xyz=0.0 0.06776001387753285 0.015000000939161373 rpy=-1.5707963 0.0 0.0
- joint right_hip_yaw: limit lower=-0.087266463 upper=1.5707963 effort=1 velocity=20 -> lower=-0.087266463 upper=1.5707963 effort=80 velocity=5; origin xyz=-0.02550000162875169 0.0025000011415515153 0.019359999918275368 rpy=9.282041333256968e-08 1.5707963000000005 0.0 -> xyz=-0.02550000162875169 0.012500001141551514 0.019359999918275368 rpy=9.282041333256968e-08 1.5707963000000005 0.0
- joint right_knee_pitch: axis 0 0 1 -> 0 0 -1; child ankle_pitch_right -> right_knee_pitch_motor; limit lower=-1.0471976 upper=1.0471976 effort=1 velocity=20 -> lower=-1.5707963 upper=1.5707963 effort=80 velocity=5; origin xyz=0.01882501239711481 -9.39161338975314e-10 -0.04221000153916135 rpy=-1.5707963 0.0 1.5707963 -> xyz=0.018825 0 0.02221 rpy=1.5707963 0 -1.5707963; parent knee_pitch_right -> knee_pitch_left
- joint right_shoulder_pitch: child shoulder_yaw_right -> right_shoulder_yaw_2; limit lower=-1.5707963 upper=1.5707963 effort=1 velocity=20 -> lower=-1.7453293 upper=1.7453293 effort=80 velocity=5; origin xyz=-0.07813646375169968 -0.0003355559182753147 0.04305328991827533 rpy=1.5707963 2.220446049250313e-16 1.5707963 -> xyz=-0.07825018475169968 -0.0003268979182753165 0.04615118291827534 rpy=1.5707963 2.220446049250313e-16 1.5707963
- joint right_shoulder_yaw: axis 0 0 -1 -> 0 0 1; limit lower=-1.5707963 upper=1.5707963 effort=1 velocity=20 -> lower=-1.134464 upper=0.87266463 effort=80 velocity=5; origin xyz=-0.018825 -0.01629921 -0.03 rpy=3.1415927 -1.5707963 0 -> xyz=-0.018825 -0.01629921 -0.03 rpy=0 -1.5707963 0; parent shoulder_yaw_right -> right_shoulder_yaw_2

Commit message: Updated robot.urdf and robot.xml for the stompymicro robot.

File: sim/resources/stompymicro/robot.urdf (robot description, URDF)
Before this commit: robot opus, 18 links, 17 joints
Joints:
- removed joint righ_elbow_yaw
- added joint right_elbow_yaw: type revolute, parent right_shoulder_yaw_motor, child right_hand, origin xyz=-0.030003116165437632 -0.06434189265302206 -0.00015000392836930906 rpy=3.141592518707449 -1.961380480253183e-08 2.7052603000000013, axis 0 0 1, limit lower=-1.5707963 upper=1.5707963 effort=80 velocity=5
- joint left_ankle_pitch: limit lower=-1.5707963 upper=1.5707963 effort=80 velocity=5 -> lower=-1.0471976 upper=1.0471976 effort=2 velocity=10
- joint left_hip_pitch: limit lower=-1.5707963 upper=1.5707963 effort=80 velocity=5 -> lower=-1.5707963 upper=1.5707963 effort=2 velocity=10
- joint left_hip_roll: limit lower=-0.78539816 upper=0.78539816 effort=80 velocity=5 -> lower=-0.78539816 upper=0.78539816 effort=2 velocity=10
- joint left_hip_yaw: limit lower=-1.5707963 upper=0.087266463 effort=80 velocity=5 -> lower=-1.5707963 upper=0.087266463 effort=2 velocity=10
- joint left_knee_pitch: limit lower=-1.5707963 upper=1.5707963 effort=80 velocity=5 -> lower=-1.0471976 upper=0 effort=2 velocity=10
- joint right_ankle_pitch: limit lower=-1.5707963 upper=1.5707963 effort=80 velocity=5 -> lower=-1.0471976 upper=1.0471976 effort=2 velocity=10
- joint right_hip_pitch: limit lower=-1.5707963 upper=1.5707963 effort=80 velocity=5 -> lower=-1.5707963 upper=1.5707963 effort=2 velocity=10
- joint right_hip_roll: limit lower=-0.78539816 upper=0.78539816 effort=80 velocity=5 -> lower=-0.78539816 upper=0.78539816 effort=2 velocity=10
- joint right_hip_yaw: limit lower=-0.087266463 upper=1.5707963 effort=80 velocity=5 -> lower=-0.087266463 upper=1.5707963 effort=2 velocity=10
- joint right_knee_pitch: limit lower=-1.5707963 upper=1.5707963 effort=80 velocity=5 -> lower=0 upper=1.0471976 effort=2 velocity=10

Commit message: Set matching effort and velocity values in urdf vs joints.py

File: sim/resources/stompymicro/robot.urdf (robot description, URDF)
Before this commit: robot opus, 18 links, 17 joints
Joints:
- joint left_ankle_pitch: limit lower=-1.0471976 upper=1.0471976 effort=2 velocity=10 -> lower=-1.5707963 upper=1.5707963 effort=80 velocity=5
- joint left_hip_pitch: limit lower=-1.5707963 upper=1.5707963 effort=2 velocity=10 -> lower=-1.5707963 upper=1.5707963 effort=80 velocity=5
- joint left_hip_roll: limit lower=-0.78539816 upper=0.78539816 effort=2 velocity=10 -> lower=-0.78539816 upper=0.78539816 effort=80 velocity=5
- joint left_hip_yaw: limit lower=-1.5707963 upper=0.087266463 effort=2 velocity=10 -> lower=-1.5707963 upper=0.087266463 effort=80 velocity=5
- joint left_knee_pitch: limit lower=-1.0471976 upper=0 effort=2 velocity=10 -> lower=-1.5707963 upper=1.5707963 effort=80 velocity=5
- joint right_ankle_pitch: limit lower=-1.0471976 upper=1.0471976 effort=2 velocity=10 -> lower=-1.5707963 upper=1.5707963 effort=80 velocity=5
- joint right_hip_pitch: limit lower=-1.5707963 upper=1.5707963 effort=2 velocity=10 -> lower=-1.5707963 upper=1.5707963 effort=80 velocity=5
- joint right_hip_roll: limit lower=-0.78539816 upper=0.78539816 effort=2 velocity=10 -> lower=-0.78539816 upper=0.78539816 effort=80 velocity=5
- joint right_hip_yaw: limit lower=-0.087266463 upper=1.5707963 effort=2 velocity=10 -> lower=-0.087266463 upper=1.5707963 effort=80 velocity=5
- joint right_knee_pitch: limit lower=0 upper=1.0471976 effort=2 velocity=10 -> lower=-1.5707963 upper=1.5707963 effort=80 velocity=5
