Commit message: update robot

File: sim/resources/stompypro/robot_fixed.urdf (robot description, URDF)
Before this commit: robot robot, 20 links, 19 joints
Joints:
- joint L_ankle_y: limit lower=-0.698 upper=0.698 effort=17 velocity=5 -> lower=-0.698 upper=0.698 effort=50 velocity=10
- joint L_hip_x: limit lower=-0.523 upper=2.093 effort=60 velocity=5 -> lower=-0.523 upper=2.093 effort=150 velocity=10
- joint L_hip_y: limit lower=-3.14 upper=3.14 effort=120 velocity=5 -> lower=-3.14 upper=3.14 effort=150 velocity=10
- joint L_hip_z: limit lower=-3.14 upper=3.14 effort=60 velocity=5 -> lower=-3.14 upper=3.14 effort=100 velocity=10
- joint L_knee: limit lower=-1.919 upper=1.919 effort=120 velocity=5 -> lower=-1.919 upper=1.919 effort=150 velocity=10
- joint R_ankle_y: limit lower=-0.698 upper=0.698 effort=17 velocity=5 -> lower=-0.698 upper=0.698 effort=50 velocity=10
- joint R_hip_x: limit lower=-2.093 upper=0.523 effort=60 velocity=5 -> lower=-2.093 upper=0.523 effort=150 velocity=10
- joint R_hip_y: limit lower=-3.14 upper=3.14 effort=120 velocity=5 -> lower=-3.14 upper=3.14 effort=150 velocity=10
- joint R_hip_z: limit lower=-3.14 upper=3.14 effort=60 velocity=5 -> lower=-3.14 upper=3.14 effort=100 velocity=10
- joint R_knee: limit lower=-1.919 upper=1.919 effort=120 velocity=5 -> lower=-1.919 upper=1.919 effort=150 velocity=10

Commit message: changing the setup

File: sim/resources/stompypro/robot_fixed.urdf (robot description, URDF)
Before this commit: robot robot, 20 links, 19 joints
Joints:
- joint L_ankle_y: limit lower=-0.698 upper=0.698 effort=17 velocity=5 -> lower=-0.698 upper=0.698 effort=100 velocity=10
- joint L_hip_x: limit lower=-0.523 upper=2.093 effort=60 velocity=5 -> lower=-0.523 upper=2.093 effort=100 velocity=10
- joint L_hip_y: limit lower=-3.14 upper=3.14 effort=120 velocity=5 -> lower=-3.14 upper=3.14 effort=250 velocity=10
- joint L_hip_z: limit lower=-3.14 upper=3.14 effort=60 velocity=5 -> lower=-3.14 upper=3.14 effort=100 velocity=10
- joint L_knee: limit lower=-1.919 upper=1.919 effort=120 velocity=5 -> lower=-1.919 upper=1.919 effort=250 velocity=10
- joint R_ankle_y: limit lower=-0.698 upper=0.698 effort=17 velocity=5 -> lower=-0.698 upper=0.698 effort=100 velocity=10
- joint R_hip_x: limit lower=-2.093 upper=0.523 effort=60 velocity=5 -> lower=-2.093 upper=0.523 effort=100 velocity=10
- joint R_hip_y: limit lower=-3.14 upper=3.14 effort=120 velocity=5 -> lower=-3.14 upper=3.14 effort=250 velocity=10
- joint R_hip_z: limit lower=-3.14 upper=3.14 effort=60 velocity=5 -> lower=-3.14 upper=3.14 effort=100 velocity=10
- joint R_knee: limit lower=-1.919 upper=1.919 effort=120 velocity=5 -> lower=-1.919 upper=1.919 effort=250 velocity=10

Commit message: adjusting to the robstride specs

File: sim/resources/stompypro/robot_fixed.urdf (robot description, URDF)
Before this commit: robot robot, 20 links, 19 joints
Joints:
- joint L_ankle_y: limit lower=-0.698 upper=0.698 effort=100 velocity=10 -> lower=-0.698 upper=0.698 effort=17 velocity=10
- joint L_hip_x: limit lower=-0.523 upper=2.093 effort=100 velocity=10 -> lower=-0.523 upper=2.093 effort=60 velocity=10
- joint L_hip_y: limit lower=-3.14 upper=3.14 effort=250 velocity=10 -> lower=-3.14 upper=3.14 effort=120 velocity=10
- joint L_hip_z: limit lower=-3.14 upper=3.14 effort=100 velocity=10 -> lower=-3.14 upper=3.14 effort=60 velocity=10
- joint L_knee: limit lower=-1.919 upper=1.919 effort=250 velocity=10 -> lower=-1.919 upper=1.919 effort=120 velocity=10
- joint R_ankle_y: limit lower=-0.698 upper=0.698 effort=100 velocity=10 -> lower=-0.698 upper=0.698 effort=17 velocity=10
- joint R_hip_x: limit lower=-2.093 upper=0.523 effort=100 velocity=10 -> lower=-2.093 upper=0.523 effort=60 velocity=10
- joint R_hip_y: limit lower=-3.14 upper=3.14 effort=250 velocity=10 -> lower=-3.14 upper=3.14 effort=120 velocity=10
- joint R_hip_z: limit lower=-3.14 upper=3.14 effort=100 velocity=10 -> lower=-3.14 upper=3.14 effort=60 velocity=10
- joint R_knee: limit lower=-1.919 upper=1.919 effort=250 velocity=10 -> lower=-1.919 upper=1.919 effort=120 velocity=10

Commit message: working setup

File: sim/resources/stompypro/robot_fixed.urdf (robot description, URDF)
Before this commit: robot robot, 20 links, 19 joints
Joints:
- joint L_hip_x: limit lower=-0.523 upper=2.093 effort=60 velocity=10 -> lower=-0.523 upper=2.093 effort=100 velocity=10
- joint L_hip_y: limit lower=-3.14 upper=3.14 effort=120 velocity=10 -> lower=-3.14 upper=3.14 effort=250 velocity=10
- joint L_hip_z: limit lower=-3.14 upper=3.14 effort=60 velocity=10 -> lower=-3.14 upper=3.14 effort=100 velocity=10
- joint L_knee: limit lower=-1.919 upper=1.919 effort=120 velocity=10 -> lower=-1.919 upper=1.919 effort=250 velocity=10
- joint R_hip_x: limit lower=-2.093 upper=0.523 effort=60 velocity=10 -> lower=-2.093 upper=0.523 effort=100 velocity=10
- joint R_hip_y: limit lower=-3.14 upper=3.14 effort=120 velocity=10 -> lower=-3.14 upper=3.14 effort=250 velocity=10
- joint R_hip_z: limit lower=-3.14 upper=3.14 effort=60 velocity=10 -> lower=-3.14 upper=3.14 effort=100 velocity=10
- joint R_knee: limit lower=-1.919 upper=1.919 effort=120 velocity=10 -> lower=-1.919 upper=1.919 effort=250 velocity=10

Commit message: Improvements to sim2sim (#102)
* add walking checkpoint

* working config

* working pd

* fix the setup

* saving simple setup

* changing the setup

* check the new setup

* getting stable results

* setup works

* testing new setup

* change default position, save better rad setup

* more balanced setup

* adjusting to the robstride specs

* working setup

---------

Co-authored-by: WT-MM <wesley.maa@gmail.com>

File: sim/resources/stompypro/robot_fixed.urdf (robot description, URDF)
Before this commit: robot robot, 20 links, 19 joints
Joints:
- joint L_ankle_y: limit lower=-0.698 upper=0.698 effort=50 velocity=10 -> lower=-0.698 upper=0.698 effort=17 velocity=10
- joint L_hip_x: limit lower=-0.523 upper=2.093 effort=150 velocity=10 -> lower=-0.523 upper=2.093 effort=100 velocity=10
- joint L_hip_y: limit lower=-3.14 upper=3.14 effort=150 velocity=10 -> lower=-3.14 upper=3.14 effort=250 velocity=10
- joint L_knee: limit lower=-1.919 upper=1.919 effort=150 velocity=10 -> lower=-1.919 upper=1.919 effort=250 velocity=10
- joint R_ankle_y: limit lower=-0.698 upper=0.698 effort=50 velocity=10 -> lower=-0.698 upper=0.698 effort=17 velocity=10
- joint R_hip_x: limit lower=-2.093 upper=0.523 effort=150 velocity=10 -> lower=-2.093 upper=0.523 effort=100 velocity=10
- joint R_hip_y: limit lower=-3.14 upper=3.14 effort=150 velocity=10 -> lower=-3.14 upper=3.14 effort=250 velocity=10
- joint R_knee: limit lower=-1.919 upper=1.919 effort=150 velocity=10 -> lower=-1.919 upper=1.919 effort=250 velocity=10

Commit message: add imu link

File: sim/resources/stompypro/robot_fixed.urdf (robot description, URDF)
Before this commit: robot robot, 20 links, 19 joints
Links:
- added link imu_link
Joints:
- added joint imu_joint: type fixed, parent base, child imu_link, origin xyz=-0.04452 -0.01891 0.27756 rpy=0 0 0

Commit message: add visual placement and proper index, first training

File: sim/resources/stompypro/robot_fixed.urdf (robot description, URDF)
Before this commit: robot robot, 21 links, 20 joints
Links:
- link imu_link: geometry visual box size=0.1 0.1 0.1
Joints:
- joint imu_joint: origin xyz=-0.04452 -0.01891 0.27756 rpy=0 0 0 -> xyz=0.0 0.0 0.0 rpy=0 0 0

Commit message: Revert "Merge branch 'pawel/imu_setup' of github.com:kscalelabs/sim into onnx_setup"
This reverts commit 10bdc9bf2f3bea2b4ec1456febc85103b7ae4f37, reversing
changes made to 606d79114366cafe4b69d37cb2aa9eff167e1529.

File: sim/resources/stompypro/robot_fixed.urdf (robot description, URDF)
Before this commit: robot robot, 21 links, 20 joints
Links:
- removed link imu_link
Joints:
- removed joint imu_joint

Commit message: robust with new imu

File: sim/resources/stompypro/robot_fixed.urdf (robot description, URDF)
Before this commit: robot robot, 21 links, 20 joints
Joints:
- joint imu_joint: origin xyz=0.0 0.0 0.0 rpy=0 0 0 -> xyz=0.0 0.0 0.55 rpy=0 0 0

Commit message: add imu link (#109)
* add imu link

* add visual placement and proper index, first training

* robust with new imu

* update imu placement

* format

File: sim/resources/stompypro/robot_fixed.urdf (robot description, URDF)
Before this commit: robot robot, 20 links, 19 joints
Links:
- added link imu_link; visual box size=0.1 0.1 0.1
Joints:
- added joint imu_joint: type fixed, parent base, child imu_link, origin xyz=0.0 0.0 0.55 rpy=0 0 0

Commit message: new assets

File: sim/resources/stompypro/robot_fixed.urdf (robot description, URDF)
Before this commit: robot robot, 21 links, 20 joints
Links:
- removed link L_leg
- removed link trunk
- added link L_finger, mass 0.737286180296128; collision mesh filename=meshes/L_finger.STL; visual mesh filename=meshes/L_finger.STL
- added link L_hip, mass 0.83376821073388; collision mesh filename=meshes/L_hip.STL; visual mesh filename=meshes/L_hip.STL
- added link R_finger, mass 0.869674405890661; collision mesh filename=meshes/R_finger.STL; visual mesh filename=meshes/R_finger.STL
- link L_buttock: mass 1.2990888 -> 0.717874293135761; geometry collision mesh filename=meshes/L_buttock.STL; visual mesh filename=meshes/L_buttock.STL
- link L_calf: mass 1.544772 -> 1.01528348517359; geometry collision mesh filename=meshes/L_calf.STL; visual mesh filename=meshes/L_calf.STL
- link L_clav: mass 1.1246895 -> 0.556581229687908; geometry collision mesh filename=meshes/L_clav.STL; visual mesh filename=meshes/L_clav.STL
- link L_farm: mass 0.66002606 -> 0.344651145281825; geometry collision mesh filename=meshes/L_farm.STL; visual mesh filename=meshes/L_farm.STL
- link L_foot: mass 0.54237266 -> 0.550460500951221; geometry collision mesh filename=meshes/L_foot.STL; visual mesh filename=meshes/L_foot.STL
- link L_scapula: mass 0.65454544 -> 0.338558086149021; geometry collision mesh filename=meshes/L_scapula.STL; visual mesh filename=meshes/L_scapula.STL
- link L_thigh: mass 1.9399504 -> 0.798828442920691; geometry collision mesh filename=meshes/L_thigh.STL; visual mesh filename=meshes/L_thigh.STL
- link L_uarm: mass 0.58244405 -> 0.277294237289419; geometry collision mesh filename=meshes/L_uarm.STL; visual mesh filename=meshes/L_uarm.STL
- link R_buttock: mass 1.2990888 -> 0.716812635597912; geometry collision mesh filename=meshes/R_buttock.STL; visual mesh filename=meshes/R_buttock.STL
- link R_calf: mass 1.544772 -> 1.01514022175102; geometry collision mesh filename=meshes/R_calf.STL; visual mesh filename=meshes/R_calf.STL
- link R_clav: mass 1.1246895 -> 0.556580211071974; geometry collision mesh filename=meshes/R_clav.STL; visual mesh filename=meshes/R_clav.STL
- link R_farm: mass 0.66002606 -> 0.333434347202916; geometry collision mesh filename=meshes/R_farm.STL; visual mesh filename=meshes/R_farm.STL
- link R_foot: mass 0.54237266 -> 0.549121604771221; geometry collision mesh filename=meshes/R_foot.STL; visual mesh filename=meshes/R_foot.STL
- link R_leg: mass 1.3398346 -> 0.827134269923993; geometry collision mesh filename=meshes/R_leg.STL; visual mesh filename=meshes/R_leg.STL
- link R_scapula: mass 0.65454544 -> 0.33855519445856; geometry collision mesh filename=meshes/R_scapula.STL; visual mesh filename=meshes/R_scapula.STL
- link R_thigh: mass 1.9399504 -> 0.79742290295527; geometry collision mesh filename=meshes/R_thigh.STL; visual mesh filename=meshes/R_thigh.STL
- link R_uarm: mass 0.58244405 -> 0.277293520071397; geometry collision mesh filename=meshes/R_uarm.STL; visual mesh filename=meshes/R_uarm.STL
- link base: mass 0.001 -> 8.62540645323623; geometry collision mesh filename=meshes/body_base.STL; visual mesh filename=meshes/body_base.STL
- link imu_link: geometry visual box size=0.2 0.2 0.2
Joints:
- removed joint floating_base
- added joint L_hand_x: type fixed, parent L_farm, child L_finger, origin xyz=0 0.164 0 rpy=1.5707963267949 0 -1.5707963267949, axis -1 0 0
- added joint R_hand_x: type fixed, parent R_farm, child R_finger, origin xyz=-0.00399999999999999 0.164 0 rpy=0.00107337749648937 0 -1.5707963267949, axis -1 0 0
- joint L_ankle_y: axis 0.0 1.0 0.0 -> -1 0 0; origin xyz=0 0 -0.3 rpy=0.0 0.0 0.0 -> xyz=0 0.300033748101774 0 rpy=1.57079632679433 0 -0.0149988751526712
- joint L_elbow_x: axis 1.0 0 0.0 -> -1 0 0; limit lower=-1.9199 upper=1.9199 effort=17 velocity=0 -> (none); origin xyz=0 0 -0.23 rpy=0.0 0.0 0.0 -> xyz=-0.116 0 0 rpy=0 -0.00107337747433267 1.5707963267949
- joint L_hip_x: axis 1.0 0.0 0.0 -> 0 0 1; child L_leg -> L_hip; limit lower=-0.523 upper=2.093 effort=100 velocity=10 -> lower=-2.093 upper=0.523 effort=100 velocity=10; origin xyz=0 0 0 rpy=0.0 0.0 0.0 -> xyz=0 0 0 rpy=0 0 0
- joint L_hip_y: axis 0.0 1.0 0 -> -1 0 0; origin xyz=0 0.1577 0 rpy=0 0 0 -> xyz=0 0.1572 0 rpy=1.5707963267949 0 -1.5707963267949; parent trunk -> base
- joint L_hip_z: axis 0.0 0.0 1.0 -> -1 0 0; origin xyz=0 0 0 rpy=0.0 0 0.0 -> xyz=0 -0.13525 0 rpy=1.5707963267949 0 1.5707963267949; parent L_leg -> L_hip
- joint L_knee: axis 0.0 1.0 0.0 -> -0.999887518980808 0.0149983127852693 0; origin xyz=0 0 -0.3 rpy=0.0 0.0 0.0 -> xyz=-0.16475 0 0.00650000000000001 rpy=1.5707963267949 1.55579745164248 3.14159265358946
- joint L_shoulder_x: axis 1.0 0.0 0.0 -> -1 0 0; limit lower=0 upper=3.1416 effort=60 velocity=0 -> (none); origin xyz=0 0 0 rpy=0.0 0.0 0.0 -> xyz=0 0 0 rpy=3.14159265358979 0 1.5707963267949
- joint L_shoulder_y: axis 0.0 1.0 0.0 -> -1 0 0; limit lower=-3.1416 upper=3.1416 effort=60 velocity=0 -> (none); origin xyz=0 0.255 0.45 rpy=0 0 0 -> xyz=0 0.255 0.45 rpy=0 0 -1.5707963267949; parent trunk -> base
- joint L_shoulder_z: axis 0.0 0.0 1.0 -> -1 0 0; limit lower=-3.14 upper=3.14 effort=17 velocity=0 -> (none); origin xyz=0 0 0 rpy=0.0 0.0 0.0 -> xyz=1.19643736612081E-05 0 0.113943721548401 rpy=1.56972294932056 1.5707963267949 0
- joint R_ankle_y: axis 0.0 1.0 0.0 -> -1 0 0; origin xyz=0 0 -0.3 rpy=0.0 0.0 0.0 -> xyz=0 0.300020415972074 0 rpy=1.57079634708826 0 -3.12992651620125
- joint R_elbow_x: axis 1.0 0 0.0 -> -1 0 0; limit lower=-1.9199 upper=1.9199 effort=17 velocity=0 -> (none); origin xyz=0 0 -0.23 rpy=0.0 0.0 0.0 -> xyz=-0.1155 0.00349999798375654 0 rpy=0 0.0010733774846464 1.5707963267949
- joint R_hip_x: axis 1.0 0.0 0.0 -> 0.999247470344691 -0.0387877945974834 0; origin xyz=0 0 0 rpy=0.0 0.0 0.0 -> xyz=0 0 0 rpy=0 0 0
- joint R_hip_y: axis 0.0 1.0 0 -> 0 0 1; origin xyz=0 -0.1577 0 rpy=0 0 0 -> xyz=0.00525 -0.1572 0 rpy=-1.5707963267949 0.0387975271824028 0; parent trunk -> base
- joint R_hip_z: axis 0.0 0.0 1.0 -> -1 0 0; origin xyz=0 0 0 rpy=0.0 0 0.0 -> xyz=0 0.135351856285756 0 rpy=0 0 -1.6095938539773
- joint R_knee: axis 0.0 1.0 0.0 -> -0.999931951391002 -0.0116658727656092 0; origin xyz=0 0 -0.3 rpy=0.0 0.0 0.0 -> xyz=-0.16475 0 0.00650000000000001 rpy=1.5707963267949 -1.55913018940661 0
- joint R_shoulder_x: axis 1.0 0.0 0.0 -> 0 0 -1; limit lower=-3.1416 upper=0 effort=60 velocity=0 -> (none); origin xyz=0 0 0 rpy=0.0 0.0 0.0 -> xyz=0 0 0 rpy=0 1.5707963267949 0
- joint R_shoulder_y: axis 0.0 1.0 0.0 -> 0 0 1; limit lower=-3.1416 upper=3.1416 effort=60 velocity=0 -> (none); origin xyz=0 -0.255 0.45 rpy=0 0 0 -> xyz=0.000261964373661241 -0.255 0.4500562784516 rpy=1.5707963267949 0 3.14159265358979; parent trunk -> base
- joint R_shoulder_z: axis 0.0 0.0 1.0 -> -1 0 0; limit lower=-3.14 upper=3.14 effort=17 velocity=0 -> (none); origin xyz=0 0 0 rpy=0.0 0.0 0.0 -> xyz=0 -0.114 0.000249999999999991 rpy=1.57186970427954 0 1.5707963267949
- joint imu_joint: origin xyz=0.0 0.0 0.55 rpy=0 0 0 -> xyz=0.0 0.0 0.35 rpy=0 0 0

Commit message: updates, left leg works

File: sim/resources/stompypro/robot_fixed.urdf (robot description, URDF)
Before this commit: robot robot, 21 links, 20 joints
Links:
- removed link L_leg
- removed link trunk
- added link L_finger, mass 0.737286180296128; collision mesh filename=meshes/L_finger.STL; visual mesh filename=meshes/L_finger.STL
- added link L_hip, mass 0.83376821073388; collision mesh filename=meshes/L_hip.STL; visual mesh filename=meshes/L_hip.STL
- added link R_finger, mass 0.869674405890661; collision mesh filename=meshes/R_finger.STL; visual mesh filename=meshes/R_finger.STL
- link L_buttock: mass 1.2990888 -> 0.717874293135761; geometry collision mesh filename=meshes/L_buttock.STL; visual mesh filename=meshes/L_buttock.STL
- link L_calf: mass 1.544772 -> 1.01528348517359; geometry collision mesh filename=meshes/L_calf.STL; visual mesh filename=meshes/L_calf.STL
- link L_clav: mass 1.1246895 -> 0.556581229687908; geometry collision mesh filename=meshes/L_clav.STL; visual mesh filename=meshes/L_clav.STL
- link L_farm: mass 0.66002606 -> 0.344651145281825; geometry collision mesh filename=meshes/L_farm.STL; visual mesh filename=meshes/L_farm.STL
- link L_foot: mass 0.54237266 -> 0.550460500951221; geometry collision mesh filename=meshes/L_foot.STL; visual mesh filename=meshes/L_foot.STL
- link L_scapula: mass 0.65454544 -> 0.338558086149021; geometry collision mesh filename=meshes/L_scapula.STL; visual mesh filename=meshes/L_scapula.STL
- link L_thigh: mass 1.9399504 -> 0.798828442920691; geometry collision mesh filename=meshes/L_thigh.STL; visual mesh filename=meshes/L_thigh.STL
- link L_uarm: mass 0.58244405 -> 0.277294237289419; geometry collision mesh filename=meshes/L_uarm.STL; visual mesh filename=meshes/L_uarm.STL
- link R_buttock: mass 1.2990888 -> 0.716812635597912; geometry collision mesh filename=meshes/R_buttock.STL; visual mesh filename=meshes/R_buttock.STL
- link R_calf: mass 1.544772 -> 1.01514022175102; geometry collision mesh filename=meshes/R_calf.STL; visual mesh filename=meshes/R_calf.STL
- link R_clav: mass 1.1246895 -> 0.556580211071974; geometry collision mesh filename=meshes/R_clav.STL; visual mesh filename=meshes/R_clav.STL
- link R_farm: mass 0.66002606 -> 0.333434347202916; geometry collision mesh filename=meshes/R_farm.STL; visual mesh filename=meshes/R_farm.STL
- link R_foot: mass 0.54237266 -> 0.549121604771221; geometry collision mesh filename=meshes/R_foot.STL; visual mesh filename=meshes/R_foot.STL
- link R_leg: mass 1.3398346 -> 0.827134269923993; geometry collision mesh filename=meshes/R_leg.STL; visual mesh filename=meshes/R_leg.STL
- link R_scapula: mass 0.65454544 -> 0.33855519445856; geometry collision mesh filename=meshes/R_scapula.STL; visual mesh filename=meshes/R_scapula.STL
- link R_thigh: mass 1.9399504 -> 0.79742290295527; geometry collision mesh filename=meshes/R_thigh.STL; visual mesh filename=meshes/R_thigh.STL
- link R_uarm: mass 0.58244405 -> 0.277293520071397; geometry collision mesh filename=meshes/R_uarm.STL; visual mesh filename=meshes/R_uarm.STL
- link base: mass 0.001 -> 8.62540645323623; geometry collision mesh filename=meshes/body_base.STL; visual mesh filename=meshes/body_base.STL
Joints:
- removed joint floating_base
- added joint L_hand_x: type fixed, parent L_farm, child L_finger, origin xyz=0 0.164 0 rpy=1.5707963267949 0 -1.5707963267949, axis -1 0 0
- added joint R_hand_x: type fixed, parent R_farm, child R_finger, origin xyz=-0.00399999999999999 0.164 0 rpy=0.00107337749648937 0 -1.5707963267949, axis -1 0 0
- joint L_ankle_y: axis 0.0 1.0 0.0 -> -1 0 0; origin xyz=0 0 -0.3 rpy=0.0 0.0 0.0 -> xyz=0 0.300033748101774 0 rpy=1.57079632679433 0 -0.0149988751526712
- joint L_elbow_x: axis 1.0 0 0.0 -> -1 0 0; limit lower=-1.9199 upper=1.9199 effort=17 velocity=0 -> (none); origin xyz=0 0 -0.23 rpy=0.0 0.0 0.0 -> xyz=-0.116 0 0 rpy=0 -0.00107337747433267 1.5707963267949
- joint L_hip_x: axis 1.0 0.0 0.0 -> 0 0 1; child L_leg -> L_hip; limit lower=-0.523 upper=2.093 effort=100 velocity=10 -> lower=-2.093 upper=0.523 effort=100 velocity=10; origin xyz=0 0 0 rpy=0.0 0.0 0.0 -> xyz=0 0 0 rpy=0 0 0
- joint L_hip_y: axis 0.0 1.0 0 -> -1 0 0; origin xyz=0 0.1577 0 rpy=0 0 0 -> xyz=0 0.1572 0 rpy=1.5707963267949 0 -1.5707963267949; parent trunk -> base
- joint L_hip_z: axis 0.0 0.0 1.0 -> -1 0 0; origin xyz=0 0 0 rpy=0.0 0 0.0 -> xyz=0 -0.13525 0 rpy=1.5707963267949 0 1.5707963267949; parent L_leg -> L_hip
- joint L_knee: axis 0.0 1.0 0.0 -> -0.999887518980808 0.0149983127852693 0; origin xyz=0 0 -0.3 rpy=0.0 0.0 0.0 -> xyz=-0.16475 0 0.00650000000000001 rpy=1.5707963267949 1.55579745164248 3.14159265358946
- joint L_shoulder_x: axis 1.0 0.0 0.0 -> -1 0 0; limit lower=0 upper=3.1416 effort=60 velocity=0 -> (none); origin xyz=0 0 0 rpy=0.0 0.0 0.0 -> xyz=0 0 0 rpy=3.14159265358979 0 1.5707963267949
- joint L_shoulder_y: axis 0.0 1.0 0.0 -> -1 0 0; limit lower=-3.1416 upper=3.1416 effort=60 velocity=0 -> (none); origin xyz=0 0.255 0.45 rpy=0 0 0 -> xyz=0 0.255 0.45 rpy=0 0 -1.5707963267949; parent trunk -> base
- joint L_shoulder_z: axis 0.0 0.0 1.0 -> -1 0 0; limit lower=-3.14 upper=3.14 effort=17 velocity=0 -> (none); origin xyz=0 0 0 rpy=0.0 0.0 0.0 -> xyz=1.19643736612081E-05 0 0.113943721548401 rpy=1.56972294932056 1.5707963267949 0
- joint R_ankle_y: axis 0.0 1.0 0.0 -> -1 0 0; origin xyz=0 0 -0.3 rpy=0.0 0.0 0.0 -> xyz=0 0.300020415972074 0 rpy=1.57079634708826 0 -3.12992651620125
- joint R_elbow_x: axis 1.0 0 0.0 -> -1 0 0; limit lower=-1.9199 upper=1.9199 effort=17 velocity=0 -> (none); origin xyz=0 0 -0.23 rpy=0.0 0.0 0.0 -> xyz=-0.1155 0.00349999798375654 0 rpy=0 0.0010733774846464 1.5707963267949
- joint R_hip_x: axis 1.0 0.0 0.0 -> 0.999247470344691 -0.0387877945974834 0; origin xyz=0 0 0 rpy=0.0 0.0 0.0 -> xyz=0 0 0 rpy=0 0 0
- joint R_hip_y: axis 0.0 1.0 0 -> 0 0 1; origin xyz=0 -0.1577 0 rpy=0 0 0 -> xyz=0.00525 -0.1572 0 rpy=-1.5707963267949 0.0387975271824028 0; parent trunk -> base
- joint R_hip_z: axis 0.0 0.0 1.0 -> -1 0 0; origin xyz=0 0 0 rpy=0.0 0 0.0 -> xyz=0 0.135351856285756 0 rpy=0 0 -1.6095938539773
- joint R_knee: axis 0.0 1.0 0.0 -> -0.999931951391002 -0.0116658727656092 0; origin xyz=0 0 -0.3 rpy=0.0 0.0 0.0 -> xyz=-0.16475 0 0.00650000000000001 rpy=1.5707963267949 -1.55913018940661 0
- joint R_shoulder_x: axis 1.0 0.0 0.0 -> 0 0 -1; limit lower=-3.1416 upper=0 effort=60 velocity=0 -> (none); origin xyz=0 0 0 rpy=0.0 0.0 0.0 -> xyz=0 0 0 rpy=0 1.5707963267949 0
- joint R_shoulder_y: axis 0.0 1.0 0.0 -> 0 0 1; limit lower=-3.1416 upper=3.1416 effort=60 velocity=0 -> (none); origin xyz=0 -0.255 0.45 rpy=0 0 0 -> xyz=0.000261964373661241 -0.255 0.4500562784516 rpy=1.5707963267949 0 3.14159265358979; parent trunk -> base
- joint R_shoulder_z: axis 0.0 0.0 1.0 -> -1 0 0; limit lower=-3.14 upper=3.14 effort=17 velocity=0 -> (none); origin xyz=0 0 0 rpy=0.0 0.0 0.0 -> xyz=0 -0.114 0.000249999999999991 rpy=1.57186970427954 0 1.5707963267949
- joint imu_joint: origin xyz=0.0 0.0 0.55 rpy=0 0 0 -> xyz=0.0 0.0 0.35 rpy=0 0 0

Commit message: scales, cycle gait, joints and friction

File: sim/resources/stompypro/robot_fixed.urdf (robot description, URDF)
Before this commit: robot k-bot, 22 links, 21 joints
Joints:
- joint L_ankle_y: limit lower=-0.698 upper=0.698 effort=17 velocity=10 -> lower=-0.498 upper=0.498 effort=17 velocity=10
- joint R_ankle_y: limit lower=-0.698 upper=0.698 effort=17 velocity=10 -> lower=-0.398 upper=0.398 effort=17 velocity=10
