Commit message: update efforts

File: sim/resources/stompypro/robot_fixed.urdf (robot description, URDF)
Before this commit: robot k-bot, 22 links, 21 joints
Links:
- link imu_link: geometry visual box size=0.1 0.3 0.1
Joints:
- joint L_ankle_y: limit lower=-0.498 upper=0.498 effort=17 velocity=10 -> lower=-0.498 upper=0.498 effort=100 velocity=10
- joint R_ankle_y: limit lower=-0.398 upper=0.398 effort=17 velocity=10 -> lower=-0.398 upper=0.398 effort=100 velocity=10

Commit message: save imu vis

File: sim/resources/stompypro/robot_fixed.urdf (robot description, URDF)
Before this commit: robot k-bot, 22 links, 21 joints
Links:
- link R_finger: mass 0.869674405890661 -> 0.739674405890661
- link imu_link: geometry visual box size=0.3 0.01 0.01

Commit message: update the urdf

File: sim/resources/stompypro/robot_fixed.urdf (robot description, URDF)
Before this commit: robot k-bot, 22 links, 21 joints
Joints:
- joint L_ankle_y: axis -1 0 0 -> 1 0 0
- joint L_knee: axis -0.999887518980808 0.0149983127852693 0 -> -1 0 0; limit lower=-1.919 upper=1.919 effort=250 velocity=10 -> lower=-1.919 upper=0 effort=250 velocity=10
- joint R_ankle_y: axis -1 0 0 -> 1 0 0; limit lower=-0.398 upper=0.398 effort=100 velocity=10 -> lower=-0.498 upper=0.498 effort=100 velocity=10
- joint R_hip_x: axis 0.999247470344691 -0.0387877945974834 0 -> 1 0 0
- joint R_hip_y: axis 0 0 1 -> 0 0 -1
- joint R_knee: axis -0.999931951391002 -0.0116658727656092 0 -> 1 0 0; limit lower=-1.919 upper=1.919 effort=250 velocity=10 -> lower=0 upper=1.919 effort=250 velocity=10

Commit message: update join position

File: sim/resources/stompypro/robot_fixed.urdf (robot description, URDF)
Before this commit: robot k-bot, 22 links, 21 joints
Links:
- link base: mass 8.62540645323623 -> 13.62540645323623

Commit message: removign pushing allows for lower kps

File: sim/resources/stompypro/robot_fixed.urdf (robot description, URDF)
Before this commit: robot k-bot, 22 links, 21 joints
Joints:
- joint L_ankle_y: limit lower=-0.498 upper=0.498 effort=100 velocity=10 -> lower=-0.498 upper=0.498 effort=50 velocity=10
- joint L_hip_y: limit lower=-3.14 upper=3.14 effort=250 velocity=10 -> lower=-3.14 upper=3.14 effort=120 velocity=10
- joint L_knee: limit lower=-1.919 upper=0 effort=250 velocity=10 -> lower=-1.919 upper=0 effort=120 velocity=10
- joint R_ankle_y: limit lower=-0.498 upper=0.498 effort=100 velocity=10 -> lower=-0.498 upper=0.498 effort=50 velocity=10
- joint R_hip_y: limit lower=-3.14 upper=3.14 effort=250 velocity=10 -> lower=-3.14 upper=3.14 effort=120 velocity=10
- joint R_knee: limit lower=0 upper=1.919 effort=250 velocity=10 -> lower=0 upper=1.919 effort=120 velocity=10
