Commit message: update zeroth

File: sim/resources/zeroth/robot.urdf (robot description, URDF)
Before this commit: robot zeroth, 12 links, 11 joints
Links:
- removed link Part_76
- removed link Robot_-_STS3250_v1
- removed link Robot_-_STS3250_v1_2
- removed link Rotor
- removed link Rotor_2
- removed link foot_bracket_for_5dof_leg_v9
- removed link foot_bracket_for_5dof_leg_v9_2
- removed link leg_top_bracket_v8_1
- removed link leg_top_bracket_v8_1_2
- removed link leg_top_bracket_v9
- removed link leg_top_bracket_v9_2
- added link Document, mass 1.036095351; collision mesh filename=meshes/Document.stl; visual mesh filename=meshes/Document.stl
- added link SERVO-DUAL_v2, mass 0.110875259; collision mesh filename=meshes/SERVO-DUAL_v2.stl; visual mesh filename=meshes/SERVO-DUAL_v2.stl
- added link SERVO-DUAL_v2(Mirror), mass 0.110875424; collision mesh filename=meshes/SERVO-DUAL_v2(Mirror).stl; visual mesh filename=meshes/SERVO-DUAL_v2(Mirror).stl
- added link SERVO-DUAL_v2(Mirror)_1, mass 0.165984684; collision mesh filename=meshes/SERVO-DUAL_v2(Mirror)_1.stl; visual mesh filename=meshes/SERVO-DUAL_v2(Mirror)_1.stl
- added link SERVO-DUAL_v2(Mirror)_3, mass 0.22693714599999998; collision mesh filename=meshes/SERVO-DUAL_v2(Mirror)_3.stl; visual mesh filename=meshes/SERVO-DUAL_v2(Mirror)_3.stl
- added link SERVO-DUAL_v2(Mirror)_4, mass 0.145867186; collision mesh filename=meshes/SERVO-DUAL_v2(Mirror)_4.stl; visual mesh filename=meshes/SERVO-DUAL_v2(Mirror)_4.stl
- added link SERVO-DUAL_v2_1, mass 0.16598466899999997; collision mesh filename=meshes/SERVO-DUAL_v2_1.stl; visual mesh filename=meshes/SERVO-DUAL_v2_1.stl
- added link SERVO-DUAL_v2_2, mass 0.166182934; collision mesh filename=meshes/SERVO-DUAL_v2_2.stl; visual mesh filename=meshes/SERVO-DUAL_v2_2.stl
- added link SERVO-DUAL_v2_2_2, mass 0.166182928; collision mesh filename=meshes/SERVO-DUAL_v2_2_2.stl; visual mesh filename=meshes/SERVO-DUAL_v2_2_2.stl
- added link SERVO-DUAL_v2_4, mass 0.226937274; collision mesh filename=meshes/SERVO-DUAL_v2_4.stl; visual mesh filename=meshes/SERVO-DUAL_v2_4.stl
- added link SERVO-DUAL_v2_5, mass 0.145867171; collision mesh filename=meshes/SERVO-DUAL_v2_5.stl; visual mesh filename=meshes/SERVO-DUAL_v2_5.stl
- added link Z-BOT2_MASTER-v24_DEC07-ASSY_v3, mass 0.016645284; collision mesh filename=meshes/Z-BOT2_MASTER-v24_DEC07-ASSY_v3.stl; visual mesh filename=meshes/Z-BOT2_MASTER-v24_DEC07-ASSY_v3.stl
- added link Z-BOT2_MASTER-v24_DEC07-ASSY_v3_2, mass 0.016645284; collision mesh filename=meshes/Z-BOT2_MASTER-v24_DEC07-ASSY_v3_2.stl; visual mesh filename=meshes/Z-BOT2_MASTER-v24_DEC07-ASSY_v3_2.stl
- added link Z-BOT2_MASTER-v24_DEC07-ASSY_v3_3, mass 0.030093227; collision mesh filename=meshes/Z-BOT2_MASTER-v24_DEC07-ASSY_v3_3.stl; visual mesh filename=meshes/Z-BOT2_MASTER-v24_DEC07-ASSY_v3_3.stl
- added link Z-BOT2_MASTER-v24_DEC07-ASSY_v3_4, mass 0.030093227; collision mesh filename=meshes/Z-BOT2_MASTER-v24_DEC07-ASSY_v3_4.stl; visual mesh filename=meshes/Z-BOT2_MASTER-v24_DEC07-ASSY_v3_4.stl
- added link Z-BOT2_MASTER-v24_DEC07-ASSY_v3_5, mass 0.102093376; collision mesh filename=meshes/Z-BOT2_MASTER-v24_DEC07-ASSY_v3_5.stl; visual mesh filename=meshes/Z-BOT2_MASTER-v24_DEC07-ASSY_v3_5.stl
- added link Z-BOT2_MASTER-v24_DEC07-ASSY_v3_6, mass 0.102093376; collision mesh filename=meshes/Z-BOT2_MASTER-v24_DEC07-ASSY_v3_6.stl; visual mesh filename=meshes/Z-BOT2_MASTER-v24_DEC07-ASSY_v3_6.stl
Joints:
- added joint left_elbow_yaw: type revolute, parent SERVO-DUAL_v2_2, child SERVO-DUAL_v2_1, origin xyz=-0.018825 0.09368378999999999 -0.023450655999999997 rpy=3.1415926071795868 1.5707963 0.0, axis 0 0 1, limit lower=-2.268928 upper=1.5707963 effort=80 velocity=5
- added joint left_shoulder_pitch: type revolute, parent Z-BOT2_MASTER-v24_DEC07-ASSY_v3, child SERVO-DUAL_v2_2, origin xyz=0.017067737 -0.0048184479 0.018826238 rpy=3.1415927 1.5707963 0, axis 0 0 1, limit lower=-3.1415927 upper=3.1415927 effort=80 velocity=5
- added joint left_shoulder_yaw: type revolute, parent Document, child Z-BOT2_MASTER-v24_DEC07-ASSY_v3, origin xyz=0.057194730000000006 0.016280631268824133 0.021094319501615166 rpy=1.5707963000000003 0.0 0.0, axis 0 0 1, limit lower=-0.17453293 upper=1.3962634 effort=80 velocity=5
- added joint right_elbow_yaw: type revolute, parent SERVO-DUAL_v2_2_2, child SERVO-DUAL_v2(Mirror)_1, origin xyz=-0.018825 -0.09368378999999999 -0.023450655999999997 rpy=0.0 -1.5707963 0.0, axis 0 0 1, limit lower=-1.5707963 upper=2.268928 effort=80 velocity=5
- added joint right_shoulder_pitch: type revolute, parent Z-BOT2_MASTER-v24_DEC07-ASSY_v3_2, child SERVO-DUAL_v2_2_2, origin xyz=-0.017067737 -0.0048184479 0.018826238 rpy=0 1.5707963 0, axis 0 0 1, limit lower=-3.1415927 upper=3.1415927 effort=80 velocity=5
- added joint right_shoulder_yaw: type revolute, parent Document, child Z-BOT2_MASTER-v24_DEC07-ASSY_v3_2, origin xyz=-0.056366071000000004 0.016280631268824133 0.021094319501615166 rpy=1.5707963000000003 0.0 0.0, axis 0 0 1, limit lower=-1.3962634 upper=0.17453293 effort=80 velocity=5
- joint floating_base: child Part_76 -> Document
- joint left_ankle_pitch: child foot_bracket_for_5dof_leg_v9 -> Z-BOT2_MASTER-v24_DEC07-ASSY_v3_5; origin xyz=-0.09999999473730714 -3.719999999707291e-08 -7.499219426298359e-05 rpy=-3.1415926071795863 0.0 0.0 -> xyz=-3.6496522071854942e-09 -0.09960050419999995 -6.451933117575595e-05 rpy=-3.1415926071795863 0.0 0.0; parent leg_top_bracket_v8_1 -> SERVO-DUAL_v2_4
- joint left_hip_pitch: child leg_top_bracket_v9 -> SERVO-DUAL_v2_5; limit lower=-1.5707963 upper=1.5707963 effort=80 velocity=5 -> lower=-1.8325957 upper=1.7453293 effort=80 velocity=5; origin xyz=0.018525040302885504 -4.922427119732897e-07 0.0183599908378569 rpy=1.570796353589794 4.641020678874952e-08 -1.5707963000000005 -> xyz=0.010290707000000003 0.0316618118359243 -0.02465886601719911 rpy=3.141592626794896 -1.5707962889011906 0.0; parent Robot_-_STS3250_v1 -> SERVO-DUAL_v2
- joint left_hip_roll: child Rotor -> Z-BOT2_MASTER-v24_DEC07-ASSY_v3_3; limit lower=-0.78539816 upper=0.78539816 effort=80 velocity=5 -> lower=-1.0471976 upper=1.0471976 effort=80 velocity=5; origin xyz=-0.0353001417379795 -0.0036199730613269685 -0.07354320094310968 rpy=-0.005235926794896062 2.67948967458409e-08 0.0 -> xyz=0.042980284550000004 -0.00014490883999999926 -0.0579460267 rpy=-3.1415926071795863 0.0 0.0; parent Part_76 -> Document
- joint left_hip_yaw: child Robot_-_STS3250_v1 -> SERVO-DUAL_v2; limit lower=-0.087266463 upper=1.5707963 effort=80 velocity=5 -> lower=-1.9198622 upper=0.17453293 effort=80 velocity=5; origin xyz=0.0 -0.018009991 -0.020898149999999997 rpy=-1.5707963000000003 0.0 0.0 -> xyz=0.0082500076 -0.024599356 0.056607331 rpy=1.5707963 0 0; parent Rotor -> Z-BOT2_MASTER-v24_DEC07-ASSY_v3_3
- joint left_knee_pitch: axis 0 0 -1 -> 0 0 1; child leg_top_bracket_v8_1 -> SERVO-DUAL_v2_4; limit lower=-1.5707963 upper=1.5707963 effort=80 velocity=5 -> lower=-0.17453293 upper=2.9670597 effort=80 velocity=5; origin xyz=-0.12916282413730715 -1.9999999954778414e-09 0.0372749282506018 rpy=0.0 0.0 0.0 -> xyz=0.021500004396296457 -0.10043832342856604 -0.000289528907266242 rpy=-4.6410205422728156e-08 0.0 4.6410206666284834e-08; parent leg_top_bracket_v9 -> SERVO-DUAL_v2_5
- joint right_ankle_pitch: child foot_bracket_for_5dof_leg_v9_2 -> Z-BOT2_MASTER-v24_DEC07-ASSY_v3_6; origin xyz=0.09999999915897508 -5.7487026731006386e-08 2.5007553905526114e-05 rpy=-3.141592607179616 2.6794969798515922e-08 -5.535897937836154e-07 -> xyz=-8.175391336129323e-10 0.09960050362638555 -6.451866882414142e-05 rpy=-3.141592653589792 0.0 -4.641020678874952e-08; parent leg_top_bracket_v8_1_2 -> SERVO-DUAL_v2(Mirror)_3
- joint right_hip_pitch: child leg_top_bracket_v9_2 -> SERVO-DUAL_v2(Mirror)_4; limit lower=-1.5707963 upper=1.5707963 effort=80 velocity=5 -> lower=-1.7453293 upper=1.8325957 effort=80 velocity=5; origin xyz=0.01852495960295464 -4.235463209323331e-09 0.018359997984461623 rpy=-1.5707963535897924 -4.64102059005711e-08 1.5707963000000003 -> xyz=-0.010290707000000003 0.0316618118359243 -0.02465886601719911 rpy=2.6794896194407875e-08 -1.5707962889011906 0.0; parent Robot_-_STS3250_v1_2 -> SERVO-DUAL_v2(Mirror)
- joint right_hip_roll: child Rotor_2 -> Z-BOT2_MASTER-v24_DEC07-ASSY_v3_4; limit lower=-0.78539816 upper=0.78539816 effort=80 velocity=5 -> lower=-1.0471976 upper=1.0471976 effort=80 velocity=5; origin xyz=0.035299859288700844 -0.0036199727372057573 -0.0735432024963366 rpy=-0.005235980384690442 -2.6794896301751692e-08 2.220446049250313e-16 -> xyz=-0.04269607545 -0.00014490883999999926 -0.0579460267 rpy=-3.1415926071795863 0.0 0.0; parent Part_76 -> Document
- joint right_hip_yaw: child Robot_-_STS3250_v1_2 -> SERVO-DUAL_v2(Mirror); limit lower=-1.5707963 upper=0.087266463 effort=80 velocity=5 -> lower=-0.17453293 upper=1.9198622 effort=80 velocity=5; origin xyz=0.0 -0.018009991 -0.020898149999999997 rpy=-1.5707963000000003 0.0 0.0 -> xyz=-0.0082500076 -0.024599356 0.056607331 rpy=1.5707963 0 0; parent Rotor_2 -> Z-BOT2_MASTER-v24_DEC07-ASSY_v3_4
- joint right_knee_pitch: axis 0 0 -1 -> 0 0 1; child leg_top_bracket_v8_1_2 -> SERVO-DUAL_v2(Mirror)_3; limit lower=-1.5707963 upper=1.5707963 effort=80 velocity=5 -> lower=-2.9670597 upper=0.17453293 effort=80 velocity=5; origin xyz=0.12916282526269282 1.999999997212565e-09 0.0003749122493981972 rpy=-3.1415926071795863 0.0 0.0 -> xyz=0.021499999495586064 0.10043832500000001 -0.00028952709273386 rpy=0.0 0.0 0.0; parent leg_top_bracket_v9_2 -> SERVO-DUAL_v2(Mirror)_4

File: sim/resources/zeroth/robot_fixed.urdf (robot description, URDF)
Before this commit: robot zeroth, 12 links, 11 joints
Links:
- removed link Part_76
- removed link Robot_-_STS3250_v1
- removed link Robot_-_STS3250_v1_2
- removed link Rotor
- removed link Rotor_2
- removed link foot_bracket_for_5dof_leg_v9
- removed link foot_bracket_for_5dof_leg_v9_2
- removed link leg_top_bracket_v8_1
- removed link leg_top_bracket_v8_1_2
- removed link leg_top_bracket_v9
- removed link leg_top_bracket_v9_2
- added link Document, mass 1.036095351; collision mesh filename=meshes/Document.stl; visual mesh filename=meshes/Document.stl
- added link SERVO-DUAL_v2, mass 0.110875259; collision mesh filename=meshes/SERVO-DUAL_v2.stl; visual mesh filename=meshes/SERVO-DUAL_v2.stl
- added link SERVO-DUAL_v2(Mirror), mass 0.110875424; collision mesh filename=meshes/SERVO-DUAL_v2(Mirror).stl; visual mesh filename=meshes/SERVO-DUAL_v2(Mirror).stl
- added link SERVO-DUAL_v2(Mirror)_1, mass 0.165984684; collision mesh filename=meshes/SERVO-DUAL_v2(Mirror)_1.stl; visual mesh filename=meshes/SERVO-DUAL_v2(Mirror)_1.stl
- added link SERVO-DUAL_v2(Mirror)_3, mass 0.22693714599999998; collision mesh filename=meshes/SERVO-DUAL_v2(Mirror)_3.stl; visual mesh filename=meshes/SERVO-DUAL_v2(Mirror)_3.stl
- added link SERVO-DUAL_v2(Mirror)_4, mass 0.145867186; collision mesh filename=meshes/SERVO-DUAL_v2(Mirror)_4.stl; visual mesh filename=meshes/SERVO-DUAL_v2(Mirror)_4.stl
- added link SERVO-DUAL_v2_1, mass 0.16598466899999997; collision mesh filename=meshes/SERVO-DUAL_v2_1.stl; visual mesh filename=meshes/SERVO-DUAL_v2_1.stl
- added link SERVO-DUAL_v2_2, mass 0.166182934; collision mesh filename=meshes/SERVO-DUAL_v2_2.stl; visual mesh filename=meshes/SERVO-DUAL_v2_2.stl
- added link SERVO-DUAL_v2_2_2, mass 0.166182928; collision mesh filename=meshes/SERVO-DUAL_v2_2_2.stl; visual mesh filename=meshes/SERVO-DUAL_v2_2_2.stl
- added link SERVO-DUAL_v2_4, mass 0.226937274; collision mesh filename=meshes/SERVO-DUAL_v2_4.stl; visual mesh filename=meshes/SERVO-DUAL_v2_4.stl
- added link SERVO-DUAL_v2_5, mass 0.145867171; collision mesh filename=meshes/SERVO-DUAL_v2_5.stl; visual mesh filename=meshes/SERVO-DUAL_v2_5.stl
- added link Z-BOT2_MASTER-v24_DEC07-ASSY_v3, mass 0.016645284; collision mesh filename=meshes/Z-BOT2_MASTER-v24_DEC07-ASSY_v3.stl; visual mesh filename=meshes/Z-BOT2_MASTER-v24_DEC07-ASSY_v3.stl
- added link Z-BOT2_MASTER-v24_DEC07-ASSY_v3_2, mass 0.016645284; collision mesh filename=meshes/Z-BOT2_MASTER-v24_DEC07-ASSY_v3_2.stl; visual mesh filename=meshes/Z-BOT2_MASTER-v24_DEC07-ASSY_v3_2.stl
- added link Z-BOT2_MASTER-v24_DEC07-ASSY_v3_3, mass 0.030093227; collision mesh filename=meshes/Z-BOT2_MASTER-v24_DEC07-ASSY_v3_3.stl; visual mesh filename=meshes/Z-BOT2_MASTER-v24_DEC07-ASSY_v3_3.stl
- added link Z-BOT2_MASTER-v24_DEC07-ASSY_v3_4, mass 0.030093227; collision mesh filename=meshes/Z-BOT2_MASTER-v24_DEC07-ASSY_v3_4.stl; visual mesh filename=meshes/Z-BOT2_MASTER-v24_DEC07-ASSY_v3_4.stl
- added link Z-BOT2_MASTER-v24_DEC07-ASSY_v3_5, mass 0.102093376; collision mesh filename=meshes/Z-BOT2_MASTER-v24_DEC07-ASSY_v3_5.stl; visual mesh filename=meshes/Z-BOT2_MASTER-v24_DEC07-ASSY_v3_5.stl
- added link Z-BOT2_MASTER-v24_DEC07-ASSY_v3_6, mass 0.102093376; collision mesh filename=meshes/Z-BOT2_MASTER-v24_DEC07-ASSY_v3_6.stl; visual mesh filename=meshes/Z-BOT2_MASTER-v24_DEC07-ASSY_v3_6.stl
Joints:
- added joint left_elbow_yaw: type fixed, parent SERVO-DUAL_v2_2, child SERVO-DUAL_v2_1, origin xyz=-0.018825 0.09368378999999999 -0.023450655999999997 rpy=3.1415926071795868 1.5707963 0.0, axis 0 0 1, limit lower=-2.268928 upper=1.5707963 effort=80 velocity=5
- added joint left_shoulder_pitch: type fixed, parent Z-BOT2_MASTER-v24_DEC07-ASSY_v3, child SERVO-DUAL_v2_2, origin xyz=0.017067737 -0.0048184479 0.018826238 rpy=3.1415927 1.5707963 0, axis 0 0 1, limit lower=-3.1415927 upper=3.1415927 effort=80 velocity=5
- added joint left_shoulder_yaw: type fixed, parent Document, child Z-BOT2_MASTER-v24_DEC07-ASSY_v3, origin xyz=0.057194730000000006 0.016280631268824133 0.021094319501615166 rpy=1.5707963000000003 0.0 0.0, axis 0 0 1, limit lower=-0.17453293 upper=1.3962634 effort=80 velocity=5
- added joint right_elbow_yaw: type fixed, parent SERVO-DUAL_v2_2_2, child SERVO-DUAL_v2(Mirror)_1, origin xyz=-0.018825 -0.09368378999999999 -0.023450655999999997 rpy=0.0 -1.5707963 0.0, axis 0 0 1, limit lower=-1.5707963 upper=2.268928 effort=80 velocity=5
- added joint right_shoulder_pitch: type fixed, parent Z-BOT2_MASTER-v24_DEC07-ASSY_v3_2, child SERVO-DUAL_v2_2_2, origin xyz=-0.017067737 -0.0048184479 0.018826238 rpy=0 1.5707963 0, axis 0 0 1, limit lower=-3.1415927 upper=3.1415927 effort=80 velocity=5
- added joint right_shoulder_yaw: type fixed, parent Document, child Z-BOT2_MASTER-v24_DEC07-ASSY_v3_2, origin xyz=-0.056366071000000004 0.016280631268824133 0.021094319501615166 rpy=1.5707963000000003 0.0 0.0, axis 0 0 1, limit lower=-1.3962634 upper=0.17453293 effort=80 velocity=5
- joint floating_base: child Part_76 -> Document; origin xyz=0 0 0 rpy=0 0 -1.5707963267948966 -> xyz=0 0 0 rpy=0 0 0
- joint left_ankle_pitch: child foot_bracket_for_5dof_leg_v9 -> Z-BOT2_MASTER-v24_DEC07-ASSY_v3_5; origin xyz=-0.09999999473730714 -3.719999999707291e-08 -7.499219426298359e-05 rpy=-3.1415926071795863 0.0 0.0 -> xyz=-3.6496522071854942e-09 -0.09960050419999995 -6.451933117575595e-05 rpy=-3.1415926071795863 0.0 0.0; parent leg_top_bracket_v8_1 -> SERVO-DUAL_v2_4
- joint left_hip_pitch: child leg_top_bracket_v9 -> SERVO-DUAL_v2_5; limit lower=-1.5707963 upper=1.5707963 effort=10 velocity=10 -> lower=-1.8325957 upper=1.7453293 effort=10 velocity=10; origin xyz=0.018525040302885504 -4.922427119732897e-07 0.0183599908378569 rpy=1.570796353589794 4.641020678874952e-08 -1.5707963000000005 -> xyz=0.010290707000000003 0.0316618118359243 -0.02465886601719911 rpy=3.141592626794896 -1.5707962889011906 0.0; parent Robot_-_STS3250_v1 -> SERVO-DUAL_v2
- joint left_hip_roll: child Rotor -> Z-BOT2_MASTER-v24_DEC07-ASSY_v3_3; limit lower=-0.78539816 upper=0.78539816 effort=10 velocity=10 -> lower=-1.0471976 upper=1.0471976 effort=10 velocity=10; origin xyz=-0.0353001417379795 -0.0036199730613269685 -0.07354320094310968 rpy=-0.005235926794896062 2.67948967458409e-08 0.0 -> xyz=0.042980284550000004 -0.00014490883999999926 -0.0579460267 rpy=-3.1415926071795863 0.0 0.0; parent Part_76 -> Document
- joint left_hip_yaw: child Robot_-_STS3250_v1 -> SERVO-DUAL_v2; limit lower=-0.087266463 upper=1.5707963 effort=10 velocity=10 -> lower=-1.9198622 upper=0.17453293 effort=10 velocity=10; origin xyz=0.0 -0.018009991 -0.020898149999999997 rpy=-1.5707963000000003 0.0 0.0 -> xyz=0.0082500076 -0.024599356 0.056607331 rpy=1.5707963 0 0; parent Rotor -> Z-BOT2_MASTER-v24_DEC07-ASSY_v3_3
- joint left_knee_pitch: axis 0 0 -1 -> 0 0 1; child leg_top_bracket_v8_1 -> SERVO-DUAL_v2_4; limit lower=-1.57 upper=0 effort=10 velocity=10 -> lower=0 upper=1.57 effort=10 velocity=10; origin xyz=-0.12916282413730715 -1.9999999954778414e-09 0.0372749282506018 rpy=0.0 0.0 0.0 -> xyz=0.021500004396296457 -0.10043832342856604 -0.000289528907266242 rpy=-4.6410205422728156e-08 0.0 4.6410206666284834e-08; parent leg_top_bracket_v9 -> SERVO-DUAL_v2_5
- joint right_ankle_pitch: child foot_bracket_for_5dof_leg_v9_2 -> Z-BOT2_MASTER-v24_DEC07-ASSY_v3_6; origin xyz=0.09999999915897508 -5.7487026731006386e-08 2.5007553905526114e-05 rpy=-3.141592607179616 2.6794969798515922e-08 -5.535897937836154e-07 -> xyz=-8.175391336129323e-10 0.09960050362638555 -6.451866882414142e-05 rpy=-3.141592653589792 0.0 -4.641020678874952e-08; parent leg_top_bracket_v8_1_2 -> SERVO-DUAL_v2(Mirror)_3
- joint right_hip_pitch: child leg_top_bracket_v9_2 -> SERVO-DUAL_v2(Mirror)_4; limit lower=-1.5707963 upper=1.5707963 effort=10 velocity=10 -> lower=-1.7453293 upper=1.8325957 effort=10 velocity=10; origin xyz=0.01852495960295464 -4.235463209323331e-09 0.018359997984461623 rpy=-1.5707963535897924 -4.64102059005711e-08 1.5707963000000003 -> xyz=-0.010290707000000003 0.0316618118359243 -0.02465886601719911 rpy=2.6794896194407875e-08 -1.5707962889011906 0.0; parent Robot_-_STS3250_v1_2 -> SERVO-DUAL_v2(Mirror)
- joint right_hip_roll: child Rotor_2 -> Z-BOT2_MASTER-v24_DEC07-ASSY_v3_4; limit lower=-0.78539816 upper=0.78539816 effort=10 velocity=10 -> lower=-1.0471976 upper=1.0471976 effort=10 velocity=10; origin xyz=0.035299859288700844 -0.0036199727372057573 -0.0735432024963366 rpy=-0.005235980384690442 -2.6794896301751692e-08 2.220446049250313e-16 -> xyz=-0.04269607545 -0.00014490883999999926 -0.0579460267 rpy=-3.1415926071795863 0.0 0.0; parent Part_76 -> Document
- joint right_hip_yaw: child Robot_-_STS3250_v1_2 -> SERVO-DUAL_v2(Mirror); limit lower=-1.5707963 upper=0.087266463 effort=10 velocity=10 -> lower=-0.17453293 upper=1.9198622 effort=10 velocity=10; origin xyz=0.0 -0.018009991 -0.020898149999999997 rpy=-1.5707963000000003 0.0 0.0 -> xyz=-0.0082500076 -0.024599356 0.056607331 rpy=1.5707963 0 0; parent Rotor_2 -> Z-BOT2_MASTER-v24_DEC07-ASSY_v3_4
- joint right_knee_pitch: axis 0 0 -1 -> 0 0 1; child leg_top_bracket_v8_1_2 -> SERVO-DUAL_v2(Mirror)_3; limit lower=0 upper=1.57 effort=10 velocity=10 -> lower=-1.57 upper=0 effort=10 velocity=10; origin xyz=0.12916282526269282 1.999999997212565e-09 0.0003749122493981972 rpy=-3.1415926071795863 0.0 0.0 -> xyz=0.021499999495586064 0.10043832500000001 -0.00028952709273386 rpy=0.0 0.0 0.0; parent leg_top_bracket_v9_2 -> SERVO-DUAL_v2(Mirror)_4

Commit message: add proper height and parameters

File: sim/resources/zeroth/robot.urdf (robot description, URDF)
Before this commit: robot z-02_urdf_assembly, 18 links, 17 joints
Joints:
- joint floating_base: origin xyz=0 0 0 rpy=0 0 0 -> xyz=0 0 0 rpy=0 0 1.57

File: sim/resources/zeroth/robot_fixed.urdf (robot description, URDF)
Before this commit: robot z-02_urdf_assembly, 18 links, 17 joints
Joints:
- joint floating_base: origin xyz=0 0 0 rpy=0 0 0 -> xyz=0 0 0 rpy=0 0 1.57
