Commit message: updated urdf from onshape

File: sim/resources/zbot2/robot.urdf (robot description, URDF)
Before this commit: robot assembly_1, 20 links, 19 joints
Links:
- link FINGER_1: mass 0.023485225999999998 -> 0.045310716
- link FINGER_1_1: mass 0.023485229 -> 0.045310724000000004
- link FK-AP-019-25T_11_16: mass 0.10041221239999999 -> 0.1408833525
- link FK-AP-019-25T_11_5: mass 0.1004122084 -> 0.1408833515
- link FOOT: mass 0.054831927 -> 0.096390673
- link FOOT_1: mass 0.054831945 -> 0.096390725
- link L-ARM_1: mass 0.0930900236 -> 0.1697714245
- link R-ARM-1: mass 0.0930898796 -> 0.1697709975
- link SJ-WK00-0021TOPCABINETCASE_104_7: mass 0.042114028 -> 0.045121527999999994
- link SJ-WK00-0023BOTTOMCASE_12_12: mass 0.068115593 -> 0.120162816
- link SJ-WK00-0023BOTTOMCASE_12_13: mass 0.081325173 -> 0.081865261
- link SJ-WK00-0023BOTTOMCASE_12_8: mass 0.068115596 -> 0.120162817
- link U-HIP: mass 0.016331226 -> 0.047132399
- link U-HIP_1: mass 0.016331226 -> 0.047132399
- link WJ-DP00-0002-FK-AP-020_7_10: mass 0.042114023 -> 0.045121525999999995
- link WJ-DP00-0002-FK-AP-020_7_8: mass 0.081325175 -> 0.081865261
- link Z-BOT2-MASTER-SHOULDER2: mass 0.0083497418 -> 0.0240976
- link Z-BOT2-MASTER-SHOULDER2_1: mass 0.0083497418 -> 0.0240976
- link Z-BOT2_MASTER-BODY-SKELETON: mass 0.9136450087000001 -> 1.5916352207
Joints:
- joint left_ankle_pitch: limit lower=-1.5707963 upper=1.5707963 effort=80 velocity=5 -> lower=-0.26179939 upper=2.8797933 effort=80 velocity=5

Commit message: upload latest urdf

File: sim/resources/zbot2/robot.urdf (robot description, URDF)
Before this commit: robot assembly_1, 20 links, 19 joints
Links:
- removed link FINGER_1_1
- removed link FK-AP-019-25T_11_16
- removed link FK-AP-019-25T_11_5
- removed link FOOT_1
- removed link SJ-WK00-0021TOPCABINETCASE_104_7
- removed link SJ-WK00-0023BOTTOMCASE_12_12
- removed link SJ-WK00-0023BOTTOMCASE_12_13
- removed link SJ-WK00-0023BOTTOMCASE_12_8
- removed link U-HIP
- removed link U-HIP_1
- removed link WJ-DP00-0002-FK-AP-020_7_10
- removed link WJ-DP00-0002-FK-AP-020_7_8
- removed link Z-BOT2-MASTER-SHOULDER2_1
- added link FINGER_1_2, mass 0.022322296; collision mesh filename=meshes/FINGER_1_2.stl; visual mesh filename=meshes/FINGER_1_2.stl
- added link FK-AP-019-25T_11, mass 0.14822332759999998; collision mesh filename=meshes/FK-AP-019-25T_11.stl; visual mesh filename=meshes/FK-AP-019-25T_11.stl
- added link FK-AP-019-25T_11_2, mass 0.1482233276; collision mesh filename=meshes/FK-AP-019-25T_11_2.stl; visual mesh filename=meshes/FK-AP-019-25T_11_2.stl
- added link FOOT_2, mass 0.09495736199999999; collision mesh filename=meshes/FOOT_2.stl; visual mesh filename=meshes/FOOT_2.stl
- added link U-HIP-L, mass 0.016091061; collision mesh filename=meshes/U-HIP-L.stl; visual mesh filename=meshes/U-HIP-L.stl
- added link U-HIP-R, mass 0.016091061; collision mesh filename=meshes/U-HIP-R.stl; visual mesh filename=meshes/U-HIP-R.stl
- added link WJ-DP00-0002-FK-AP-020_7, mass 0.066367059; collision mesh filename=meshes/WJ-DP00-0002-FK-AP-020_7.stl; visual mesh filename=meshes/WJ-DP00-0002-FK-AP-020_7.stl
- added link WJ-DP00-0002-FK-AP-020_7_2, mass 0.066367059; collision mesh filename=meshes/WJ-DP00-0002-FK-AP-020_7_2.stl; visual mesh filename=meshes/WJ-DP00-0002-FK-AP-020_7_2.stl
- added link WJ-DP00-0002-FK-AP-020_7_3, mass 0.091986251; collision mesh filename=meshes/WJ-DP00-0002-FK-AP-020_7_3.stl; visual mesh filename=meshes/WJ-DP00-0002-FK-AP-020_7_3.stl
- added link WJ-DP00-0002-FK-AP-020_7_4, mass 0.091986251; collision mesh filename=meshes/WJ-DP00-0002-FK-AP-020_7_4.stl; visual mesh filename=meshes/WJ-DP00-0002-FK-AP-020_7_4.stl
- added link WJ-DP00-0002-FK-AP-020_7_5, mass 0.1298739283; collision mesh filename=meshes/WJ-DP00-0002-FK-AP-020_7_5.stl; visual mesh filename=meshes/WJ-DP00-0002-FK-AP-020_7_5.stl
- added link WJ-DP00-0002-FK-AP-020_7_6, mass 0.1298739283; collision mesh filename=meshes/WJ-DP00-0002-FK-AP-020_7_6.stl; visual mesh filename=meshes/WJ-DP00-0002-FK-AP-020_7_6.stl
- added link Z-BOT2-MASTER-SHOULDER2_2, mass 0.0082269514; collision mesh filename=meshes/Z-BOT2-MASTER-SHOULDER2_2.stl; visual mesh filename=meshes/Z-BOT2-MASTER-SHOULDER2_2.stl
- link FINGER_1: mass 0.045310716 -> 0.022322296
- link FOOT: mass 0.096390673 -> 0.09495736199999999
- link L-ARM_1: mass 0.1697714245 -> 0.113768642
- link R-ARM-1: mass 0.1697709975 -> 0.113768495
- link Z-BOT2-MASTER-SHOULDER2: mass 0.0240976 -> 0.0082269514
- link Z-BOT2_MASTER-BODY-SKELETON: mass 1.5916352207 -> 1.00556824628
Joints:
- removed joint left_ankle_pitch
- removed joint left_elbow_yaw
- removed joint left_gripper
- removed joint left_hip_pitch
- removed joint left_hip_roll
- removed joint left_hip_yaw
- removed joint left_knee_pitch
- removed joint left_shoulder_pitch
- removed joint left_shoulder_yaw
- removed joint right_ankle_pitch
- removed joint right_elbow_yaw
- removed joint right_gripper
- removed joint right_hip_pitch
- removed joint right_hip_roll
- removed joint right_hip_yaw
- removed joint right_knee_pitch
- removed joint right_shoulder_pitch
- removed joint right_shoulder_yaw
- added joint L_Ankle_Pitch: type revolute, parent WJ-DP00-0002-FK-AP-020_7_5, child FOOT, origin xyz=0.09999999987006428 3.364079596487879e-09 -0.0001999952684794198 rpy=-3.141592653589792 4.641020900919557e-08 1.5707964071795835, axis 0 0 1, limit lower=-1.5707963 upper=1.5707963 effort=80 velocity=5
- added joint L_Elbow_Pitch: type revolute, parent FK-AP-019-25T_11, child R-ARM-1, origin xyz=0.09298379437380097 -0.01879971801611121 -0.018600374777602353 rpy=-1.570796346410206 -1.5707963071795867 0.0, axis 0 0 1, limit lower=0 upper=0 effort=80 velocity=5
- added joint L_Hand_Pitch: type revolute, parent R-ARM-1, child FINGER_1, origin xyz=-0.011778207168971242 0.06620574802540724 0.037339718524295344 rpy=-3.141592653589792 -4.641020678874952e-08 0.3490658, axis 0 0 1, limit lower=0 upper=0 effort=80 velocity=5
- added joint L_Hip_Pitch: type revolute, parent WJ-DP00-0002-FK-AP-020_7, child WJ-DP00-0002-FK-AP-020_7_3, origin xyz=-0.007399653999999995 -0.032 -0.017899999999999996 rpy=1.5707963 0.0 -1.5707963, axis 0 0 1, limit lower=0 upper=0 effort=80 velocity=5
- added joint L_Hip_Roll: type revolute, parent Z-BOT2_MASTER-BODY-SKELETON, child U-HIP-L, origin xyz=0.04280822375832449 0.007735076030833816 -0.08441842862429541 rpy=3.1415926071795863 -2.220446049250313e-15 3.1415926071795863, axis 0 0 1, limit lower=0 upper=0 effort=80 velocity=5
- added joint L_Hip_Yaw: type revolute, parent U-HIP-L, child WJ-DP00-0002-FK-AP-020_7, origin xyz=0 0.018699662 0.0564 rpy=-1.5707963 0 0, axis 0 0 1, limit lower=0 upper=0 effort=80 velocity=5
- added joint L_Knee_Pitch: type revolute, parent WJ-DP00-0002-FK-AP-020_7_3, child WJ-DP00-0002-FK-AP-020_7_5, origin xyz=0.10000000066047848 0.009999997542907974 -0.0002597236558159702 rpy=4.641020790984154e-08 4.641020678874952e-08 2.6469779601696886e-23, axis 0 0 1, limit lower=-1.0471976 upper=2.7925268 effort=80 velocity=5
- added joint L_Shoulder_Pitch: type revolute, parent Z-BOT2_MASTER-BODY-SKELETON, child Z-BOT2-MASTER-SHOULDER2, origin xyz=0.05599502633660092 -0.009609988350796515 -0.00952781042498181 rpy=1.5707963999999994 0.0 -3.1415926071795863, axis 0 0 1, limit lower=0 upper=0 effort=80 velocity=5
- added joint L_Shoulder_Roll: type revolute, parent Z-BOT2-MASTER-SHOULDER2, child FK-AP-019-25T_11, origin xyz=-0.019845 -0.0049 0.0188 rpy=-1.5707963 0 -1.5707963, axis 0 0 1, limit lower=0 upper=0 effort=80 velocity=5
- added joint R_Ankle_Pitch: type revolute, parent WJ-DP00-0002-FK-AP-020_7_6, child FOOT_2, origin xyz=0.09999999987006428 3.364079596487879e-09 4.731520579850934e-09 rpy=-3.141592560769378 -4.6410206566704915e-08 -1.5707963000000027, axis 0 0 1, limit lower=0 upper=0 effort=80 velocity=5
- added joint R_Elbow_Pitch: type revolute, parent FK-AP-019-25T_11_2, child L-ARM_1, origin xyz=0.09298379516154365 0.018799715578725902 -0.018600375932454845 rpy=1.570796273205104 -1.570796288901191 0.0, axis 0 0 1, limit lower=0 upper=0 effort=80 velocity=5
- added joint R_Hand_Pitch: type revolute, parent L-ARM_1, child FINGER_1_2, origin xyz=-0.011778203442038957 -0.06620574861365118 0.037339718524295344 rpy=-3.141592653589792 4.6410207010794124e-08 -0.3490658, axis 0 0 1, limit lower=0 upper=0 effort=80 velocity=5
- added joint R_Hip_Pitch: type revolute, parent WJ-DP00-0002-FK-AP-020_7_2, child WJ-DP00-0002-FK-AP-020_7_4, origin xyz=0.007399655009421977 -0.03199999927137579 0.0188997194 rpy=-1.5707963 0.0 -1.5707963071795867, axis 0 0 1, limit lower=0 upper=0 effort=80 velocity=5
- added joint R_Hip_Roll: type revolute, parent Z-BOT2_MASTER-BODY-SKELETON, child U-HIP-R, origin xyz=-0.04286813624167551 0.007735076030833816 -0.08441842862429541 rpy=3.1415926071795863 -2.220446049250313e-15 3.1415926071795863, axis 0 0 1, limit lower=0 upper=0 effort=80 velocity=5
- added joint R_Hip_Yaw: type revolute, parent U-HIP-R, child WJ-DP00-0002-FK-AP-020_7_2, origin xyz=0 -0.018699662 0.0564 rpy=-1.5707963 0 0, axis 0 0 -1, limit lower=0 upper=0 effort=80 velocity=5
- added joint R_Knee_Pitch: type revolute, parent WJ-DP00-0002-FK-AP-020_7_4, child WJ-DP00-0002-FK-AP-020_7_6, origin xyz=0.10000000042471463 -0.00999999754290798 -0.00025971514418403357 rpy=4.641020790984154e-08 -4.641020678874952e-08 -2.6469779601696886e-23, axis 0 0 1, limit lower=0 upper=0 effort=80 velocity=5
- added joint R_Shoulder_Pitch: type revolute, parent Z-BOT2_MASTER-BODY-SKELETON, child Z-BOT2-MASTER-SHOULDER2_2, origin xyz=-0.05599497353346345 -0.009609990641140206 -0.009527810424981806 rpy=-1.5707963071795867 0.0 9.282041324443213e-08, axis 0 0 1, limit lower=0 upper=0 effort=80 velocity=5
- added joint R_Shoulder_Roll: type revolute, parent Z-BOT2-MASTER-SHOULDER2_2, child FK-AP-019-25T_11_2, origin xyz=-0.019845 0.0049 0.0188 rpy=1.5707963 0 1.5707963, axis 0 0 1, limit lower=0 upper=0 effort=80 velocity=5
- joint floating_base: origin xyz=0 0 0 rpy=0 0 1.57 -> xyz=0 0 0 rpy=0 0 0

File: sim/resources/zbot2/robot_fixed.urdf (robot description, URDF)
Before this commit: robot assembly_1, 20 links, 19 joints
Links:
- removed link FINGER_1_1
- removed link FK-AP-019-25T_11_16
- removed link FK-AP-019-25T_11_5
- removed link FOOT_1
- removed link SJ-WK00-0021TOPCABINETCASE_104_7
- removed link SJ-WK00-0023BOTTOMCASE_12_12
- removed link SJ-WK00-0023BOTTOMCASE_12_13
- removed link SJ-WK00-0023BOTTOMCASE_12_8
- removed link U-HIP
- removed link U-HIP_1
- removed link WJ-DP00-0002-FK-AP-020_7_10
- removed link WJ-DP00-0002-FK-AP-020_7_8
- removed link Z-BOT2-MASTER-SHOULDER2_1
- added link FINGER_1_2, mass 0.022322296; collision mesh filename=meshes/FINGER_1_2.stl; visual mesh filename=meshes/FINGER_1_2.stl
- added link FK-AP-019-25T_11, mass 0.14822332759999998; collision mesh filename=meshes/FK-AP-019-25T_11.stl; visual mesh filename=meshes/FK-AP-019-25T_11.stl
- added link FK-AP-019-25T_11_2, mass 0.1482233276; collision mesh filename=meshes/FK-AP-019-25T_11_2.stl; visual mesh filename=meshes/FK-AP-019-25T_11_2.stl
- added link FOOT_2, mass 0.09495736199999999; collision mesh filename=meshes/FOOT_2.stl; visual mesh filename=meshes/FOOT_2.stl
- added link U-HIP-L, mass 0.016091061; collision mesh filename=meshes/U-HIP-L.stl; visual mesh filename=meshes/U-HIP-L.stl
- added link U-HIP-R, mass 0.016091061; collision mesh filename=meshes/U-HIP-R.stl; visual mesh filename=meshes/U-HIP-R.stl
- added link WJ-DP00-0002-FK-AP-020_7, mass 0.066367059; collision mesh filename=meshes/WJ-DP00-0002-FK-AP-020_7.stl; visual mesh filename=meshes/WJ-DP00-0002-FK-AP-020_7.stl
- added link WJ-DP00-0002-FK-AP-020_7_2, mass 0.066367059; collision mesh filename=meshes/WJ-DP00-0002-FK-AP-020_7_2.stl; visual mesh filename=meshes/WJ-DP00-0002-FK-AP-020_7_2.stl
- added link WJ-DP00-0002-FK-AP-020_7_3, mass 0.091986251; collision mesh filename=meshes/WJ-DP00-0002-FK-AP-020_7_3.stl; visual mesh filename=meshes/WJ-DP00-0002-FK-AP-020_7_3.stl
- added link WJ-DP00-0002-FK-AP-020_7_4, mass 0.091986251; collision mesh filename=meshes/WJ-DP00-0002-FK-AP-020_7_4.stl; visual mesh filename=meshes/WJ-DP00-0002-FK-AP-020_7_4.stl
- added link WJ-DP00-0002-FK-AP-020_7_5, mass 0.1298739283; collision mesh filename=meshes/WJ-DP00-0002-FK-AP-020_7_5.stl; visual mesh filename=meshes/WJ-DP00-0002-FK-AP-020_7_5.stl
- added link WJ-DP00-0002-FK-AP-020_7_6, mass 0.1298739283; collision mesh filename=meshes/WJ-DP00-0002-FK-AP-020_7_6.stl; visual mesh filename=meshes/WJ-DP00-0002-FK-AP-020_7_6.stl
- added link Z-BOT2-MASTER-SHOULDER2_2, mass 0.0082269514; collision mesh filename=meshes/Z-BOT2-MASTER-SHOULDER2_2.stl; visual mesh filename=meshes/Z-BOT2-MASTER-SHOULDER2_2.stl
- link FINGER_1: mass 0.045310716 -> 0.022322296
- link FOOT: mass 0.096390673 -> 0.09495736199999999
- link L-ARM_1: mass 0.1697714245 -> 0.113768642
- link R-ARM-1: mass 0.1697709975 -> 0.113768495
- link Z-BOT2-MASTER-SHOULDER2: mass 0.0240976 -> 0.0082269514
- link Z-BOT2_MASTER-BODY-SKELETON: mass 1.5916352207 -> 1.00556824628
Joints:
- removed joint left_ankle_pitch
- removed joint left_elbow_yaw
- removed joint left_gripper
- removed joint left_hip_pitch
- removed joint left_hip_roll
- removed joint left_hip_yaw
- removed joint left_knee_pitch
- removed joint left_shoulder_pitch
- removed joint left_shoulder_yaw
- removed joint right_ankle_pitch
- removed joint right_elbow_yaw
- removed joint right_gripper
- removed joint right_hip_pitch
- removed joint right_hip_roll
- removed joint right_hip_yaw
- removed joint right_knee_pitch
- removed joint right_shoulder_pitch
- removed joint right_shoulder_yaw
- added joint L_Ankle_Pitch: type revolute, parent WJ-DP00-0002-FK-AP-020_7_5, child FOOT, origin xyz=0.09999999987006428 3.364079596487879e-09 -0.0001999952684794198 rpy=-3.141592653589792 4.641020900919557e-08 1.5707964071795835, axis 0 0 1, limit lower=-1.5708 upper=1.5708 effort=1.0 velocity=10
- added joint L_Elbow_Pitch: type fixed, parent FK-AP-019-25T_11, child R-ARM-1, origin xyz=0.09298379437380097 -0.01879971801611121 -0.018600374777602353 rpy=-1.570796346410206 -1.5707963071795867 0.0, axis 0 0 1, limit lower=0 upper=0 effort=80 velocity=5
- added joint L_Hand_Pitch: type fixed, parent R-ARM-1, child FINGER_1, origin xyz=-0.011778207168971242 0.06620574802540724 0.037339718524295344 rpy=-3.141592653589792 -4.641020678874952e-08 0.3490658, axis 0 0 1, limit lower=0 upper=0 effort=80 velocity=5
- added joint L_Hip_Pitch: type revolute, parent WJ-DP00-0002-FK-AP-020_7, child WJ-DP00-0002-FK-AP-020_7_3, origin xyz=-0.007399653999999995 -0.032 -0.017899999999999996 rpy=1.5707963 0.0 -1.5707963, axis 0 0 1, limit lower=-1.8326 upper=1.74533 effort=1.0 velocity=10
- added joint L_Hip_Roll: type revolute, parent Z-BOT2_MASTER-BODY-SKELETON, child U-HIP-L, origin xyz=0.04280822375832449 0.007735076030833816 -0.08441842862429541 rpy=3.1415926071795863 -2.220446049250313e-15 3.1415926071795863, axis 0 0 1, limit lower=-1.0472 upper=1.0472 effort=1.0 velocity=10
- added joint L_Hip_Yaw: type revolute, parent U-HIP-L, child WJ-DP00-0002-FK-AP-020_7, origin xyz=0 0.018699662 0.0564 rpy=-1.5707963 0 0, axis 0 0 1, limit lower=-1.91986 upper=0.174533 effort=1.0 velocity=10
- added joint L_Knee_Pitch: type revolute, parent WJ-DP00-0002-FK-AP-020_7_3, child WJ-DP00-0002-FK-AP-020_7_5, origin xyz=0.10000000066047848 0.009999997542907974 -0.0002597236558159702 rpy=4.641020790984154e-08 4.641020678874952e-08 2.6469779601696886e-23, axis 0 0 1, limit lower=-0.174533 upper=2.96706 effort=1.0 velocity=10
- added joint L_Shoulder_Pitch: type fixed, parent Z-BOT2_MASTER-BODY-SKELETON, child Z-BOT2-MASTER-SHOULDER2, origin xyz=0.05599502633660092 -0.009609988350796515 -0.00952781042498181 rpy=1.5707963999999994 0.0 -3.1415926071795863, axis 0 0 1, limit lower=0 upper=0 effort=80 velocity=5
- added joint L_Shoulder_Roll: type fixed, parent Z-BOT2-MASTER-SHOULDER2, child FK-AP-019-25T_11, origin xyz=-0.019845 -0.0049 0.0188 rpy=-1.5707963 0 -1.5707963, axis 0 0 1, limit lower=0 upper=0 effort=80 velocity=5
- added joint R_Ankle_Pitch: type revolute, parent WJ-DP00-0002-FK-AP-020_7_6, child FOOT_2, origin xyz=0.09999999987006428 3.364079596487879e-09 4.731520579850934e-09 rpy=-3.141592560769378 -4.6410206566704915e-08 -1.5707963000000027, axis 0 0 1, limit lower=-1.5708 upper=1.5708 effort=1.0 velocity=10
- added joint R_Elbow_Pitch: type fixed, parent FK-AP-019-25T_11_2, child L-ARM_1, origin xyz=0.09298379516154365 0.018799715578725902 -0.018600375932454845 rpy=1.570796273205104 -1.570796288901191 0.0, axis 0 0 1, limit lower=0 upper=0 effort=80 velocity=5
- added joint R_Hand_Pitch: type fixed, parent L-ARM_1, child FINGER_1_2, origin xyz=-0.011778203442038957 -0.06620574861365118 0.037339718524295344 rpy=-3.141592653589792 4.6410207010794124e-08 -0.3490658, axis 0 0 1, limit lower=0 upper=0 effort=80 velocity=5
- added joint R_Hip_Pitch: type revolute, parent WJ-DP00-0002-FK-AP-020_7_2, child WJ-DP00-0002-FK-AP-020_7_4, origin xyz=0.007399655009421977 -0.03199999927137579 0.0188997194 rpy=-1.5707963 0.0 -1.5707963071795867, axis 0 0 1, limit lower=-1.74533 upper=1.8326 effort=1.0 velocity=10
- added joint R_Hip_Roll: type revolute, parent Z-BOT2_MASTER-BODY-SKELETON, child U-HIP-R, origin xyz=-0.04286813624167551 0.007735076030833816 -0.08441842862429541 rpy=3.1415926071795863 -2.220446049250313e-15 3.1415926071795863, axis 0 0 1, limit lower=-1.0472 upper=1.0472 effort=1.0 velocity=10
- added joint R_Hip_Yaw: type revolute, parent U-HIP-R, child WJ-DP00-0002-FK-AP-020_7_2, origin xyz=0 -0.018699662 0.0564 rpy=-1.5707963 0 0, axis 0 0 -1, limit lower=-0.174533 upper=1.91986 effort=1.0 velocity=10
- added joint R_Knee_Pitch: type revolute, parent WJ-DP00-0002-FK-AP-020_7_4, child WJ-DP00-0002-FK-AP-020_7_6, origin xyz=0.10000000042471463 -0.00999999754290798 -0.00025971514418403357 rpy=4.641020790984154e-08 -4.641020678874952e-08 -2.6469779601696886e-23, axis 0 0 1, limit lower=-0.174533 upper=2.96706 effort=1.0 velocity=10
- added joint R_Shoulder_Pitch: type fixed, parent Z-BOT2_MASTER-BODY-SKELETON, child Z-BOT2-MASTER-SHOULDER2_2, origin xyz=-0.05599497353346345 -0.009609990641140206 -0.009527810424981806 rpy=-1.5707963071795867 0.0 9.282041324443213e-08, axis 0 0 1, limit lower=0 upper=0 effort=80 velocity=5
- added joint R_Shoulder_Roll: type fixed, parent Z-BOT2-MASTER-SHOULDER2_2, child FK-AP-019-25T_11_2, origin xyz=-0.019845 0.0049 0.0188 rpy=1.5707963 0 1.5707963, axis 0 0 1, limit lower=0 upper=0 effort=80 velocity=5
- joint floating_base: origin xyz=0 0 0 rpy=0 0 1.57 -> xyz=0 0 0 rpy=0 0 0

Commit message: update imu placement and xmls

File: sim/resources/zbot2/robot.urdf (robot description, URDF)
Before this commit: robot z-bot2_al_limits, 20 links, 19 joints
Links:
- removed link base
Joints:
- removed joint floating_base

File: sim/resources/zbot2/robot_fixed.urdf (robot description, URDF)
Before this commit: robot z-bot2_al_limits, 20 links, 19 joints
Joints:
- joint floating_base: type fixed -> floating

Commit message: update urdf limits

File: sim/resources/zbot2/robot.urdf (robot description, URDF)
Before this commit: robot z-bot2_al_limits, 19 links, 18 joints
Links:
- added link base, mass 0.001
Joints:
- added joint floating_base: type fixed, parent base, child Z-BOT2_MASTER-BODY-SKELETON, origin xyz=0 0 0 rpy=0 0 1.57
- joint L_Ankle_Pitch: limit lower=-1.5707963 upper=1.5707963 effort=80 velocity=5 -> lower=-0.9 upper=0.9 effort=80 velocity=5
- joint L_Hip_Pitch: limit lower=0 upper=0 effort=80 velocity=5 -> lower=-1.54 upper=1.0 effort=80 velocity=5
- joint L_Hip_Roll: limit lower=0 upper=0 effort=80 velocity=5 -> lower=-0.7 upper=0.7 effort=80 velocity=5
- joint L_Hip_Yaw: limit lower=0 upper=0 effort=80 velocity=5 -> lower=-1.54 upper=0.157 effort=80 velocity=5
- joint L_Knee_Pitch: limit lower=-1.0471976 upper=2.7925268 effort=80 velocity=5 -> lower=0 upper=1.57 effort=80 velocity=5
- joint R_Ankle_Pitch: limit lower=0 upper=0 effort=80 velocity=5 -> lower=-0.9 upper=0.9 effort=80 velocity=5
- joint R_Hip_Pitch: limit lower=0 upper=0 effort=80 velocity=5 -> lower=-1.0 upper=1.54 effort=80 velocity=5
- joint R_Hip_Roll: limit lower=0 upper=0 effort=80 velocity=5 -> lower=-0.7 upper=0.7 effort=80 velocity=5
- joint R_Hip_Yaw: limit lower=0 upper=0 effort=80 velocity=5 -> lower=-1.54 upper=0.157 effort=80 velocity=5
- joint R_Knee_Pitch: limit lower=0 upper=0 effort=80 velocity=5 -> lower=-1.57 upper=0 effort=80 velocity=5

File: sim/resources/zbot2/robot_fixed.urdf (robot description, URDF)
Before this commit: robot z-bot2_al_limits, 20 links, 19 joints
Joints:
- joint L_Ankle_Pitch: limit lower=-0.9 upper=0.9 effort=3.0 velocity=10 -> lower=-0.9 upper=0.9 effort=3.0 velocity=15
- joint L_Hip_Pitch: limit lower=-0.9 upper=0.9 effort=3.0 velocity=10 -> lower=-1.54 upper=1.0 effort=3.0 velocity=15
- joint L_Hip_Roll: limit lower=-0.9 upper=0.9 effort=3.0 velocity=10 -> lower=-0.7 upper=0.7 effort=3.0 velocity=15
- joint L_Hip_Yaw: limit lower=-0.9 upper=0.9 effort=3.0 velocity=10 -> lower=-1.54 upper=0.157 effort=3.0 velocity=15
- joint L_Knee_Pitch: limit lower=-0.9 upper=0.9 effort=3.0 velocity=10 -> lower=0 upper=1.57 effort=3.0 velocity=15
- joint R_Ankle_Pitch: limit lower=-0.9 upper=0.9 effort=3.0 velocity=10 -> lower=-0.9 upper=0.9 effort=3.0 velocity=15
- joint R_Hip_Pitch: limit lower=-0.9 upper=0.9 effort=3.0 velocity=10 -> lower=-1.0 upper=1.54 effort=3.0 velocity=15
- joint R_Hip_Roll: limit lower=-0.9 upper=0.9 effort=3.0 velocity=10 -> lower=-0.7 upper=0.7 effort=3.0 velocity=15
- joint R_Hip_Yaw: limit lower=-0.9 upper=0.9 effort=3.0 velocity=10 -> lower=-1.54 upper=0.157 effort=3.0 velocity=15
- joint R_Knee_Pitch: limit lower=-0.9 upper=0.9 effort=3.0 velocity=10 -> lower=-1.57 upper=0 effort=3.0 velocity=15
