Commit message: good behavior

File: sim/resources/zbot2/robot.urdf (robot description, URDF)
Before this commit: robot z-bot2_al_limits, 20 links, 19 joints
Links:
- removed link FK-AP-019-25T_11
- removed link FK-AP-019-25T_11_2
- removed link L-ARM_1
- removed link R-ARM-1
- removed link WJ-DP00-0002-FK-AP-020_7
- removed link WJ-DP00-0002-FK-AP-020_7_2
- removed link WJ-DP00-0002-FK-AP-020_7_3
- removed link WJ-DP00-0002-FK-AP-020_7_4
- removed link WJ-DP00-0002-FK-AP-020_7_5
- removed link WJ-DP00-0002-FK-AP-020_7_6
- added link 3215_1Flange, mass 0.181960114; collision mesh filename=meshes/3215_1Flange.stl; visual mesh filename=meshes/3215_1Flange.stl
- added link 3215_1Flange_2, mass 0.181960114; collision mesh filename=meshes/3215_1Flange_2.stl; visual mesh filename=meshes/3215_1Flange_2.stl
- added link 3215_BothFlange, mass 0.068295303; collision mesh filename=meshes/3215_BothFlange.stl; visual mesh filename=meshes/3215_BothFlange.stl
- added link 3215_BothFlange_2, mass 0.068295303; collision mesh filename=meshes/3215_BothFlange_2.stl; visual mesh filename=meshes/3215_BothFlange_2.stl
- added link 3215_BothFlange_3, mass 0.14333659199999998; collision mesh filename=meshes/3215_BothFlange_3.stl; visual mesh filename=meshes/3215_BothFlange_3.stl
- added link 3215_BothFlange_4, mass 0.14333659199999998; collision mesh filename=meshes/3215_BothFlange_4.stl; visual mesh filename=meshes/3215_BothFlange_4.stl
- added link 3215_BothFlange_5, mass 0.128212813; collision mesh filename=meshes/3215_BothFlange_5.stl; visual mesh filename=meshes/3215_BothFlange_5.stl
- added link 3215_BothFlange_6, mass 0.128212813; collision mesh filename=meshes/3215_BothFlange_6.stl; visual mesh filename=meshes/3215_BothFlange_6.stl
- added link L-ARM-MIRROR_1, mass 0.186073123; collision mesh filename=meshes/L-ARM-MIRROR_1.stl; visual mesh filename=meshes/L-ARM-MIRROR_1.stl
- added link R-ARM-MIRROR-1, mass 0.186072694; collision mesh filename=meshes/R-ARM-MIRROR-1.stl; visual mesh filename=meshes/R-ARM-MIRROR-1.stl
- link FINGER_1: mass 0.022322296 -> 0.044317970000000005
- link FINGER_1_2: mass 0.022322296 -> 0.044317970000000005
- link FOOT: mass 0.09495736199999999 -> 0.27814003
- link FOOT_2: mass 0.09495736199999999 -> 0.27814003
- link U-HIP-L: mass 0.016091061 -> 0.047132399
- link U-HIP-R: mass 0.016091061 -> 0.047132399
- link Z-BOT2-MASTER-SHOULDER2: mass 0.0082269514 -> 0.0240976
- link Z-BOT2-MASTER-SHOULDER2_2: mass 0.0082269514 -> 0.0240976
- link Z-BOT2_MASTER-BODY-SKELETON: mass 1.00556824628 -> 1.5482792056799994
Joints:
- removed joint L_Elbow_Pitch
- removed joint L_Hand_Pitch
- removed joint L_Shoulder_Roll
- removed joint R_Elbow_Pitch
- removed joint R_Hand_Pitch
- removed joint R_Shoulder_Roll
- added joint L_Elbow_Yaw: type revolute, parent 3215_1Flange, child R-ARM-MIRROR-1, origin xyz=0.09298379430410703 0.018799717128502175 -0.018600374924981792 rpy=1.5707963000000005 2.220446049250313e-16 3.1415926, axis 0 0 -1, limit lower=0 upper=0 effort=80 velocity=5
- added joint L_Gripper: type revolute, parent R-ARM-MIRROR-1, child FINGER_1, origin xyz=-0.06620574753840905 -0.011778206850776778 0.00025971726760990604 rpy=3.141592609978465 1.5873225178708594e-08 1.9198622000000003, axis 0 0 1, limit lower=0 upper=0 effort=80 velocity=5
- added joint L_Shoulder_Yaw: type revolute, parent Z-BOT2_MASTER-BODY-SKELETON, child Z-BOT2-MASTER-SHOULDER2, origin xyz=0.05599502633660092 -0.009609988350796515 -0.00952781042498181 rpy=1.5707963999999994 0.0 -3.1415926071795863, axis 0 0 1, limit lower=0 upper=0 effort=80 velocity=5
- added joint R_Elbow_Yaw: type revolute, parent 3215_1Flange_2, child L-ARM-MIRROR_1, origin xyz=0.09298379437380097 -0.018799718976802476 -0.018600374222947996 rpy=-1.570796346410206 -1.5707963071795867 0.0, axis 0 0 1, limit lower=0 upper=0 effort=80 velocity=5
- added joint R_Gripper: type revolute, parent L-ARM-MIRROR_1, child FINGER_1_2, origin xyz=-0.011778204959700955 0.06620574806126743 -0.00025971899999999853 rpy=0.0 0.0 0.3490658, axis 0 0 1, limit lower=0 upper=0 effort=80 velocity=5
- added joint R_Shoulder_Yaw: type revolute, parent Z-BOT2_MASTER-BODY-SKELETON, child Z-BOT2-MASTER-SHOULDER2_2, origin xyz=-0.05599497353346345 -0.009609990641140206 -0.009527810424981806 rpy=-1.5707963071795867 0.0 9.282041324443213e-08, axis 0 0 1, limit lower=0 upper=0 effort=80 velocity=5
- joint L_Ankle_Pitch: limit lower=-0.9 upper=0.9 effort=80 velocity=5 -> lower=0 upper=0 effort=80 velocity=5; parent WJ-DP00-0002-FK-AP-020_7_5 -> 3215_BothFlange_5
- joint L_Hip_Pitch: child WJ-DP00-0002-FK-AP-020_7_3 -> 3215_BothFlange_3; limit lower=-1.54 upper=1.0 effort=80 velocity=5 -> lower=0 upper=0 effort=80 velocity=5; parent WJ-DP00-0002-FK-AP-020_7 -> 3215_BothFlange
- joint L_Hip_Roll: limit lower=-0.7 upper=0.7 effort=80 velocity=5 -> lower=0 upper=0 effort=80 velocity=5
- joint L_Hip_Yaw: child WJ-DP00-0002-FK-AP-020_7 -> 3215_BothFlange; limit lower=-1.54 upper=0.157 effort=80 velocity=5 -> lower=0 upper=0 effort=80 velocity=5
- joint L_Knee_Pitch: child WJ-DP00-0002-FK-AP-020_7_5 -> 3215_BothFlange_5; limit lower=0 upper=1.57 effort=80 velocity=5 -> lower=0 upper=0 effort=80 velocity=5; parent WJ-DP00-0002-FK-AP-020_7_3 -> 3215_BothFlange_3
- joint L_Shoulder_Pitch: child Z-BOT2-MASTER-SHOULDER2 -> 3215_1Flange; origin xyz=0.05599502633660092 -0.009609988350796515 -0.00952781042498181 rpy=1.5707963999999994 0.0 -3.1415926071795863 -> xyz=-0.019845 -0.0049 0.0188 rpy=-1.5707963 0 -1.5707963; parent Z-BOT2_MASTER-BODY-SKELETON -> Z-BOT2-MASTER-SHOULDER2
- joint R_Ankle_Pitch: limit lower=-0.9 upper=0.9 effort=80 velocity=5 -> lower=0 upper=0 effort=80 velocity=5; parent WJ-DP00-0002-FK-AP-020_7_6 -> 3215_BothFlange_6
- joint R_Hip_Pitch: child WJ-DP00-0002-FK-AP-020_7_4 -> 3215_BothFlange_4; limit lower=-1.0 upper=1.54 effort=80 velocity=5 -> lower=0 upper=0 effort=80 velocity=5; parent WJ-DP00-0002-FK-AP-020_7_2 -> 3215_BothFlange_2
- joint R_Hip_Roll: limit lower=-0.7 upper=0.7 effort=80 velocity=5 -> lower=0 upper=0 effort=80 velocity=5
- joint R_Hip_Yaw: child WJ-DP00-0002-FK-AP-020_7_2 -> 3215_BothFlange_2; limit lower=-1.54 upper=0.157 effort=80 velocity=5 -> lower=0 upper=0 effort=80 velocity=5
- joint R_Knee_Pitch: child WJ-DP00-0002-FK-AP-020_7_6 -> 3215_BothFlange_6; limit lower=-1.57 upper=0 effort=80 velocity=5 -> lower=0 upper=0 effort=80 velocity=5; parent WJ-DP00-0002-FK-AP-020_7_4 -> 3215_BothFlange_4
- joint R_Shoulder_Pitch: child Z-BOT2-MASTER-SHOULDER2_2 -> 3215_1Flange_2; origin xyz=-0.05599497353346345 -0.009609990641140206 -0.009527810424981806 rpy=-1.5707963071795867 0.0 9.282041324443213e-08 -> xyz=-0.019845 0.0049 0.0188 rpy=1.5707963 0 1.5707963; parent Z-BOT2_MASTER-BODY-SKELETON -> Z-BOT2-MASTER-SHOULDER2_2
- joint floating_base: origin xyz=0 0 0 rpy=0 0 1.57 -> xyz=0 0 0 rpy=0 0 0

File: sim/resources/zbot2/robot_fixed.urdf (robot description, URDF)
Before this commit: robot z-bot2_al_limits, 20 links, 19 joints
Links:
- removed link FK-AP-019-25T_11
- removed link FK-AP-019-25T_11_2
- removed link L-ARM_1
- removed link R-ARM-1
- removed link WJ-DP00-0002-FK-AP-020_7
- removed link WJ-DP00-0002-FK-AP-020_7_2
- removed link WJ-DP00-0002-FK-AP-020_7_3
- removed link WJ-DP00-0002-FK-AP-020_7_4
- removed link WJ-DP00-0002-FK-AP-020_7_5
- removed link WJ-DP00-0002-FK-AP-020_7_6
- added link 3215_1Flange, mass 0.181960114; collision mesh filename=meshes/3215_1Flange.stl; visual mesh filename=meshes/3215_1Flange.stl
- added link 3215_1Flange_2, mass 0.181960114; collision mesh filename=meshes/3215_1Flange_2.stl; visual mesh filename=meshes/3215_1Flange_2.stl
- added link 3215_BothFlange, mass 0.068295303; collision mesh filename=meshes/3215_BothFlange.stl; visual mesh filename=meshes/3215_BothFlange.stl
- added link 3215_BothFlange_2, mass 0.068295303; collision mesh filename=meshes/3215_BothFlange_2.stl; visual mesh filename=meshes/3215_BothFlange_2.stl
- added link 3215_BothFlange_3, mass 0.14333659199999998; collision mesh filename=meshes/3215_BothFlange_3.stl; visual mesh filename=meshes/3215_BothFlange_3.stl
- added link 3215_BothFlange_4, mass 0.14333659199999998; collision mesh filename=meshes/3215_BothFlange_4.stl; visual mesh filename=meshes/3215_BothFlange_4.stl
- added link 3215_BothFlange_5, mass 0.128212813; collision mesh filename=meshes/3215_BothFlange_5.stl; visual mesh filename=meshes/3215_BothFlange_5.stl
- added link 3215_BothFlange_6, mass 0.128212813; collision mesh filename=meshes/3215_BothFlange_6.stl; visual mesh filename=meshes/3215_BothFlange_6.stl
- added link L-ARM-MIRROR_1, mass 0.186073123; collision mesh filename=meshes/L-ARM-MIRROR_1.stl; visual mesh filename=meshes/L-ARM-MIRROR_1.stl
- added link R-ARM-MIRROR-1, mass 0.186072694; collision mesh filename=meshes/R-ARM-MIRROR-1.stl; visual mesh filename=meshes/R-ARM-MIRROR-1.stl
- link FINGER_1: mass 0.022322296 -> 0.044317970000000005
- link FINGER_1_2: mass 0.022322296 -> 0.044317970000000005
- link FOOT: mass 0.09495736199999999 -> 0.27814003
- link FOOT_2: mass 0.09495736199999999 -> 0.27814003
- link U-HIP-L: mass 0.016091061 -> 0.047132399
- link U-HIP-R: mass 0.016091061 -> 0.047132399
- link Z-BOT2-MASTER-SHOULDER2: mass 0.0082269514 -> 0.0240976
- link Z-BOT2-MASTER-SHOULDER2_2: mass 0.0082269514 -> 0.0240976
- link Z-BOT2_MASTER-BODY-SKELETON: mass 1.00556824628 -> 1.5482792056799994
Joints:
- removed joint L_Elbow_Pitch
- removed joint L_Hand_Pitch
- removed joint L_Shoulder_Roll
- removed joint R_Elbow_Pitch
- removed joint R_Hand_Pitch
- removed joint R_Shoulder_Roll
- added joint L_Elbow_Yaw: type fixed, parent 3215_1Flange, child R-ARM-MIRROR-1, origin xyz=0.09298379430410703 0.018799717128502175 -0.018600374924981792 rpy=1.5707963000000005 2.220446049250313e-16 3.1415926, axis 0 0 -1, limit lower=0 upper=0 effort=80 velocity=5
- added joint L_Gripper: type fixed, parent R-ARM-MIRROR-1, child FINGER_1, origin xyz=-0.06620574753840905 -0.011778206850776778 0.00025971726760990604 rpy=3.141592609978465 1.5873225178708594e-08 1.9198622000000003, axis 0 0 1, limit lower=0 upper=0 effort=80 velocity=5
- added joint L_Shoulder_Yaw: type fixed, parent Z-BOT2_MASTER-BODY-SKELETON, child Z-BOT2-MASTER-SHOULDER2, origin xyz=0.05599502633660092 -0.009609988350796515 -0.00952781042498181 rpy=1.5707963999999994 0.0 -3.1415926071795863, axis 0 0 1, limit lower=0 upper=0 effort=80 velocity=5
- added joint R_Elbow_Yaw: type fixed, parent 3215_1Flange_2, child L-ARM-MIRROR_1, origin xyz=0.09298379437380097 -0.018799718976802476 -0.018600374222947996 rpy=-1.570796346410206 -1.5707963071795867 0.0, axis 0 0 1, limit lower=0 upper=0 effort=80 velocity=5
- added joint R_Gripper: type fixed, parent L-ARM-MIRROR_1, child FINGER_1_2, origin xyz=-0.011778204959700955 0.06620574806126743 -0.00025971899999999853 rpy=0.0 0.0 0.3490658, axis 0 0 1, limit lower=0 upper=0 effort=80 velocity=5
- added joint R_Shoulder_Yaw: type fixed, parent Z-BOT2_MASTER-BODY-SKELETON, child Z-BOT2-MASTER-SHOULDER2_2, origin xyz=-0.05599497353346345 -0.009609990641140206 -0.009527810424981806 rpy=-1.5707963071795867 0.0 9.282041324443213e-08, axis 0 0 1, limit lower=0 upper=0 effort=80 velocity=5
- joint L_Ankle_Pitch: limit lower=-0.9 upper=0.9 effort=3.0 velocity=15 -> lower=-0.9 upper=0.9 effort=1.91 velocity=15; parent WJ-DP00-0002-FK-AP-020_7_5 -> 3215_BothFlange_5
- joint L_Hip_Pitch: child WJ-DP00-0002-FK-AP-020_7_3 -> 3215_BothFlange_3; limit lower=-1.54 upper=1.0 effort=3.0 velocity=15 -> lower=-1.54 upper=1.0 effort=1.91 velocity=15; parent WJ-DP00-0002-FK-AP-020_7 -> 3215_BothFlange
- joint L_Hip_Roll: limit lower=-0.7 upper=0.7 effort=3.0 velocity=15 -> lower=-0.7 upper=0.7 effort=1.91 velocity=15
- joint L_Hip_Yaw: child WJ-DP00-0002-FK-AP-020_7 -> 3215_BothFlange; limit lower=-1.54 upper=0.157 effort=3.0 velocity=15 -> lower=-1.54 upper=0.157 effort=1.91 velocity=15
- joint L_Knee_Pitch: child WJ-DP00-0002-FK-AP-020_7_5 -> 3215_BothFlange_5; limit lower=0 upper=1.57 effort=3.0 velocity=15 -> lower=0 upper=1.57 effort=1.91 velocity=15; parent WJ-DP00-0002-FK-AP-020_7_3 -> 3215_BothFlange_3
- joint L_Shoulder_Pitch: child Z-BOT2-MASTER-SHOULDER2 -> 3215_1Flange; origin xyz=0.05599502633660092 -0.009609988350796515 -0.00952781042498181 rpy=1.5707963999999994 0.0 -3.1415926071795863 -> xyz=-0.019845 -0.0049 0.0188 rpy=-1.5707963 0 -1.5707963; parent Z-BOT2_MASTER-BODY-SKELETON -> Z-BOT2-MASTER-SHOULDER2
- joint R_Ankle_Pitch: limit lower=-0.9 upper=0.9 effort=3.0 velocity=15 -> lower=-0.9 upper=0.9 effort=1.91 velocity=15; parent WJ-DP00-0002-FK-AP-020_7_6 -> 3215_BothFlange_6
- joint R_Hip_Pitch: child WJ-DP00-0002-FK-AP-020_7_4 -> 3215_BothFlange_4; limit lower=-1.0 upper=1.54 effort=3.0 velocity=15 -> lower=-1.0 upper=1.54 effort=1.91 velocity=15; parent WJ-DP00-0002-FK-AP-020_7_2 -> 3215_BothFlange_2
- joint R_Hip_Roll: limit lower=-0.7 upper=0.7 effort=3.0 velocity=15 -> lower=-0.7 upper=0.7 effort=1.91 velocity=15
- joint R_Hip_Yaw: child WJ-DP00-0002-FK-AP-020_7_2 -> 3215_BothFlange_2; limit lower=-1.54 upper=0.157 effort=3.0 velocity=15 -> lower=-1.54 upper=0.157 effort=1.91 velocity=15
- joint R_Knee_Pitch: child WJ-DP00-0002-FK-AP-020_7_6 -> 3215_BothFlange_6; limit lower=-1.57 upper=0 effort=3.0 velocity=15 -> lower=-1.57 upper=0 effort=1.91 velocity=15; parent WJ-DP00-0002-FK-AP-020_7_4 -> 3215_BothFlange_4
- joint R_Shoulder_Pitch: child Z-BOT2-MASTER-SHOULDER2_2 -> 3215_1Flange_2; origin xyz=-0.05599497353346345 -0.009609990641140206 -0.009527810424981806 rpy=-1.5707963071795867 0.0 9.282041324443213e-08 -> xyz=-0.019845 0.0049 0.0188 rpy=1.5707963 0 1.5707963; parent Z-BOT2_MASTER-BODY-SKELETON -> Z-BOT2-MASTER-SHOULDER2_2
