Commit message: updated fixed urdf

File: sim/resources/zbot2/robot_fixed.urdf (robot description, URDF)
Before this commit: robot assembly_1, 20 links, 19 joints
Joints:
- joint left_ankle_pitch: limit lower=-1.5708 upper=1.5708 effort=80.0 velocity=10.0 -> lower=-1.5708 upper=1.5708 effort=10 velocity=10
- joint left_elbow_yaw: limit lower=-2.0944 upper=1.5708 effort=80.0 velocity=10.0 -> lower=-2.0943951 upper=1.5707963 effort=80 velocity=5; type revolute -> fixed
- joint left_gripper: limit lower=-0.872665 upper=0.349066 effort=80.0 velocity=10.0 -> lower=-0.87266463 upper=0.34906585 effort=80 velocity=5; type revolute -> fixed
- joint left_hip_pitch: limit lower=-1.8326 upper=1.74533 effort=80.0 velocity=10.0 -> lower=-1.8326 upper=1.74533 effort=10 velocity=10
- joint left_hip_roll: limit lower=-1.0472 upper=1.0472 effort=80.0 velocity=10.0 -> lower=-1.0472 upper=1.0472 effort=10 velocity=10
- joint left_hip_yaw: limit lower=-1.91986 upper=0.174533 effort=80.0 velocity=10.0 -> lower=-1.91986 upper=0.174533 effort=10 velocity=10
- joint left_knee_pitch: limit lower=-0.174533 upper=2.96706 effort=80.0 velocity=10.0 -> lower=-0.174533 upper=2.96706 effort=10 velocity=10
- joint left_shoulder_pitch: limit lower=-3.14159 upper=3.14159 effort=80.0 velocity=10.0 -> lower=-3.1415927 upper=3.1415927 effort=80 velocity=5; type revolute -> fixed
- joint left_shoulder_yaw: limit lower=-0.349066 upper=1.22173 effort=80.0 velocity=10.0 -> lower=-0.34906585 upper=1.2217305 effort=80 velocity=5; type revolute -> fixed
- joint right_ankle_pitch: limit lower=-1.5708 upper=1.5708 effort=80.0 velocity=10.0 -> lower=-1.5708 upper=1.5708 effort=10 velocity=10
- joint right_elbow_yaw: limit lower=-1.5708 upper=2.0944 effort=80.0 velocity=10.0 -> lower=-1.5707963 upper=2.0943951 effort=80 velocity=5; type revolute -> fixed
- joint right_gripper: limit lower=-0.349066 upper=0.872665 effort=80.0 velocity=10.0 -> lower=-0.34906585 upper=0.87266463 effort=80 velocity=5; type revolute -> fixed
- joint right_hip_pitch: limit lower=-1.74533 upper=1.8326 effort=80.0 velocity=10.0 -> lower=-1.74533 upper=1.8326 effort=10 velocity=10
- joint right_hip_roll: limit lower=-1.0472 upper=1.0472 effort=80.0 velocity=10.0 -> lower=-1.0472 upper=1.0472 effort=10 velocity=10
- joint right_hip_yaw: limit lower=-0.174533 upper=1.91986 effort=80.0 velocity=10.0 -> lower=-0.174533 upper=1.91986 effort=10 velocity=10
- joint right_knee_pitch: limit lower=-0.174533 upper=2.96706 effort=80.0 velocity=10.0 -> lower=-0.174533 upper=2.96706 effort=10 velocity=10
- joint right_shoulder_pitch: limit lower=-3.14159 upper=3.14159 effort=80.0 velocity=10.0 -> lower=-3.1415927 upper=3.1415927 effort=80 velocity=5; type revolute -> fixed
- joint right_shoulder_yaw: limit lower=-1.22173 upper=0.349066 effort=80.0 velocity=10.0 -> lower=-1.2217305 upper=0.34906585 effort=80 velocity=5; type revolute -> fixed

Commit message: updated urdf

File: sim/resources/zbot2/robot_fixed.urdf (robot description, URDF)
Before this commit: robot assembly_1, 20 links, 19 joints
Joints:
- joint left_ankle_pitch: limit lower=-1.5708 upper=1.5708 effort=10 velocity=10 -> lower=-1.5708 upper=1.5708 effort=1 velocity=20
- joint left_hip_pitch: limit lower=-1.8326 upper=1.74533 effort=10 velocity=10 -> lower=-1.8326 upper=1.74533 effort=1 velocity=20
- joint left_hip_roll: limit lower=-1.0472 upper=1.0472 effort=10 velocity=10 -> lower=-1.0472 upper=1.0472 effort=1 velocity=20
- joint left_hip_yaw: limit lower=-1.91986 upper=0.174533 effort=10 velocity=10 -> lower=-1.91986 upper=0.174533 effort=1 velocity=20
- joint left_knee_pitch: limit lower=-0.174533 upper=2.96706 effort=10 velocity=10 -> lower=-0.174533 upper=2.96706 effort=1 velocity=20
- joint right_ankle_pitch: limit lower=-1.5708 upper=1.5708 effort=10 velocity=10 -> lower=-1.5708 upper=1.5708 effort=1 velocity=20
- joint right_hip_pitch: limit lower=-1.74533 upper=1.8326 effort=10 velocity=10 -> lower=-1.74533 upper=1.8326 effort=1 velocity=20
- joint right_hip_roll: limit lower=-1.0472 upper=1.0472 effort=10 velocity=10 -> lower=-1.0472 upper=1.0472 effort=1 velocity=20
- joint right_hip_yaw: limit lower=-0.174533 upper=1.91986 effort=10 velocity=10 -> lower=-0.174533 upper=1.91986 effort=1 velocity=20
- joint right_knee_pitch: limit lower=-0.174533 upper=2.96706 effort=10 velocity=10 -> lower=-0.174533 upper=2.96706 effort=1 velocity=20

Commit message: larger kps

File: sim/resources/zbot2/robot_fixed.urdf (robot description, URDF)
Before this commit: robot assembly_1, 20 links, 19 joints
Joints:
- joint left_ankle_pitch: limit lower=-1.5708 upper=1.5708 effort=1 velocity=20 -> lower=-1.5708 upper=1.5708 effort=1.0 velocity=10
- joint left_hip_pitch: limit lower=-1.8326 upper=1.74533 effort=1 velocity=20 -> lower=-1.8326 upper=1.74533 effort=1.0 velocity=10
- joint left_hip_roll: limit lower=-1.0472 upper=1.0472 effort=1 velocity=20 -> lower=-1.0472 upper=1.0472 effort=1.0 velocity=10
- joint left_hip_yaw: limit lower=-1.91986 upper=0.174533 effort=1 velocity=20 -> lower=-1.91986 upper=0.174533 effort=1.0 velocity=10
- joint left_knee_pitch: limit lower=-0.174533 upper=2.96706 effort=1 velocity=20 -> lower=-0.174533 upper=2.96706 effort=1.0 velocity=10
- joint right_ankle_pitch: limit lower=-1.5708 upper=1.5708 effort=1 velocity=20 -> lower=-1.5708 upper=1.5708 effort=1.0 velocity=10
- joint right_hip_pitch: limit lower=-1.74533 upper=1.8326 effort=1 velocity=20 -> lower=-1.74533 upper=1.8326 effort=1.0 velocity=10
- joint right_hip_roll: limit lower=-1.0472 upper=1.0472 effort=1 velocity=20 -> lower=-1.0472 upper=1.0472 effort=1.0 velocity=10
- joint right_hip_yaw: limit lower=-0.174533 upper=1.91986 effort=1 velocity=20 -> lower=-0.174533 upper=1.91986 effort=1.0 velocity=10
- joint right_knee_pitch: limit lower=-0.174533 upper=2.96706 effort=1 velocity=20 -> lower=-0.174533 upper=2.96706 effort=1.0 velocity=10

Commit message: add projected gravity

File: sim/resources/zbot2/robot_fixed.urdf (robot description, URDF)
Before this commit: robot z-bot2_al_limits, 20 links, 19 joints
Joints:
- joint L_Ankle_Pitch: limit lower=-1.5708 upper=1.5708 effort=1.0 velocity=10 -> lower=-0.9 upper=0.9 effort=1.0 velocity=10
- joint L_Hip_Pitch: limit lower=-1.8326 upper=1.74533 effort=1.0 velocity=10 -> lower=-0.9 upper=0.9 effort=1.0 velocity=10
- joint L_Hip_Roll: limit lower=-1.0472 upper=1.0472 effort=1.0 velocity=10 -> lower=-0.9 upper=0.9 effort=1.0 velocity=10
- joint L_Hip_Yaw: limit lower=-1.91986 upper=0.174533 effort=1.0 velocity=10 -> lower=-0.9 upper=0.9 effort=1.0 velocity=10
- joint L_Knee_Pitch: limit lower=-0.174533 upper=2.96706 effort=1.0 velocity=10 -> lower=-0.9 upper=0.9 effort=1.0 velocity=10
- joint R_Ankle_Pitch: limit lower=-1.5708 upper=1.5708 effort=1.0 velocity=10 -> lower=-0.9 upper=0.9 effort=1.0 velocity=10
- joint R_Hip_Pitch: limit lower=-1.74533 upper=1.8326 effort=1.0 velocity=10 -> lower=-0.9 upper=0.9 effort=1.0 velocity=10
- joint R_Hip_Roll: limit lower=-1.0472 upper=1.0472 effort=1.0 velocity=10 -> lower=-0.9 upper=0.9 effort=1.0 velocity=10
- joint R_Hip_Yaw: limit lower=-0.174533 upper=1.91986 effort=1.0 velocity=10 -> lower=-0.9 upper=0.9 effort=1.0 velocity=10
- joint R_Knee_Pitch: limit lower=-0.174533 upper=2.96706 effort=1.0 velocity=10 -> lower=-0.9 upper=0.9 effort=1.0 velocity=10

Commit message: save well behaved policy

File: sim/resources/zbot2/robot_fixed.urdf (robot description, URDF)
Before this commit: robot z-bot2_al_limits, 20 links, 19 joints
Joints:
- joint L_Ankle_Pitch: limit lower=-0.9 upper=0.9 effort=1.0 velocity=10 -> lower=-0.9 upper=0.9 effort=3.0 velocity=10
- joint L_Hip_Pitch: limit lower=-0.9 upper=0.9 effort=1.0 velocity=10 -> lower=-0.9 upper=0.9 effort=3.0 velocity=10
- joint L_Hip_Roll: limit lower=-0.9 upper=0.9 effort=1.0 velocity=10 -> lower=-0.9 upper=0.9 effort=3.0 velocity=10
- joint L_Hip_Yaw: limit lower=-0.9 upper=0.9 effort=1.0 velocity=10 -> lower=-0.9 upper=0.9 effort=3.0 velocity=10
- joint L_Knee_Pitch: limit lower=-0.9 upper=0.9 effort=1.0 velocity=10 -> lower=-0.9 upper=0.9 effort=3.0 velocity=10
- joint R_Ankle_Pitch: limit lower=-0.9 upper=0.9 effort=1.0 velocity=10 -> lower=-0.9 upper=0.9 effort=3.0 velocity=10
- joint R_Hip_Pitch: limit lower=-0.9 upper=0.9 effort=1.0 velocity=10 -> lower=-0.9 upper=0.9 effort=3.0 velocity=10
- joint R_Hip_Roll: limit lower=-0.9 upper=0.9 effort=1.0 velocity=10 -> lower=-0.9 upper=0.9 effort=3.0 velocity=10
- joint R_Hip_Yaw: limit lower=-0.9 upper=0.9 effort=1.0 velocity=10 -> lower=-0.9 upper=0.9 effort=3.0 velocity=10
- joint R_Knee_Pitch: limit lower=-0.9 upper=0.9 effort=1.0 velocity=10 -> lower=-0.9 upper=0.9 effort=3.0 velocity=10

Commit message: 50hz policy stable on flat

File: sim/resources/zbot2/robot_fixed.urdf (robot description, URDF)
Before this commit: robot z-bot2_fe_urdf, 20 links, 19 joints
Joints:
- joint L_Ankle_Pitch: limit lower=-0.9 upper=0.9 effort=1.91 velocity=15 -> lower=-0.9 upper=0.9 effort=1.91 velocity=2
- joint L_Hip_Pitch: limit lower=-1.54 upper=1.0 effort=1.91 velocity=15 -> lower=-1.54 upper=1.0 effort=1.91 velocity=2
- joint L_Hip_Roll: limit lower=-0.7 upper=0.7 effort=1.91 velocity=15 -> lower=-0.7 upper=0.7 effort=1.91 velocity=2
- joint L_Hip_Yaw: limit lower=-1.54 upper=0.157 effort=1.91 velocity=15 -> lower=-1.54 upper=0.157 effort=1.91 velocity=2
- joint L_Knee_Pitch: limit lower=0 upper=1.57 effort=1.91 velocity=15 -> lower=0 upper=1.57 effort=1.91 velocity=2
- joint R_Ankle_Pitch: limit lower=-0.9 upper=0.9 effort=1.91 velocity=15 -> lower=-0.9 upper=0.9 effort=1.91 velocity=2
- joint R_Hip_Pitch: limit lower=-1.0 upper=1.54 effort=1.91 velocity=15 -> lower=-1.0 upper=1.54 effort=1.91 velocity=2
- joint R_Hip_Roll: limit lower=-0.7 upper=0.7 effort=1.91 velocity=15 -> lower=-0.7 upper=0.7 effort=1.91 velocity=2
- joint R_Hip_Yaw: limit lower=-1.54 upper=0.157 effort=1.91 velocity=15 -> lower=-1.54 upper=0.157 effort=1.91 velocity=2
- joint R_Knee_Pitch: limit lower=-1.57 upper=0 effort=1.91 velocity=15 -> lower=-1.57 upper=0 effort=1.91 velocity=2
- joint floating_base: origin xyz=0 0 0 rpy=0 0 1.57 -> xyz=0 0 0 rpy=0 0 1.5707963

Commit message: update pos

File: sim/resources/zbot2/robot_fixed.urdf (robot description, URDF)
Before this commit: robot z-bot2_fe_urdf, 20 links, 19 joints
Joints:
- joint L_Hip_Roll: limit lower=-0.7 upper=0.7 effort=1.91 velocity=2 -> lower=-0.0 upper=0.0 effort=1.91 velocity=2
- joint L_Hip_Yaw: limit lower=-1.54 upper=0.157 effort=1.91 velocity=2 -> lower=0.0 upper=0.0 effort=1.91 velocity=2
- joint R_Hip_Roll: limit lower=-0.7 upper=0.7 effort=1.91 velocity=2 -> lower=-0.0 upper=0.0 effort=1.91 velocity=2
- joint R_Hip_Yaw: limit lower=-1.54 upper=0.157 effort=1.91 velocity=2 -> lower=0 upper=0 effort=1.91 velocity=2

Commit message: remove pos, ease up terrain

File: sim/resources/zbot2/robot_fixed.urdf (robot description, URDF)
Before this commit: robot z-bot2_fe_urdf, 20 links, 19 joints
Joints:
- joint L_Hip_Roll: limit lower=-0.0 upper=0.0 effort=1.91 velocity=2 -> lower=-0.7 upper=0.7 effort=1.91 velocity=2
- joint L_Hip_Yaw: limit lower=0.0 upper=0.0 effort=1.91 velocity=2 -> lower=-1.54 upper=0.157 effort=1.91 velocity=2
- joint R_Hip_Roll: limit lower=-0.0 upper=0.0 effort=1.91 velocity=2 -> lower=-0.7 upper=0.7 effort=1.91 velocity=2
- joint R_Hip_Yaw: limit lower=0 upper=0 effort=1.91 velocity=2 -> lower=-1.54 upper=0.157 effort=1.91 velocity=2
