Commit message: fix, name joints, height

File: sim/resources/kbot2/robot_fixed.urdf (robot description, URDF)
Before this commit: robot k-bot-v2, 22 links, 21 joints
Joints:
- joint left_elbow_02: type revolute -> fixed
- joint left_shoulder_pitch_03: type revolute -> fixed
- joint left_shoulder_roll_03: type revolute -> fixed
- joint left_shoulder_yaw_02: type revolute -> fixed
- joint left_wrist_02: type revolute -> fixed
- joint right_elbow_02: type revolute -> fixed
- joint right_shoulder_pitch_03: type revolute -> fixed
- joint right_shoulder_roll_03: type revolute -> fixed
- joint right_shoulder_yaw_02: type revolute -> fixed
- joint right_wrist_02: type revolute -> fixed

Commit message: new

File: sim/resources/kbot2/robot_fixed.urdf (robot description, URDF)
Before this commit: robot k-bot-v2, 22 links, 21 joints
Links:
- link L_Hip_Yaw_RS03: mass 2.67808146 -> 2.67808111
Joints:
- joint floating_base: origin xyz=0.0 0.0009999996829318347 -7.963267107333194e-07 rpy=0.00 0.00 0.00 -> xyz=0 0 0 rpy=0.00 0.00 0.00
- joint left_ankle_02: origin xyz=-0.026 -0.2925 0.003 rpy=0 0 0 -> xyz=-0.026 -0.2925 0.004 rpy=0 0 0
- joint left_elbow_02: axis 0 0 1 -> (none); limit lower=-2.5307274 upper=0 effort=17 velocity=12.566 -> (none); origin xyz=-0.019000000085993334 -0.00999752800444823 -0.13702813751982898 rpy=1.570796400123929 -0.09599312679489658 1.570796324214841 -> xyz=-0.018000000085993336 -0.009997528000000009 -0.13702813759282043 rpy=1.570796400123929 -0.09599312679489658 1.570796324214841
- joint left_hip_pitch_04: origin xyz=-0.056495156388220724 1.548108519327779e-05 -0.07179286928519331 rpy=-1.5707963 4.6410206566704915e-08 -1.5707963535897922 -> xyz=-0.05549515638822072 1.5481058398381098e-05 -0.07179286925839841 rpy=-1.5707963 4.6410206566704915e-08 -1.5707963535897922
- joint left_hip_roll_03: origin xyz=-0.02425 0.03 -0.0660000000267949 rpy=0 -1.5707963 0 -> xyz=-0.02525 0.03 -0.066 rpy=0 -1.5707963 0
- joint left_hip_yaw_03: origin xyz=8.737654313262573e-09 0.1430000033427469 -0.025250003435317102 rpy=-1.5707962071795865 0.0 3.1415926071795863 -> xyz=8.691244106351359e-09 0.1420000033427469 -0.02525000331570179 rpy=-1.5707962071795865 0.0 3.1415926071795863
- joint left_knee_04: origin xyz=-0.02099999837519743 0.020999999640192304 -0.21200000204019234 rpy=1.5707963 0.0 1.5707963 -> xyz=-0.01999999837519743 0.020999999613397408 -0.21200000201339744 rpy=1.5707963 0.0 1.5707963
- joint left_shoulder_pitch_03: axis 0 0 1 -> (none); limit lower=-3.4906585 upper=1.9198622 effort=60 velocity=6.283 -> (none); origin xyz=-0.12394516500822303 -0.0021481216530753566 0.3387071333530755 rpy=-1.5707963 4.6410206566704915e-08 -1.5707963535897922 -> xyz=-0.12294516500822303 -0.002148121679870253 0.3387071333798704 rpy=-1.5707963 4.6410206566704915e-08 -1.5707963535897922
- joint left_shoulder_roll_03: axis 0 0 1 -> (none); limit lower=-0.48869219 upper=1.6580628 effort=60 velocity=6.283 -> (none); origin xyz=-0.02425 -2.6794896579307448e-11 -0.0800000000267949 rpy=-1.5707963 0 1.5707963 -> xyz=-0.02525 0 -0.08 rpy=-1.5707963 0 1.5707963
- joint left_shoulder_yaw_02: axis 0 0 1 -> (none); limit lower=-1.7453293 upper=1.7453293 effort=17 velocity=12.566 -> (none); origin xyz=0.14250000111248584 0.012713926047757364 -0.03020093770906647 rpy=-1.5707962267948243 -2.6794896301751692e-08 1.5707963267948966 -> xyz=0.14150000111248584 0.012713926047757361 -0.0302009376090664 rpy=-1.5707962267948243 -2.6794896301751692e-08 1.5707963267948966
- joint left_wrist_02: axis 0 0 1 -> (none); limit lower=-1.5707963 upper=1.5707963 effort=17 velocity=12.566 -> (none); origin xyz=0.017350000572946937 -0.10300000033493621 0.017999999565063794 rpy=-1.5707963071795865 -1.5707963 0.0 -> xyz=0.017350000553331628 -0.10200000033493621 0.017999999565063794 rpy=-1.5707963071795865 -1.5707963 0.0
- joint right_ankle_02: origin xyz=-0.025999999999999995 0.292499995396667 0.03300001483027525 rpy=9.282041333256967e-08 0.0 0.0 -> xyz=-0.025999999999999995 0.29249999530384657 0.034000014830275246 rpy=9.282041333256967e-08 0.0 0.0
- joint right_elbow_02: axis 0 0 1 -> (none); limit lower=0 upper=2.5307274 effort=17 velocity=12.566 -> (none); origin xyz=-0.01900000056016338 0.010007317759360172 -0.13702727562463635 rpy=-1.5707963646886025 -2.6794893859261038e-08 -1.5707962535897928 -> xyz=-0.018000000560163383 0.010007317832565275 -0.13702727566253006 rpy=-1.5707963646886025 -2.6794893859261038e-08 -1.5707962535897928
- joint right_hip_pitch_04: origin xyz=0.0565048409105324 1.547891480672564e-05 -0.07179286928519331 rpy=1.5707963 -4.641020634466031e-08 -1.5707963535897922 -> xyz=0.0555048409105324 1.5478941601622387e-05 -0.07179286925839841 rpy=1.5707963 -4.641020634466031e-08 -1.5707963535897922
- joint right_hip_roll_03: origin xyz=-0.024250000000000004 -0.030000000046410204 -0.0659999999732051 rpy=3.1415927 1.5707963 0 -> xyz=-0.02525 -0.03 -0.066 rpy=3.1415927 1.5707963 0
- joint right_hip_yaw_03: origin xyz=8.900090130537314e-09 0.14300000421300732 -0.025249999952628055 rpy=-1.5707963071795867 -4.6410206566704915e-08 3.141592560769381 -> xyz=8.807269719079969e-09 0.14200000421300732 -0.025249999933012746 rpy=-1.5707963071795867 -4.6410206566704915e-08 3.141592560769381
- joint right_knee_04: limit lower=-2.6005406 upper=0.078539816 effort=120 velocity=6.283 -> lower=-2.6703538 upper=0 effort=120 velocity=6.283; origin xyz=0.021099998493035996 0.02034023431476345 -0.212648350120343 rpy=-1.5707962070772346 -0.08726646299999974 1.5707962976557508 -> xyz=0.020099998493036002 0.020340234333468515 -0.2126483500010809 rpy=-1.5707962073561919 2.220446049250313e-16 1.5707963040449164
- joint right_shoulder_pitch_03: axis 0 0 1 -> (none); limit lower=-3.4906585 upper=1.9198622 effort=60 velocity=6.283 -> (none); origin xyz=0.12395483289078238 -0.002148124546924123 0.338707134112055 rpy=1.5707963071795872 -4.6410206566704915e-08 -1.5707963535897917 -> xyz=0.12295483289078238 -0.002148124520129227 0.3387071341316703 rpy=1.5707963071795872 -4.6410206566704915e-08 -1.5707963535897917
- joint right_shoulder_roll_03: axis 0 0 1 -> (none); limit lower=-1.6580628 upper=0.48869219 effort=60 velocity=6.283 -> (none); origin xyz=-0.02425 0.0 -0.0800000000267949 rpy=0 -1.5707963 0 -> xyz=-0.02525 0 -0.08 rpy=0 -1.5707963 0
- joint right_shoulder_yaw_02: axis 0 0 1 -> (none); limit lower=-1.7453293 upper=1.7453293 effort=17 velocity=12.566 -> (none); origin xyz=-0.013027815851142209 -0.14250000289956488 -0.030245284794312124 rpy=1.5707963996335306 -0.008726650000000058 3.141592595346938 -> xyz=-0.013027815793534982 -0.14150000289956488 -0.030245284867147983 rpy=1.5707963996335306 -0.008726650000000058 3.141592595346938
- joint right_wrist_02: axis 0 0 1 -> (none); limit lower=-1.5707963 upper=1.5707963 effort=17 velocity=12.566 -> (none); origin xyz=0.017349999519873475 0.10300000033493621 0.017999999565063797 rpy=1.5707963999999996 1.5707963000000005 0.0 -> xyz=0.017349999446668374 0.10200000033493621 0.017999999565063794 rpy=1.5707963999999996 1.5707963000000005 0.0

Commit message: bigger lims

File: sim/resources/kbot2/robot_fixed.urdf (robot description, URDF)
Before this commit: robot k-bot-v2, 22 links, 21 joints
Joints:
- joint left_ankle_02: limit lower=-0.78539816 upper=0.29670597 effort=17 velocity=12.566 -> lower=-1.2217 upper=0.7330 effort=17 velocity=12.566
- joint left_hip_pitch_04: limit lower=-1.5707963 upper=1.9198622 effort=120 velocity=6.283 -> lower=-2.0071 upper=2.3562 effort=120 velocity=6.283
- joint left_hip_roll_03: limit lower=-0.20943951 upper=2.6179939 effort=60 velocity=6.283 -> lower=-0.6457 upper=3.0543 effort=60 velocity=6.283
- joint left_hip_yaw_03: limit lower=-1.5707963 upper=1.9198622 effort=60 velocity=6.283 -> lower=-2.0071 upper=2.3562 effort=60 velocity=6.283
- joint left_knee_04: limit lower=0 upper=2.6703538 effort=120 velocity=6.283 -> lower=-0.4363 upper=3.1067 effort=120 velocity=6.283
- joint right_ankle_02: limit lower=-0.29670597 upper=0.78539816 effort=17 velocity=12.566 -> lower=-0.7330 upper=1.2217 effort=17 velocity=12.566
- joint right_hip_pitch_04: limit lower=-1.9198622 upper=1.5707963 effort=120 velocity=6.283 -> lower=-2.3562 upper=2.0071 effort=120 velocity=6.283
- joint right_hip_roll_03: limit lower=-2.6179939 upper=0.20943951 effort=60 velocity=6.283 -> lower=-3.0543 upper=0.6457 effort=60 velocity=6.283
- joint right_hip_yaw_03: limit lower=-1.5707963 upper=1.9198622 effort=60 velocity=6.283 -> lower=-2.0071 upper=2.3562 effort=60 velocity=6.283
- joint right_knee_04: limit lower=-2.6703538 upper=0 effort=120 velocity=6.283 -> lower=-0.4363 upper=3.1067 effort=120 velocity=6.283
