Commit message: updated urdf

File: sim/resources/gpr_headless/old/robot_fixed.urdf (robot description, URDF)
Before this commit: robot k-bot_sim, 23 links, 22 joints
Links:
- link arm1_top: geometry collision mesh filename=meshes/arm1_top.stl; visual mesh filename=meshes/arm1_top.stl
- link arm1_top_2: geometry collision mesh filename=meshes/arm1_top_2.stl; visual mesh filename=meshes/arm1_top_2.stl
- link arm2_shell: geometry collision mesh filename=meshes/arm2_shell.stl; visual mesh filename=meshes/arm2_shell.stl
- link arm2_shell_2: geometry collision mesh filename=meshes/arm2_shell_2.stl; visual mesh filename=meshes/arm2_shell_2.stl
- link arm3_shell: geometry collision mesh filename=meshes/arm3_shell.stl; visual mesh filename=meshes/arm3_shell.stl
- link arm3_shell2: geometry collision mesh filename=meshes/arm3_shell2.stl; visual mesh filename=meshes/arm3_shell2.stl
- link body1-part: geometry collision mesh filename=meshes/body1-part.stl; visual mesh filename=meshes/body1-part.stl
- link foot1: geometry collision mesh filename=meshes/foot1.stl; visual mesh filename=meshes/foot1.stl
- link foot3: geometry collision mesh filename=meshes/foot3.stl; visual mesh filename=meshes/foot3.stl
- link hand_shell: geometry collision mesh filename=meshes/hand_shell.stl; visual mesh filename=meshes/hand_shell.stl
- link hand_shell_2: geometry collision mesh filename=meshes/hand_shell_2.stl; visual mesh filename=meshes/hand_shell_2.stl
- link imu: geometry collision mesh filename=meshes/imu.stl; visual mesh filename=meshes/imu.stl
- link leg0_shell: geometry collision mesh filename=meshes/leg0_shell.stl; visual mesh filename=meshes/leg0_shell.stl
- link leg0_shell_2: geometry collision mesh filename=meshes/leg0_shell_2.stl; visual mesh filename=meshes/leg0_shell_2.stl
- link leg1_shell: geometry collision mesh filename=meshes/leg1_shell.stl; visual mesh filename=meshes/leg1_shell.stl
- link leg1_shell3: geometry collision mesh filename=meshes/leg1_shell3.stl; visual mesh filename=meshes/leg1_shell3.stl
- link leg2_shell: geometry collision mesh filename=meshes/leg2_shell.stl; visual mesh filename=meshes/leg2_shell.stl
- link leg2_shell_2: geometry collision mesh filename=meshes/leg2_shell_2.stl; visual mesh filename=meshes/leg2_shell_2.stl
- link leg3_shell1: geometry collision mesh filename=meshes/leg3_shell1.stl; visual mesh filename=meshes/leg3_shell1.stl
- link leg3_shell11: geometry collision mesh filename=meshes/leg3_shell11.stl; visual mesh filename=meshes/leg3_shell11.stl
- link shoulder: geometry collision mesh filename=meshes/shoulder.stl; visual mesh filename=meshes/shoulder.stl
- link shoulder_2: geometry collision mesh filename=meshes/shoulder_2.stl; visual mesh filename=meshes/shoulder_2.stl
Joints:
- joint floating_base: origin xyz=0.0 0.0009999996829318347 -7.963267107333194e-07 rpy=1.57 0.00 0.00 -> xyz=0 0 0 rpy=-1.57 3.14 0
- joint left_elbow_02: origin xyz=-0.027 -4.64102069112142e-11 -0.09799999974544849 rpy=-3.1415926071795863 -1.5707963 0.0 -> xyz=-0.026000000000000002 0.0 -0.09799999977224338 rpy=-3.1415926071795863 -1.5707963 0.0
- joint left_shoulder_pitch_03: origin xyz=-1.0603758999999933e-05 0.018089562004361112 0.18849980999999996 rpy=3.1415926071795868 -2.220446049250313e-15 3.1415926071795868 -> xyz=-0.0071262490312895945 0.2868887861013424 -0.1871062947956447 rpy=-2.220446049250311e-16 0.0 1.9915984595047395e-16
- joint left_shoulder_roll_03: axis 0 0 -1 -> 0 0 1; limit lower=-3.6302848 upper=0.47996554 effort=60 velocity=6.283 -> lower=-0.47996554 upper=3.6302848 effort=60 velocity=6.283; origin xyz=0.023511964 5.6278358217861975e-05 -0.06749999990621787 rpy=1.5707963 0.0 1.5707963 -> xyz=0.022511964 5.627838501275855e-05 -0.06749999993301277 rpy=1.5707963 0.0 1.5707963
- joint left_shoulder_yaw_02: origin xyz=-0.14049999999999996 -1.5083317163881439e-09 -0.023499999129165863 rpy=-1.5707963535897926 -2.6794894969484062e-08 -1.5707962803846895 -> xyz=-0.13949999999999996 -1.4619215099879723e-09 -0.02349999915596076 rpy=-4.641020604450649e-08 1.5707962732050293 0.0
- joint left_wrist_02: limit lower=-3.1415927 upper=3.1415927 effort=17 velocity=12.566 -> lower=0 upper=6.2831853 effort=17 velocity=12.566; origin xyz=-0.18249999999999997 -1.5083317163881439e-09 0.021500000870834136 rpy=-1.5707963535897926 -2.6794894969484062e-08 -1.5707962803846895 -> xyz=-0.18149999999999997 -1.4619215099879723e-09 0.02150000084403924 rpy=-4.641020604450649e-08 1.5707962732050293 0.0
- joint right_elbow_02: origin xyz=2.0814131093671585e-10 -0.027000000000000003 0.0975 rpy=-1.5707963071795865 1.5707963 0.0 -> xyz=0.026000000000000002 0.0 0.09750000022775662 rpy=-3.1415926071795863 1.5707963 0.0
- joint right_shoulder_pitch_03: origin xyz=-1.0603759e-05 0.018089564 -0.18850019 rpy=0.0 0.0 -3.1415926071795863 -> xyz=-0.007126249031289128 0.28688879614942864 0.18789370520435525 rpy=3.1415925999999996 -2.4424906541753444e-15 -9.282041357749904e-08
- joint right_shoulder_roll_03: origin xyz=0.023511963999999996 -5.627835821786203e-05 -0.06749999985980766 rpy=1.5707963999999996 -2.220446049250313e-16 -1.5707963000000003 -> xyz=0.022511964 -5.627838501275855e-05 -0.06749999993301277 rpy=1.5707963999999996 -2.220446049250313e-16 -1.5707963000000003
- joint right_shoulder_yaw_02: origin xyz=-0.14049999999999999 4.64102069112142e-11 0.02249999912916586 rpy=-3.1415926071795863 1.5707963 0.0 -> xyz=-0.13949999999999999 4.64102069112142e-11 0.02249999912916586 rpy=-3.1415926071795863 1.5707963 0.0
- joint right_wrist_02: limit lower=-3.1415927 upper=3.1415927 effort=17 velocity=12.566 -> lower=0 upper=6.2831853 effort=17 velocity=12.566; origin xyz=-0.18249999999999997 -1.5083317161660992e-09 0.021500000870834136 rpy=1.5707963535897933 -2.679489807810853e-08 1.5707963732051022 -> xyz=-0.18149999999999997 -1.4619215099879723e-09 0.02150000084403924 rpy=-4.641020604450649e-08 1.5707962732050293 0.0
