Commit message: latest

File: sim/resources/gpr_vel/robot_fixed.urdf (robot description, URDF)
Before this commit: robot k-bot_sim, 22 links, 21 joints
Joints:
- joint left_hip_pitch_04: limit lower=-1.570796 upper=1.570796 effort=120 velocity=6.283 -> lower=-1.570796 upper=1.570796 effort=100 velocity=6.283
- joint left_hip_roll_03: limit lower=-3.185226 upper=0.349066 effort=60 velocity=6.283 -> lower=-3.185226 upper=0.349066 effort=50 velocity=6.283
- joint left_hip_yaw_03: limit lower=-1.570796 upper=1.570796 effort=60 velocity=6.283 -> lower=-1.570796 upper=1.570796 effort=50 velocity=6.283
- joint left_knee_04: limit lower=0 upper=2.094395 effort=120 velocity=6.283 -> lower=0 upper=2.094395 effort=100 velocity=6.283
- joint left_shoulder_pitch_03: limit lower=0 upper=3.141593 effort=60 velocity=6.283 -> lower=0 upper=3.141593 effort=50 velocity=6.283
- joint left_shoulder_roll_03: limit lower=-3.630285 upper=0.479966 effort=60 velocity=6.283 -> lower=-3.630285 upper=0.479966 effort=50 velocity=6.283
- joint right_hip_pitch_04: limit lower=-1.570796 upper=1.570796 effort=120 velocity=6.283 -> lower=-1.570796 upper=1.570796 effort=100 velocity=6.283
- joint right_hip_roll_03: limit lower=-0.349066 upper=3.185226 effort=60 velocity=6.283 -> lower=-0.349066 upper=3.185226 effort=50 velocity=6.283
- joint right_hip_yaw_03: limit lower=-1.570796 upper=1.570796 effort=60 velocity=6.283 -> lower=-1.570796 upper=1.570796 effort=50 velocity=6.283
- joint right_knee_04: limit lower=-2.094395 upper=0 effort=120 velocity=6.283 -> lower=-2.094395 upper=0 effort=100 velocity=6.283
- joint right_shoulder_pitch_03: limit lower=-3.141593 upper=0 effort=60 velocity=6.283 -> lower=-3.141593 upper=0 effort=50 velocity=6.283
- joint right_shoulder_roll_03: limit lower=-0.479966 upper=3.630285 effort=60 velocity=6.283 -> lower=-0.479966 upper=3.630285 effort=50 velocity=6.283

Commit message: switch to old urdf

File: sim/resources/gpr_vel/robot_fixed.urdf (robot description, URDF)
Before this commit: robot k-bot_sim, 22 links, 21 joints
Links:
- removed link imu
- removed link leg3_shell1
- removed link leg3_shell11
- added link base, mass 0.001
- added link leg3_shell2, mass 1.179677561; collision mesh filename=meshes/leg3_shell2.stl; visual mesh filename=meshes/leg3_shell2.stl
- added link leg3_shell22, mass 1.179683991; collision mesh filename=meshes/leg3_shell22.stl; visual mesh filename=meshes/leg3_shell22.stl
- link arm1_top: mass 0.572732 -> 0.6485195170000001; geometry collision mesh filename=meshes/arm1_top.stl; visual mesh filename=meshes/arm1_top.stl
- link arm1_top_2: mass 0.572732 -> 0.648518913; geometry collision mesh filename=meshes/arm1_top_2.stl; visual mesh filename=meshes/arm1_top_2.stl
- link arm2_shell: mass 0.510678 -> 0.51101595; geometry collision mesh filename=meshes/arm2_shell.stl; visual mesh filename=meshes/arm2_shell.stl
- link arm2_shell_2: mass 0.510678 -> 0.51101595; geometry collision mesh filename=meshes/arm2_shell_2.stl; visual mesh filename=meshes/arm2_shell_2.stl
- link arm3_shell: mass 0.578536 -> 0.57887479; geometry collision mesh filename=meshes/arm3_shell.stl; visual mesh filename=meshes/arm3_shell.stl
- link arm3_shell2: mass 0.578536 -> 0.57887479; geometry collision mesh filename=meshes/arm3_shell2.stl; visual mesh filename=meshes/arm3_shell2.stl
- link body1-part: mass 9.415838 -> 11.417627727; geometry collision mesh filename=meshes/body1-part.stl; visual mesh filename=meshes/body1-part.stl
- link foot1: mass 0.582091 -> 0.54574734; geometry collision mesh filename=meshes/foot1.stl; visual mesh filename=meshes/foot1.stl
- link foot3: mass 0.582091 -> 0.5457471700000001; geometry collision mesh filename=meshes/foot3.stl; visual mesh filename=meshes/foot3.stl
- link hand_shell: mass 0.793063 -> 0.7933517460000001; geometry collision mesh filename=meshes/hand_shell.stl; visual mesh filename=meshes/hand_shell.stl
- link hand_shell_2: mass 0.793063 -> 0.7933517460000001; geometry collision mesh filename=meshes/hand_shell_2.stl; visual mesh filename=meshes/hand_shell_2.stl
- link leg0_shell: mass 1.323448 -> 1.3234480570000002; geometry collision mesh filename=meshes/leg0_shell.stl; visual mesh filename=meshes/leg0_shell.stl
- link leg0_shell_2: mass 1.323448 -> 1.3234480570000002; geometry collision mesh filename=meshes/leg0_shell_2.stl; visual mesh filename=meshes/leg0_shell_2.stl
- link leg1_shell: mass 1.264352 -> 1.360769512; geometry collision mesh filename=meshes/leg1_shell.stl; visual mesh filename=meshes/leg1_shell.stl
- link leg1_shell3: mass 1.264352 -> 1.360769362; geometry collision mesh filename=meshes/leg1_shell3.stl; visual mesh filename=meshes/leg1_shell3.stl
- link leg2_shell: mass 1.820923 -> 1.820922667; geometry collision mesh filename=meshes/leg2_shell.stl; visual mesh filename=meshes/leg2_shell.stl
- link leg2_shell_2: mass 1.820923 -> 1.820922667; geometry collision mesh filename=meshes/leg2_shell_2.stl; visual mesh filename=meshes/leg2_shell_2.stl
- link shoulder: mass 1.107356 -> 1.10769407; geometry collision mesh filename=meshes/shoulder.stl; visual mesh filename=meshes/shoulder.stl
- link shoulder_2: mass 1.107354 -> 1.10769287; geometry collision mesh filename=meshes/shoulder_2.stl; visual mesh filename=meshes/shoulder_2.stl
Joints:
- removed joint imu_link
- removed joint left_ankle_02
- removed joint left_elbow_02
- removed joint left_hip_pitch_04
- removed joint left_hip_roll_03
- removed joint left_hip_yaw_03
- removed joint left_knee_04
- removed joint left_shoulder_pitch_03
- removed joint left_shoulder_roll_03
- removed joint left_shoulder_yaw_02
- removed joint left_wrist_02
- removed joint right_ankle_02
- removed joint right_elbow_02
- removed joint right_hip_pitch_04
- removed joint right_hip_roll_03
- removed joint right_hip_yaw_03
- removed joint right_knee_04
- removed joint right_shoulder_pitch_03
- removed joint right_shoulder_roll_03
- removed joint right_shoulder_yaw_02
- removed joint right_wrist_02
- added joint L_ankle: type revolute, parent leg3_shell2, child foot1, origin xyz=0.0 -0.30000000004641003 0.07019999118206069 rpy=9.282041357749903e-08 0.0 0.0, axis 0 0 -1, limit lower=-0.6981317 upper=0.6981317 effort=17 velocity=1000
- added joint L_elbow: type fixed, parent arm2_shell, child arm3_shell, origin xyz=-0.026 0.0 -0.09799999977224338 rpy=-3.1415926071795863 -1.5707963 0.0, axis 0 0 1, limit lower=-2.5307274 upper=0 effort=80 velocity=5
- added joint L_hip_x: type revolute, parent leg0_shell, child leg1_shell, origin xyz=0.026499999999999965 -1.516591136963008e-09 -0.06950000151659115 rpy=-1.5707963 0.0 1.5707963, axis 0 0 1, limit lower=-0.34906585 upper=3.1852259 effort=40 velocity=1000
- added joint L_hip_y: type revolute, parent body1-part, child leg0_shell, origin xyz=-1.0608503738440467e-05 -0.43201043179234816 0.08770000686486729 rpy=-3.1415925071795874 4.641020723283873e-08 -3.1415926535897913, axis 0 0 1, limit lower=-1.5707963 upper=1.5707963 effort=60 velocity=1000
- added joint L_hip_z: type revolute, parent leg1_shell, child leg2_shell, origin xyz=-0.15649999999999997 0.00011981393 0.02749999848340886 rpy=-0.0 1.5707963 0.0, axis 0 0 1, limit lower=-1.5707963 upper=1.5707963 effort=40 velocity=1000
- added joint L_knee: type revolute, parent leg2_shell, child leg3_shell2, origin xyz=0.0 0.0342 -0.14250000009378214 rpy=1.5707963 0.0 0.0, axis 0 0 1, limit lower=-1.57 upper=0 effort=60 velocity=1000
- added joint L_shoulder_x: type fixed, parent shoulder, child arm1_top, origin xyz=0.022511964 5.627838501275897e-05 -0.06749999993301277 rpy=1.5707963 2.220446049250313e-16 1.5707963, axis 0 0 -1, limit lower=-0.47996554 upper=3.6302848 effort=80 velocity=5
- added joint L_shoulder_y: type fixed, parent body1-part, child shoulder, origin xyz=-1.0603759e-05 0.018089562050771318 0.18749980999999996 rpy=3.1415926071795868 -2.220446049250313e-15 3.1415926071795868, axis 0 0 1, limit lower=0 upper=3.1415927 effort=80 velocity=5
- added joint L_shoulder_z: type fixed, parent arm1_top, child arm2_shell, origin xyz=-0.13949999999999996 -1.461921509987972e-09 -0.023499999155960766 rpy=-4.641020604450648e-08 1.5707962732050293 0.0, axis 0 0 1, limit lower=-1.5707963 upper=1.5707963 effort=80 velocity=5
- added joint L_wrist: type fixed, parent arm3_shell, child hand_shell, origin xyz=-0.18149999999999994 -1.461921509987972e-09 0.021500000844039233 rpy=-4.641020604450648e-08 1.5707962732050293 0.0, axis 0 0 1, limit lower=0 upper=6.2831853 effort=80 velocity=5
- added joint R_ankle: type revolute, parent leg3_shell22, child foot3, origin xyz=1.0767167917674625e-08 -0.29999999865410376 0.027200000000000002 rpy=-3.1415926071795868 0.0 -3.1415926071795868, axis 0 0 -1, limit lower=-0.6981317 upper=0.6981317 effort=17 velocity=1000
- added joint R_elbow: type fixed, parent arm2_shell_2, child arm3_shell2, origin xyz=0.026 0.0 0.09750000022775662 rpy=-3.1415926071795863 1.5707963 0.0, axis 0 0 1, limit lower=0 upper=2.5307274 effort=80 velocity=5
- added joint R_hip_x: type revolute, parent leg0_shell_2, child leg1_shell3, origin xyz=0.026499999999999965 -1.516591136963008e-09 -0.06900000151659115 rpy=1.5707963 -4.641020678874952e-08 -1.5707963535897917, axis 0 0 1, limit lower=-0.34906585 upper=3.1852259 effort=40 velocity=1000
- added joint R_hip_y: type revolute, parent body1-part, child leg0_shell_2, origin xyz=-1.0600340183049505e-05 -0.4320104467591277 -0.08819999313513191 rpy=9.99999991702083e-08 4.641020723283873e-08 -3.1415926535897913, axis 0 0 1, limit lower=-1.5707963 upper=1.5707963 effort=60 velocity=1000
- added joint R_hip_z: type revolute, parent leg1_shell3, child leg2_shell_2, origin xyz=-0.15649999999999997 -0.00011981393 0.02749999848340886 rpy=-3.1415926535897922 -1.5707962732050305 0.0, axis 0 0 1, limit lower=-1.5707963 upper=1.5707963 effort=40 velocity=1000
- added joint R_knee: type revolute, parent leg2_shell_2, child leg3_shell22, origin xyz=0.0 0.0342 -0.14250000009378214 rpy=1.5707963 0.0 0.0, axis 0 0 -1, limit lower=-1.57 upper=0 effort=60 velocity=1000
- added joint R_shoulder_x: type fixed, parent shoulder_2, child arm1_top_2, origin xyz=0.022511964 -5.627838501275897e-05 -0.06749999993301277 rpy=1.5707963999999996 2.220446049250313e-16 -1.5707963000000003, axis 0 0 1, limit lower=-0.47996554 upper=3.6302848 effort=80 velocity=5
- added joint R_shoulder_y: type fixed, parent body1-part, child shoulder_2, origin xyz=-1.0603759e-05 0.018089564 -0.18750019 rpy=0.0 0.0 -3.1415926071795863, axis 0 0 1, limit lower=-3.1415927 upper=0 effort=80 velocity=5
- added joint R_shoulder_z: type fixed, parent arm1_top_2, child arm2_shell_2, origin xyz=-0.13949999999999999 0.0 0.02249999915596076 rpy=-3.1415926071795863 1.5707963 0.0, axis 0 0 -1, limit lower=-1.5707963 upper=1.5707963 effort=80 velocity=5
- added joint R_wrist: type fixed, parent arm3_shell2, child hand_shell_2, origin xyz=-0.18149999999999994 -1.461921509987972e-09 0.021500000844039233 rpy=-4.641020604450648e-08 1.5707962732050293 0.0, axis 0 0 1, limit lower=0 upper=6.2831853 effort=80 velocity=5
- added joint floating_base: type fixed, parent base, child body1-part, origin xyz=0 0 0 rpy=-1.57 3.14 0
