Commit message: update headless normal

File: sim/resources/gpr_headless/old_real/robot_fixed.urdf (robot description, URDF)
Before this commit: robot k-bot_sim, 23 links, 22 joints
Joints:
- joint floating_base: origin xyz=0.0 0.0009999996829318347 -7.963267107333194e-07 rpy=1.57 0.00 0.00 -> xyz=0.0 0.0009999996829318347 0 rpy=1.57 0.00 0.00
- joint left_ankle_02: limit lower=-0.6981317 upper=0.6981317 effort=17 velocity=12.566 -> lower=-1.2217307 upper=1.2217307 effort=17 velocity=12.566
- joint left_hip_pitch_04: limit lower=-1.5707963 upper=1.5707963 effort=120 velocity=6.283 -> lower=-2.0943953 upper=2.0943953 effort=120 velocity=6.283
- joint left_hip_roll_03: limit lower=-3.1852259 upper=0.34906585 effort=60 velocity=6.283 -> lower=-3.7088249 upper=0.8726648 effort=60 velocity=6.283
- joint left_hip_yaw_03: limit lower=-1.5707963 upper=1.5707963 effort=60 velocity=6.283 -> lower=-2.0943953 upper=2.0943953 effort=60 velocity=6.283
- joint left_knee_04: limit lower=0 upper=2.0943951 effort=120 velocity=6.283 -> lower=-0.523599 upper=2.6179941 effort=120 velocity=6.283
- joint right_ankle_02: limit lower=-0.6981317 upper=0.6981317 effort=17 velocity=12.566 -> lower=-1.2217307 upper=1.2217307 effort=17 velocity=12.566
- joint right_hip_pitch_04: limit lower=-1.5707963 upper=1.5707963 effort=120 velocity=6.283 -> lower=-2.0943953 upper=2.0943953 effort=120 velocity=6.283
- joint right_hip_roll_03: limit lower=-0.34906585 upper=3.1852259 effort=60 velocity=6.283 -> lower=-0.8726648 upper=3.7088249 effort=60 velocity=6.283
- joint right_hip_yaw_03: limit lower=-1.5707963 upper=1.5707963 effort=60 velocity=6.283 -> lower=-2.0943953 upper=2.0943953 effort=60 velocity=6.283
- joint right_knee_04: limit lower=-2.0943951 upper=0 effort=120 velocity=6.283 -> lower=-2.6179941 upper=0.523599 effort=120 velocity=6.283

File: sim/resources/gpr_headless/robot_fixed.urdf (robot description, URDF)
Before this commit: robot k-bot_sim, 23 links, 22 joints
Links:
- removed link base
- added link floating_base_link, mass 0.001; visual sphere radius=0.01
- link arm1_top: mass 0.5727323900000001 -> 0.572732; geometry visual mesh filename=meshes/arm1_top.stl
- link arm1_top_2: mass 0.57273186 -> 0.572732; geometry visual mesh filename=meshes/arm1_top_2.stl
- link arm2_shell: mass 0.51067762 -> 0.510678; geometry collision mesh filename=meshes/arm2_shell.collision.stl; visual mesh filename=meshes/arm2_shell.stl
- link arm2_shell_2: mass 0.51067762 -> 0.510678; geometry collision mesh filename=meshes/arm2_shell_2.collision.stl; visual mesh filename=meshes/arm2_shell_2.stl
- link arm3_shell: mass 0.5785364000000001 -> 0.578536; geometry visual mesh filename=meshes/arm3_shell.stl
- link arm3_shell2: mass 0.5785364000000001 -> 0.578536; geometry visual mesh filename=meshes/arm3_shell2.stl
- link body1-part: mass 9.12867194 -> 9.415838; geometry collision mesh filename=meshes/body1-part.collision.stl; visual mesh filename=meshes/body1-part.stl
- link foot1: mass 0.58209124 -> 0.582091; geometry collision mesh filename=meshes/foot1.collision.stl; visual mesh filename=meshes/foot1.stl
- link foot3: mass 0.58209108 -> 0.582091; geometry collision mesh filename=meshes/foot3.collision.stl; visual mesh filename=meshes/foot3.stl
- link hand_shell: mass 0.7930633560000001 -> 0.793063; geometry collision mesh filename=meshes/hand_shell.collision.stl; visual mesh filename=meshes/hand_shell.stl
- link hand_shell_2: mass 0.7930633560000001 -> 0.793063; geometry collision mesh filename=meshes/hand_shell_2.collision.stl; visual mesh filename=meshes/hand_shell_2.stl
- link imu: mass 0.01 -> 0.010000
- link leg0_shell: mass 1.3234480570000002 -> 1.323448; geometry collision mesh filename=meshes/leg0_shell.collision.stl; visual mesh filename=meshes/leg0_shell.stl
- link leg0_shell_2: mass 1.3234480570000002 -> 1.323448; geometry collision mesh filename=meshes/leg0_shell_2.collision.stl; visual mesh filename=meshes/leg0_shell_2.stl
- link leg1_shell: mass 1.2643519300000001 -> 1.264352; geometry visual mesh filename=meshes/leg1_shell.stl
- link leg1_shell3: mass 1.26435173 -> 1.264352; geometry visual mesh filename=meshes/leg1_shell3.stl
- link leg2_shell: mass 1.820922667 -> 1.820923; geometry visual mesh filename=meshes/leg2_shell.stl
- link leg2_shell_2: mass 1.820922667 -> 1.820923; geometry visual mesh filename=meshes/leg2_shell_2.stl
- link leg3_shell1: mass 1.10995541 -> 1.109955; geometry collision mesh filename=meshes/leg3_shell1.collision.stl; visual mesh filename=meshes/leg3_shell1.stl
- link leg3_shell11: mass 1.10996161 -> 1.109962; geometry collision mesh filename=meshes/leg3_shell11.collision.stl; visual mesh filename=meshes/leg3_shell11.stl
- link shoulder: mass 1.1073556900000001 -> 1.107356; geometry collision mesh filename=meshes/shoulder.collision.stl; visual mesh filename=meshes/shoulder.stl
- link shoulder_2: mass 1.10735447 -> 1.107354; geometry collision mesh filename=meshes/shoulder_2.collision.stl; visual mesh filename=meshes/shoulder_2.stl
Joints:
- removed joint floating_base
- added joint floating_base_joint: type fixed, parent floating_base_link, child body1-part, origin xyz=0 0 0 rpy=1.57 0.00 0.00
- joint imu_link: origin xyz=0.039989396 -0.12791044000000001 -2.6794896579307448e-11 rpy=-1.5707963 0 0 -> xyz=0.039989 -0.127910 0 rpy=-1.570796 0 0
- joint left_ankle_02: limit lower=-1.2217307 upper=1.2217307 effort=17 velocity=12.566 -> lower=-0.698132 upper=0.698132 effort=17 velocity=12.566; origin xyz=0.0 -0.30000000013923045 0.009499991182060727 rpy=9.282041333256967e-08 0.0 0.0 -> xyz=0 -0.300000 0.009500 rpy=0 0 0
- joint left_elbow_02: limit lower=-2.5307274 upper=0 effort=17 velocity=12.566 -> lower=-2.530727 upper=0 effort=17 velocity=12.566; origin xyz=-0.027 -4.64102069112142e-11 -0.09799999974544849 rpy=-3.1415926071795863 -1.5707963 0.0 -> xyz=-0.027000 0 -0.098000 rpy=-3.141593 -1.570796 0
- joint left_hip_pitch_04: limit lower=-2.0943953 upper=2.0943953 effort=120 velocity=6.283 -> lower=-1.570796 upper=1.570796 effort=120 velocity=6.283; origin xyz=-1.0608550148631657e-05 -0.43201043164593794 0.0887000068648673 rpy=-3.1415925071795874 4.641020678874952e-08 -3.1415926535897913 -> xyz=-0.000011 -0.432010 0.088700 rpy=-3.141593 0 -3.141593
- joint left_hip_roll_03: limit lower=-3.7088249 upper=0.8726648 effort=60 velocity=6.283 -> lower=-3.185226 upper=0.349066 effort=60 velocity=6.283; origin xyz=0.027499999999999972 -1.543386042968109e-09 -0.06950000154338605 rpy=-1.5707963 0.0 1.5707963 -> xyz=0.027500 0 -0.069500 rpy=-1.570796 0 1.570796
- joint left_hip_yaw_03: limit lower=-2.0943953 upper=2.0943953 effort=60 velocity=6.283 -> lower=-1.570796 upper=1.570796 effort=60 velocity=6.283; origin xyz=-0.15749999999999997 0.00011981393 0.027499998456613956 rpy=-0.0 1.5707963 0.0 -> xyz=-0.157500 0.000120 0.027500 rpy=0 1.570796 0
- joint left_knee_04: limit lower=-0.523599 upper=2.6179941 effort=120 velocity=6.283 -> lower=0 upper=2.094395 effort=120 velocity=6.283; origin xyz=0.0 -0.026999999999999993 -0.14250000111820607 rpy=1.5707963999999996 0.0 0.0 -> xyz=0 -0.027000 -0.142500 rpy=1.570796 0 0
- joint left_shoulder_pitch_03: limit lower=0 upper=3.1415927 effort=60 velocity=6.283 -> lower=0 upper=3.141593 effort=60 velocity=6.283; origin xyz=-1.0603758999999933e-05 0.018089562004361112 0.18849980999999996 rpy=3.1415926071795868 -2.220446049250313e-15 3.1415926071795868 -> xyz=-0.000011 0.018090 0.188500 rpy=3.141593 0 3.141593
- joint left_shoulder_roll_03: limit lower=-3.6302848 upper=0.47996554 effort=60 velocity=6.283 -> lower=-3.630285 upper=0.479966 effort=60 velocity=6.283; origin xyz=0.023511964 5.6278358217861975e-05 -0.06749999990621787 rpy=1.5707963 0.0 1.5707963 -> xyz=0.023512 0.000056 -0.067500 rpy=1.570796 0 1.570796
- joint left_shoulder_yaw_02: limit lower=-1.5707963 upper=1.5707963 effort=17 velocity=12.566 -> lower=-1.570796 upper=1.570796 effort=17 velocity=12.566; origin xyz=-0.14049999999999996 -1.5083317163881439e-09 -0.023499999129165863 rpy=-1.5707963535897926 -2.6794894969484062e-08 -1.5707962803846895 -> xyz=-0.140500 0 -0.023500 rpy=-1.570796 0 -1.570796
- joint left_wrist_02: limit lower=-3.1415927 upper=3.1415927 effort=17 velocity=12.566 -> lower=-3.141593 upper=3.141593 effort=17 velocity=12.566; origin xyz=-0.18249999999999997 -1.5083317163881439e-09 0.021500000870834136 rpy=-1.5707963535897926 -2.6794894969484062e-08 -1.5707962803846895 -> xyz=-0.182500 0 0.021500 rpy=-1.570796 0 -1.570796
- joint right_ankle_02: axis 0 0 -1 -> 0 0 1.0; limit lower=-1.2217307 upper=1.2217307 effort=17 velocity=12.566 -> lower=-0.698132 upper=0.698132 effort=17 velocity=12.566; origin xyz=2.153907282807268e-18 -0.3000000000464102 -0.035500000000000004 rpy=3.1415927 0 3.1415927 -> xyz=0 -0.300000 -0.035500 rpy=3.141593 0 3.141593
- joint right_elbow_02: limit lower=0 upper=2.5307274 effort=17 velocity=12.566 -> lower=0 upper=2.530727 effort=17 velocity=12.566; origin xyz=2.0814131093671585e-10 -0.027000000000000003 0.0975 rpy=-1.5707963071795865 1.5707963 0.0 -> xyz=0 -0.027000 0.097500 rpy=-1.570796 1.570796 0
- joint right_hip_pitch_04: limit lower=-2.0943953 upper=2.0943953 effort=120 velocity=6.283 -> lower=-1.570796 upper=1.570796 effort=120 velocity=6.283; origin xyz=-1.0600293772844438e-05 -0.4320104468591277 -0.08919999313513188 rpy=9.99999991702083e-08 4.641020678874952e-08 -3.1415926535897913 -> xyz=-0.000011 -0.432010 -0.089200 rpy=0 0 -3.141593
- joint right_hip_roll_03: limit lower=-0.8726648 upper=3.7088249 effort=60 velocity=6.283 -> lower=-0.349066 upper=3.185226 effort=60 velocity=6.283; origin xyz=0.027499999999999972 -1.5433860431346424e-09 -0.06900000154338605 rpy=1.5707963 -4.641020634466031e-08 -1.5707963535897922 -> xyz=0.027500 0 -0.069000 rpy=1.570796 0 -1.570796
- joint right_hip_yaw_03: limit lower=-2.0943953 upper=2.0943953 effort=60 velocity=6.283 -> lower=-1.570796 upper=1.570796 effort=60 velocity=6.283; origin xyz=-0.15749999999999997 -0.00011981393000000101 0.027499998536998718 rpy=-3.1415926535897922 -1.5707962732050302 0.0 -> xyz=-0.157500 -0.000120 0.027500 rpy=-3.141593 -1.570796 0
- joint right_knee_04: limit lower=-2.6179941 upper=0.523599 effort=120 velocity=6.283 -> lower=-2.094395 upper=0 effort=120 velocity=6.283; origin xyz=0.0 -0.026999999999999993 -0.14250000111820607 rpy=1.5707963999999996 0.0 0.0 -> xyz=0 -0.027000 -0.142500 rpy=1.570796 0 0
- joint right_shoulder_pitch_03: limit lower=-3.1415927 upper=0 effort=60 velocity=6.283 -> lower=-3.141593 upper=0 effort=60 velocity=6.283; origin xyz=-1.0603759e-05 0.018089564 -0.18850019 rpy=0.0 0.0 -3.1415926071795863 -> xyz=-0.000011 0.018090 -0.188500 rpy=0 0 -3.141593
- joint right_shoulder_roll_03: limit lower=-0.47996554 upper=3.6302848 effort=60 velocity=6.283 -> lower=-0.479966 upper=3.630285 effort=60 velocity=6.283; origin xyz=0.023511963999999996 -5.627835821786203e-05 -0.06749999985980766 rpy=1.5707963999999996 -2.220446049250313e-16 -1.5707963000000003 -> xyz=0.023512 -0.000056 -0.067500 rpy=1.570796 0 -1.570796
- joint right_shoulder_yaw_02: limit lower=-1.5707963 upper=1.5707963 effort=17 velocity=12.566 -> lower=-1.570796 upper=1.570796 effort=17 velocity=12.566; origin xyz=-0.14049999999999999 4.64102069112142e-11 0.02249999912916586 rpy=-3.1415926071795863 1.5707963 0.0 -> xyz=-0.140500 0 0.022500 rpy=-3.141593 1.570796 0
- joint right_wrist_02: limit lower=-3.1415927 upper=3.1415927 effort=17 velocity=12.566 -> lower=-3.141593 upper=3.141593 effort=17 velocity=12.566; origin xyz=-0.18249999999999997 -1.5083317161660992e-09 0.021500000870834136 rpy=1.5707963535897933 -2.679489807810853e-08 1.5707963732051022 -> xyz=-0.182500 0 0.021500 rpy=1.570796 0 1.570796
