Commit message: save

File: sim/resources/gpr_headless/robot_fixed.urdf (robot description, URDF)
Before this commit: robot k-bot_naked, 23 links, 22 joints
Joints:
- joint floating_base: origin xyz=0 0 0 rpy=-1.57 0 0 -> xyz=0 0 0 rpy=-1.57 3.14 0

Commit message: flexible lims

File: sim/resources/gpr_headless/robot_fixed.urdf (robot description, URDF)
Before this commit: robot k-bot_sim, 23 links, 22 joints
Joints:
- joint left_ankle_02: limit lower=-0.6981317 upper=0.6981317 effort=17 velocity=12.566 -> lower=-1.2217307 upper=1.2217307 effort=17 velocity=12.566
- joint left_hip_pitch_04: limit lower=-1.5707963 upper=1.5707963 effort=120 velocity=6.283 -> lower=-2.0943953 upper=2.0943953 effort=120 velocity=6.283
- joint left_hip_roll_03: limit lower=-3.1852259 upper=0.34906585 effort=60 velocity=6.283 -> lower=-3.7088249 upper=0.8726648 effort=60 velocity=6.283
- joint left_hip_yaw_03: limit lower=-1.5707963 upper=1.5707963 effort=60 velocity=6.283 -> lower=-2.0943953 upper=2.0943953 effort=60 velocity=6.283
- joint left_knee_04: limit lower=0 upper=2.0943951 effort=120 velocity=6.283 -> lower=-0.523599 upper=2.6179941 effort=120 velocity=6.283
- joint right_ankle_02: limit lower=-0.6981317 upper=0.6981317 effort=17 velocity=12.566 -> lower=-1.2217307 upper=1.2217307 effort=17 velocity=12.566
- joint right_hip_pitch_04: limit lower=-1.5707963 upper=1.5707963 effort=120 velocity=6.283 -> lower=-2.0943953 upper=2.0943953 effort=120 velocity=6.283
- joint right_hip_roll_03: limit lower=-0.34906585 upper=3.1852259 effort=60 velocity=6.283 -> lower=-0.8726648 upper=3.7088249 effort=60 velocity=6.283
- joint right_hip_yaw_03: limit lower=-1.5707963 upper=1.5707963 effort=60 velocity=6.283 -> lower=-2.0943953 upper=2.0943953 effort=60 velocity=6.283
- joint right_knee_04: limit lower=-2.0943951 upper=0 effort=120 velocity=6.283 -> lower=-2.6179941 upper=0.523599 effort=120 velocity=6.283

Commit message: fiz heights

File: sim/resources/gpr_headless/robot_fixed.urdf (robot description, URDF)
Before this commit: robot k-bot_sim, 23 links, 22 joints
Joints:
- joint floating_base: origin xyz=0.0 0.0009999996829318347 -7.963267107333194e-07 rpy=1.57 0.00 0.00 -> xyz=0.0 0.0009999996829318347 0 rpy=1.57 0.00 0.00

Commit message: update urdfs

File: sim/resources/gpr_headless/robot_fixed.urdf (robot description, URDF)
Before this commit: robot k-bot_sim, 23 links, 22 joints
Links:
- link floating_base_link: mass 0.001 -> None; geometry 
Joints:
- joint floating_base_joint: origin xyz=0 0 0 rpy=1.57 0.00 0.00 -> xyz=0 0 0 rpy=1.57 0 3.14
- joint left_ankle_02: limit lower=-0.698132 upper=0.698132 effort=17 velocity=12.566 -> lower=-0.698132 upper=0.698132 effort=17 velocity=18.0
- joint left_hip_pitch_04: limit lower=-1.570796 upper=1.570796 effort=120 velocity=6.283 -> lower=-1.570796 upper=1.570796 effort=80 velocity=18.0
- joint left_hip_roll_03: limit lower=-3.185226 upper=0.349066 effort=60 velocity=6.283 -> lower=-3.185226 upper=0.349066 effort=40 velocity=18.0
- joint left_hip_yaw_03: limit lower=-1.570796 upper=1.570796 effort=60 velocity=6.283 -> lower=-1.570796 upper=1.570796 effort=40 velocity=18.0
- joint left_knee_04: limit lower=0 upper=2.094395 effort=120 velocity=6.283 -> lower=-1.57 upper=0 effort=80 velocity=18.0
- joint right_ankle_02: limit lower=-0.698132 upper=0.698132 effort=17 velocity=12.566 -> lower=-0.698132 upper=0.698132 effort=17 velocity=18.0
- joint right_hip_pitch_04: limit lower=-1.570796 upper=1.570796 effort=120 velocity=6.283 -> lower=-1.570796 upper=1.570796 effort=80 velocity=18.0
- joint right_hip_roll_03: limit lower=-0.349066 upper=3.185226 effort=60 velocity=6.283 -> lower=-0.349066 upper=3.185226 effort=40 velocity=18.0
- joint right_hip_yaw_03: limit lower=-1.570796 upper=1.570796 effort=60 velocity=6.283 -> lower=-1.570796 upper=1.570796 effort=40 velocity=18.0
- joint right_knee_04: limit lower=-2.094395 upper=0 effort=120 velocity=6.283 -> lower=-1.57 upper=0 effort=80 velocity=18.0
