Commit message: save updates

File: sim/resources/gpr_headless_latency_pos/robot_fixed.urdf (robot description, URDF)
Before this commit: robot k-bot_sim, 23 links, 22 joints
Joints:
- joint left_ankle_02: limit lower=-0.698132 upper=0.698132 effort=17 velocity=18.0 -> lower=-0.698132 upper=0.698132 effort=17 velocity=18
- joint left_hip_pitch_04: limit lower=-1.570796 upper=1.570796 effort=80 velocity=18.0 -> lower=-1.570796 upper=1.570796 effort=60 velocity=18
- joint left_hip_roll_03: limit lower=-3.185226 upper=0.349066 effort=40 velocity=18.0 -> lower=-3.185226 upper=0.349066 effort=40 velocity=18
- joint left_hip_yaw_03: limit lower=-1.570796 upper=1.570796 effort=40 velocity=18.0 -> lower=-1.570796 upper=1.570796 effort=40 velocity=18
- joint left_knee_04: limit lower=-1.57 upper=0 effort=80 velocity=18.0 -> lower=0 upper=2.094395 effort=60 velocity=18
- joint right_ankle_02: limit lower=-0.698132 upper=0.698132 effort=17 velocity=18.0 -> lower=-0.698132 upper=0.698132 effort=17 velocity=18
- joint right_hip_pitch_04: limit lower=-1.570796 upper=1.570796 effort=80 velocity=18.0 -> lower=-1.570796 upper=1.570796 effort=60 velocity=18
- joint right_hip_roll_03: limit lower=-0.349066 upper=3.185226 effort=40 velocity=18.0 -> lower=-0.349066 upper=3.185226 effort=40 velocity=18
- joint right_hip_yaw_03: limit lower=-1.570796 upper=1.570796 effort=40 velocity=18.0 -> lower=-1.570796 upper=1.570796 effort=40 velocity=18
- joint right_knee_04: limit lower=-1.57 upper=0 effort=80 velocity=18.0 -> lower=-2.094395 upper=0 effort=60 velocity=18
