Commit message: update kbot urdf, will probably break everything cause joint names are all different

File: sim/resources/gpr/robot.urdf (robot description, URDF)
Before this commit: robot gpr, 22 links, 21 joints
Links:
- link body1-part: mass 11.923537116999997 -> 11.417627727
- link shoulder_2: mass 0.80769287 -> 1.10769287
Joints:
- removed joint L_ankle_y
- removed joint L_hip_x
- removed joint L_hip_y
- removed joint L_hip_z
- removed joint L_knee
- removed joint R_ankle_y
- removed joint R_hip_x
- removed joint R_hip_y
- removed joint R_hip_z
- removed joint R_knee
- removed joint Revolute_1
- removed joint Revolute_15
- removed joint Revolute_16
- removed joint Revolute_2
- removed joint Revolute_3
- removed joint Revolute_4
- removed joint Revolute_5
- removed joint Revolute_6
- removed joint Revolute_7
- removed joint Revolute_8
- added joint keft_elbow_02: type revolute, parent arm2_shell, child arm3_shell, origin xyz=-0.026000000000000002 0.0 -0.09799999977224338 rpy=-3.1415926071795863 -1.5707963 0.0, axis 0 0 1, limit lower=-2.5307274 upper=0 effort=17 velocity=720
- added joint left_ankle_02: type revolute, parent leg3_shell2, child foot1, origin xyz=0.0 -0.30000000004641003 0.07019999118206069 rpy=9.282041357749903e-08 0.0 0.0, axis 0 0 1, limit lower=-0.6981317 upper=0.6981317 effort=17 velocity=720
- added joint left_hip_pitch_04: type revolute, parent body1-part, child leg0_shell, origin xyz=-1.0608503738424868e-05 -0.43201043179234816 0.08770000686486731 rpy=-3.1415925071795874 4.641020678874952e-08 -3.1415926535897913, axis 0 0 1, limit lower=-1.5707963 upper=1.5707963 effort=120 velocity=360
- added joint left_hip_roll_03: type revolute, parent leg0_shell, child leg1_shell, origin xyz=0.02649999999999997 -1.5165911463888016e-09 -0.06950000151659115 rpy=-1.5707963 0.0 1.5707963, axis 0 0 1, limit lower=-3.1852259 upper=0.34906585 effort=60 velocity=360
- added joint left_hip_yaw_03: type revolute, parent leg1_shell, child leg2_shell, origin xyz=-0.15649999999999997 0.00011981393 0.027499998483408852 rpy=-0.0 1.5707963 0.0, axis 0 0 1, limit lower=-1.5707963 upper=1.5707963 effort=60 velocity=360
- added joint left_knee_04: type revolute, parent leg2_shell, child leg3_shell2, origin xyz=0.0 0.0342 -0.14250000009378214 rpy=1.5707963000000003 0.0 0.0, axis 0 0 1, limit lower=-2.0943951 upper=0 effort=120 velocity=360
- added joint left_shoulder_pitch_03: type revolute, parent body1-part, child shoulder, origin xyz=-1.0603759e-05 0.018089562050771318 0.18749980999999996 rpy=3.1415926071795868 -2.220446049250313e-15 3.1415926071795868, axis 0 0 1, limit lower=0 upper=3.1415927 effort=60 velocity=360
- added joint left_shoulder_roll_03: type revolute, parent shoulder, child arm1_top, origin xyz=0.022511964 5.627838501275855e-05 -0.06749999993301277 rpy=1.5707963 0.0 1.5707963, axis 0 0 1, limit lower=-0.47996554 upper=3.6302848 effort=60 velocity=360
- added joint left_shoulder_yaw_02: type revolute, parent arm1_top, child arm2_shell, origin xyz=-0.13949999999999996 -1.4619215099879723e-09 -0.02349999915596076 rpy=-4.641020604450649e-08 1.5707962732050293 0.0, axis 0 0 1, limit lower=-1.5707963 upper=1.5707963 effort=17 velocity=720
- added joint left_wrist_02: type revolute, parent arm3_shell, child hand_shell, origin xyz=-0.18149999999999997 -1.4619215099879723e-09 0.02150000084403924 rpy=-4.641020604450649e-08 1.5707962732050293 0.0, axis 0 0 1, limit lower=0 upper=6.2831853 effort=17 velocity=720
- added joint right_ankle_02: type revolute, parent leg3_shell22, child foot3, origin xyz=1.0767167917674625e-08 -0.2999999986541038 0.027200000000000002 rpy=-3.1415926071795868 2.220446049250313e-16 -3.1415926071795868, axis 0 0 1, limit lower=-0.6981317 upper=0.6981317 effort=17 velocity=720
- added joint right_elbow_02: type revolute, parent arm2_shell_2, child arm3_shell2, origin xyz=0.026000000000000002 0.0 0.09750000022775662 rpy=-3.1415926071795863 1.5707963 0.0, axis 0 0 1, limit lower=0 upper=2.5307274 effort=17 velocity=720
- added joint right_hip_pitch_04: type revolute, parent body1-part, child leg0_shell_2, origin xyz=-1.0600340183051227e-05 -0.4320104467591277 -0.08819999313513188 rpy=9.99999991702083e-08 4.641020678874952e-08 -3.1415926535897913, axis 0 0 1, limit lower=-1.5707963 upper=1.5707963 effort=120 velocity=360
- added joint right_hip_roll_03: type revolute, parent leg0_shell_2, child leg1_shell3, origin xyz=0.02649999999999997 -1.5165911463888016e-09 -0.06900000151659115 rpy=1.5707963 -4.641020634466031e-08 -1.5707963535897922, axis 0 0 1, limit lower=-0.34906585 upper=3.1852259 effort=60 velocity=360
- added joint right_hip_yaw_03: type revolute, parent leg1_shell3, child leg2_shell_2, origin xyz=-0.15649999999999997 -0.00011981393 0.027499998483408852 rpy=-3.1415926535897922 -1.5707962732050302 0.0, axis 0 0 1, limit lower=-1.5707963 upper=1.5707963 effort=60 velocity=360
- added joint right_knee_04: type revolute, parent leg2_shell_2, child leg3_shell22, origin xyz=0.0 0.0342 -0.14250000009378214 rpy=1.5707963000000003 0.0 0.0, axis 0 0 1, limit lower=0 upper=2.0943951 effort=120 velocity=360
- added joint right_shoulder_pitch_03: type revolute, parent body1-part, child shoulder_2, origin xyz=-1.0603759e-05 0.018089564 -0.18750019 rpy=0.0 0.0 -3.1415926071795863, axis 0 0 1, limit lower=-3.1415927 upper=0 effort=60 velocity=360
- added joint right_shoulder_roll_03: type revolute, parent shoulder_2, child arm1_top_2, origin xyz=0.022511964 -5.627838501275855e-05 -0.06749999993301277 rpy=1.5707963999999996 -2.220446049250313e-16 -1.5707963000000003, axis 0 0 1, limit lower=-0.47996554 upper=3.6302848 effort=60 velocity=360
- added joint right_shoulder_yaw_02: type revolute, parent arm1_top_2, child arm2_shell_2, origin xyz=-0.13949999999999999 0.0 0.022499999155960758 rpy=-3.1415926071795863 1.5707963 0.0, axis 0 0 1, limit lower=-1.5707963 upper=1.5707963 effort=17 velocity=720
- added joint right_wrist_02: type revolute, parent arm3_shell2, child hand_shell_2, origin xyz=-0.18149999999999997 -1.4619215099879723e-09 0.02150000084403924 rpy=-4.641020604450649e-08 1.5707962732050293 0.0, axis 0 0 1, limit lower=0 upper=6.2831853 effort=17 velocity=720
- joint floating_base: origin xyz=0 0 0 rpy=-1.57 3.14 0 -> xyz=0 0 0 rpy=1.57 0.00 0.00

File: sim/resources/gpr/robot_fixed.urdf (robot description, URDF)
Before this commit: robot gpr, 23 links, 22 joints
Links:
- removed link imu_link
- link body1-part: mass 11.923537116999997 -> 11.417627727
- link shoulder_2: mass 0.80769287 -> 1.10769287
Joints:
- removed joint L_ankle_y
- removed joint L_hip_x
- removed joint L_hip_y
- removed joint L_hip_z
- removed joint L_knee
- removed joint R_ankle_y
- removed joint R_hip_x
- removed joint R_hip_y
- removed joint R_hip_z
- removed joint R_knee
- removed joint Revolute_1
- removed joint Revolute_15
- removed joint Revolute_16
- removed joint Revolute_2
- removed joint Revolute_3
- removed joint Revolute_4
- removed joint Revolute_5
- removed joint Revolute_6
- removed joint Revolute_7
- removed joint Revolute_8
- removed joint imu_joint
- added joint keft_elbow_02: type fixed, parent arm2_shell, child arm3_shell, origin xyz=-0.026000000000000002 0.0 -0.09799999977224338 rpy=-3.1415926071795863 -1.5707963 0.0, axis 0 0 1, limit lower=-2.5307274 upper=0 effort=17 velocity=720
- added joint left_ankle_02: type revolute, parent leg3_shell2, child foot1, origin xyz=0.0 -0.30000000004641003 0.07019999118206069 rpy=9.282041357749903e-08 0.0 0.0, axis 0 0 1, limit lower=-0.6981317 upper=0.6981317 effort=17 velocity=10
- added joint left_hip_pitch_04: type revolute, parent body1-part, child leg0_shell, origin xyz=-1.0608503738424868e-05 -0.43201043179234816 0.08770000686486731 rpy=-3.1415925071795874 4.641020678874952e-08 -3.1415926535897913, axis 0 0 1, limit lower=-1.5707963 upper=1.5707963 effort=120 velocity=10
- added joint left_hip_roll_03: type revolute, parent leg0_shell, child leg1_shell, origin xyz=0.02649999999999997 -1.5165911463888016e-09 -0.06950000151659115 rpy=-1.5707963 0.0 1.5707963, axis 0 0 1, limit lower=-3.1852259 upper=0.34906585 effort=60 velocity=10
- added joint left_hip_yaw_03: type revolute, parent leg1_shell, child leg2_shell, origin xyz=-0.15649999999999997 0.00011981393 0.027499998483408852 rpy=-0.0 1.5707963 0.0, axis 0 0 1, limit lower=-1.5707963 upper=1.5707963 effort=60 velocity=10
- added joint left_knee_04: type revolute, parent leg2_shell, child leg3_shell2, origin xyz=0.0 0.0342 -0.14250000009378214 rpy=1.5707963000000003 0.0 0.0, axis 0 0 1, limit lower=-1.57 upper=0 effort=60 velocity=10
- added joint left_shoulder_pitch_03: type fixed, parent body1-part, child shoulder, origin xyz=-1.0603759e-05 0.018089562050771318 0.18749980999999996 rpy=3.1415926071795868 -2.220446049250313e-15 3.1415926071795868, axis 0 0 1, limit lower=0 upper=3.1415927 effort=60 velocity=360
- added joint left_shoulder_roll_03: type fixed, parent shoulder, child arm1_top, origin xyz=0.022511964 5.627838501275855e-05 -0.06749999993301277 rpy=1.5707963 0.0 1.5707963, axis 0 0 1, limit lower=-0.47996554 upper=3.6302848 effort=60 velocity=360
- added joint left_shoulder_yaw_02: type fixed, parent arm1_top, child arm2_shell, origin xyz=-0.13949999999999996 -1.4619215099879723e-09 -0.02349999915596076 rpy=-4.641020604450649e-08 1.5707962732050293 0.0, axis 0 0 1, limit lower=-1.5707963 upper=1.5707963 effort=17 velocity=720
- added joint left_wrist_02: type fixed, parent arm3_shell, child hand_shell, origin xyz=-0.18149999999999997 -1.4619215099879723e-09 0.02150000084403924 rpy=-4.641020604450649e-08 1.5707962732050293 0.0, axis 0 0 1, limit lower=0 upper=6.2831853 effort=17 velocity=720
- added joint right_ankle_02: type revolute, parent leg3_shell22, child foot3, origin xyz=1.0767167917674625e-08 -0.2999999986541038 0.027200000000000002 rpy=-3.1415926071795868 2.220446049250313e-16 -3.1415926071795868, axis 0 0 1, limit lower=-0.6981317 upper=0.6981317 effort=17 velocity=10
- added joint right_elbow_02: type fixed, parent arm2_shell_2, child arm3_shell2, origin xyz=0.026000000000000002 0.0 0.09750000022775662 rpy=-3.1415926071795863 1.5707963 0.0, axis 0 0 1, limit lower=0 upper=2.5307274 effort=17 velocity=720
- added joint right_hip_pitch_04: type revolute, parent body1-part, child leg0_shell_2, origin xyz=-1.0600340183051227e-05 -0.4320104467591277 -0.08819999313513188 rpy=9.99999991702083e-08 4.641020678874952e-08 -3.1415926535897913, axis 0 0 1, limit lower=-1.5707963 upper=1.5707963 effort=120 velocity=10
- added joint right_hip_roll_03: type revolute, parent leg0_shell_2, child leg1_shell3, origin xyz=0.02649999999999997 -1.5165911463888016e-09 -0.06900000151659115 rpy=1.5707963 -4.641020634466031e-08 -1.5707963535897922, axis 0 0 1, limit lower=-0.34906585 upper=3.1852259 effort=60 velocity=10
- added joint right_hip_yaw_03: type revolute, parent leg1_shell3, child leg2_shell_2, origin xyz=-0.15649999999999997 -0.00011981393 0.027499998483408852 rpy=-3.1415926535897922 -1.5707962732050302 0.0, axis 0 0 1, limit lower=-1.5707963 upper=1.5707963 effort=60 velocity=10
- added joint right_knee_04: type revolute, parent leg2_shell_2, child leg3_shell22, origin xyz=0.0 0.0342 -0.14250000009378214 rpy=1.5707963000000003 0.0 0.0, axis 0 0 1, limit lower=0 upper=1.57 effort=60 velocity=10
- added joint right_shoulder_pitch_03: type fixed, parent body1-part, child shoulder_2, origin xyz=-1.0603759e-05 0.018089564 -0.18750019 rpy=0.0 0.0 -3.1415926071795863, axis 0 0 1, limit lower=-3.1415927 upper=0 effort=60 velocity=360
- added joint right_shoulder_roll_03: type fixed, parent shoulder_2, child arm1_top_2, origin xyz=0.022511964 -5.627838501275855e-05 -0.06749999993301277 rpy=1.5707963999999996 -2.220446049250313e-16 -1.5707963000000003, axis 0 0 1, limit lower=-0.47996554 upper=3.6302848 effort=60 velocity=360
- added joint right_shoulder_yaw_02: type fixed, parent arm1_top_2, child arm2_shell_2, origin xyz=-0.13949999999999999 0.0 0.022499999155960758 rpy=-3.1415926071795863 1.5707963 0.0, axis 0 0 1, limit lower=-1.5707963 upper=1.5707963 effort=17 velocity=720
- added joint right_wrist_02: type fixed, parent arm3_shell2, child hand_shell_2, origin xyz=-0.18149999999999997 -1.4619215099879723e-09 0.02150000084403924 rpy=-4.641020604450649e-08 1.5707962732050293 0.0, axis 0 0 1, limit lower=0 upper=6.2831853 effort=17 velocity=720
- joint floating_base: origin xyz=0 0 0 rpy=-1.57 3.14 0 -> xyz=0 0 0 rpy=1.57 0.00 0.00
