Commit message: new setup, fix mapping todo

File: sim/resources/gpr/robot.urdf (robot description, URDF)
Before this commit: robot kbot, 22 links, 21 joints
Links:
- removed link base
- removed link leg3_shell2
- removed link leg3_shell22
- added link imu, mass 0.010000; visual mesh filename=meshes/imu.stl
- added link leg3_shell1, mass 1.109955; collision mesh filename=meshes/leg3_shell1.collision.stl; visual mesh filename=meshes/leg3_shell1.stl
- added link leg3_shell11, mass 1.109962; collision mesh filename=meshes/leg3_shell11.collision.stl; visual mesh filename=meshes/leg3_shell11.stl
- link arm1_top: mass 0.6485195170000001 -> 0.572732; geometry visual mesh filename=meshes/arm1_top.stl
- link arm1_top_2: mass 0.648518913 -> 0.572732; geometry visual mesh filename=meshes/arm1_top_2.stl
- link arm2_shell: mass 0.51101595 -> 0.510678; geometry collision mesh filename=meshes/arm2_shell.collision.stl; visual mesh filename=meshes/arm2_shell.stl
- link arm2_shell_2: mass 0.51101595 -> 0.510678; geometry collision mesh filename=meshes/arm2_shell_2.collision.stl; visual mesh filename=meshes/arm2_shell_2.stl
- link arm3_shell: mass 0.57887479 -> 0.578536; geometry visual mesh filename=meshes/arm3_shell.stl
- link arm3_shell2: mass 0.57887479 -> 0.578536; geometry visual mesh filename=meshes/arm3_shell2.stl
- link body1-part: mass 11.417627727 -> 9.415838; geometry collision mesh filename=meshes/body1-part.collision.stl; visual mesh filename=meshes/body1-part.stl
- link foot1: mass 0.54574734 -> 0.582091; geometry collision mesh filename=meshes/foot1.collision.stl; visual mesh filename=meshes/foot1.stl
- link foot3: mass 0.5457471700000001 -> 0.582091; geometry collision mesh filename=meshes/foot3.collision.stl; visual mesh filename=meshes/foot3.stl
- link hand_shell: mass 0.7933517460000001 -> 0.793063; geometry collision mesh filename=meshes/hand_shell.collision.stl; visual mesh filename=meshes/hand_shell.stl
- link hand_shell_2: mass 0.7933517460000001 -> 0.793063; geometry collision mesh filename=meshes/hand_shell_2.collision.stl; visual mesh filename=meshes/hand_shell_2.stl
- link leg0_shell: mass 1.3234480570000002 -> 1.323448; geometry collision mesh filename=meshes/leg0_shell.collision.stl; visual mesh filename=meshes/leg0_shell.stl
- link leg0_shell_2: mass 1.3234480570000002 -> 1.323448; geometry collision mesh filename=meshes/leg0_shell_2.collision.stl; visual mesh filename=meshes/leg0_shell_2.stl
- link leg1_shell: mass 1.360769512 -> 1.264352; geometry visual mesh filename=meshes/leg1_shell.stl
- link leg1_shell3: mass 1.360769362 -> 1.264352; geometry visual mesh filename=meshes/leg1_shell3.stl
- link leg2_shell: mass 1.820922667 -> 1.820923; geometry visual mesh filename=meshes/leg2_shell.stl
- link leg2_shell_2: mass 1.820922667 -> 1.820923; geometry visual mesh filename=meshes/leg2_shell_2.stl
- link shoulder: mass 1.10769407 -> 1.107356; geometry collision mesh filename=meshes/shoulder.collision.stl; visual mesh filename=meshes/shoulder.stl
- link shoulder_2: mass 1.10769287 -> 1.107354; geometry collision mesh filename=meshes/shoulder_2.collision.stl; visual mesh filename=meshes/shoulder_2.stl
Joints:
- removed joint L_ankle
- removed joint L_elbow
- removed joint L_hip_x
- removed joint L_hip_y
- removed joint L_hip_z
- removed joint L_knee
- removed joint L_shoulder_x
- removed joint L_shoulder_y
- removed joint L_shoulder_z
- removed joint L_wrist
- removed joint R_ankle
- removed joint R_elbow
- removed joint R_hip_x
- removed joint R_hip_y
- removed joint R_hip_z
- removed joint R_knee
- removed joint R_shoulder_x
- removed joint R_shoulder_y
- removed joint R_shoulder_z
- removed joint R_wrist
- removed joint floating_base
- added joint imu_link: type fixed, parent body1-part, child imu, origin xyz=0.040000 0 -0.131000 rpy=0 0 0
- added joint left_ankle_02: type revolute, parent leg3_shell1, child foot1, origin xyz=0 -0.300000 0.009500 rpy=0 0 0, axis 0 0 -1, limit lower=-0.698132 upper=0.698132 effort=17 velocity=12.566
- added joint left_elbow_02: type revolute, parent arm2_shell, child arm3_shell, origin xyz=-0.027000 0 -0.098000 rpy=-3.141593 -1.570796 0, axis 0 0 1, limit lower=-2.530727 upper=0 effort=17 velocity=12.566
- added joint left_hip_pitch_04: type revolute, parent body1-part, child leg0_shell, origin xyz=-0.000002 -0.091000 -0.430001 rpy=1.570000 0 3.140000, axis 0 0 1, limit lower=-1.570796 upper=1.570796 effort=120 velocity=6.283
- added joint left_hip_roll_03: type revolute, parent leg0_shell, child leg1_shell, origin xyz=0.027500 0 -0.069500 rpy=-1.570796 0 1.570796, axis 0 0 1, limit lower=-3.185226 upper=0.349066 effort=60 velocity=6.283
- added joint left_hip_yaw_03: type revolute, parent leg1_shell, child leg2_shell, origin xyz=-0.157500 0.000120 0.027500 rpy=0 1.570796 0, axis 0 0 1, limit lower=-1.570796 upper=1.570796 effort=60 velocity=6.283
- added joint left_knee_04: type revolute, parent leg2_shell, child leg3_shell1, origin xyz=0 -0.027000 -0.142500 rpy=1.570796 0 0, axis 0 0 -1, limit lower=0 upper=2.094395 effort=120 velocity=6.283
- added joint left_shoulder_pitch_03: type revolute, parent body1-part, child shoulder, origin xyz=0.000002 -0.191000 0.019999 rpy=1.570000 0 -3.140000, axis 0 0 1, limit lower=0 upper=3.141593 effort=60 velocity=6.283
- added joint left_shoulder_roll_03: type revolute, parent shoulder, child arm1_top, origin xyz=0.023512 0.000056 -0.067500 rpy=1.570796 0 1.570796, axis 0 0 -1, limit lower=-3.630285 upper=0.479966 effort=60 velocity=6.283
- added joint left_shoulder_yaw_02: type revolute, parent arm1_top, child arm2_shell, origin xyz=-0.140500 0 -0.023500 rpy=-1.570796 0 -1.570796, axis 0 0 1, limit lower=-1.570796 upper=1.570796 effort=17 velocity=12.566
- added joint left_wrist_02: type revolute, parent arm3_shell, child hand_shell, origin xyz=-0.182500 0 0.021500 rpy=-1.570796 0 -1.570796, axis 0 0 1, limit lower=-3.141593 upper=3.141593 effort=17 velocity=12.566
- added joint right_ankle_02: type revolute, parent leg3_shell11, child foot3, origin xyz=0 -0.300000 -0.035500 rpy=3.141593 0 3.141593, axis 0 0 1.0, limit lower=-0.698132 upper=0.698132 effort=17 velocity=12.566
- added joint right_elbow_02: type revolute, parent arm2_shell_2, child arm3_shell2, origin xyz=0 -0.027000 0.097500 rpy=-1.570796 1.570796 0, axis 0 0 1, limit lower=0 upper=2.530727 effort=17 velocity=12.566
- added joint right_hip_pitch_04: type revolute, parent body1-part, child leg0_shell_2, origin xyz=0.000002 0.091000 -0.430001 rpy=-1.570000 0 3.140000, axis 0 0 1, limit lower=-1.570796 upper=1.570796 effort=120 velocity=6.283
- added joint right_hip_roll_03: type revolute, parent leg0_shell_2, child leg1_shell3, origin xyz=0.027500 0 -0.069000 rpy=1.570796 0 -1.570796, axis 0 0 1, limit lower=-0.349066 upper=3.185226 effort=60 velocity=6.283
- added joint right_hip_yaw_03: type revolute, parent leg1_shell3, child leg2_shell_2, origin xyz=-0.157500 -0.000120 0.027500 rpy=-3.141593 -1.570796 0, axis 0 0 1, limit lower=-1.570796 upper=1.570796 effort=60 velocity=6.283
- added joint right_knee_04: type revolute, parent leg2_shell_2, child leg3_shell11, origin xyz=0 -0.027000 -0.142500 rpy=1.570796 0 0, axis 0 0 -1, limit lower=-2.094395 upper=0 effort=120 velocity=6.283
- added joint right_shoulder_pitch_03: type revolute, parent body1-part, child shoulder_2, origin xyz=-0.000002 0.191000 0.019999 rpy=-1.570000 0 -3.140000, axis 0 0 1, limit lower=-3.141593 upper=0 effort=60 velocity=6.283
- added joint right_shoulder_roll_03: type revolute, parent shoulder_2, child arm1_top_2, origin xyz=0.023512 -0.000056 -0.067500 rpy=1.570796 0 -1.570796, axis 0 0 1, limit lower=-0.479966 upper=3.630285 effort=60 velocity=6.283
- added joint right_shoulder_yaw_02: type revolute, parent arm1_top_2, child arm2_shell_2, origin xyz=-0.140500 0 0.022500 rpy=-3.141593 1.570796 0, axis 0 0 -1, limit lower=-1.570796 upper=1.570796 effort=17 velocity=12.566
- added joint right_wrist_02: type revolute, parent arm3_shell2, child hand_shell_2, origin xyz=-0.182500 0 0.021500 rpy=1.570796 0 1.570796, axis 0 0 1, limit lower=-3.141593 upper=3.141593 effort=17 velocity=12.566

File: sim/resources/gpr/robot_fixed.urdf (robot description, URDF)
Before this commit: robot kbot, 22 links, 21 joints
Links:
- removed link leg3_shell2
- removed link leg3_shell22
- added link leg3_shell1, mass 1.109955; collision mesh filename=meshes/leg3_shell1.collision.stl; visual mesh filename=meshes/leg3_shell1.stl
- added link leg3_shell11, mass 1.109962; collision mesh filename=meshes/leg3_shell11.collision.stl; visual mesh filename=meshes/leg3_shell11.stl
- link arm1_top: mass 0.6485195170000001 -> 0.572732; geometry visual mesh filename=meshes/arm1_top.stl
- link arm1_top_2: mass 0.648518913 -> 0.572732; geometry visual mesh filename=meshes/arm1_top_2.stl
- link arm2_shell: mass 0.51101595 -> 0.510678; geometry collision mesh filename=meshes/arm2_shell.collision.stl; visual mesh filename=meshes/arm2_shell.stl
- link arm2_shell_2: mass 0.51101595 -> 0.510678; geometry collision mesh filename=meshes/arm2_shell_2.collision.stl; visual mesh filename=meshes/arm2_shell_2.stl
- link arm3_shell: mass 0.57887479 -> 0.578536; geometry visual mesh filename=meshes/arm3_shell.stl
- link arm3_shell2: mass 0.57887479 -> 0.578536; geometry visual mesh filename=meshes/arm3_shell2.stl
- link body1-part: mass 11.417627727 -> 9.415838; geometry collision mesh filename=meshes/body1-part.collision.stl; visual mesh filename=meshes/body1-part.stl
- link foot1: mass 0.54574734 -> 0.582091; geometry collision mesh filename=meshes/foot1.collision.stl; visual mesh filename=meshes/foot1.stl
- link foot3: mass 0.5457471700000001 -> 0.582091; geometry collision mesh filename=meshes/foot3.collision.stl; visual mesh filename=meshes/foot3.stl
- link hand_shell: mass 0.7933517460000001 -> 0.793063; geometry collision mesh filename=meshes/hand_shell.collision.stl; visual mesh filename=meshes/hand_shell.stl
- link hand_shell_2: mass 0.7933517460000001 -> 0.793063; geometry collision mesh filename=meshes/hand_shell_2.collision.stl; visual mesh filename=meshes/hand_shell_2.stl
- link leg0_shell: mass 1.3234480570000002 -> 1.323448; geometry collision mesh filename=meshes/leg0_shell.collision.stl; visual mesh filename=meshes/leg0_shell.stl
- link leg0_shell_2: mass 1.3234480570000002 -> 1.323448; geometry collision mesh filename=meshes/leg0_shell_2.collision.stl; visual mesh filename=meshes/leg0_shell_2.stl
- link leg1_shell: mass 1.360769512 -> 1.264352; geometry visual mesh filename=meshes/leg1_shell.stl
- link leg1_shell3: mass 1.360769362 -> 1.264352; geometry visual mesh filename=meshes/leg1_shell3.stl
- link leg2_shell: mass 1.820922667 -> 1.820923; geometry visual mesh filename=meshes/leg2_shell.stl
- link leg2_shell_2: mass 1.820922667 -> 1.820923; geometry visual mesh filename=meshes/leg2_shell_2.stl
- link shoulder: mass 1.10769407 -> 1.107356; geometry collision mesh filename=meshes/shoulder.collision.stl; visual mesh filename=meshes/shoulder.stl
- link shoulder_2: mass 1.10769287 -> 1.107354; geometry collision mesh filename=meshes/shoulder_2.collision.stl; visual mesh filename=meshes/shoulder_2.stl
Joints:
- removed joint L_ankle
- removed joint L_elbow
- removed joint L_hip_x
- removed joint L_hip_y
- removed joint L_hip_z
- removed joint L_knee
- removed joint L_shoulder_x
- removed joint L_shoulder_y
- removed joint L_shoulder_z
- removed joint L_wrist
- removed joint R_ankle
- removed joint R_elbow
- removed joint R_hip_x
- removed joint R_hip_y
- removed joint R_hip_z
- removed joint R_knee
- removed joint R_shoulder_x
- removed joint R_shoulder_y
- removed joint R_shoulder_z
- removed joint R_wrist
- added joint left_ankle_02: type revolute, parent leg3_shell1, child foot1, origin xyz=0 -0.300000 0.009500 rpy=0 0 0, axis 0 0 -1, limit lower=-0.698132 upper=0.698132 effort=17 velocity=12.566
- added joint left_elbow_02: type fixed, parent arm2_shell, child arm3_shell, origin xyz=-0.027000 0 -0.098000 rpy=-3.141593 -1.570796 0, axis 0 0 1, limit lower=-2.530727 upper=0 effort=17 velocity=12.566
- added joint left_hip_pitch_04: type revolute, parent body1-part, child leg0_shell, origin xyz=-0.000002 -0.091000 -0.430001 rpy=1.570000 0 3.140000, axis 0 0 1, limit lower=-1.570796 upper=1.570796 effort=60 velocity=6.283
- added joint left_hip_roll_03: type revolute, parent leg0_shell, child leg1_shell, origin xyz=0.027500 0 -0.069500 rpy=-1.570796 0 1.570796, axis 0 0 1, limit lower=-3.185226 upper=0.349066 effort=40 velocity=6.283
- added joint left_hip_yaw_03: type revolute, parent leg1_shell, child leg2_shell, origin xyz=-0.157500 0.000120 0.027500 rpy=0 1.570796 0, axis 0 0 1, limit lower=-1.570796 upper=1.570796 effort=40 velocity=6.283
- added joint left_knee_04: type revolute, parent leg2_shell, child leg3_shell1, origin xyz=0 -0.027000 -0.142500 rpy=1.570796 0 0, axis 0 0 -1, limit lower=0 upper=2.094395 effort=60 velocity=6.283
- added joint left_shoulder_pitch_03: type fixed, parent body1-part, child shoulder, origin xyz=0.000002 -0.191000 0.019999 rpy=1.570000 0 -3.140000, axis 0 0 1, limit lower=0 upper=3.141593 effort=60 velocity=6.283
- added joint left_shoulder_roll_03: type fixed, parent shoulder, child arm1_top, origin xyz=0.023512 0.000056 -0.067500 rpy=1.570796 0 1.570796, axis 0 0 -1, limit lower=-3.630285 upper=0.479966 effort=60 velocity=6.283
- added joint left_shoulder_yaw_02: type fixed, parent arm1_top, child arm2_shell, origin xyz=-0.140500 0 -0.023500 rpy=-1.570796 0 -1.570796, axis 0 0 1, limit lower=-1.570796 upper=1.570796 effort=17 velocity=12.566
- added joint left_wrist_02: type fixed, parent arm3_shell, child hand_shell, origin xyz=-0.182500 0 0.021500 rpy=-1.570796 0 -1.570796, axis 0 0 1, limit lower=-3.141593 upper=3.141593 effort=17 velocity=12.566
- added joint right_ankle_02: type revolute, parent leg3_shell11, child foot3, origin xyz=0 -0.300000 -0.035500 rpy=3.141593 0 3.141593, axis 0 0 1.0, limit lower=-0.698132 upper=0.698132 effort=17 velocity=12.566
- added joint right_elbow_02: type fixed, parent arm2_shell_2, child arm3_shell2, origin xyz=0 -0.027000 0.097500 rpy=-1.570796 1.570796 0, axis 0 0 1, limit lower=0 upper=2.530727 effort=17 velocity=12.566
- added joint right_hip_pitch_04: type revolute, parent body1-part, child leg0_shell_2, origin xyz=0.000002 0.091000 -0.430001 rpy=-1.570000 0 3.140000, axis 0 0 1, limit lower=-1.570796 upper=1.570796 effort=60 velocity=6.283
- added joint right_hip_roll_03: type revolute, parent leg0_shell_2, child leg1_shell3, origin xyz=0.027500 0 -0.069000 rpy=1.570796 0 -1.570796, axis 0 0 1, limit lower=-0.349066 upper=3.185226 effort=40 velocity=6.283
- added joint right_hip_yaw_03: type revolute, parent leg1_shell3, child leg2_shell_2, origin xyz=-0.157500 -0.000120 0.027500 rpy=-3.141593 -1.570796 0, axis 0 0 1, limit lower=-1.570796 upper=1.570796 effort=40 velocity=6.283
- added joint right_knee_04: type revolute, parent leg2_shell_2, child leg3_shell11, origin xyz=0 -0.027000 -0.142500 rpy=1.570796 0 0, axis 0 0 -1, limit lower=-2.094395 upper=0 effort=60 velocity=6.283
- added joint right_shoulder_pitch_03: type fixed, parent body1-part, child shoulder_2, origin xyz=-0.000002 0.191000 0.019999 rpy=-1.570000 0 -3.140000, axis 0 0 1, limit lower=-3.141593 upper=0 effort=60 velocity=6.283
- added joint right_shoulder_roll_03: type fixed, parent shoulder_2, child arm1_top_2, origin xyz=0.023512 -0.000056 -0.067500 rpy=1.570796 0 -1.570796, axis 0 0 1, limit lower=-0.479966 upper=3.630285 effort=60 velocity=6.283
- added joint right_shoulder_yaw_02: type fixed, parent arm1_top_2, child arm2_shell_2, origin xyz=-0.140500 0 0.022500 rpy=-3.141593 1.570796 0, axis 0 0 -1, limit lower=-1.570796 upper=1.570796 effort=17 velocity=12.566
- added joint right_wrist_02: type fixed, parent arm3_shell2, child hand_shell_2, origin xyz=-0.182500 0 0.021500 rpy=1.570796 0 1.570796, axis 0 0 1, limit lower=-3.141593 upper=3.141593 effort=17 velocity=12.566
- joint floating_base: origin xyz=0 0 0 rpy=-1.57 3.14 0 -> xyz=0 0 0 rpy=0 0 3.14

Commit message: add headless

File: sim/resources/gpr/robot.urdf (robot description, URDF)
Before this commit: robot k-bot_sim, 22 links, 21 joints
Links:
- removed link imu
- added link floating_base_link
Joints:
- removed joint imu_link
- added joint floating_base_joint: type fixed, parent floating_base_link, child body1-part, origin xyz=0 0 0 rpy=1.57 0 3.14
- joint left_hip_pitch_04: origin xyz=-0.000002 -0.091000 -0.430001 rpy=1.570000 0 3.140000 -> xyz=-0.000011 -0.432010 0.088700 rpy=-3.141593 0 -3.141593
- joint left_shoulder_pitch_03: origin xyz=0.000002 -0.191000 0.019999 rpy=1.570000 0 -3.140000 -> xyz=-0.000011 0.018090 0.188500 rpy=3.141593 0 3.141593
- joint right_hip_pitch_04: origin xyz=0.000002 0.091000 -0.430001 rpy=-1.570000 0 3.140000 -> xyz=-0.000011 -0.432010 -0.089200 rpy=0 0 -3.141593
- joint right_shoulder_pitch_03: origin xyz=-0.000002 0.191000 0.019999 rpy=-1.570000 0 -3.140000 -> xyz=-0.000011 0.018090 -0.188500 rpy=0 0 -3.141593

File: sim/resources/gpr/robot_fixed.urdf (robot description, URDF)
Before this commit: robot k-bot_sim, 22 links, 21 joints
Links:
- removed link base
- added link floating_base_link
Joints:
- removed joint floating_base
- added joint floating_base_joint: type fixed, parent floating_base_link, child body1-part, origin xyz=0 0 0 rpy=1.57 0 3.14
- joint left_hip_pitch_04: origin xyz=-0.000002 -0.091000 -0.430001 rpy=1.570000 0 3.140000 -> xyz=-0.000011 -0.432010 0.088700 rpy=-3.141593 0 -3.141593
- joint left_shoulder_pitch_03: origin xyz=0.000002 -0.191000 0.019999 rpy=1.570000 0 -3.140000 -> xyz=-0.000011 0.018090 0.188500 rpy=3.141593 0 3.141593
- joint right_hip_pitch_04: origin xyz=0.000002 0.091000 -0.430001 rpy=-1.570000 0 3.140000 -> xyz=-0.000011 -0.432010 -0.089200 rpy=0 0 -3.141593
- joint right_shoulder_pitch_03: origin xyz=-0.000002 0.191000 0.019999 rpy=-1.570000 0 -3.140000 -> xyz=-0.000011 0.018090 -0.188500 rpy=0 0 -3.141593

Commit message: update to the limits, no merging joints

File: sim/resources/gpr/robot.urdf (robot description, URDF)
Before this commit: robot k-bot_sim, 22 links, 21 joints
Links:
- added link imu, mass 0.010000; visual mesh filename=meshes/imu.stl
Joints:
- added joint imu_link: type fixed, parent body1-part, child imu, origin xyz=0.039989 -0.127910 0 rpy=-1.570796 0 0

File: sim/resources/gpr/robot_fixed.urdf (robot description, URDF)
Before this commit: robot k-bot_sim, 22 links, 21 joints
Links:
- added link imu, mass 0.010000; visual mesh filename=meshes/imu.stl
Joints:
- added joint imu_link: type fixed, parent body1-part, child imu, origin xyz=0.039989 -0.127910 0 rpy=-1.570796 0 0
