Commit message: update values

File: sim/resources/gpr/robot_fixed.urdf (robot description, URDF)
Before this commit: robot gpr, 22 links, 21 joints
Joints:
- joint L_ankle_y: limit lower=-0.6981317 upper=0.6981317 effort=17 velocity=10 -> lower=-0.6981317 upper=0.6981317 effort=26 velocity=10
- joint R_ankle_y: limit lower=-0.6981317 upper=0.6981317 effort=17 velocity=10 -> lower=-0.6981317 upper=0.6981317 effort=26 velocity=10

Commit message: update to even lower efforts

File: sim/resources/gpr/robot_fixed.urdf (robot description, URDF)
Before this commit: robot gpr, 22 links, 21 joints
Joints:
- joint L_ankle_y: limit lower=-0.6981317 upper=0.6981317 effort=26 velocity=10 -> lower=-0.6981317 upper=0.6981317 effort=17 velocity=10
- joint L_hip_x: limit lower=-0.34906585 upper=3.1852259 effort=60 velocity=10 -> lower=-0.34906585 upper=3.1852259 effort=20 velocity=10
- joint L_hip_y: limit lower=-1.5707963 upper=1.5707963 effort=120 velocity=10 -> lower=-1.5707963 upper=1.5707963 effort=40 velocity=10
- joint L_hip_z: limit lower=-1.5707963 upper=1.5707963 effort=60 velocity=10 -> lower=-1.5707963 upper=1.5707963 effort=20 velocity=10
- joint L_knee: limit lower=-1.57 upper=0 effort=120 velocity=10 -> lower=-1.57 upper=0 effort=40 velocity=10
- joint R_ankle_y: limit lower=-0.6981317 upper=0.6981317 effort=26 velocity=10 -> lower=-0.6981317 upper=0.6981317 effort=17 velocity=10
- joint R_hip_x: limit lower=-0.34906585 upper=3.1852259 effort=60 velocity=10 -> lower=-0.34906585 upper=3.1852259 effort=20 velocity=10
- joint R_hip_y: limit lower=-1.5707963 upper=1.5707963 effort=120 velocity=10 -> lower=-1.5707963 upper=1.5707963 effort=40 velocity=10
- joint R_hip_z: limit lower=-1.5707963 upper=1.5707963 effort=60 velocity=10 -> lower=-1.5707963 upper=1.5707963 effort=20 velocity=10
- joint R_knee: limit lower=0 upper=1.57 effort=120 velocity=10 -> lower=0 upper=1.57 effort=40 velocity=10

Commit message: new params

File: sim/resources/gpr/robot_fixed.urdf (robot description, URDF)
Before this commit: robot gpr, 22 links, 21 joints
Joints:
- joint L_hip_y: limit lower=-1.5707963 upper=1.5707963 effort=40 velocity=10 -> lower=-1.5707963 upper=1.5707963 effort=30 velocity=10
- joint L_knee: limit lower=-1.57 upper=0 effort=40 velocity=10 -> lower=-1.57 upper=0 effort=30 velocity=10
- joint R_hip_y: limit lower=-1.5707963 upper=1.5707963 effort=40 velocity=10 -> lower=-1.5707963 upper=1.5707963 effort=30 velocity=10
- joint R_knee: limit lower=0 upper=1.57 effort=40 velocity=10 -> lower=0 upper=1.57 effort=30 velocity=10

Commit message: low efforts

File: sim/resources/gpr/robot_fixed.urdf (robot description, URDF)
Before this commit: robot gpr, 22 links, 21 joints
Joints:
- joint L_ankle_y: limit lower=-0.6981317 upper=0.6981317 effort=17 velocity=10 -> lower=-0.6981317 upper=0.6981317 effort=10 velocity=10
- joint L_hip_x: limit lower=-0.34906585 upper=3.1852259 effort=20 velocity=10 -> lower=-0.34906585 upper=3.1852259 effort=10 velocity=10
- joint L_hip_y: limit lower=-1.5707963 upper=1.5707963 effort=40 velocity=10 -> lower=-1.5707963 upper=1.5707963 effort=20 velocity=10
- joint L_hip_z: limit lower=-1.5707963 upper=1.5707963 effort=20 velocity=10 -> lower=-1.5707963 upper=1.5707963 effort=10 velocity=10
- joint L_knee: limit lower=-1.57 upper=0 effort=40 velocity=10 -> lower=-1.57 upper=0 effort=20 velocity=10
- joint R_ankle_y: limit lower=-0.6981317 upper=0.6981317 effort=17 velocity=10 -> lower=-0.6981317 upper=0.6981317 effort=10 velocity=10
- joint R_hip_x: limit lower=-0.34906585 upper=3.1852259 effort=20 velocity=10 -> lower=-0.34906585 upper=3.1852259 effort=10 velocity=10
- joint R_hip_y: limit lower=-1.5707963 upper=1.5707963 effort=40 velocity=10 -> lower=-1.5707963 upper=1.5707963 effort=20 velocity=10
- joint R_hip_z: limit lower=-1.5707963 upper=1.5707963 effort=20 velocity=10 -> lower=-1.5707963 upper=1.5707963 effort=10 velocity=10
- joint R_knee: limit lower=0 upper=1.57 effort=40 velocity=10 -> lower=0 upper=1.57 effort=20 velocity=10

Commit message: adjust parameters

File: sim/resources/gpr/robot_fixed.urdf (robot description, URDF)
Before this commit: robot gpr, 22 links, 21 joints
Joints:
- joint L_ankle_y: limit lower=-0.6981317 upper=0.6981317 effort=10 velocity=10 -> lower=-0.6981317 upper=0.6981317 effort=17 velocity=10
- joint L_hip_x: limit lower=-0.34906585 upper=3.1852259 effort=10 velocity=10 -> lower=-0.34906585 upper=3.1852259 effort=20 velocity=10
- joint L_hip_y: limit lower=-1.5707963 upper=1.5707963 effort=20 velocity=10 -> lower=-1.5707963 upper=1.5707963 effort=40 velocity=10
- joint L_hip_z: limit lower=-1.5707963 upper=1.5707963 effort=10 velocity=10 -> lower=-1.5707963 upper=1.5707963 effort=20 velocity=10
- joint L_knee: limit lower=-1.57 upper=0 effort=20 velocity=10 -> lower=-1.57 upper=0 effort=40 velocity=10
- joint R_ankle_y: limit lower=-0.6981317 upper=0.6981317 effort=10 velocity=10 -> lower=-0.6981317 upper=0.6981317 effort=17 velocity=10
- joint R_hip_x: limit lower=-0.34906585 upper=3.1852259 effort=10 velocity=10 -> lower=-0.34906585 upper=3.1852259 effort=20 velocity=10
- joint R_hip_y: limit lower=-1.5707963 upper=1.5707963 effort=20 velocity=10 -> lower=-1.5707963 upper=1.5707963 effort=40 velocity=10
- joint R_hip_z: limit lower=-1.5707963 upper=1.5707963 effort=10 velocity=10 -> lower=-1.5707963 upper=1.5707963 effort=20 velocity=10
- joint R_knee: limit lower=0 upper=1.57 effort=20 velocity=10 -> lower=0 upper=1.57 effort=40 velocity=10

Commit message: gpr - smaller efforts, updates to export (#126)
update efforts and export

File: sim/resources/gpr/robot_fixed.urdf (robot description, URDF)
Before this commit: robot gpr, 22 links, 21 joints
Joints:
- joint L_hip_x: limit lower=-0.34906585 upper=3.1852259 effort=60 velocity=10 -> lower=-0.34906585 upper=3.1852259 effort=20 velocity=10
- joint L_hip_y: limit lower=-1.5707963 upper=1.5707963 effort=120 velocity=10 -> lower=-1.5707963 upper=1.5707963 effort=40 velocity=10
- joint L_hip_z: limit lower=-1.5707963 upper=1.5707963 effort=60 velocity=10 -> lower=-1.5707963 upper=1.5707963 effort=20 velocity=10
- joint L_knee: limit lower=-1.57 upper=0 effort=120 velocity=10 -> lower=-1.57 upper=0 effort=40 velocity=10
- joint R_hip_x: limit lower=-0.34906585 upper=3.1852259 effort=60 velocity=10 -> lower=-0.34906585 upper=3.1852259 effort=20 velocity=10
- joint R_hip_y: limit lower=-1.5707963 upper=1.5707963 effort=120 velocity=10 -> lower=-1.5707963 upper=1.5707963 effort=40 velocity=10
- joint R_hip_z: limit lower=-1.5707963 upper=1.5707963 effort=60 velocity=10 -> lower=-1.5707963 upper=1.5707963 effort=20 velocity=10
- joint R_knee: limit lower=0 upper=1.57 effort=120 velocity=10 -> lower=0 upper=1.57 effort=40 velocity=10

Commit message: more power

File: sim/resources/gpr/robot_fixed.urdf (robot description, URDF)
Before this commit: robot gpr, 22 links, 21 joints
Joints:
- joint L_hip_x: limit lower=-0.34906585 upper=3.1852259 effort=20 velocity=10 -> lower=-0.34906585 upper=3.1852259 effort=40 velocity=10
- joint L_hip_y: limit lower=-1.5707963 upper=1.5707963 effort=40 velocity=10 -> lower=-1.5707963 upper=1.5707963 effort=60 velocity=10
- joint L_hip_z: limit lower=-1.5707963 upper=1.5707963 effort=20 velocity=10 -> lower=-1.5707963 upper=1.5707963 effort=40 velocity=10
- joint L_knee: limit lower=-1.57 upper=0 effort=40 velocity=10 -> lower=-1.57 upper=0 effort=60 velocity=10
- joint R_hip_x: limit lower=-0.34906585 upper=3.1852259 effort=20 velocity=10 -> lower=-0.34906585 upper=3.1852259 effort=40 velocity=10
- joint R_hip_y: limit lower=-1.5707963 upper=1.5707963 effort=40 velocity=10 -> lower=-1.5707963 upper=1.5707963 effort=60 velocity=10
- joint R_hip_z: limit lower=-1.5707963 upper=1.5707963 effort=20 velocity=10 -> lower=-1.5707963 upper=1.5707963 effort=40 velocity=10
- joint R_knee: limit lower=0 upper=1.57 effort=40 velocity=10 -> lower=0 upper=1.57 effort=60 velocity=10

Commit message: update friction parameters

File: sim/resources/gpr/robot_fixed.urdf (robot description, URDF)
Before this commit: robot gpr, 22 links, 21 joints
Joints:
- joint L_ankle_y: limit lower=-0.6981317 upper=0.6981317 effort=17 velocity=10 -> lower=-0.6981317 upper=0.6981317 effort=20 velocity=10
- joint L_hip_x: limit lower=-0.34906585 upper=3.1852259 effort=20 velocity=10 -> lower=-0.34906585 upper=3.1852259 effort=40 velocity=10
- joint L_hip_y: limit lower=-1.5707963 upper=1.5707963 effort=40 velocity=10 -> lower=-1.5707963 upper=1.5707963 effort=60 velocity=10
- joint L_hip_z: limit lower=-1.5707963 upper=1.5707963 effort=20 velocity=10 -> lower=-1.5707963 upper=1.5707963 effort=40 velocity=10
- joint L_knee: limit lower=-1.57 upper=0 effort=40 velocity=10 -> lower=-1.57 upper=0 effort=60 velocity=10
- joint R_ankle_y: limit lower=-0.6981317 upper=0.6981317 effort=17 velocity=10 -> lower=-0.6981317 upper=0.6981317 effort=20 velocity=10
- joint R_hip_x: limit lower=-0.34906585 upper=3.1852259 effort=20 velocity=10 -> lower=-0.34906585 upper=3.1852259 effort=40 velocity=10
- joint R_hip_y: limit lower=-1.5707963 upper=1.5707963 effort=40 velocity=10 -> lower=-1.5707963 upper=1.5707963 effort=60 velocity=10
- joint R_hip_z: limit lower=-1.5707963 upper=1.5707963 effort=20 velocity=10 -> lower=-1.5707963 upper=1.5707963 effort=40 velocity=10
- joint R_knee: limit lower=0 upper=1.57 effort=40 velocity=10 -> lower=0 upper=1.57 effort=60 velocity=10

Commit message: add imu back

File: sim/resources/gpr/robot_fixed.urdf (robot description, URDF)
Before this commit: robot gpr, 22 links, 21 joints
Links:
- added link imu_link; visual box size=0.3 0.01 0.01
Joints:
- added joint imu_joint: type fixed, parent base, child imu_link, origin xyz=0.0 0.0 -0.13 rpy=0 0 0

Commit message: update efforts

File: sim/resources/gpr/robot_fixed.urdf (robot description, URDF)
Before this commit: robot gpr, 23 links, 22 joints
Links:
- removed link imu_link
Joints:
- removed joint imu_joint
- joint L_hip_x: limit lower=-0.34906585 upper=3.1852259 effort=20 velocity=10 -> lower=-0.34906585 upper=3.1852259 effort=40 velocity=10
- joint L_hip_y: limit lower=-1.5707963 upper=1.5707963 effort=40 velocity=10 -> lower=-1.5707963 upper=1.5707963 effort=60 velocity=10
- joint L_hip_z: limit lower=-1.5707963 upper=1.5707963 effort=20 velocity=10 -> lower=-1.5707963 upper=1.5707963 effort=40 velocity=10
- joint L_knee: limit lower=-1.57 upper=0 effort=40 velocity=10 -> lower=-1.57 upper=0 effort=60 velocity=10
- joint R_hip_x: limit lower=-0.34906585 upper=3.1852259 effort=20 velocity=10 -> lower=-0.34906585 upper=3.1852259 effort=40 velocity=10
- joint R_hip_y: limit lower=-1.5707963 upper=1.5707963 effort=40 velocity=10 -> lower=-1.5707963 upper=1.5707963 effort=60 velocity=10
- joint R_hip_z: limit lower=-1.5707963 upper=1.5707963 effort=20 velocity=10 -> lower=-1.5707963 upper=1.5707963 effort=40 velocity=10
- joint R_knee: limit lower=0 upper=1.57 effort=40 velocity=10 -> lower=0 upper=1.57 effort=60 velocity=10

Commit message: increase velocity

File: sim/resources/gpr/robot_fixed.urdf (robot description, URDF)
Before this commit: robot gpr, 22 links, 21 joints
Joints:
- joint L_ankle_y: limit lower=-0.6981317 upper=0.6981317 effort=17 velocity=10 -> lower=-0.6981317 upper=0.6981317 effort=17 velocity=15
- joint L_hip_x: limit lower=-0.34906585 upper=3.1852259 effort=40 velocity=10 -> lower=-0.34906585 upper=3.1852259 effort=40 velocity=15
- joint L_hip_y: limit lower=-1.5707963 upper=1.5707963 effort=60 velocity=10 -> lower=-1.5707963 upper=1.5707963 effort=100 velocity=15
- joint L_hip_z: limit lower=-1.5707963 upper=1.5707963 effort=40 velocity=10 -> lower=-1.5707963 upper=1.5707963 effort=40 velocity=15
- joint L_knee: limit lower=-1.57 upper=0 effort=60 velocity=10 -> lower=-1.57 upper=0 effort=100 velocity=15
- joint R_ankle_y: limit lower=-0.6981317 upper=0.6981317 effort=17 velocity=10 -> lower=-0.6981317 upper=0.6981317 effort=17 velocity=15
- joint R_hip_x: limit lower=-0.34906585 upper=3.1852259 effort=40 velocity=10 -> lower=-0.34906585 upper=3.1852259 effort=40 velocity=15
- joint R_hip_y: limit lower=-1.5707963 upper=1.5707963 effort=60 velocity=10 -> lower=-1.5707963 upper=1.5707963 effort=100 velocity=15
- joint R_hip_z: limit lower=-1.5707963 upper=1.5707963 effort=40 velocity=10 -> lower=-1.5707963 upper=1.5707963 effort=40 velocity=15
- joint R_knee: limit lower=0 upper=1.57 effort=60 velocity=10 -> lower=0 upper=1.57 effort=100 velocity=15

Commit message: imu

File: sim/resources/gpr/robot_fixed.urdf (robot description, URDF)
Before this commit: robot gpr, 22 links, 21 joints
Links:
- added link imu_link; visual box size=0.05 0.05 0.05
Joints:
- added joint imu_joint: type fixed, parent body1-part, child imu_link, origin xyz=-0.008 -0.32 0 rpy=0 0 0

Commit message: imu

File: sim/resources/gpr/robot_fixed.urdf (robot description, URDF)
Before this commit: robot gpr, 23 links, 22 joints
Links:
- link imu_link: geometry visual box size=0.3 0.01 0.01
Joints:
- joint imu_joint: origin xyz=-0.008 -0.32 0 rpy=0 0 0 -> xyz=0.03 0.0 -0.08 rpy=0 0 0; parent body1-part -> base

Commit message: Update kinfer module (#134)
* kinfer module

* ppo schema

* fix typo

* get jit

* save

* lint

* move schema definition

* fmt

* fix schema

* minor fixes

* fix names

* tensors

* squeeze

* fix imports

* pin 3.8 compatible kinfer

* lint

* joints

* update local kinfer

* update metadata + path

* clean and rename

* lint

* rename

* push kinfer

* new names

* policy runs

* joint name ordering

* stands

* clean

* lint

* cycle time

* noise to default

* change noise behavior

* less noise

* fix noise

* lint

* get name from schema

* fix

* lint

* more info from schema

* imu

* imu

* add imu missing warning

* remove default randomization

File: sim/resources/gpr/robot_fixed.urdf (robot description, URDF)
Before this commit: robot gpr, 22 links, 21 joints
Links:
- added link imu_link; visual box size=0.3 0.01 0.01
Joints:
- added joint imu_joint: type fixed, parent base, child imu_link, origin xyz=0.03 0.0 -0.08 rpy=0 0 0

Commit message: fixed limits

File: sim/resources/gpr/robot_fixed.urdf (robot description, URDF)
Before this commit: robot gpr, 23 links, 22 joints
Joints:
- joint R_knee: limit lower=0 upper=1.57 effort=100 velocity=15 -> lower=-1.57 upper=0 effort=100 velocity=15

Commit message: update limit

File: sim/resources/gpr/robot_fixed.urdf (robot description, URDF)
Before this commit: robot gpr, 23 links, 22 joints
Joints:
- joint L_hip_x: limit lower=-0.34906585 upper=3.1852259 effort=40 velocity=15 -> lower=-3.1852259 upper=0.34906585 effort=40 velocity=15

Commit message: latest

File: sim/resources/gpr/robot_fixed.urdf (robot description, URDF)
Before this commit: robot kbot, 23 links, 22 joints
Joints:
- joint floating_base: origin xyz=0 0 0 rpy=1.57 0.00 0.00 -> xyz=0 0 0 rpy=-1.57 3.14 0

Commit message: s

File: sim/resources/gpr/robot_fixed.urdf (robot description, URDF)
Before this commit: robot kbot, 23 links, 22 joints
Joints:
- joint floating_base: origin xyz=0 0 0 rpy=-1.57 3.14 0 -> xyz=0 0 0 rpy=-1.57 3.14 3.14

Commit message: new urdf

File: sim/resources/gpr/robot_fixed.urdf (robot description, URDF)
Before this commit: robot kbot, 23 links, 22 joints
Links:
- removed link leg3_shell2
- removed link leg3_shell22
- added link leg3_shell1, mass 1.10995541; collision mesh filename=meshes/leg3_shell1.stl; visual mesh filename=meshes/leg3_shell1.stl
- added link leg3_shell11, mass 1.10996161; collision mesh filename=meshes/leg3_shell11.stl; visual mesh filename=meshes/leg3_shell11.stl
- link arm1_top: mass 0.6485195170000001 -> 0.5727323900000001
- link arm1_top_2: mass 0.648518913 -> 0.57273186
- link arm2_shell: mass 0.51101595 -> 0.51067762
- link arm2_shell_2: mass 0.51101595 -> 0.51067762
- link arm3_shell: mass 0.57887479 -> 0.5785364000000001
- link arm3_shell2: mass 0.57887479 -> 0.5785364000000001
- link body1-part: mass 9.415837554000001 -> 9.12867194
- link hand_shell: mass 0.7933517460000001 -> 0.7930633560000001
- link hand_shell_2: mass 0.7933517460000001 -> 0.7930633560000001
- link leg1_shell: mass 1.360769512 -> 1.2643519300000001
- link leg1_shell3: mass 1.360769362 -> 1.26435173
- link shoulder: mass 1.10769407 -> 1.1073556900000001
- link shoulder_2: mass 1.10769287 -> 1.10735447
Joints:
- joint floating_base: origin xyz=0 0 0 rpy=-1.57 3.14 3.14 -> xyz=0 0 0 rpy=-1.57 0 0
- joint imu_link: origin xyz=-0.047126255760769356 0.14188879185640826 0.0003937090896153101 rpy=1.5707963999999994 0.0 3.1415926071795863 -> xyz=0.039989396 -0.12791044000000001 -2.6794896579307448e-11 rpy=-1.5707963 0 0
- joint left_ankle_02: axis 0 0 1 -> 0 0 -1; origin xyz=0.0 -0.30000000004641003 0.07019999118206069 rpy=9.282041357749903e-08 0.0 0.0 -> xyz=0.0 -0.30000000013923045 0.009499991182060727 rpy=9.282041333256967e-08 0.0 0.0; parent leg3_shell2 -> leg3_shell1
- joint left_hip_pitch_04: origin xyz=-0.0071262559999999975 -0.16321120617636828 -0.08730629129474379 rpy=1.0000000028043132e-07 0.0 0.0 -> xyz=-1.0608550148631657e-05 -0.43201043164593794 0.0887000068648673 rpy=-3.1415925071795874 4.641020678874952e-08 -3.1415926535897913
- joint left_hip_roll_03: origin xyz=0.02649999999999997 -1.5165911463888016e-09 -0.06950000151659115 rpy=-1.5707963 0.0 1.5707963 -> xyz=0.027499999999999972 -1.543386042968109e-09 -0.06950000154338605 rpy=-1.5707963 0.0 1.5707963
- joint left_hip_yaw_03: origin xyz=-0.15649999999999997 0.00011981393 0.027499998483408852 rpy=-0.0 1.5707963 0.0 -> xyz=-0.15749999999999997 0.00011981393 0.027499998456613956 rpy=-0.0 1.5707963 0.0
- joint left_knee_04: axis 0 0 1 -> 0 0 -1; child leg3_shell2 -> leg3_shell1; limit lower=-2.0943951 upper=0 effort=120 velocity=6.283 -> lower=0 upper=2.0943951 effort=120 velocity=6.283; origin xyz=0.0 0.0342 -0.14250000009378214 rpy=1.5707963000000003 0.0 0.0 -> xyz=0.0 -0.026999999999999993 -0.14250000111820607 rpy=1.5707963999999996 0.0 0.0
- joint right_ankle_02: axis 0 0 1 -> 0 0 -1; origin xyz=1.0767167917674625e-08 -0.2999999986541038 0.027200000000000002 rpy=-3.1415926071795868 2.220446049250313e-16 -3.1415926071795868 -> xyz=2.153907282807268e-18 -0.3000000000464102 -0.035500000000000004 rpy=3.1415927 0 3.1415927; parent leg3_shell22 -> leg3_shell11
- joint right_hip_pitch_04: origin xyz=-0.0071262559999999975 -0.16321121297959254 0.08859370870525608 rpy=-3.141592599999999 0.0 0.0 -> xyz=-1.0600293772844438e-05 -0.4320104468591277 -0.08919999313513188 rpy=9.99999991702083e-08 4.641020678874952e-08 -3.1415926535897913
- joint right_hip_roll_03: origin xyz=0.02649999999999997 -1.5165911463888016e-09 -0.06900000151659115 rpy=1.5707963 -4.641020634466031e-08 -1.5707963535897922 -> xyz=0.027499999999999972 -1.5433860431346424e-09 -0.06900000154338605 rpy=1.5707963 -4.641020634466031e-08 -1.5707963535897922
- joint right_hip_yaw_03: origin xyz=-0.15649999999999997 -0.00011981393 0.027499998483408852 rpy=-3.1415926535897922 -1.5707962732050302 0.0 -> xyz=-0.15749999999999997 -0.00011981393000000101 0.027499998536998718 rpy=-3.1415926535897922 -1.5707962732050302 0.0
- joint right_knee_04: axis 0 0 1 -> 0 0 -1; child leg3_shell22 -> leg3_shell11; limit lower=0 upper=2.0943951 effort=120 velocity=6.283 -> lower=-2.0943951 upper=0 effort=120 velocity=6.283; origin xyz=0.0 0.0342 -0.14250000009378214 rpy=1.5707963000000003 0.0 0.0 -> xyz=0.0 -0.026999999999999993 -0.14250000111820607 rpy=1.5707963999999996 0.0 0.0
- joint right_shoulder_yaw_02: axis 0 0 1 -> 0 0 -1; origin xyz=-0.13949999999999999 0.0 0.022499999155960758 rpy=-3.1415926071795863 1.5707963 0.0 -> xyz=-0.13949999999999999 4.64102069112142e-11 0.02249999912916586 rpy=-3.1415926071795863 1.5707963 0.0

Commit message: save the setup with higher kps

File: sim/resources/gpr/robot_fixed.urdf (robot description, URDF)
Before this commit: robot k-bot_sim, 23 links, 22 joints
Joints:
- joint left_ankle_02: limit lower=-0.698132 upper=0.698132 effort=17 velocity=12.566 -> lower=-0.698132 upper=0.698132 effort=17 velocity=18
- joint left_hip_pitch_04: limit lower=-1.570796 upper=1.570796 effort=60 velocity=6.283 -> lower=-1.570796 upper=1.570796 effort=60 velocity=18
- joint left_hip_roll_03: limit lower=-3.185226 upper=0.349066 effort=40 velocity=6.283 -> lower=-3.185226 upper=0.349066 effort=40 velocity=18
- joint left_hip_yaw_03: limit lower=-1.570796 upper=1.570796 effort=40 velocity=6.283 -> lower=-1.570796 upper=1.570796 effort=40 velocity=18
- joint left_knee_04: limit lower=0 upper=2.094395 effort=60 velocity=6.283 -> lower=0 upper=2.094395 effort=60 velocity=18
- joint right_ankle_02: limit lower=-0.698132 upper=0.698132 effort=17 velocity=12.566 -> lower=-0.698132 upper=0.698132 effort=17 velocity=18
- joint right_hip_pitch_04: limit lower=-1.570796 upper=1.570796 effort=60 velocity=6.283 -> lower=-1.570796 upper=1.570796 effort=60 velocity=18
- joint right_hip_roll_03: limit lower=-0.349066 upper=3.185226 effort=40 velocity=6.283 -> lower=-0.349066 upper=3.185226 effort=40 velocity=18
- joint right_hip_yaw_03: limit lower=-1.570796 upper=1.570796 effort=40 velocity=6.283 -> lower=-1.570796 upper=1.570796 effort=40 velocity=18
- joint right_knee_04: limit lower=-2.094395 upper=0 effort=60 velocity=6.283 -> lower=-2.094395 upper=0 effort=60 velocity=18

File: sim/resources/zbot2/robot_fixed.urdf (robot description, URDF)
Before this commit: robot z-bot2_fe_urdf, 20 links, 19 joints
Joints:
- joint floating_base: origin xyz=0 0 0 rpy=0 0 1.5707963 -> xyz=0 0 0 rpy=0 0 0
