Commit message: Pos and vel targets with latency (#144)
* slow walk

* better gait

* update xml

* update to terrain too

* testing original rewards

* add uneven terrain

* mv

* urdf

* s

* fix imu

* first run

* policy

* sim2sim

* latest

* xml

* s

* new urdf

* new class

* fix path

* more path

* same name

* save

* updated urdf

* fix new urdf

* flexible lims

* lower res sim + 50hz policy

* fix signs?

* fiz heights

* rename

* termination contacts and flipping some signs just cause

* nvm lol

* ONE. MORE. TRYgit status!

* headless xml

* policy

* lint

* loosen

* lint

* no ang vel, shorter history, higher effort lim, 200hz sim time

* separate pd decimation

* new setup

* minor rewrite

* parameterize export

* temp latency config

* oneshot lol

* use buffers

* ang vel

* fix

* higher drop

* draft

* clean

* pd decimatino

* motor randomizations (and link mass)

* initialize vars

* param optimization

* clean

* lint

* ignore

* ang vel

* match noise

* fix pd init

* curriculum + energy rewards

* update urdf

* backup

* save

* output positions and velocities

* fix playing

* export num_joints

* mv

* up to date with vel-test-ideal

* port in vel-test-ideal

* fix play

* fix

* add new updated urdf for latency env

* fix headless latency run

* move latency env to separate base class

* update headless normal

* fix headless

* update logging

* headless ideal training config

* add termination contacts and reduce noise

* update urdfs

* add termination contacts

* update termination conds

* update term height

* increase height

* increase term height

* really high term

* kneel less noisy

* port in old vel setup

* register vel

* noise

* add headless pos

* fix

* fix vel play

* higher kp kds

* wean off traj + more noise

* slightly bigger pushes

* rewards etc

* more smoothing, slightly easier

* clean up

File: sim/resources/gpr/robot_fixed.urdf (robot description, URDF)
Before this commit: robot gpr, 23 links, 22 joints
Links:
- removed link imu_link
- removed link leg3_shell2
- removed link leg3_shell22
- added link imu, mass 0.01; collision mesh filename=meshes/imu.stl; visual mesh filename=meshes/imu.stl
- added link leg3_shell1, mass 1.10995541; collision mesh filename=meshes/leg3_shell1.stl; visual mesh filename=meshes/leg3_shell1.stl
- added link leg3_shell11, mass 1.10996161; collision mesh filename=meshes/leg3_shell11.stl; visual mesh filename=meshes/leg3_shell11.stl
- link arm1_top: mass 0.6485195170000001 -> 0.5727323900000001
- link arm1_top_2: mass 0.648518913 -> 0.57273186
- link arm2_shell: mass 0.51101595 -> 0.51067762
- link arm2_shell_2: mass 0.51101595 -> 0.51067762
- link arm3_shell: mass 0.57887479 -> 0.5785364000000001
- link arm3_shell2: mass 0.57887479 -> 0.5785364000000001
- link body1-part: mass 11.923537116999997 -> 9.12867194
- link foot1: mass 0.54574734 -> 0.58209124
- link foot3: mass 0.5457471700000001 -> 0.58209108
- link hand_shell: mass 0.7933517460000001 -> 0.7930633560000001
- link hand_shell_2: mass 0.7933517460000001 -> 0.7930633560000001
- link leg1_shell: mass 1.360769512 -> 1.2643519300000001
- link leg1_shell3: mass 1.360769362 -> 1.26435173
- link shoulder: mass 1.10769407 -> 1.1073556900000001
- link shoulder_2: mass 0.80769287 -> 1.10735447
Joints:
- removed joint L_ankle_y
- removed joint L_hip_x
- removed joint L_hip_y
- removed joint L_hip_z
- removed joint L_knee
- removed joint R_ankle_y
- removed joint R_hip_x
- removed joint R_hip_y
- removed joint R_hip_z
- removed joint R_knee
- removed joint Revolute_1
- removed joint Revolute_15
- removed joint Revolute_16
- removed joint Revolute_2
- removed joint Revolute_3
- removed joint Revolute_4
- removed joint Revolute_5
- removed joint Revolute_6
- removed joint Revolute_7
- removed joint Revolute_8
- removed joint imu_joint
- added joint imu_link: type fixed, parent body1-part, child imu, origin xyz=0.039989396 -0.12791044000000001 -2.6794896579307448e-11 rpy=-1.5707963 0 0
- added joint left_ankle_02: type revolute, parent leg3_shell1, child foot1, origin xyz=0.0 -0.30000000013923045 0.009499991182060727 rpy=9.282041333256967e-08 0.0 0.0, axis 0 0 -1, limit lower=-0.6981317 upper=0.6981317 effort=17 velocity=12.566
- added joint left_elbow_02: type fixed, parent arm2_shell, child arm3_shell, origin xyz=-0.026000000000000002 0.0 -0.09799999977224338 rpy=-3.1415926071795863 -1.5707963 0.0, axis 0 0 1, limit lower=-2.5307274 upper=0 effort=17 velocity=12.566
- added joint left_hip_pitch_04: type revolute, parent body1-part, child leg0_shell, origin xyz=-1.0608550148631657e-05 -0.43201043164593794 0.0887000068648673 rpy=-3.1415925071795874 4.641020678874952e-08 -3.1415926535897913, axis 0 0 1, limit lower=-1.5707963 upper=1.5707963 effort=120 velocity=6.283
- added joint left_hip_roll_03: type revolute, parent leg0_shell, child leg1_shell, origin xyz=0.027499999999999972 -1.543386042968109e-09 -0.06950000154338605 rpy=-1.5707963 0.0 1.5707963, axis 0 0 1, limit lower=-3.1852259 upper=0.34906585 effort=60 velocity=6.283
- added joint left_hip_yaw_03: type revolute, parent leg1_shell, child leg2_shell, origin xyz=-0.15749999999999997 0.00011981393 0.027499998456613956 rpy=-0.0 1.5707963 0.0, axis 0 0 1, limit lower=-1.5707963 upper=1.5707963 effort=60 velocity=6.283
- added joint left_knee_04: type revolute, parent leg2_shell, child leg3_shell1, origin xyz=0.0 -0.026999999999999993 -0.14250000111820607 rpy=1.5707963999999996 0.0 0.0, axis 0 0 -1, limit lower=0 upper=2.0943951 effort=120 velocity=6.283
- added joint left_shoulder_pitch_03: type fixed, parent body1-part, child shoulder, origin xyz=-0.0071262490312895945 0.2868887861013424 -0.1871062947956447 rpy=-2.220446049250311e-16 0.0 1.9915984595047395e-16, axis 0 0 1, limit lower=0 upper=3.1415927 effort=60 velocity=6.283
- added joint left_shoulder_roll_03: type fixed, parent shoulder, child arm1_top, origin xyz=0.022511964 5.627838501275855e-05 -0.06749999993301277 rpy=1.5707963 0.0 1.5707963, axis 0 0 1, limit lower=-0.47996554 upper=3.6302848 effort=60 velocity=6.283
- added joint left_shoulder_yaw_02: type fixed, parent arm1_top, child arm2_shell, origin xyz=-0.13949999999999996 -1.4619215099879723e-09 -0.02349999915596076 rpy=-4.641020604450649e-08 1.5707962732050293 0.0, axis 0 0 1, limit lower=-1.5707963 upper=1.5707963 effort=17 velocity=12.566
- added joint left_wrist_02: type fixed, parent arm3_shell, child hand_shell, origin xyz=-0.18149999999999997 -1.4619215099879723e-09 0.02150000084403924 rpy=-4.641020604450649e-08 1.5707962732050293 0.0, axis 0 0 1, limit lower=0 upper=6.2831853 effort=17 velocity=12.566
- added joint right_ankle_02: type revolute, parent leg3_shell11, child foot3, origin xyz=2.153907282807268e-18 -0.3000000000464102 -0.035500000000000004 rpy=3.1415927 0 3.1415927, axis 0 0 -1, limit lower=-0.6981317 upper=0.6981317 effort=17 velocity=12.566
- added joint right_elbow_02: type fixed, parent arm2_shell_2, child arm3_shell2, origin xyz=0.026000000000000002 0.0 0.09750000022775662 rpy=-3.1415926071795863 1.5707963 0.0, axis 0 0 1, limit lower=0 upper=2.5307274 effort=17 velocity=12.566
- added joint right_hip_pitch_04: type revolute, parent body1-part, child leg0_shell_2, origin xyz=-1.0600293772844438e-05 -0.4320104468591277 -0.08919999313513188 rpy=9.99999991702083e-08 4.641020678874952e-08 -3.1415926535897913, axis 0 0 1, limit lower=-1.5707963 upper=1.5707963 effort=120 velocity=6.283
- added joint right_hip_roll_03: type revolute, parent leg0_shell_2, child leg1_shell3, origin xyz=0.027499999999999972 -1.5433860431346424e-09 -0.06900000154338605 rpy=1.5707963 -4.641020634466031e-08 -1.5707963535897922, axis 0 0 1, limit lower=-0.34906585 upper=3.1852259 effort=60 velocity=6.283
- added joint right_hip_yaw_03: type revolute, parent leg1_shell3, child leg2_shell_2, origin xyz=-0.15749999999999997 -0.00011981393000000101 0.027499998536998718 rpy=-3.1415926535897922 -1.5707962732050302 0.0, axis 0 0 1, limit lower=-1.5707963 upper=1.5707963 effort=60 velocity=6.283
- added joint right_knee_04: type revolute, parent leg2_shell_2, child leg3_shell11, origin xyz=0.0 -0.026999999999999993 -0.14250000111820607 rpy=1.5707963999999996 0.0 0.0, axis 0 0 -1, limit lower=-2.0943951 upper=0 effort=120 velocity=6.283
- added joint right_shoulder_pitch_03: type fixed, parent body1-part, child shoulder_2, origin xyz=-0.007126249031289128 0.28688879614942864 0.18789370520435525 rpy=3.1415925999999996 -2.4424906541753444e-15 -9.282041357749904e-08, axis 0 0 1, limit lower=-3.1415927 upper=0 effort=60 velocity=6.283
- added joint right_shoulder_roll_03: type fixed, parent shoulder_2, child arm1_top_2, origin xyz=0.022511964 -5.627838501275855e-05 -0.06749999993301277 rpy=1.5707963999999996 -2.220446049250313e-16 -1.5707963000000003, axis 0 0 1, limit lower=-0.47996554 upper=3.6302848 effort=60 velocity=6.283
- added joint right_shoulder_yaw_02: type fixed, parent arm1_top_2, child arm2_shell_2, origin xyz=-0.13949999999999999 4.64102069112142e-11 0.02249999912916586 rpy=-3.1415926071795863 1.5707963 0.0, axis 0 0 -1, limit lower=-1.5707963 upper=1.5707963 effort=17 velocity=12.566
- added joint right_wrist_02: type fixed, parent arm3_shell2, child hand_shell_2, origin xyz=-0.18149999999999997 -1.4619215099879723e-09 0.02150000084403924 rpy=-4.641020604450649e-08 1.5707962732050293 0.0, axis 0 0 1, limit lower=0 upper=6.2831853 effort=17 velocity=12.566
- joint floating_base: origin xyz=0 0 0 rpy=-1.57 3.14 0 -> xyz=0 0 0 rpy=-1.57 0 0
